File: gpio.sch (KiCad schematic (older format))
At the start: 3 parts, among them J1 DF40C-100DP-0.4V(51), J2 DF40C-100DP-0.4V(51), U1 LFE5U-85F-6BG381C

Commit message: SDRAM, JTAG routed - before logo delete
Connections:
- net AUDIO_R0: no longer U1.A3 (PL14C)
- net GP9: no longer U1.A2 (PL35A)
- net BTN_PWRn: no longer names the net of U1.D6 (PT6B)
- new net USB_FPGA_PULL_D+: U1.A2 (PL35A)
- new net USB_FPGA_PULL_D-: U1.A3 (PL14C)
Changed lines of the file:
@@
 Text GLabel 2550 3500 2    60   Input ~ 0
 GN9
-Text GLabel 1050 3500 0    60   Input ~ 0
+Text GLabel -600 3450 0    60   Input ~ 0
 GP9
 Text GLabel 2550 2900 2    60   Input ~ 0
@@
 Text GLabel 2550 2800 2    60   Input ~ 0
 AUDIO_L3
-Text GLabel 1050 2800 0    60   Input ~ 0
+Text GLabel -500 3300 0    60   Input ~ 0
 AUDIO_R0
 Text GLabel 1050 2600 0    60   Input ~ 0
@@
 Text Notes 950  7550 0    60   ~ 0
 GPIO route only A/B pairs as those are differential bidirectional\ndon't route C/D pairs to GPIO as those can be differential input only\nBANK0,1 are single-ended (non-differential)
-Text GLabel 2600 1800 2    60   Input ~ 0
-BTN_PWRn
 Text Notes 950  7200 0    60   ~ 0
 GP,GN 14-21 differential bidirectional connected to BANK2,3 on "ram" sheet\nGP,GN 22-27 single-ended connected to BANK1 on "gpdi" sheet
@@
 Wire Wire Line
 	4600 1150 4450 1150
+Text GLabel 1050 3500 0    60   Input ~ 0
+USB_FPGA_PULL_D+
+Text GLabel 1050 2800 0    60   Input ~ 0
+USB_FPGA_PULL_D-
+Text GLabel 5300 2550 0    60   Input ~ 0
+JTAG_TDI
+Text GLabel 5300 2650 0    60   Input ~ 0
+JTAG_TMS
+Text GLabel 5300 2750 0    60   Input ~ 0
+JTAG_TCK
+Text GLabel 5300 2850 0    60   Input ~ 0
+JTAG_TDO
+Text GLabel 5400 2550 2    60   Input ~ 0
+GPIO26
+Text GLabel 5400 2650 2    60   Input ~ 0
+GPIO19
+Text GLabel 5400 2850 2    60   Input ~ 0
+GPIO16
+Wire Wire Line
+	5300 2550 5400 2550
+Wire Wire Line
+	5400 2650 5300 2650
+Text GLabel 5400 2750 2    60   Input ~ 0
+GPIO20
+Wire Wire Line
+	5300 2750 5400 2750
+Wire Wire Line
+	5400 2850 5300 2850
 $EndSCHEMATC

Commit message: Cleaning DRC errors
Connections:
- net SD_D0 renamed SD_DAT0
- net SD_D1 renamed SD_DAT1
- net SD_D2 renamed SD_DAT2
- net SD_D3 renamed SD_DAT3
Changed lines of the file:
@@
 Text GLabel 18150 2350 0    60   Input ~ 0
 GPIO21
-Text GLabel 16500 4150 0    60   Input ~ 0
+Text GLabel 14950 6500 0    60   Input ~ 0
 CAM0_D0_N
-Text GLabel 16500 4050 0    60   Input ~ 0
+Text GLabel 14950 6400 0    60   Input ~ 0
 CAM0_D0_P
-Text GLabel 16500 3950 0    60   Input ~ 0
+Text GLabel 14950 6300 0    60   Input ~ 0
 CAM0_D1_N
-Text GLabel 16500 3850 0    60   Input ~ 0
+Text GLabel 14950 6200 0    60   Input ~ 0
 CAM0_D1_P
-Text GLabel 16500 3750 0    60   Input ~ 0
+Text GLabel 14950 6100 0    60   Input ~ 0
 CAM0_C_N
-Text GLabel 16500 3650 0    60   Input ~ 0
+Text GLabel 14950 6000 0    60   Input ~ 0
 CAM0_C_P
 Text GLabel 15100 3650 0    60   Input ~ 0
@@
 Text GLabel 14100 5950 0    60   Input ~ 0
 DSI0_D0_N
-Text GLabel 4450 1050 0    60   Input ~ 0
-SD_D2
-Text GLabel 4450 1150 0    60   Input ~ 0
-SD_D3
-Text GLabel 4450 850  0    60   Input ~ 0
-SD_D0
-Text GLabel 4450 950  0    60   Input ~ 0
-SD_D1
-Text GLabel 4600 1050 2    60   Input ~ 0
-SD_DAT2
-Text GLabel 4600 950  2    60   Input ~ 0
-SD_DAT1
-Text GLabel 4600 1300 2    60   Input ~ 0
-SD_DAT4
-Text GLabel 4600 1400 2    60   Input ~ 0
-SD_DAT5
-Text GLabel 4600 1500 2    60   Input ~ 0
-SD_DAT6
-Text GLabel 4600 1600 2    60   Input ~ 0
-SD_DAT7
-Text GLabel 4600 1150 2    60   Input ~ 0
-SD_DAT3
-Text GLabel 4600 850  2    60   Input ~ 0
-SD_DAT0
-Text GLabel 4600 1750 2    60   Input ~ 0
-SD_PWR_ON
-Wire Wire Line
-	4450 850  4600 850
-Wire Wire Line
-	4600 950  4450 950
-Wire Wire Line
-	4450 1050 4600 1050
-Wire Wire Line
-	4600 1150 4450 1150
 Text GLabel 1050 3500 0    60   Input ~ 0
 USB_FPGA_PULL_D+
 Text GLabel 1050 2800 0    60   Input ~ 0
 USB_FPGA_PULL_D-
-Text GLabel 5300 2550 0    60   Input ~ 0
-JTAG_TDI
-Text GLabel 5300 2650 0    60   Input ~ 0
-JTAG_TMS
-Text GLabel 5300 2750 0    60   Input ~ 0
-JTAG_TCK
-Text GLabel 5300 2850 0    60   Input ~ 0
-JTAG_TDO
-Text GLabel 5400 2550 2    60   Input ~ 0
-GPIO26
-Text GLabel 5400 2650 2    60   Input ~ 0
-GPIO19
-Text GLabel 5400 2850 2    60   Input ~ 0
-GPIO16
-Wire Wire Line
-	5300 2550 5400 2550
-Wire Wire Line
-	5400 2650 5300 2650
-Text GLabel 5400 2750 2    60   Input ~ 0
-GPIO20
-Wire Wire Line
-	5300 2750 5400 2750
-Wire Wire Line
-	5400 2850 5300 2850
 $EndSCHEMATC

Commit message: Routing cam and display differential
Connections:
- net GP2: no longer U1.A9 (GR_PCLK0_1)
- net PCIe_CLK_nREQ: now also U1.A9 (GR_PCLK0_1)
- net PCIe_nRST: now also U1.D9 (PT20A)
Changed lines of the file:
@@
 Text GLabel 1100 900  0    60   Input ~ 0
 GP1
-Text GLabel 1100 1000 0    60   Input ~ 0
+Text GLabel 350  600  0    60   Input ~ 0
 GP2
 Text GLabel 1100 1300 0    60   Input ~ 0
@@
 Text GLabel 18150 2350 0    60   Input ~ 0
 GPIO21
-Text GLabel 14950 6500 0    60   Input ~ 0
-CAM0_D0_N
-Text GLabel 14950 6400 0    60   Input ~ 0
-CAM0_D0_P
-Text GLabel 14950 6300 0    60   Input ~ 0
-CAM0_D1_N
-Text GLabel 14950 6200 0    60   Input ~ 0
-CAM0_D1_P
-Text GLabel 14950 6100 0    60   Input ~ 0
-CAM0_C_N
-Text GLabel 14950 6000 0    60   Input ~ 0
-CAM0_C_P
 Text GLabel 15100 3650 0    60   Input ~ 0
 CAM1_D0_N
@@
 Text GLabel 13000 5500 0    60   Input ~ 0
 DSI1_D0_N
-Text GLabel 14100 6450 0    60   Input ~ 0
-DSI0_C_P
-Text GLabel 14100 6350 0    60   Input ~ 0
-DSI0_C_N
-Text GLabel 14100 6250 0    60   Input ~ 0
-DSI0_D1_P
-Text GLabel 14100 6150 0    60   Input ~ 0
-DSI0_D1_N
-Text GLabel 14100 6050 0    60   Input ~ 0
-DSI0_D0_P
-Text GLabel 14100 5950 0    60   Input ~ 0
-DSI0_D0_N
 Text GLabel 1050 3500 0    60   Input ~ 0
 USB_FPGA_PULL_D+
 Text GLabel 1050 2800 0    60   Input ~ 0
 USB_FPGA_PULL_D-
+Text GLabel 1100 1000 0    60   Input ~ 0
+PCIe_CLK_nREQ
+Text GLabel 1100 1200 0    60   Input ~ 0
+PCIe_nRST
 $EndSCHEMATC

Commit message: connecting more pins
Connections:
- net GP8: no longer U1.A4 (PL11A)
- net USB_OTG_ID: now also U1.A4 (PL11A)
Changed lines of the file:
@@
 Text GLabel 2550 2700 2    60   Input ~ 0
 GN8
-Text GLabel 1050 2700 0    60   Input ~ 0
+Text GLabel -50  2700 0    60   Input ~ 0
 GP8
 Text GLabel 2600 1900 2    60   Input ~ 0
@@
 Text GLabel 13150 850  0    60   Input ~ 0
 ETH_1P
-Text GLabel 13900 2150 0    60   Input ~ 0
-ID_SC
-Text GLabel 13900 2250 0    60   Input ~ 0
-ID_SD
 Text GLabel 18150 2850 0    60   Input ~ 0
 GPIO26
@@
 Text GLabel 1100 1200 0    60   Input ~ 0
 PCIe_nRST
+Text GLabel 1050 2700 0    60   Input ~ 0
+USB_OTG_ID
 $EndSCHEMATC

Commit message: Connecting serdes to gpio
Changed lines of the file:
@@
 Text GLabel 18150 250  0    60   Input ~ 0
 SDA0
-Text GLabel 13100 200  0    60   Input ~ 0
-ETH_3P
-Text GLabel 13100 300  0    60   Input ~ 0
-ETH_3N
-Text GLabel 13100 450  0    60   Input ~ 0
-ETH_2N
-Text GLabel 13100 550  0    60   Input ~ 0
-ETH_2P
 Text GLabel 13150 1350 0    60   Input ~ 0
 ETH_nLED2
@@
 Text GLabel 13150 1700 0    60   Input ~ 0
 ETH_SYNC_OUT
-Text GLabel 13150 1100 0    60   Input ~ 0
-ETH_0P
 Text GLabel 13150 1250 0    60   Input ~ 0
 ETH_nLED3
 Text GLabel 7700 1400 2    60   Input ~ 0
 ETH_0N
-Text GLabel 13150 1000 0    60   Input ~ 0
-ETH_0N
-Text GLabel 13100 700  0    60   Input ~ 0
-ETH_1N
-Text GLabel 13150 850  0    60   Input ~ 0
-ETH_1P
 Text GLabel 18150 2850 0    60   Input ~ 0
 GPIO26
@@
 Text GLabel 1050 2700 0    60   Input ~ 0
 USB_OTG_ID
+Text GLabel 4550 3150 0    60   Input ~ 0
+SRX11P
+Text GLabel 4550 3250 0    60   Input ~ 0
+SRX11N
+Text GLabel 4550 3050 0    60   Input ~ 0
+STX11P
+Text GLabel 4550 2950 0    60   Input ~ 0
+STX11N
+Text GLabel 4550 2700 0    60   Input ~ 0
+SRCLK1P
+Text GLabel 4550 2800 0    60   Input ~ 0
+SRCLK1N
+Text GLabel 4700 3150 2    60   Input ~ 0
+GPIO11
+Text GLabel 4700 3250 2    60   Input ~ 0
+GPIO9
+Text GLabel 4700 3050 2    60   Input ~ 0
+GPIO10
+Text GLabel 4700 2950 2    60   Input ~ 0
+GPIO22
+Text GLabel 4700 2700 2    60   Input ~ 0
+GPIO27
+Text GLabel 4700 2800 2    60   Input ~ 0
+GPIO17
+Wire Wire Line
+	4550 2700 4700 2700
+Wire Wire Line
+	4700 2800 4550 2800
+Wire Wire Line
+	4550 2950 4700 2950
+Wire Wire Line
+	4700 3050 4550 3050
+Wire Wire Line
+	4550 3150 4700 3150
+Wire Wire Line
+	4700 3250 4550 3250
 $EndSCHEMATC

Commit message: Fixing 3.3V - CM4 needs to provide 3.3V
Connections:
- net CM4_3.3V renamed +3V3
Changed lines of the file:
@@
 Wire Wire Line
 	4700 3250 4550 3250
+Text GLabel 4850 5200 2    60   Input ~ 0
+CM4_3.3V
+$Comp
+L power:+3V3 #PWR?
+U 1 1 61646D74
+P 4650 5200
+F 0 "#PWR?" H 4650 5050 50  0001 C CNN
+F 1 "+3V3" H 4650 5340 50  0000 C CNN
+F 2 "" H 4650 5200 50  0000 C CNN
+F 3 "" H 4650 5200 50  0000 C CNN
+	1    4650 5200
+	0    -1   -1   0
+$EndComp
+Wire Wire Line
+	4650 5200 4850 5200
 $EndSCHEMATC

Commit message: Moving connectors 0.3mm away from each other
Other:
- note added: "CM4 needs to provide 3.3V to CM4 IO board"
Changed lines of the file:
@@
 Wire Wire Line
 	4700 3250 4550 3250
-Text GLabel 4850 5200 2    60   Input ~ 0
+Text GLabel 5200 4700 1    60   Input ~ 0
 CM4_3.3V
 $Comp
 L power:+3V3 #PWR?
 U 1 1 61646D74
-P 4650 5200
-F 0 "#PWR?" H 4650 5050 50  0001 C CNN
-F 1 "+3V3" H 4650 5340 50  0000 C CNN
-F 2 "" H 4650 5200 50  0000 C CNN
-F 3 "" H 4650 5200 50  0000 C CNN
-	1    4650 5200
-	0    -1   -1   0
+P 5200 4900
+F 0 "#PWR?" H 5200 4750 50  0001 C CNN
+F 1 "+3V3" H 5200 5040 50  0000 C CNN
+F 2 "" H 5200 4900 50  0000 C CNN
+F 3 "" H 5200 4900 50  0000 C CNN
+	1    5200 4900
+	-1   0    0    1
 $EndComp
 Wire Wire Line
-	4650 5200 4850 5200
+	5200 4900 5200 4700
+Text Notes 5050 5600 1    60   ~ 0
+CM4 needs to provide 3.3V to CM4 IO board
 $EndSCHEMATC

Commit message: Adding buttons
Connections:
- net AUDIO_L3 is gone; now on net LED2: U1.B3 (PL14D)
- net AUDIO_L2: no longer U1.C3 (PL17C)
- net GN9: no longer U1.B1 (PL35B)
- net LED1: now also U1.B1 (PL35B); no longer U1.C2 (PL35D)
- net LED2: no longer U1.C1 (PL38A)
- net LED3: now also U1.C1 (PL38A); no longer U1.D2 (PL38C)
- net LED4: no longer U1.D1 (PL38B)
- net LED5: no longer U1.E2 (PCLKC7_0)
- net LED7: no longer U1.H3 (PL41D)
- new net BTN1: U1.C2 (PL35D)
- new net BTN2: U1.C3 (PL17C)
Changed lines of the file:
@@
 Text GLabel 1050 3300 0    60   Input ~ 0
 GP11
-Text GLabel 2550 3500 2    60   Input ~ 0
-GN9
+Text GLabel 2550 3400 2    60   Input ~ 0
+BTN1
 Text GLabel -600 3450 0    60   Input ~ 0
 GP9
@@
 Text GLabel 2550 3000 2    60   Input ~ 0
 AUDIO_L1
+Text GLabel 3850 4250 0    60   Input ~ 0
+AUDIO_L2
 Text GLabel 1050 3000 0    60   Input ~ 0
-AUDIO_L2
-Text GLabel 2550 2800 2    60   Input ~ 0
-AUDIO_L3
+BTN2
 Text GLabel -500 3300 0    60   Input ~ 0
 AUDIO_R0
@@
 Text GLabel 1050 3400 0    60   Input ~ 0
 LED0
-Text GLabel 2550 4000 2    60   Input ~ 0
+Text GLabel 3200 3700 2    60   Input ~ 0
 LED5
+Text GLabel 2550 2800 2    60   Input ~ 0
+LED2
 Text GLabel 1050 3700 0    60   Input ~ 0
-LED2
-Text GLabel 1050 3600 0    60   Input ~ 0
 LED3
-Text GLabel 2550 3700 2    60   Input ~ 0
+Text GLabel 3200 3500 2    60   Input ~ 0
 LED4
-Text GLabel 2550 3400 2    60   Input ~ 0
-LED1
 Text GLabel 2550 3600 2    60   Input ~ 0
 LED6
-Text GLabel 2550 3800 2    60   Input ~ 0
+Text GLabel 3200 3600 2    60   Input ~ 0
 LED7
 Text Notes 950  7550 0    60   ~ 0
@@
 CM4_3.3V
 $Comp
-L power:+3V3 #PWR?
+L power:+3V3 #PWR0111
 U 1 1 61646D74
 P 5200 4900
-F 0 "#PWR?" H 5200 4750 50  0001 C CNN
+F 0 "#PWR0111" H 5200 4750 50  0001 C CNN
 F 1 "+3V3" H 5200 5040 50  0000 C CNN
 F 2 "" H 5200 4900 50  0000 C CNN
@@
 Text Notes 5050 5600 1    60   ~ 0
 CM4 needs to provide 3.3V to CM4 IO board
+Text GLabel 2550 3500 2    60   Input ~ 0
+LED1
 $EndSCHEMATC
