File: ulx3s.kicad_pcb (KiCad board)
At the start: 4 copper layers, 82.9 x 50.8 mm, 92 parts, among them J5 VJ1, U1 LFE5U-85F-6BG381C, U10 IS25LP128F-JBLE, U2 IS42S16320D-6BLI, U3 TLV62569DBV, U4 TLV62569DBV, U5 TLV62569DBV, Y1 FNETHE025

Commit message: Making all 3 DC/DC converters the same size and shape
Parts:
- moved R12 171.7 mm to (205.7, 55.5)
- moved R29 171.7 mm to (209.7, 58.0)
- moved R11 171.7 mm to (199.0, 60.2)
- moved R27 171.7 mm to (209.7, 60.4)
- moved R28 171.7 mm to (199.0, 57.9)
- moved R30 171.7 mm to (203.1, 55.5)
- moved U10 171.7 mm to (204.4, 59.0)
- moved RP2 151.2 mm to (195.7, 42.4), turned to 0 degrees
- moved RB2 150.8 mm to (192.5, 37.0), turned to 270 degrees
- moved C1 150.1 mm to (190.2, 36.2)
- moved L2 150.1 mm to (191.4, 43.0)
- moved U4 150.1 mm to (190.2, 39.2)
- moved C23 149.7 mm to (191.9, 45.5)
- moved C10 149.6 mm to (194.1, 36.4)
- moved RA2 149.6 mm to (194.1, 37.4)
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Routing:
- net GND: track 237.8 -> 225.6 mm, vias 57 -> 82
- net /power/P1V1: track 20.2 -> 11.5 mm
- net /power/FB1: track 10.7 -> 4.10 mm
- net /power/P3V3: track 16.6 -> 11.5 mm
- net /power/FB3: track 6.95 -> 4.10 mm
- net +5V: track 10.5 -> 8.28 mm, vias 1 -> 3
- net /power/FB2: track 5.28 -> 4.10 mm
- net +1V1: track 64.4 -> 65.5 mm, vias 6 -> 7
- net /power/P2V5: track 12.5 -> 11.5 mm
- net /power/PWREN: track 15.8 -> 16.6 mm, vias 1 -> 3
- net +3V3: track 47.5 -> 48.1 mm, vias 9 -> 10
- net +2V5: track 75.8 -> 75.7 mm, vias 8 -> 9

Commit message: Adding footprints
Parts:
- added J1: DF40C-100DP-0.4V(51), connectors:HRS_DF40C-100DP-0.4V(51), B.Cu at (140.4, 69.0)
- added J10: DF40C-100DP-0.4V(51), parts:HRS_DF40C-100DP-0.4V(51), B.Cu at (-75.2, 98.5)
- added J11: DF40C-100DP-0.4V(51), parts:HRS_DF40C-100DP-0.4V(51), B.Cu at (-91.2, 82.5)
- added J12: DF40C-100DP-0.4V(51), parts:HRS_DF40C-100DP-0.4V(51), B.Cu at (-59.2, 82.5)
- added J2: DF40C-100DP-0.4V(51), connectors:HRS_DF40C-100DP-0.4V(51), B.Cu at (140.4, 102.7)
- added J9: DF40C-100DP-0.4V(51), parts:HRS_DF40C-100DP-0.4V(51), B.Cu at (-75.2, 66.5)
- D1: value ORA -> ORANGE
- D2: value GRE -> GREEN
- D3: value BLU -> BLUE
- Y1: footprint oscxo:Crystal_SMD_7050_4Pads -> Crystal:Crystal_SMD_TXC_7M-4Pin_3.2x2.5mm
- moved H4 95.6 mm to (167.4, 102.9)
- moved C10 94.5 mm to (108.6, 76.7)
- moved C1 94.5 mm to (104.7, 76.5)
- moved C23 94.5 mm to (106.4, 85.8)
- moved RA2 94.5 mm to (108.6, 77.8)
- moved RB2 94.5 mm to (107.1, 77.3)
- moved RP2 94.5 mm to (110.2, 82.8)
- moved U4 94.5 mm to (104.7, 79.6)
- moved C11 94.5 mm to (108.6, 79.1)
- moved C12 94.5 mm to (108.6, 80.7)
- moved L2 94.5 mm to (106.0, 83.4)
- moved R12 86.4 mm to (130.2, 97.5)
- moved R30 86.4 mm to (127.6, 97.5)
- moved H3 78.8 mm to (118.3, 101.8)
- moved H2 63.8 mm to (167.4, 68.7)
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Routing:
- net (no net): track 783.3 -> 720.4 mm, vias 126 -> 125
- net 2V5_3V3: track 26.4 -> 12.9 mm, vias 5 -> 4
- net +3V3: track 48.1 -> 44.5 mm, vias 10 -> 9
- net LED1: track 5.52 -> 2.09 mm
- net CLK_25MHz: track 6.62 -> 4.61 mm
- net /usb/ANT_433MHz: track 5.12 -> 3.34 mm
- net BTN_PWRn: track 20.2 -> 19.7 mm
- net +2V5: track 75.7 -> 75.4 mm, vias 9 -> 8
Other:
- board size 82.9 x 50.8 mm -> 55.1 x 40 mm

Commit message: Adding labels
Parts:
- moved C34 202.3 mm to (35.3, 158.8)
- moved D28 202.3 mm to (33.2, 160.7)
- moved D29 202.3 mm to (33.2, 162.5)
- moved R31 202.3 mm to (36.1, 160.8)
- moved C2 183.4 mm to (55.0, 165.9)
- moved C22 183.4 mm to (52.7, 175.1)
- moved C3 183.4 mm to (54.9, 168.3)
- moved C4 183.4 mm to (54.9, 169.9)
- moved C5 183.4 mm to (51.0, 165.8)
- moved L1 183.4 mm to (52.3, 172.6)
- moved RA1 183.4 mm to (55.0, 167.0)
- moved RB1 183.4 mm to (53.4, 166.5)
- moved RP1 183.4 mm to (56.5, 172.0)
- moved U3 183.4 mm to (51.0, 168.8)
- moved D17 172.9 mm to (50.6, 148.5)
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
Commit message: Adding connectors
Parts:
- moved D0 1.69 mm to (104.8, 78.9)
- moved D1 1.69 mm to (106.5, 78.9)
- moved R41 1.69 mm to (104.6, 81.4)
- moved R42 1.69 mm to (106.3, 81.4)
- moved H3 1.10 mm to (146.2, 75.1)
Changed lines of the file:
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@@
   )
   (module Mounting_Holes:MountingHole_3.2mm_M3_ISO14580_Pad (layer F.Cu)
-    (at 146.213 76.221 180)
+    (at 146.213 75.12 180)
     (descr "Mounting Hole 3.2mm, M3, ISO14580")
     (tags "mounting hole 3.2mm m3 iso14580")
-    (fp_text reference H3 (at 0.025 -1.375) (layer F.SilkS) hide
+    (fp_text reference H3 (at 0.025 1.101) (layer F.SilkS) hide
       (effects (font (size 1 1) (thickness 0.15)))
     )
@@
   )
   (module LED_SMD:LED_0603_1608Metric (layer F.Cu)
-    (at 106.525 78.870001 270)
+    (at 104.830001 78.870001 270)
     (descr "LED SMD 0603 (1608 Metric), square (rectangular) end terminal, IPC_7351 nominal, (Body size source: http://www.tortai-tech.com/upload/download/2011102023233369053.pdf), generated with kicad-footprint-generator")
     (tags LED)
@@
   )
   (module LED_SMD:LED_0603_1608Metric (layer F.Cu)
-    (at 104.830001 78.870001 270)
+    (at 106.525 78.870001 270)
     (descr "LED SMD 0603 (1608 Metric), square (rectangular) end terminal, IPC_7351 nominal, (Body size source: http://www.tortai-tech.com/upload/download/2011102023233369053.pdf), generated with kicad-footprint-generator")
     (tags LED)
@@
   )
   (module Capacitor_SMD:C_0402_1005Metric (layer F.Cu)
-    (at 106.255001 81.37 90)
+    (at 104.565 81.37 90)
     (descr "Capacitor SMD 0402 (1005 Metric), square (rectangular) end terminal, IPC_7351 nominal, (Body size source: IPC-SM-782 page 76, https://www.pcb-3d.com/wordpress/wp-content/uploads/ipc-sm-782a_amendment_1_and_2.pdf), generated with kicad-footprint-generator")
     (tags capacitor)
@@
   )
   (module Capacitor_SMD:C_0402_1005Metric (layer F.Cu)
-    (at 104.565 81.369999 90)
+    (at 106.255001 81.369999 90)
     (descr "Capacitor SMD 0402 (1005 Metric), square (rectangular) end terminal, IPC_7351 nominal, (Body size source: IPC-SM-782 page 76, https://www.pcb-3d.com/wordpress/wp-content/uploads/ipc-sm-782a_amendment_1_and_2.pdf), generated with kicad-footprint-generator")
     (tags capacitor)
@@
   (gr_circle (center 97.113 75.12) (end 94.913 75.12) (layer F.Fab) (width 0.2))
   (gr_circle (center 97.113 75.12) (end 94.913 75.12) (layer B.Fab) (width 0.2))
-  (gr_circle (center 146.213 76.281) (end 144.013 76.281) (layer B.Fab) (width 0.2))
-  (gr_circle (center 146.212999 76.181) (end 144.012999 76.181) (layer F.Fab) (width 0.2))
+  (gr_circle (center 146.213 75.12) (end 148.413 75.12) (layer B.Fab) (width 0.2))
+  (gr_circle (center 146.212999 75.12) (end 148.412999 75.12) (layer F.Fab) (width 0.2))
   (gr_circle (center 97.073 109.295) (end 94.873 109.295) (layer F.Fab) (width 0.2))
   (gr_circle (center 97.073 109.295) (end 94.873 109.295) (layer B.Fab) (width 0.2))

Commit message: Before power placement
Parts:
- removed HR: HR, hrvatski_proizvod_veci:hrvatski
- removed J5: VJ1, Connector_PinHeader_2.54mm:PinHeader_1x03_P2.54mm_Vertical
- added C13: 100n, Capacitor_SMD:C_0402_1005Metric, F.Cu at (127.9, 78.4)
- added C14: 100n, Capacitor_SMD:C_0402_1005Metric, F.Cu at (128.9, 78.4)
- added C15: 100n, Capacitor_SMD:C_0402_1005Metric, F.Cu at (129.9, 78.4)
- added C18: 100n, Capacitor_SMD:C_0402_1005Metric, F.Cu at (130.9, 78.4)
- added C21: 100n, Capacitor_SMD:C_0402_1005Metric, F.Cu at (131.9, 78.4)
- added C36: 100n, Capacitor_SMD:C_0402_1005Metric, F.Cu at (132.9, 78.4)
- added C37: 100n, Capacitor_SMD:C_0402_1005Metric, F.Cu at (133.9, 78.4)
- added C38: 100n, Capacitor_SMD:C_0402_1005Metric, F.Cu at (134.9, 78.4)
- added C39: 100n, Capacitor_SMD:C_0402_1005Metric, F.Cu at (119.9, 78.4)
- added C40: 100n, Capacitor_SMD:C_0402_1005Metric, F.Cu at (120.9, 78.4)
- added C41: 100n, Capacitor_SMD:C_0402_1005Metric, F.Cu at (121.9, 78.4)
- added C42: 100n, Capacitor_SMD:C_0402_1005Metric, F.Cu at (122.9, 78.4)
- added C43: 100n, Capacitor_SMD:C_0402_1005Metric, F.Cu at (123.9, 78.4)
- added C44: 100n, Capacitor_SMD:C_0402_1005Metric, F.Cu at (124.9, 78.4)
- added C45: 100n, Capacitor_SMD:C_0402_1005Metric, F.Cu at (125.9, 78.4)
- added C54: 100n, Capacitor_SMD:C_0402_1005Metric, F.Cu at (126.9, 78.4)
- added C55: 22n, Capacitor_SMD:C_0402_1005Metric, F.Cu at (91.1, 96.6)
- added C56: 22n, Capacitor_SMD:C_0402_1005Metric, F.Cu at (117.1, 132.3)
- added C57: 22n, Capacitor_SMD:C_0402_1005Metric, F.Cu at (121.5, 132.2)
- added C58: 22n, Capacitor_SMD:C_0402_1005Metric, F.Cu at (129.1, 132.4)
- added C59: 22n, Capacitor_SMD:C_0402_1005Metric, F.Cu at (91.1, 94.6)
- added C61: 22n, Capacitor_SMD:C_0402_1005Metric, F.Cu at (91.1, 98.7)
- added C62: 22n, Capacitor_SMD:C_0402_1005Metric, F.Cu at (115.0, 132.3)
- added C63: 22n, Capacitor_SMD:C_0402_1005Metric, F.Cu at (131.3, 132.4)
- added C64: 22n, Capacitor_SMD:C_0402_1005Metric, F.Cu at (123.8, 132.3)
- added C65: 22n, Capacitor_SMD:C_0402_1005Metric, F.Cu at (127.1, 132.4)
- added C66: 22n, Capacitor_SMD:C_0402_1005Metric, F.Cu at (91.1, 93.6)
- added C67: 22n, Capacitor_SMD:C_0402_1005Metric, F.Cu at (91.1, 97.7)
- added C68: 22n, Capacitor_SMD:C_0402_1005Metric, F.Cu at (116.1, 132.3)
- added C69: 22n, Capacitor_SMD:C_0402_1005Metric, F.Cu at (132.2, 132.4)
- added C70: 22n, Capacitor_SMD:C_0402_1005Metric, F.Cu at (124.8, 132.3)
- added C71: 22n, Capacitor_SMD:C_0402_1005Metric, F.Cu at (128.1, 132.4)
- added C72: 22n, Capacitor_SMD:C_0402_1005Metric, F.Cu at (91.1, 95.6)
- added C73: 22n, Capacitor_SMD:C_0402_1005Metric, F.Cu at (118.1, 132.3)
- added C74: 22n, Capacitor_SMD:C_0402_1005Metric, F.Cu at (122.5, 132.2)
- added C75: 22n, Capacitor_SMD:C_0402_1005Metric, F.Cu at (130.2, 132.4)
- added D4: 1N914, Diode_SMD:D_SOD-323, B.Cu at (108.6, 76.0)
- added D5: 1N914, Diode_SMD:D_SOD-323, B.Cu at (108.6, 78.0)
- added D6: 1N914, Diode_SMD:D_SOD-323, B.Cu at (110.2, 80.6)
- added D7: 1N914, Diode_SMD:D_SOD-323, B.Cu at (108.2, 80.6)
- added J3: JTAG, Connector_PinSocket_2.54mm:PinSocket_2x03_P2.54mm_Vertical, F.Cu at (100.0, 102.4)
- added R1: 27, Resistor_SMD:R_0402_1005Metric, B.Cu at (111.2, 76.4)
- added R10: 4K7, Resistor_SMD:R_0402_1005Metric, B.Cu at (123.3, 79.0)
- added R13: 4K7, Resistor_SMD:R_0402_1005Metric, B.Cu at (122.1, 79.0)
- added R14: 4K7, Resistor_SMD:R_0402_1005Metric, F.Cu at (136.2, 73.8)
- added R15: 4K7, Resistor_SMD:R_0402_1005Metric, F.Cu at (136.2, 76.8)
- added R16: 100K, Resistor_SMD:R_0402_1005Metric, B.Cu at (124.4, 79.0)
- added R17: 100K, Resistor_SMD:R_0402_1005Metric, B.Cu at (121.1, 79.0)
- added R2: 27, Resistor_SMD:R_0402_1005Metric, B.Cu at (111.2, 75.4)
- added R4: 1.1K, Resistor_SMD:R_0402_1005Metric, B.Cu at (109.2, 74.5)
- added R5: 15K, Resistor_SMD:R_0402_1005Metric, B.Cu at (111.3, 77.5)
- added R6: 1.1K, Resistor_SMD:R_0402_1005Metric, B.Cu at (111.8, 80.0)
- added R7: 15K, Resistor_SMD:R_0402_1005Metric, B.Cu at (111.3, 78.5)
- added R8: 100K, Resistor_SMD:R_0402_1005Metric, B.Cu at (125.4, 79.0)
- added R9: 100K, Resistor_SMD:R_0402_1005Metric, B.Cu at (126.5, 79.0)
- C49: moved to F.Cu
- D17, D28, D29: footprint Diode_SMD:D_SOD-323_HandSoldering -> Diode_SMD:D_SOD-323
- moved C49 163.0 mm to (113.2, 75.5), turned to 90 degrees
- moved C48 160.0 mm to (105.4, 76.6), turned to 180 degrees
- moved L1 126.3 mm to (111.0, 60.7)
- moved RA1 126.3 mm to (113.6, 55.1)
- moved RP1 126.3 mm to (115.2, 60.1)
- moved C4 126.3 mm to (113.6, 58.1)
- moved C5 126.3 mm to (109.7, 53.9)
- moved U3 126.3 mm to (109.7, 56.9)
- moved C2 126.3 mm to (113.6, 54.1)
- moved C22 126.3 mm to (111.4, 63.2)
- moved C3 126.3 mm to (113.5, 56.4)
- moved RB1 126.3 mm to (112.1, 54.7)
- moved C1 125.4 mm to (128.8, 50.7)
- moved C12 125.4 mm to (132.6, 54.8)
- moved C23 125.4 mm to (130.5, 59.9)
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Connections:
- J1 pad 1: (no net) -> GND
- J1 pad 13: (no net) -> GND
- J1 pad 14: (no net) -> GND
- J1 pad 2: (no net) -> GND
- J1 pad 22: (no net) -> GND
- J1 pad 23: (no net) -> GND
- J1 pad 32: (no net) -> GND
- J1 pad 33: (no net) -> GND
- J1 pad 42: (no net) -> GND
- J1 pad 43: (no net) -> GND
- J1 pad 52: (no net) -> GND
- J1 pad 53: (no net) -> GND
- J1 pad 57: (no net) -> SD_CLK
- J1 pad 59: (no net) -> GND
- J1 pad 60: (no net) -> GND
- J1 pad 61: (no net) -> SD_D3
- J1 pad 62: (no net) -> SD_CMD
- J1 pad 63: (no net) -> SD_D0
- J1 pad 65: (no net) -> GND
- J1 pad 66: (no net) -> GND
- J1 pad 67: (no net) -> SD_D1
- J1 pad 69: (no net) -> SD_D2
- J1 pad 7: (no net) -> GND
- J1 pad 71: (no net) -> GND
- J1 pad 74: (no net) -> GND
- J1 pad 76: (no net) -> Reserved
- J1 pad 77: (no net) -> +5V
- J1 pad 79: (no net) -> +5V
- J1 pad 8: (no net) -> GND
- J1 pad 81: (no net) -> +5V
- J1 pad 83: (no net) -> +5V
- J1 pad 84: (no net) -> CM4_3.3V
- J1 pad 85: (no net) -> +5V
- J1 pad 86: (no net) -> CM4_3.3V
- J1 pad 87: (no net) -> +5V
- J1 pad 88: (no net) -> CM4_1.8V
- J1 pad 90: (no net) -> CM4_1.8V
- J1 pad 98: (no net) -> GND
- J2 pad 10: (no net) -> PCIe_CLK_P
- J2 pad 100: (no net) -> HDMI0_SCL
- J2 pad 12: (no net) -> PCIe_CLK_N
- J2 pad 13: (no net) -> GND
- J2 pad 14: (no net) -> GND
- J2 pad 16: (no net) -> PCIe_RX_P
- J2 pad 18: (no net) -> PCIe_RX_N
- J2 pad 19: (no net) -> GND
- J2 pad 20: (no net) -> GND
- J2 pad 22: (no net) -> PCIe_TX_P
- J2 pad 24: (no net) -> PCIe_TX_N
- J2 pad 25: (no net) -> GND
- J2 pad 26: (no net) -> GND
- J2 pad 3: (no net) -> USB_N
- J2 pad 31: (no net) -> GND
- J2 pad 32: (no net) -> GND
- J2 pad 37: (no net) -> GND
- J2 pad 38: (no net) -> GND
- J2 pad 4: (no net) -> Reserved
- J2 pad 43: (no net) -> HDMI1_HOTPLUG
- J2 pad 44: (no net) -> GND
- J2 pad 45: (no net) -> HDMI1_SDA
- J2 pad 46: (no net) -> HDMI1_TX2_P
- J2 pad 47: (no net) -> HDMI1_SCL
- J2 pad 48: (no net) -> HDMI1_TX2_N
- J2 pad 49: (no net) -> HDMI1_CEC
- J2 pad 5: (no net) -> USB_P
- J2 pad 50: (no net) -> GND
- J2 pad 51: (no net) -> HDMI0_CEC
- J2 pad 52: (no net) -> HDMI1_TX1_P
- J2 pad 53: (no net) -> HDMI0_HOTPLUG
- J2 pad 54: (no net) -> HDMI1_TX1_N
- J2 pad 55: (no net) -> GND
- J2 pad 56: (no net) -> GND
- J2 pad 58: (no net) -> HDMI1_TX0_P
- J2 pad 6: (no net) -> Reserved
- J2 pad 60: (no net) -> HDMI1_TX0_N
- J2 pad 61: (no net) -> GND
- J2 pad 62: (no net) -> GND
- J2 pad 64: (no net) -> HDMI1_CLK_P
- J2 pad 66: (no net) -> HDMI1_CLK_N
- J2 pad 67: (no net) -> GND
- J2 pad 68: (no net) -> GND
- J2 pad 7: (no net) -> GND
- J2 pad 70: (no net) -> HDMI0_TX2_P
- J2 pad 72: (no net) -> HDMI0_TX2_N
- J2 pad 73: (no net) -> GND
- J2 pad 74: (no net) -> GND
- J2 pad 76: (no net) -> HDMI0_TX1_P
- J2 pad 78: (no net) -> HDMI0_TX1_N
- J2 pad 79: (no net) -> GND
- J2 pad 8: (no net) -> GND
- J2 pad 80: (no net) -> GND
- J2 pad 82: (no net) -> HDMI0_TX0_P
- J2 pad 84: (no net) -> HDMI0_TX0_N
- J2 pad 85: (no net) -> GND
- J2 pad 86: (no net) -> GND
- J2 pad 88: (no net) -> HDMI0_CLK_P
- J2 pad 90: (no net) -> HDMI0_CLK_N
- J2 pad 91: (no net) -> GND
- J2 pad 92: (no net) -> GND
- J2 pad 97: (no net) -> GND
- J2 pad 98: (no net) -> GND
- J2 pad 99: (no net) -> HDMI0_SDA
- U1 pad A12: (no net) -> FPDI_D2+
- U1 pad A13: (no net) -> FPDI_D2-
- U1 pad A14: (no net) -> FPDI_D1+
- U1 pad A16: (no net) -> FPDI_D0+
- U1 pad A17: (no net) -> FPDI_CLK+
- U1 pad A7: (no net) -> GP4
- U1 pad A8: (no net) -> GN4
- U1 pad B11: (no net) -> GP0
- U1 pad B12: (no net) -> USB_FPGA_PULL_D+
- U1 pad B16: (no net) -> FPDI_D0-
- U1 pad B18: (no net) -> FPDI_CLK-
- U1 pad B8: (no net) -> GN5
- U1 pad B9: (no net) -> GP3
- U1 pad C10: (no net) -> GN3
- U1 pad C11: (no net) -> GN0
- U1 pad C12: (no net) -> USB_FPGA_PULL_D-
- U1 pad C14: (no net) -> FPDI_D1-
- U1 pad C8: (no net) -> GP5
- U1 pad H1: (no net) -> SD_D1
- U1 pad H2: (no net) -> SD_CLK
- U1 pad J1: (no net) -> SD_CMD
- U1 pad J3: (no net) -> SD_D0
- U1 pad K1: (no net) -> SD_D2
- U1 pad K2: (no net) -> SD_D3
- U1 pad R5: (no net) -> JTAG_TDI
- U1 pad T5: (no net) -> JTAG_TCK
- U1 pad U5: (no net) -> JTAG_TMS
- U1 pad V4: (no net) -> JTAG_TDO
- U1 pad W13: (no net) -> /serdes/S_6_P
- U1 pad W14: (no net) -> /serdes/S_6_N
- U1 pad W17: (no net) -> /serdes/S_7_P
- U1 pad W18: (no net) -> /serdes/S_7_N
- U1 pad W20: (no net) -> /serdes/CLK_1_N
- U1 pad W4: (no net) -> /serdes/S_2_P
- U1 pad W5: (no net) -> /serdes/S_2_N
- U1 pad W8: (no net) -> /serdes/S_3_P
- U1 pad W9: (no net) -> /serdes/S_3_N
- U1 pad Y11: (no net) -> /serdes/CLK_0_P
- U1 pad Y12: (no net) -> /serdes/CLK_0_N
- U1 pad Y14: (no net) -> /serdes/S_4_P
- U1 pad Y15: (no net) -> /serdes/S_4_N
- U1 pad Y16: (no net) -> /serdes/S_5_P
- U1 pad Y17: (no net) -> /serdes/S_5_N
- U1 pad Y19: (no net) -> /serdes/CLK_1_P
- U1 pad Y5: (no net) -> /serdes/S_0_P
- U1 pad Y6: (no net) -> /serdes/S_0_N
- U1 pad Y7: (no net) -> /serdes/S_1_P
- U1 pad Y8: (no net) -> /serdes/S_1_N
Routing:
- net (no net): track 720.4 -> 543.1 mm, vias 125 -> 105
- net GN3: track 0.00 -> 9.28 mm, vias 0 -> 1
- net SDRAM_D11: track 5.72 -> 14.9 mm
- net BTN_PWRn: track 19.7 -> 11.1 mm
- net SDRAM_DQM0: track 7.37 -> 15.9 mm
- net GP0: track 0.00 -> 8.29 mm, vias 0 -> 1
- net SDRAM_D7: track 6.40 -> 14.5 mm
- net GN5: track 0.00 -> 7.59 mm, vias 0 -> 1
- net GP5: track 0.00 -> 7.49 mm, vias 0 -> 2
- net USB_FPGA_PULL_D-: track 0.00 -> 7.37 mm, vias 0 -> 2
- net GN4: track 0.00 -> 7.33 mm, vias 0 -> 1
- net GP4: track 0.00 -> 7.11 mm, vias 0 -> 1
- net SDRAM_A5: track 5.36 -> 12.5 mm
- net USB_FPGA_PULL_D+: track 0.00 -> 7.03 mm, vias 0 -> 1
- net HDMI1_TX2_N: track 0.00 -> 6.89 mm, vias 0 -> 1
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Other:
- board text added: "v0.0.1"
- board text removed: "3V 12.5x2.5mm"
- board text removed: "KEYSTONE 3000"
- board text removed: "RS232"
- board text removed: "U8"
- board text removed: "skriptarnica.hr"
- board text removed: "v3.1.7"

Commit message: Routing
Parts:
- C56, C57, C58, C62, C63, C64, C65, C68, C69, C70, C71, C73, C74, C75: moved to B.Cu
- moved C5 62.4 mm to (141.6, 107.5), turned to 180 degrees
- moved RB1 58.7 mm to (139.2, 106.8), turned to 90 degrees
- moved C2 58.5 mm to (137.7, 107.4), turned to 0 degrees
- moved U3 57.3 mm to (141.6, 104.5), turned to 0 degrees
- moved RA1 56.6 mm to (137.6, 106.3), turned to 0 degrees
- moved C3 54.2 mm to (137.7, 105.0), turned to 0 degrees
- moved C4 51.3 mm to (137.7, 103.4), turned to 0 degrees
- moved L1 49.6 mm to (140.3, 100.7), turned to 180 degrees
- moved RP1 46.2 mm to (136.1, 101.3), turned to 180 degrees
- moved C22 45.2 mm to (139.9, 98.2), turned to 0 degrees
- moved C23 41.7 mm to (99.9, 88.4)
- moved C11 41.7 mm to (102.1, 81.6)
- moved RP2 41.7 mm to (103.7, 85.3)
- moved U4 41.7 mm to (98.2, 82.1)
- moved C1 41.7 mm to (98.2, 79.1)
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Routing:
- net +5V: track 8.28 -> 110.6 mm, vias 3 -> 6
- net (no net): track 543.1 -> 495.3 mm, vias 105 -> 93
- net SD_D1: track 3.20 -> 46.6 mm, vias 0 -> 1
- net SD_D2: track 4.58 -> 47.1 mm, vias 0 -> 1
- net SD_CLK: track 4.33 -> 45.9 mm, vias 0 -> 1
- net SD_D0: track 4.70 -> 45.8 mm, vias 1 -> 3
- net SD_CMD: track 2.96 -> 43.1 mm, vias 0 -> 1
- net SD_D3: track 3.85 -> 43.3 mm, vias 0 -> 1
- net /serdes/CLK_0_N: track 0.00 -> 31.3 mm, vias 0 -> 2
- net /serdes/CLK_0_P: track 0.00 -> 29.8 mm, vias 0 -> 2
- net /flash/FLASH_MOSI: track 4.67 -> 31.0 mm, vias 1 -> 2
- net JTAG_TMS: track 5.37 -> 31.7 mm, vias 1 -> 2
- net /flash/FLASH_SCK: track 5.57 -> 31.6 mm, vias 1 -> 2
- net /serdes/S_0_N: track 0.00 -> 24.0 mm, vias 0 -> 2
- net /serdes/S_0_P: track 0.00 -> 22.8 mm, vias 0 -> 2
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
Commit message: Routing
Parts:
- C60: moved to B.Cu
- R32, R33: moved to F.Cu
- moved D29 138.3 mm to (146.0, 92.4), turned to 90 degrees
- moved D28 135.5 mm to (144.0, 92.4), turned to 90 degrees
- moved C60 126.8 mm to (144.0, 94.5)
- moved R31 126.4 mm to (145.9, 94.6), turned to 0 degrees
- moved C34 115.5 mm to (135.7, 90.4), turned to 0 degrees
- moved R3 108.0 mm to (142.1, 94.5), turned to 0 degrees
- moved D17 107.3 mm to (142.0, 92.4), turned to 90 degrees
- moved EMARD 91.8 mm to (74.3, 137.8)
- moved C33 79.7 mm to (136.5, 88.8)
- moved fer 77.1 mm to (78.1, 156.3)
- moved C16 76.6 mm to (134.1, 89.1), turned to 180 degrees
- moved C35 74.0 mm to (133.8, 90.4), turned to 0 degrees
- moved C52 71.5 mm to (132.3, 94.5), turned to 0 degrees
- moved koncar 63.2 mm to (62.3, 156.4)
- moved R32 58.6 mm to (96.4, 99.1), turned to 315 degrees
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Connections:
- J1 pad 76: Reserved -> (no net)
- J2 pad 4: Reserved -> (no net)
- J2 pad 6: Reserved -> (no net)
Routing:
- net (no net): track 495.3 -> 448.1 mm, vias 93 -> 88
- net GP4: track 7.11 -> 13.9 mm
- net GN4: track 7.33 -> 14.1 mm
- net GP5: track 7.49 -> 13.5 mm, vias 2 -> 3
- net GN5: track 7.59 -> 13.3 mm, vias 1 -> 2
- net GP3: track 7.97 -> 2.76 mm, vias 1 -> 0
- net GN3: track 9.28 -> 5.01 mm
- net GN0: track 9.14 -> 4.89 mm
- net GP0: track 8.29 -> 4.38 mm
- net FPDI_D2-: track 3.79 -> 2.68 mm
- net USB_FPGA_PULL_D-: track 7.37 -> 6.43 mm
- net USB_FPGA_PULL_D+: track 7.03 -> 6.14 mm
Other:
- board text added: "ULX4M"
- board text removed: "ULX3S"

Commit message: SDRAM routed
Parts:
- moved R41 5.12 mm to (109.7, 81.3)
- moved D0 5.10 mm to (109.9, 78.8)
- moved R44 5.09 mm to (104.6, 81.4)
- moved D3 5.07 mm to (104.9, 78.9)
- moved Y1 1.85 mm to (106.3, 91.2)
- moved R42 1.71 mm to (108.0, 81.4)
- moved R43 1.70 mm to (106.3, 81.4)
- moved D1 1.70 mm to (108.2, 78.9)
- moved D2 1.69 mm to (106.5, 78.9)
- moved C35 0.49 mm to (133.4, 90.6)
- moved C34 0.23 mm to (135.7, 90.6)
- moved C16 0.23 mm to (134.1, 89.3)
- moved C33 0.20 mm to (136.6, 89.0)
Connections:
- U1 pad C20: SDRAM_D11 -> SDRAM_A9
- U1 pad D19: SDRAM_D10 -> SDRAM_DQM1
- U1 pad D20: SDRAM_D9 -> SDRAM_A11
- U1 pad E18: SDRAM_D12 -> SDRAM_A12
- U1 pad E19: SDRAM_D8 -> SDRAM_A6
- U1 pad E20: SDRAM_DQM1 -> SDRAM_A8
- U1 pad F18: SDRAM_D13 -> SDRAM_A5
- U1 pad F19: SDRAM_CLK -> SDRAM_A7
- U1 pad F20: SDRAM_CKE -> SDRAM_A4
- U1 pad G19: SDRAM_A12 -> SDRAM_CLK
- U1 pad G20: SDRAM_A11 -> SDRAM_CKE
- U1 pad H20: SDRAM_A9 -> SDRAM_D8
- U1 pad J16: SDRAM_D0 -> SDRAM_D13
- U1 pad J18: SDRAM_D14 -> SDRAM_D11
- U1 pad J19: SDRAM_A8 -> SDRAM_D9
- U1 pad J20: SDRAM_A7 -> SDRAM_D12
- U1 pad K18: SDRAM_A6 -> SDRAM_D10
- U1 pad K19: SDRAM_A5 -> SDRAM_D14
- U1 pad K20: SDRAM_A4 -> SDRAM_A3
- U1 pad L18: SDRAM_D1 -> SDRAM_BA0
- U1 pad L19: SDRAM_A3 -> SDRAM_A0
- U1 pad L20: SDRAM_A2 -> SDRAM_A1
- U1 pad M18: SDRAM_D2 -> SDRAM_nRAS
- U1 pad M19: SDRAM_A1 -> SDRAM_A2
- U1 pad M20: SDRAM_A0 -> SDRAM_BA1
- U1 pad N18: SDRAM_D3 -> SDRAM_nCAS
- U1 pad N20: SDRAM_BA1 -> SDRAM_nWE
- U1 pad P18: SDRAM_D4 -> SDRAM_nCS
- U1 pad P19: SDRAM_BA0 -> SDRAM_D7
- U1 pad P20: SDRAM_nCS -> SDRAM_DQM0
- U1 pad R20: SDRAM_nRAS -> SDRAM_D6
- U1 pad T17: SDRAM_D6 -> SDRAM_D5
- U1 pad T18: SDRAM_D5 -> SDRAM_D4
- U1 pad T19: SDRAM_nCAS -> SDRAM_D3
- U1 pad T20: SDRAM_nWE -> SDRAM_D1
- U1 pad U19: SDRAM_DQM0 -> SDRAM_D2
- U1 pad U20: SDRAM_D7 -> SDRAM_D0
Routing:
- net (no net): track 448.1 -> 134.8 mm, vias 88 -> 23
- net PCIe_CLK_N: track 0.00 -> 31.0 mm, vias 0 -> 2
- net PCIe_CLK_P: track 0.00 -> 30.2 mm, vias 0 -> 2
- net PCIe_TX_N: track 0.00 -> 30.2 mm, vias 0 -> 2
- net PCIe_RX_N: track 0.00 -> 30.2 mm, vias 0 -> 2
- net PCIe_RX_P: track 0.00 -> 29.7 mm, vias 0 -> 2
- net PCIe_TX_P: track 0.00 -> 29.2 mm, vias 0 -> 2
- net SDRAM_D15: track 11.0 -> 25.5 mm
- net GN15: track 13.2 -> 0.00 mm, vias 2 -> 0
- net GP15: track 12.2 -> 0.00 mm, vias 2 -> 0
- net FPDI_D2-: track 2.68 -> 14.2 mm
- net SDRAM_D10: track 4.94 -> 16.4 mm
- net SDRAM_A9: track 1.60 -> 12.9 mm
- net FPDI_CLK-: track 4.72 -> 15.8 mm
- net SDRAM_D13: track 9.40 -> 20.4 mm
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