File: ulx3s.kicad_pcb (KiCad board)
At the start: 4 copper layers, 55.1 x 40 mm, 151 parts, among them J1 DF40C-100DP-0.4V(51), J10 DF40C-100DP-0.4V(51), J11 DF40C-100DP-0.4V(51), J12 DF40C-100DP-0.4V(51), J2 DF40C-100DP-0.4V(51), J3 JTAG, J9 DF40C-100DP-0.4V(51), U1 LFE5U-85F-6BG381C, U10 IS25LP128F-JBLE, U2 IS42S16320D-6BLI, U3 TLV62569DBV, U4 TLV62569DBV, U5 TLV62569DBV, Y1 FNETHE025

Commit message: SDRAM, JTAG routed - before logo delete
Parts:
- moved R31 8.01 mm to (138.6, 91.2)
- moved R27 1.58 mm to (121.5, 108.6)
Connections:
- J1 pad 25: (no net) -> GPIO21
- J1 pad 27: (no net) -> GPIO20
- J1 pad 29: (no net) -> GPIO16
- J1 pad 31: (no net) -> GPIO12
- J3 pad 3: JTAG_TDI -> GPIO12
- J3 pad 4: JTAG_TCK -> GPIO20
- J3 pad 5: JTAG_TMS -> GPIO21
- J3 pad 6: JTAG_TDO -> GPIO16
- U1 pad A2: (no net) -> USB_FPGA_PULL_D+
- U1 pad A3: (no net) -> USB_FPGA_PULL_D-
- U1 pad B12: USB_FPGA_PULL_D+ -> (no net)
- U1 pad C12: USB_FPGA_PULL_D- -> (no net)
- U1 pad D6: BTN_PWRn -> (no net)
- U1 pad R5: JTAG_TDI -> GPIO12
- U1 pad T5: JTAG_TCK -> GPIO20
- U1 pad U18: (no net) -> BTN_PWRn
- U1 pad U5: JTAG_TMS -> GPIO21
- U1 pad V4: JTAG_TDO -> GPIO16
Routing:
- net +3V3: track 54.8 -> 150.6 mm, vias 19 -> 29
- net +5V: track 110.6 -> 172.2 mm, vias 6 -> 9
- net GPIO21: track 0.00 -> 52.3 mm, vias 0 -> 3
- net GPIO12: track 0.00 -> 47.8 mm, vias 0 -> 2
- net GPIO16: track 0.00 -> 44.6 mm, vias 0 -> 2
- net GPIO20: track 0.00 -> 42.4 mm, vias 0 -> 2
- net 2V5_3V3: track 14.6 -> 46.3 mm, vias 4 -> 5
- net JTAG_TMS: track 31.7 -> 0.00 mm, vias 2 -> 0
- net /flash/FPGA_PROGRAMN: track 26.8 -> 50.0 mm
- net JTAG_TDO: track 22.1 -> 0.00 mm, vias 1 -> 0
- net JTAG_TCK: track 19.9 -> 0.00 mm, vias 1 -> 0
- net USER_PROGRAMN: track 28.7 -> 47.1 mm
- net JTAG_TDI: track 17.7 -> 0.00 mm, vias 1 -> 0
- net USB_FPGA_D+: track 13.7 -> 27.9 mm, vias 2 -> 3
- net USB_FPGA_D-: track 11.7 -> 24.1 mm, vias 2 -> 3
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- added copper zone on B.Cu, net GND

Commit message: before graphics
Parts:
- removed EMARD (x2): emard12mm, emard:emard12mm
- removed J10, J11, J12, J9: DF40C-100DP-0.4V(51), parts:HRS_DF40C-100DP-0.4V(51)
- removed fer: fer, fer:fer4mm6
- removed koncar: koncar, koncar:koncar
Other:
- board text removed: "F2"
- board text removed: "KEEP PCB HERE USE PANEL MILL ONLY"
- board text removed: "KEEP STENCIL HERE IGNORE THIS RECTANGLE CUT"
- board text removed: "PANEL MILL"
- board text removed: "PWR"

Commit message: Graphic removed
Routing:
- net (no net): track 127.6 -> 0.00 mm, vias 22 -> 0
- net OLED_BL: track 8.07 -> 0.00 mm, vias 2 -> 0
- net GND: track 227.0 -> 221.8 mm
- net +3V3: track 150.6 -> 151.5 mm, vias 29 -> 30
- net +2V5: track 80.9 -> 80.4 mm
- net GPIO12: track 47.8 -> 47.3 mm
Other:
- board text added: "1.1V"

Commit message: Cleaning DRC errors
Parts:
- moved RV2 0.12 mm to (106.0, 74.9)
Connections:
- U3 pad 1: /power/PWREN -> +5V
- U4 pad 1: /power/PWREN -> +5V
- U5 pad 1: /power/PWREN -> +5V
Routing:
- net +5V: track 172.5 -> 199.3 mm, vias 9 -> 12
- net /power/PWREN: track 16.6 -> 0.00 mm, vias 3 -> 0
- net +2V5: track 80.4 -> 81.5 mm, vias 11 -> 10

Commit message: Adding few text labels
Parts:
- moved C53 12.9 mm to (102.4, 75.5), turned to 270 degrees
- moved R14 4.65 mm to (137.2, 78.4), turned to 90 degrees
- moved R15 1.61 mm to (136.2, 78.4), turned to 90 degrees
Routing:
- net 2V5_3V3: track 46.6 -> 50.2 mm
- net HDMI0_SCL: track 3.07 -> 6.20 mm
- net +5V: track 199.3 -> 200.7 mm, vias 12 -> 11
- net HDMI0_SDA: track 3.07 -> 4.37 mm
- net GND: track 221.9 -> 221.1 mm
Other:
- board text added: "25MHz"
- board text added: "GPDI0"
- board text added: "GPDI1"
- board text added: "PCIe"
- board text added: "SERDES"

Commit message: Routing cam and display differential
Parts:
- moved R9 0.63 mm to (126.0, 79.4)
- moved R8 0.57 mm to (125.0, 79.4)
- moved R16 0.52 mm to (124.0, 79.4)
- moved R10 0.46 mm to (123.0, 79.4)
- moved R13 0.37 mm to (122.0, 79.4)
- moved R17 0.35 mm to (121.0, 79.4)
Connections:
- J2 pad 2: (no net) -> PCIe_CLK_nREQ
- J2 pad 28: (no net) -> CAM0_D0_N
- J2 pad 30: (no net) -> CAM0_D0_P
- J2 pad 34: (no net) -> CAM0_D1_N
- J2 pad 36: (no net) -> CAM0_D1_P
- J2 pad 40: (no net) -> CAM0_C_N
- J2 pad 42: (no net) -> CAM0_C_P
- J2 pad 57: (no net) -> DSI0_D0_N
- J2 pad 59: (no net) -> DSI0_D0_P
- J2 pad 63: (no net) -> DSI0_D1_N
- J2 pad 65: (no net) -> DSI0_D1_P
- J2 pad 69: (no net) -> DSI0_C_N
- J2 pad 71: (no net) -> DSI0_C_P
- J2 pad 9: (no net) -> PCIe_nRST
- U1 pad A12: FPDI_D2+ -> CAM0_D0_P
- U1 pad A13: FPDI_D2- -> CAM0_D0_N
- U1 pad A14: FPDI_D1+ -> DSI0_D1_P
- U1 pad A16: FPDI_D0+ -> (no net)
- U1 pad A17: FPDI_CLK+ -> (no net)
- U1 pad A9: (no net) -> PCIe_CLK_nREQ
- U1 pad B12: (no net) -> CAM0_C_P
- U1 pad B13: (no net) -> CAM0_D1_P
- U1 pad B16: FPDI_D0- -> (no net)
- U1 pad B18: FPDI_CLK- -> (no net)
- U1 pad C12: (no net) -> CAM0_C_N
- U1 pad C13: (no net) -> CAM0_D1_N
- U1 pad C14: FPDI_D1- -> DSI0_D1_N
- U1 pad C18: (no net) -> FPDI_D2+
- U1 pad D12: (no net) -> DSI0_C_P
- U1 pad D13: (no net) -> DSI0_D0_P
- U1 pad D17: (no net) -> FPDI_D2-
- U1 pad D18: (no net) -> FPDI_D1+
- U1 pad D9: (no net) -> PCIe_nRST
- U1 pad E12: (no net) -> DSI0_C_N
- U1 pad E13: (no net) -> DSI0_D0_N
- U1 pad E17: (no net) -> FPDI_D1-
- U1 pad F17: (no net) -> FPDI_D0+
- U1 pad G18: (no net) -> FPDI_D0-
- U1 pad H17: (no net) -> SDRAM_A3
- U1 pad H18: (no net) -> SDRAM_D12
- U1 pad J20: SDRAM_D12 -> FPDI_CLK+
- U1 pad K20: SDRAM_A3 -> FPDI_CLK-
Routing:
- net DSI0_C_N: track 0.00 -> 23.5 mm, vias 0 -> 2
- net DSI0_C_P: track 0.00 -> 22.0 mm, vias 0 -> 2
- net CAM0_D1_N: track 0.00 -> 20.7 mm, vias 0 -> 3
- net CAM0_C_N: track 0.00 -> 19.7 mm, vias 0 -> 2
- net DSI0_D1_N: track 0.00 -> 19.3 mm, vias 0 -> 2
- net CAM0_D0_P: track 0.00 -> 19.2 mm, vias 0 -> 3
- net CAM0_D1_P: track 0.00 -> 18.9 mm, vias 0 -> 3
- net CAM0_C_P: track 0.00 -> 18.1 mm, vias 0 -> 2
- net PCIe_CLK_nREQ: track 0.00 -> 18.1 mm, vias 0 -> 3
- net DSI0_D0_P: track 0.00 -> 18.0 mm, vias 0 -> 2
- net CAM0_D0_N: track 0.00 -> 17.5 mm, vias 0 -> 3
- net DSI0_D0_N: track 0.00 -> 17.4 mm, vias 0 -> 2
- net DSI0_D1_P: track 0.00 -> 16.5 mm, vias 0 -> 1
- net PCIe_nRST: track 0.00 -> 15.8 mm, vias 0 -> 3
- net GND: track 221.1 -> 229.5 mm, vias 112 -> 122
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
Commit message: connecting more pins
Connections:
- D17 pad 2: BTN_PWRn -> (no net)
- J1 pad 100: (no net) -> nEXTRST
- J1 pad 35: (no net) -> ID_SC
- J1 pad 36: (no net) -> ID_SD
- J1 pad 75: (no net) -> SD_PWR_ON
- J1 pad 80: (no net) -> SCL0
- J1 pad 82: (no net) -> SDA0
- J1 pad 97: (no net) -> Camera_GPIO
- J2 pad 1: (no net) -> US2_ID
- U1 pad A4: (no net) -> US2_ID
- U1 pad P16: (no net) -> SCL0
- U1 pad P17: (no net) -> SDA0
- U1 pad R16: (no net) -> ID_SD
- U1 pad R17: (no net) -> ID_SC
- U1 pad R18: (no net) -> Camera_GPIO
- U1 pad U16: (no net) -> nEXTRST
- U1 pad U17: (no net) -> SD_PWR_ON
- U1 pad U18: BTN_PWRn -> (no net)
Routing:
- net ID_SC: track 0.00 -> 28.2 mm, vias 0 -> 5
- net Camera_GPIO: track 0.00 -> 25.7 mm, vias 0 -> 5
- net BTN_PWRn: track 22.5 -> 0.00 mm, vias 1 -> 0
- net nEXTRST: track 0.00 -> 19.6 mm, vias 0 -> 3
- net SD_PWR_ON: track 0.00 -> 16.9 mm, vias 0 -> 3
- net SDA0: track 0.00 -> 15.5 mm, vias 0 -> 1
- net SCL0: track 0.00 -> 14.9 mm, vias 0 -> 1
- net US2_ID: track 0.00 -> 11.0 mm, vias 0 -> 1
- net ID_SD: track 0.00 -> 10.5 mm, vias 0 -> 1
- net /flash/FPGA_PROGRAMN: track 50.0 -> 51.2 mm
- net +2V5: track 81.5 -> 82.5 mm
- net USER_PROGRAMN: track 47.1 -> 46.1 mm

Commit message: Connecting serdes to gpio
Parts:
- moved C56 1.02 mm to (116.2, 105.2)
- moved C64 1.02 mm to (120.2, 105.2)
- moved C70 1.02 mm to (119.2, 105.2)
- moved C73 1.02 mm to (115.2, 105.2)
- moved C58 0.21 mm to (123.2, 105.2)
- moved C63 0.21 mm to (125.2, 105.2)
- moved C65 0.21 mm to (121.2, 105.2)
- moved C69 0.21 mm to (126.2, 105.2)
- moved C71 0.21 mm to (122.2, 105.2)
- moved C75 0.21 mm to (124.2, 105.2)
- moved C57 0.20 mm to (117.2, 105.2)
- moved C62 0.20 mm to (113.2, 105.2)
- moved C68 0.20 mm to (114.2, 105.2)
- moved C74 0.20 mm to (118.2, 105.2)
Connections:
- C56 pad 1: (no net) -> ETH_2P
- C57 pad 1: (no net) -> ETH_1P
- C58 pad 1: (no net) -> GPIO10
- C62 pad 1: (no net) -> ETH_3P
- C63 pad 1: (no net) -> GPIO27
- C64 pad 1: (no net) -> ETH_0P
- C65 pad 1: (no net) -> GPIO11
- C68 pad 2: (no net) -> ETH_3N
- C69 pad 2: (no net) -> GPIO17
- C70 pad 2: (no net) -> ETH_0N
- C71 pad 2: (no net) -> GPIO9
- C73 pad 2: (no net) -> ETH_2N
- C74 pad 2: (no net) -> ETH_1N
- C75 pad 2: (no net) -> GPIO22
- J1 pad 10: (no net) -> ETH_0N
- J1 pad 11: (no net) -> ETH_2P
- J1 pad 12: (no net) -> ETH_0P
- J1 pad 3: (no net) -> ETH_3P
- J1 pad 38: (no net) -> GPIO11
- J1 pad 4: (no net) -> ETH_1P
- J1 pad 40: (no net) -> GPIO9
- J1 pad 44: (no net) -> GPIO10
- J1 pad 46: (no net) -> GPIO22
- J1 pad 48: (no net) -> GPIO27
- J1 pad 5: (no net) -> ETH_3N
- J1 pad 50: (no net) -> GPIO17
- J1 pad 6: (no net) -> ETH_1N
- J1 pad 9: (no net) -> ETH_2N
Routing:
- net GPIO21: track 52.6 -> 42.5 mm
- net ETH_2P: track 0.00 -> 8.73 mm
- net ETH_2N: track 0.00 -> 7.99 mm
- net ETH_3N: track 0.00 -> 6.52 mm
- net ETH_3P: track 0.00 -> 6.15 mm
- net GPIO16: track 44.6 -> 50.7 mm
- net +3V3: track 150.6 -> 156.3 mm, vias 30 -> 28
- net ETH_0P: track 0.00 -> 5.53 mm
- net ETH_0N: track 0.00 -> 4.99 mm
- net ETH_1N: track 0.00 -> 4.45 mm
- net ETH_1P: track 0.00 -> 3.50 mm
- net GPIO17: track 0.00 -> 3.46 mm
- net /flash/FLASH_MISO: track 26.4 -> 23.1 mm
- net GPIO27: track 0.00 -> 2.92 mm
- net GPIO20: track 42.4 -> 45.1 mm
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