File: ulx3s.kicad_pcb (KiCad board)
At the start: 4 copper layers, 55.1 x 40 mm, 143 parts, among them J1 DF40C-100DP-0.4V(51), J2 DF40C-100DP-0.4V(51), J3 JTAG, U1 LFE5U-85F-6BG381C, U10 IS25LP128F-JBLE, U2 IS42S16320D-6BLI, U3 TLV62569DBV, U4 TLV62569DBV, U5 TLV62569DBV, Y1 FNETHE025

Commit message: 4 to 6 layers
Other:
- copper layers 4 -> 6
Changed lines of the file:
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@@
     (1 In1.Cu signal)
     (2 In2.Cu signal)
+    (3 In3.Cu signal)
+    (4 In4.Cu signal)
     (31 B.Cu signal)
     (32 B.Adhes user)

Commit message: Initial 6 layer board
Routing:
- added copper zone on POWER.Cu, net +1V1
- added copper zone on POWER.Cu, net +2V5
- added copper zone on POWER.Cu, net +3V3
- added copper zone on POWER.Cu, net 2V5_3V3
- added copper zone on GND1.Cu, net GND
- added copper zone on GND2.Cu, net GND
- removed copper zone on In1.Cu, net +1V1
- removed copper zone on In1.Cu, net +2V5
- removed copper zone on In1.Cu, net +3V3
- removed copper zone on In1.Cu, net 2V5_3V3
- removed copper zone on B.Cu, net GND
- removed copper zone on F.Cu, net GND
- removed copper zone on In2.Cu, net GND
Other:
- board text added: "v0.0.2"
- board text removed: "v0.0.1"

Commit message: Fixing routing errors
Connections:
- C16 pad 1: +3V3 -> CM4_3.3V
- C20 pad 1: +3V3 -> CM4_3.3V
- C25 pad 1: +3V3 -> CM4_3.3V
- C31 pad 1: +3V3 -> CM4_3.3V
- C32 pad 1: +3V3 -> CM4_3.3V
- C33 pad 1: +3V3 -> CM4_3.3V
- C34 pad 1: +3V3 -> CM4_3.3V
- C35 pad 1: +3V3 -> CM4_3.3V
- C46 pad 1: +3V3 -> CM4_3.3V
- C50 pad 1: +3V3 -> CM4_3.3V
- C51 pad 1: +3V3 -> CM4_3.3V
- C52 pad 1: +3V3 -> CM4_3.3V
- J3 pad 2: +3V3 -> CM4_3.3V
- R11 pad 1: +3V3 -> CM4_3.3V
- R12 pad 1: +3V3 -> CM4_3.3V
- R16 pad 1: +3V3 -> CM4_3.3V
- R27 pad 1: +3V3 -> CM4_3.3V
- R28 pad 1: +3V3 -> CM4_3.3V
- R29 pad 1: +3V3 -> CM4_3.3V
- R30 pad 1: +3V3 -> CM4_3.3V
- R31 pad 1: +3V3 -> CM4_3.3V
- R32 pad 1: +3V3 -> CM4_3.3V
- R33 pad 1: +3V3 -> CM4_3.3V
- R8 pad 1: +3V3 -> CM4_3.3V
- RP3 pad 2: +3V3 -> CM4_3.3V
- RV3 pad 2: +3V3 -> CM4_3.3V
- U1 pad F11: +3V3 -> CM4_3.3V
- U1 pad F12: +3V3 -> CM4_3.3V
- U1 pad H14: +3V3 -> CM4_3.3V
- U1 pad H15: +3V3 -> CM4_3.3V
- U1 pad J15: +3V3 -> CM4_3.3V
- U1 pad L14: +3V3 -> CM4_3.3V
- U1 pad L15: +3V3 -> CM4_3.3V
- U1 pad L6: +3V3 -> CM4_3.3V
- U1 pad L7: +3V3 -> CM4_3.3V
- U1 pad M15: +3V3 -> CM4_3.3V
- U1 pad M6: +3V3 -> CM4_3.3V
- U1 pad P10: +3V3 -> CM4_3.3V
- U1 pad P9: +3V3 -> CM4_3.3V
- U1 pad T2: +3V3 -> CM4_3.3V
- U1 pad T3: +3V3 -> CM4_3.3V
- U1 pad T4: +3V3 -> CM4_3.3V
- U1 pad U2: +3V3 -> CM4_3.3V
- U10 pad 8: +3V3 -> CM4_3.3V
- U2 pad A7: +3V3 -> CM4_3.3V
- U2 pad A9: +3V3 -> CM4_3.3V
- U2 pad B3: +3V3 -> CM4_3.3V
- U2 pad C7: +3V3 -> CM4_3.3V
- U2 pad D3: +3V3 -> CM4_3.3V
- U2 pad E7: +3V3 -> CM4_3.3V
- U2 pad J9: +3V3 -> CM4_3.3V
- Y1 pad 1: +3V3 -> CM4_3.3V
- Y1 pad 4: +3V3 -> CM4_3.3V
Routing:
- net +3V3: track 156.3 -> 0.00 mm, vias 28 -> 0
- net CM4_3.3V: track 0.40 -> 127.4 mm, vias 0 -> 30
- net +5V: track 198.7 -> 166.7 mm, vias 11 -> 12
- net GND: track 229.2 -> 260.2 mm, vias 122 -> 151
- net SD_D1: track 47.2 -> 21.4 mm
- net SD_D2: track 47.1 -> 21.5 mm
- net ID_SC: track 28.9 -> 7.31 mm, vias 5 -> 3
- net SD_CMD: track 46.0 -> 27.9 mm
- net 2V5_3V3: track 49.3 -> 40.2 mm
- net USER_PROGRAMN: track 46.1 -> 37.1 mm
- net SD_PWR_ON: track 16.9 -> 15.5 mm
- net GPIO21: track 42.5 -> 41.1 mm
- net HDMI0_SDA: track 4.37 -> 3.41 mm
- net GPIO12: track 49.6 -> 48.7 mm
- net Camera_GPIO: track 26.2 -> 25.5 mm
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- added copper zone on POWER.Cu, net +5V
- added copper zone on POWER.Cu, net CM4_3.3V

Commit message: All signals are now connected - DRC shows no errors
Routing:
- net SD_D2: track 21.5 -> 46.4 mm, vias 1 -> 2
- net SD_D1: track 21.4 -> 46.0 mm, vias 1 -> 2
- net SD_CMD: track 27.9 -> 44.6 mm
- net USER_PROGRAMN: track 37.1 -> 46.7 mm
- net GND: track 260.2 -> 268.5 mm, vias 151 -> 152
- net +2V5: track 83.7 -> 90.7 mm
- net ID_SC: track 7.31 -> 13.5 mm
- net CM4_3.3V: track 127.4 -> 130.0 mm
- net +5V: track 166.7 -> 169.2 mm
- removed copper zone on POWER.Cu, net +3V3
Other:
- board text added: "ULX4M-LS"
- board text removed: "ULX4M"

Commit message: Adding buttons
Parts:
- added R18: 130, Capacitor_SMD:C_0402_1005Metric, B.Cu at (95.5, 85.9)
- added SW1: SW_Push, Switch_EVPAA:Switch_EVPAA, F.Cu at (99.1, 83.5)
- added SW2: SW_Push, Switch_EVPAA:Switch_EVPAA, F.Cu at (102.1, 86.5)
Connections:
- U1 pad B1: (no net) -> LED1
- U1 pad B3: (no net) -> LED2
- U1 pad C1: LED2 -> LED3
- U1 pad C2: LED1 -> BTN2
- U1 pad C3: (no net) -> BTN1
- U1 pad D2: LED3 -> (no net)
Routing:
- net BTN1: track 0.00 -> 20.9 mm, vias 0 -> 2
- net Net-(R18-Pad1): track 0.00 -> 15.9 mm, vias 0 -> 1
- net BTN2: track 0.00 -> 13.4 mm
- net LED2: track 8.53 -> 10.2 mm
- net LED3: track 10.9 -> 9.74 mm
- net LED1: track 9.11 -> 7.99 mm
- net CM4_3.3V: track 130.0 -> 130.7 mm, vias 30 -> 31
- net GND: vias 152 -> 151

Commit message: Connecting more GPIOs, improving routing
Parts:
- added AE1: Antenna, Connector_Coaxial:CoaxialSwitch_Hirose_MS-156C3_Horizontal, F.Cu at (147.2, 104.5)
- moved C34 8.71 mm to (133.2, 99.0)
- moved C33 8.69 mm to (140.9, 96.5)
- moved C16 8.36 mm to (133.8, 97.7), turned to 0 degrees
- moved C52 7.21 mm to (139.5, 93.8)
- moved U2 4.70 mm to (136.8, 93.2)
- moved C35 4.66 mm to (137.0, 93.5)
- moved radiona 1.37 mm to (136.7, 98.8), turned to 0 degrees
Connections:
- J1 pad 24: (no net) -> GPIO26
- J1 pad 26: (no net) -> GPIO19
- J1 pad 28: (no net) -> GPIO13
- J1 pad 30: (no net) -> GPIO6
- J1 pad 34: (no net) -> GPIO5
- J1 pad 37: (no net) -> GPIO7
- J1 pad 39: (no net) -> GPIO8
- J1 pad 41: (no net) -> GPIO25
- J1 pad 45: (no net) -> GPIO24
- J1 pad 47: (no net) -> GPIO23
- J1 pad 49: (no net) -> GPIO18
- J1 pad 51: (no net) -> GPIO15
- J1 pad 54: (no net) -> GPIO4
- J1 pad 55: (no net) -> GPIO14
- J1 pad 56: (no net) -> GPIO3
- J1 pad 58: (no net) -> GPIO2
- U1 pad H16: (no net) -> GPIO5
- U1 pad J5: (no net) -> GPIO3
- U1 pad K4: (no net) -> GPIO4
- U1 pad K5: (no net) -> GPIO2
- U1 pad L4: (no net) -> GPIO14
- U1 pad L5: (no net) -> GPIO15
- U1 pad N3: (no net) -> GPIO24
- U1 pad N4: (no net) -> GPIO23
- U1 pad N5: (no net) -> GPIO18
- U1 pad P3: (no net) -> GPIO7
- U1 pad P4: (no net) -> GPIO8
- U1 pad P5: (no net) -> GPIO25
- U1 pad R1: (no net) -> GPIO6
- U1 pad T1: (no net) -> GPIO13
- U1 pad U1: (no net) -> GPIO19
- U1 pad V1: (no net) -> GPIO26
- U2 pad A2: SDRAM_D15 -> SDRAM_D14
- U2 pad B1: SDRAM_D14 -> SDRAM_D15
Routing:
- net GPIO14: track 0.00 -> 28.9 mm, vias 0 -> 2
- net GPIO3: track 0.00 -> 28.6 mm, vias 0 -> 2
- net GPIO2: track 0.00 -> 28.4 mm, vias 0 -> 2
- net GPIO4: track 0.00 -> 28.0 mm, vias 0 -> 2
- net GPIO24: track 0.00 -> 28.0 mm, vias 0 -> 2
- net GPIO15: track 0.00 -> 27.5 mm, vias 0 -> 2
- net GPIO18: track 0.00 -> 26.5 mm, vias 0 -> 2
- net GPIO23: track 0.00 -> 26.2 mm, vias 0 -> 2
- net GPIO5: track 0.00 -> 24.1 mm, vias 0 -> 3
- net GPIO25: track 0.00 -> 23.2 mm, vias 0 -> 2
- net GPIO7: track 0.00 -> 22.7 mm, vias 0 -> 2
- net GPIO19: track 0.00 -> 22.2 mm, vias 0 -> 2
- net GPIO8: track 0.00 -> 22.1 mm, vias 0 -> 2
- net GPIO13: track 0.00 -> 22.1 mm, vias 0 -> 2
- net GPIO6: track 0.00 -> 21.7 mm, vias 0 -> 2
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
Commit message: Connecting all GPIOs, connecting SDCARD
Parts:
- C46, C58, C63, C65, C69, C71, C75: moved to F.Cu
- moved C65 36.3 mm to (139.4, 73.8), turned to 0 degrees
- moved C71 35.0 mm to (139.4, 74.8), turned to 180 degrees
- moved C58 33.6 mm to (139.4, 75.8), turned to 0 degrees
- moved C75 32.2 mm to (139.4, 76.8), turned to 180 degrees
- moved C63 30.9 mm to (139.4, 77.8), turned to 0 degrees
- moved C69 29.5 mm to (139.4, 78.8), turned to 180 degrees
- moved R14 0.26 mm to (137.0, 78.4)
- moved R15 0.24 mm to (135.9, 78.4)
Connections:
- C58 pad 1: GPIO10 -> DSI1_D1_N
- C63 pad 1: GPIO27 -> DSI1_C_P
- C65 pad 1: GPIO11 -> DSI1_D0_P
- C69 pad 2: GPIO17 -> DSI1_C_N
- C71 pad 2: GPIO9 -> DSI1_D0_N
- C75 pad 2: GPIO22 -> DSI1_D1_P
- J1 pad 48: GPIO27 -> GP16
- J1 pad 50: GPIO17 -> GN16
- J1 pad 57: SD_CLK -> GPIO15
- J1 pad 61: SD_D3 -> GPIO14
- J1 pad 63: SD_D0 -> GPIO4
- J1 pad 67: SD_D1 -> GPIO3
- J1 pad 69: SD_D2 -> GPIO2
- J2 pad 75: (no net) -> DSI1_D0_N
- J2 pad 77: (no net) -> DSI1_D0_P
- J2 pad 81: (no net) -> DSI1_D1_N
- J2 pad 83: (no net) -> DSI1_D1_P
- J2 pad 87: (no net) -> DSI1_C_N
- J2 pad 89: (no net) -> DSI1_C_P
- J2 pad 93: (no net) -> DSI1_D2_N
- J2 pad 94: (no net) -> DSI1_D3_N
- J2 pad 95: (no net) -> DSI1_D2_P
- J2 pad 96: (no net) -> DSI1_D3_P
- U1 pad A18: (no net) -> DSI1_D3_P
- U1 pad A19: (no net) -> DSI1_D2_P
- U1 pad B19: (no net) -> DSI1_D3_N
- U1 pad B20: (no net) -> DSI1_D2_N
- U1 pad G16: (no net) -> GPIO9
- U1 pad H1: SD_D1 -> GPIO3
- U1 pad H2: SD_CLK -> GPIO15
- U1 pad J3: SD_D0 -> GPIO4
- U1 pad K1: SD_D2 -> GPIO2
- U1 pad K2: SD_D3 -> GPIO14
- U1 pad L16: (no net) -> GPIO11
- U1 pad M17: (no net) -> GN16
- U1 pad N16: (no net) -> GP16
- U1 pad N17: (no net) -> GPIO10
- U1 pad U18: (no net) -> GPIO22
Routing:
- net /serdes/S_7_P: track 4.63 -> 83.6 mm, vias 1 -> 3
- net /serdes/S_7_N: track 4.37 -> 81.6 mm, vias 1 -> 3
- net /serdes/S_5_P: track 3.24 -> 72.0 mm, vias 1 -> 3
- net /serdes/CLK_1_P: track 3.44 -> 72.0 mm, vias 1 -> 3
- net /serdes/S_5_N: track 3.07 -> 71.1 mm, vias 1 -> 3
- net /serdes/CLK_1_N: track 4.28 -> 71.1 mm, vias 1 -> 3
- net GPIO9: track 2.18 -> 61.6 mm, vias 0 -> 3
- net GPIO2: track 28.4 -> 76.8 mm, vias 2 -> 5
- net GPIO3: track 28.6 -> 76.3 mm, vias 2 -> 4
- net GPIO4: track 28.0 -> 71.9 mm, vias 2 -> 5
- net SD_D2: track 43.8 -> 0.00 mm, vias 2 -> 0
- net GPIO15: track 27.5 -> 71.2 mm, vias 2 -> 3
- net SD_CLK: track 43.3 -> 0.00 mm, vias 1 -> 0
- net GPIO14: track 28.9 -> 72.1 mm, vias 2 -> 3
- net SD_D0: track 42.7 -> 0.00 mm, vias 3 -> 0
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Other:
- board text added: "03.11.2021. v0.0.2"
- board text removed: "v0.0.2"
