File: usb.sch (KiCad schematic (older format))
At the start: 24 parts, among them J4 CONN_02X03, U1 LFE5U-85F-6BG381C, U6 FT231XQ, Y1 FNETHE025

Commit message: More removing
Parts:
- removed AE1: 433MHz, TestPoint:TestPoint_Pad_D1.0mm, symbol Device:Antenna
- removed J4: CONN_02X03, Socket_Strips:Socket_Strip_Straight_2x03, symbol Connector_Generic:Conn_02x03_Odd_Even
- removed R49, R50: 27, Resistor_SMD:R_0603_1608Metric, symbol Device:R
- removed R9: 15k, Resistor_SMD:R_0603_1608Metric, symbol Device:R
- removed U6: FT231XQ, ft231x:FT231X-QFN-20-1EP_4x4mm_P0.5mm_EP2x2mm, symbol ftdi:FT231XQ
- removed US1: MICRO_USB, usb_otg:USB-MICRO-B-FCI-10118192-0001LF, symbol usb_otg:USB_OTG
Connections:
- wire segments 74 -> 49

Commit message: Sync sch and pcb
Parts:
- removed D8: STPS2L40AF, Diode_SMD:D_SMA, symbol Device:D_Schottky_Small
Connections:
- net labels removed: FTD+, FTD-
- wire segments 49 -> 38
- no-connect marks 2 -> 1
Changed lines of the file:
@@
 $EndDescr
-$Comp
-L Device:D_Schottky_Small D8
-U 1 1 58D6C83A
-P 2300 1700
-F 0 "D8" H 2350 1650 50  0000 L CNN
-F 1 "STPS2L40AF" H 1800 1650 50  0000 L CNN
-F 2 "Diode_SMD:D_SMA" V 2300 1700 60  0001 C CNN
-F 3 "" V 2300 1700 60  0000 C CNN
-F 4 "www.st.com" H 2300 1700 50  0001 C CNN "MNF1_URL"
-F 5 "STPS2L30AF" H 2300 1700 60  0001 C CNN "MPN"
-F 6 "511-STPS2L40AF" H 2300 1700 60  0001 C CNN "Mouser"
-F 7 "497-12310-1-ND" H 2300 1700 50  0001 C CNN "Digikey"
-F 8 "69AH2828" H 2300 1700 50  0001 C CNN "Newark"
-F 9 "STPS2L30AF" H 2300 1700 50  0001 C CNN "AvnetEU"
-F 10 "C111630" H 2300 1700 50  0001 C CNN "LCSC"
-F 11 "0.22121$" H 2300 1700 50  0001 C CNN "price100_AvnetEU"
-F 12 "FV008" H 2300 1700 50  0001 C CNN "Koncar"
-	1    2300 1700
-	-1   0    0    1
-$EndComp
-$Comp
-L power:+5V #PWR0107
-U 1 1 58D6C83B
-P 2800 1700
-F 0 "#PWR0107" H 2800 1550 50  0001 C CNN
-F 1 "+5V" H 2800 1840 50  0000 C CNN
-F 2 "" H 2800 1700 60  0000 C CNN
-F 3 "" H 2800 1700 60  0000 C CNN
-	1    2800 1700
-	0    1    1    0
-$EndComp
 $Comp
 L Device:Jumper_NC_Small D9
@@
 	0    1    1    0
 $EndComp
-$Comp
-L power:GND #PWR0104
-U 1 1 58D6C842
-P 1850 2100
-F 0 "#PWR0104" H 1850 1850 50  0001 C CNN
-F 1 "GND" H 1850 1950 50  0000 C CNN
-F 2 "" H 1850 2100 50  0000 C CNN
-F 3 "" H 1850 2100 50  0000 C CNN
-	1    1850 2100
-	0    -1   -1   0
-$EndComp
 Text GLabel 3000 1800 2    60   Input ~ 0
 USB_FTDI_D-
@@
 Text GLabel 3000 2850 2    60   Input ~ 0
 USB_FPGA_D+
-NoConn ~ 1850 2000
 $Comp
 L power:GND #PWR0102
@@
 USB5V
 Wire Wire Line
-	1800 1700 1950 1700
-Wire Wire Line
-	2400 1700 2800 1700
-Wire Wire Line
 	2750 2650 2800 2650
-Wire Wire Line
-	1800 2100 1850 2100
-Wire Wire Line
-	1800 1800 2150 1800
-Wire Wire Line
-	1800 1900 2150 1900
-Wire Wire Line
-	1800 2000 1850 2000
-Wire Wire Line
-	2150 1500 1950 1500
-Wire Wire Line
-	1950 1500 1950 1700
-Connection ~ 1950 1700
 Text GLabel 4850 3400 0    60   Input ~ 0
 nRESET
@@
 Text GLabel 9150 5100 0    60   Input ~ 0
 JTAG_TMS
-Wire Wire Line
-	2450 1800 3000 1800
-Wire Wire Line
-	2450 1900 3000 1900
-Text Label 1850 1800 0    60   ~ 0
-FTD-
-Text Label 1850 1900 0    60   ~ 0
-FTD+
 Text Notes 2850 3250 0    60   ~ 0
 USB_FPGA connected to\nBANK1 on "gpdi" sheet and\nBANK2 on "ram" sheet
@@
 D+,D- 15k pulldown \nfor host mode
 Wire Wire Line
-	1950 1700 2200 1700
-Wire Wire Line
 	2650 3200 2700 3200

Commit message: More removal, spliting modules
Parts:
- removed D20, D21: 3.6V, Diode_SMD:D_SOD-323_HandSoldering, symbol Device:D_Zener_Small_ALT
- removed D23, D24, D25, D26: 1N914, Diode_SMD:D_SOD-323_HandSoldering, symbol Device:D
- removed D9: 0, jumper:D_SMA_Jumper_NC, symbol Device:Jumper_NC_Small
- removed R40, R54: 1.1k, Resistor_SMD:R_0603_1608Metric, symbol Device:R
- removed R52, R53: 27, Resistor_SMD:R_0603_1608Metric, symbol Device:R
- removed R63, R64: 15k, Resistor_SMD:R_0603_1608Metric, symbol Device:R
- removed US2: MICRO_USB, usb_otg:USB-MICRO-B-FCI-10118192-0001LF, symbol usb_otg:USB_OTG
Connections:
- wire segments 38 -> 13

Commit message: Adding footprints
Parts:
- Y1: footprint oscxo:Crystal_SMD_7050_4Pads -> Crystal:Crystal_SMD_TXC_7M-4Pin_3.2x2.5mm
Changed lines of the file:
@@
 F 0 "Y1" H 5575 1650 50  0000 L CNN
 F 1 "FNETHE025" H 5575 1575 50  0000 L CNN
-F 2 "oscxo:Crystal_SMD_7050_4Pads" H 5450 1450 50  0001 C CNN
+F 2 "Crystal:Crystal_SMD_TXC_7M-4Pin_3.2x2.5mm" H 5450 1450 50  0001 C CNN
 F 3 "https://www.diodes.com/assets/Datasheets/FNETHE025.pdf" H 5450 1450 50  0001 C CNN
 F 4 "www.diodes.com" H 5450 1450 60  0001 C CNN "MNF1_URL"

Commit message: Before power placement
Parts:
- added D4, D5, D6, D7: 1N914, Diode_SMD:D_SOD-323, symbol Device:D_Small
- added J3: JTAG, Connector_PinSocket_2.54mm:PinSocket_2x03_P2.54mm_Vertical, symbol Connector_Generic:Conn_02x03_Odd_Even
- added R1, R2: 27, Resistor_SMD:R_0402_1005Metric, symbol Device:R_Small
- added R4, R6: 1.1K, Resistor_SMD:R_0402_1005Metric, symbol Device:R_Small
- added R5, R7: 15K, Resistor_SMD:R_0402_1005Metric, symbol Device:R_Small
Connections:
- net labels added: USB_N, USB_OTG_ID, USB_P
- net labels removed: +5V, US2VBUS
- wire segments 13 -> 37
Other:
- note removed: "D8,D9: Schottky 2A/30V \nLow drop Vfmax=0.375V\nParts reduction: Only D8 is required.\nD9 D51 D52 can be 1206\n1A polyfuses or 0-ohm/2A jumpers"
- note removed: "STPS2L40AF"
- note removed: "warning:\nULX3S has different pinout\nfor simpler PCB routing and\nbecause FT230X has weak CTS\ndrive capability. (Undocumented,\nFLEAfpga mail from 13-Nov-2015)\nULX2S pinout was:\nTCK = DSR\nTMS = RI\nTDI = CTS\nTDO = DCD\n"

Commit message: Cleaning DRC errors
Connections:
- net JTAG_TCK renamed GPIO20
- net JTAG_TDI renamed GPIO12
- net JTAG_TDO renamed GPIO16
- net JTAG_TMS renamed GPIO21
Changed lines of the file:
@@
 Wire Wire Line
 	7550 5500 7600 5500
+Text GLabel 9600 5150 0    60   Input ~ 0
+JTAG_TDI
+Text GLabel 9600 5250 0    60   Input ~ 0
+JTAG_TMS
+Text GLabel 9600 5350 0    60   Input ~ 0
+JTAG_TCK
+Text GLabel 9600 5450 0    60   Input ~ 0
+JTAG_TDO
+Text GLabel 9700 5450 2    60   Input ~ 0
+GPIO16
+Wire Wire Line
+	9600 5150 9700 5150
+Wire Wire Line
+	9700 5250 9600 5250
+Text GLabel 9700 5350 2    60   Input ~ 0
+GPIO20
+Wire Wire Line
+	9600 5350 9700 5350
+Wire Wire Line
+	9700 5450 9600 5450
+Text GLabel 9700 5250 2    60   Input ~ 0
+GPIO21
+Text GLabel 9700 5150 2    60   Input ~ 0
+GPIO12
+Text GLabel 5250 5100 0    60   Input ~ 0
+SD_D2
+Text GLabel 5250 5200 0    60   Input ~ 0
+SD_D3
+Text GLabel 5250 4900 0    60   Input ~ 0
+SD_D0
+Text GLabel 5250 5000 0    60   Input ~ 0
+SD_D1
+Text GLabel 5400 5100 2    60   Input ~ 0
+SD_DAT2
+Text GLabel 5400 5000 2    60   Input ~ 0
+SD_DAT1
+Text GLabel 5400 5350 2    60   Input ~ 0
+SD_DAT4
+Text GLabel 5400 5450 2    60   Input ~ 0
+SD_DAT5
+Text GLabel 5400 5550 2    60   Input ~ 0
+SD_DAT6
+Text GLabel 5400 5650 2    60   Input ~ 0
+SD_DAT7
+Text GLabel 5400 5200 2    60   Input ~ 0
+SD_DAT3
+Text GLabel 5400 4900 2    60   Input ~ 0
+SD_DAT0
+Text GLabel 5400 5800 2    60   Input ~ 0
+SD_PWR_ON
+Wire Wire Line
+	5250 4900 5400 4900
+Wire Wire Line
+	5400 5000 5250 5000
+Wire Wire Line
+	5250 5100 5400 5100
+Wire Wire Line
+	5400 5200 5250 5200
 $EndSCHEMATC

Commit message: connecting more pins
Changed lines of the file:
@@
 Text GLabel 5400 4900 2    60   Input ~ 0
 SD_DAT0
-Text GLabel 5400 5800 2    60   Input ~ 0
-SD_PWR_ON
 Wire Wire Line
 	5250 4900 5400 4900

Commit message: Connecting more GPIOs, improving routing
Connections:
- net FTDI_RXD: no longer U1.L4 (PL56C)
- net FTDI_nRXLED: no longer U1.L5 (PL56D)
- net OLED_CLK: no longer U1.P4 (GPLL0C_IN)
- net OLED_MOSI: no longer U1.P3 (GPLL0T_IN)
- net SD_CD: no longer U1.N5 (PL83B)
- net SD_WP: no longer U1.P5 (PL83D)
- net WIFI_EN: no longer U1.J5 (PL50B)
- net WIFI_GPIO19: no longer U1.N4 (PL83C)
- net WIFI_GPIO21: no longer U1.K5 (VREF1_6)
- net WIFI_GPIO27: no longer U1.N3 (PL86A)
- net WIFI_TXD: no longer U1.K4 (PL56A)
- new net GPIO14: U1.L4 (PL56C)
- new net GPIO15: U1.L5 (PL56D)
- new net GPIO18: U1.N5 (PL83B)
- new net GPIO2: U1.K5 (VREF1_6)
- new net GPIO23: U1.N4 (PL83C)
- new net GPIO24: U1.N3 (PL86A)
- new net GPIO25: U1.P5 (PL83D)
- new net GPIO3: U1.J5 (PL50B)
- new net GPIO4: U1.K4 (PL56A)
- new net GPIO7: U1.P3 (GPLL0T_IN)
- new net GPIO8: U1.P4 (GPLL0C_IN)
Changed lines of the file:
@@
 Text GLabel 10150 2650 2    60   Input ~ 0
 FTDI_TXD
-Text GLabel 8650 1950 0    60   Input ~ 0
+Text GLabel 7550 1950 0    60   Input ~ 0
 FTDI_RXD
 Text GLabel 10150 2450 2    60   Input ~ 0
@@
 Text GLabel 10150 2550 2    60   Input ~ 0
 FTDI_nDTR
-Text GLabel 8650 2050 0    60   Input ~ 0
+Text GLabel 7550 2050 0    60   Input ~ 0
 WIFI_TXD
 Text GLabel 10150 1550 2    60   Input ~ 0
@@
 Text GLabel 10150 1450 2    60   Input ~ 0
 WIFI_GPIO0
-Text GLabel 10150 1650 2    60   Input ~ 0
+Text GLabel 10850 1650 2    60   Input ~ 0
 WIFI_EN
 Text GLabel 10150 2850 2    60   Input ~ 0
 OLED_RES
-Text GLabel 8650 2750 0    60   Input ~ 0
+Text GLabel 8200 2750 0    60   Input ~ 0
 OLED_MOSI
-Text GLabel 10150 2750 2    60   Input ~ 0
+Text GLabel 11250 2750 2    60   Input ~ 0
 OLED_CLK
 Text GLabel 8650 2850 0    60   Input ~ 0
@@
 Text GLabel 10150 1850 2    60   Input ~ 0
 SD_CMD
-Text GLabel 10150 2150 2    60   Input ~ 0
+Text GLabel 11150 2150 2    60   Input ~ 0
 SD_WP
-Text GLabel 10150 2250 2    60   Input ~ 0
-SD_CD
 Text Notes 7200 3150 0    60   ~ 0
 WiFi programming pins:\nTXD RXD RTS DTR
@@
 Text Notes 6300 2500 0    60   ~ 0
 WIFI_GPIO15 v1.7 WIFI_GPIO17 <v3.1
-Text GLabel 8650 2150 0    60   Input ~ 0
-WIFI_GPIO19
-Text GLabel 8650 2450 0    60   Input ~ 0
+Text GLabel 7750 2450 0    60   Input ~ 0
 WIFI_GPIO27
 Text Notes 7450 1400 0    60   ~ 0
@@
 NC v1.7
 NoConn ~ 8650 2950
-Text GLabel 10150 1950 2    60   Input ~ 0
+Text GLabel 11500 1950 2    60   Input ~ 0
 FTDI_nRXLED
 Text Notes 10950 2000 0    60   ~ 0
@@
 Text Notes 6700 2200 0    60   ~ 0
 NC v1.7 WIFI_GPIO5 <v3.1
-Text GLabel 10150 2050 2    60   Input ~ 0
+Text GLabel 11100 2050 2    60   Input ~ 0
 WIFI_GPIO21
 Text Notes 10950 2100 0    60   ~ 0
@@
 Wire Wire Line
 	5400 5200 5250 5200
+Text GLabel 8650 2750 0    60   Input ~ 0
+GPIO7
+Text GLabel 10150 2750 2    60   Input ~ 0
+GPIO8
+Text GLabel 10150 2150 2    60   Input ~ 0
+GPIO25
+Text GLabel 10150 2250 2    60   Input ~ 0
+GPIO18
+Text GLabel 10150 1950 2    60   Input ~ 0
+GPIO15
+Text GLabel 8650 2150 0    60   Input ~ 0
+GPIO23
+Text GLabel 10750 2250 2    60   Input ~ 0
+SD_CD
+Text GLabel 8650 2450 0    60   Input ~ 0
+GPIO24
+Text GLabel 7700 2150 0    60   Input ~ 0
+WIFI_GPIO19
+Text GLabel 8650 1950 0    60   Input ~ 0
+GPIO14
+Text GLabel 8650 2050 0    60   Input ~ 0
+GPIO4
+Text GLabel 10150 1650 2    60   Input ~ 0
+GPIO3
+Text GLabel 10150 2050 2    60   Input ~ 0
+GPIO2
 $EndSCHEMATC
