File: usb.sch (KiCad schematic (older format))
At the start: 16 parts, among them J3 JTAG, U1 LFE5U-85F-6BG381C, Y1 FNETHE025

Commit message: Tuning PCie
Parts:
- added P1: USB_OTG, usb_otg:USB-MICRO-B-FCI-10118192-0001LF, symbol usb_otg:USB_OTG
Connections:
- wire segments 60 -> 61
Other:
- moved on the sheet: R19
Changed lines of the file:
@@
 L power:GND #PWR0113
 U 1 1 61CF3ABC
-P 875 2525
-F 0 "#PWR0113" H 875 2275 50  0001 C CNN
-F 1 "GND" H 875 2375 50  0000 C CNN
-F 2 "" H 875 2525 50  0001 C CNN
-F 3 "" H 875 2525 50  0001 C CNN
-	1    875  2525
+P 575 2525
+F 0 "#PWR0113" H 575 2275 50  0001 C CNN
+F 1 "GND" H 575 2375 50  0000 C CNN
+F 2 "" H 575 2525 50  0001 C CNN
+F 3 "" H 575 2525 50  0001 C CNN
+	1    575  2525
 	1    0    0    -1
 $EndComp
@@
 $EndComp
 Wire Wire Line
-	1275 2325 1325 2325
-Wire Wire Line
 	1325 2325 1325 2525
-Wire Wire Line
-	1275 2225 1375 2225
-Wire Wire Line
-	1375 2125 1275 2125
-Wire Wire Line
-	1275 2025 1375 2025
 $Comp
 L power:+5V #PWR?
@@
 	-1   0    0    -1
 $EndComp
-Wire Wire Line
-	1275 1925 1400 1925
 Wire Wire Line
 	1400 1925 1400 1775
@@
 L Device:R_Small R19
 U 1 1 618ED2BD
-P 1175 2225
-F 0 "R19" V 1225 2075 50  0000 C CNN
-F 1 "4k7" V 1175 2225 39  0000 C CNN
-F 2 "Resistor_SMD:R_0402_1005Metric" H 1175 2225 50  0001 C CNN
-F 3 "~" H 1175 2225 50  0001 C CNN
-	1    1175 2225
-	0    -1   -1   0
+P 2625 1975
+F 0 "R19" V 2675 1825 50  0000 C CNN
+F 1 "4k7" V 2625 1975 39  0000 C CNN
+F 2 "Resistor_SMD:R_0402_1005Metric" H 2625 1975 50  0001 C CNN
+F 3 "~" H 2625 1975 50  0001 C CNN
+	1    2625 1975
+	1    0    0    -1
 $EndComp
 $Comp
 L power:+3V3 #PWR08
 U 1 1 619019AA
-P 975 2225
-F 0 "#PWR08" H 975 2075 50  0001 C CNN
-F 1 "+3V3" H 975 2365 50  0000 C CNN
-F 2 "" H 975 2225 50  0001 C CNN
-F 3 "" H 975 2225 50  0001 C CNN
-	1    975  2225
-	0    -1   -1   0
+P 2625 2225
+F 0 "#PWR08" H 2625 2075 50  0001 C CNN
+F 1 "+3V3" H 2625 2365 50  0000 C CNN
+F 2 "" H 2625 2225 50  0001 C CNN
+F 3 "" H 2625 2225 50  0001 C CNN
+	1    2625 2225
+	-1   0    0    1
 $EndComp
-Wire Wire Line
-	975  2225 1075 2225
 Text GLabel 10150 1950 2    60   Input ~ 0
 GPIO9
@@
 Text GLabel 8650 2050 0    60   Input ~ 0
 GPIO10
+$Comp
+L usb_otg:USB_OTG P1
+U 1 1 65056ABD
+P 675 2125
+F 0 "P1" V 250 2047 50  0000 C CNN
+F 1 "USB_OTG" V 341 2047 50  0000 C CNN
+F 2 "usb_otg:USB-MICRO-B-FCI-10118192-0001LF" V 625 2025 50  0001 C CNN
+F 3 "" V 625 2025 50  0000 C CNN
+	1    675  2125
+	0    -1   1    0
+$EndComp
+Wire Wire Line
+	975  2125 1375 2125
+Wire Wire Line
+	975  2025 1375 2025
+Wire Wire Line
+	975  1925 1400 1925
+Wire Wire Line
+	975  2325 1325 2325
+Wire Wire Line
+	975  2225 1375 2225
+Text GLabel 2625 1800 1    60   Input ~ 0
+USB_OTG_ID
+Wire Wire Line
+	2625 1875 2625 1800
+Wire Wire Line
+	2625 2225 2625 2075
 $EndSCHEMATC
