File: usb.sch (KiCad schematic (older format))
At the start: 17 parts, among them J3 JTAG, P1 USB_OTG, U1 LFE5U-85F-6BG381C, Y1 FNETHE025

Commit message: Chaning RGMII_RX_CLK to H2, removing H5, adding pulldown to pin 33 fix #35
Connections:
- net RGMII_REF_CLK: no longer U1.H2 (PCLKT6_0)
- new net RGMII_RX_CLK: U1.H2 (PCLKT6_0)
Changed lines of the file:
@@
 Text GLabel 10150 1850 2    50   Output ~ 0
 RGMII_RX_DV
-Text GLabel 8650 1350 0    50   Output ~ 0
+Text GLabel 7325 1375 0    50   Output ~ 0
 RGMII_REF_CLK
 Text GLabel 10150 2650 2    50   Output ~ 0
@@
 Wire Wire Line
 	2625 2225 2625 2075
+Text GLabel 8650 1350 0    50   Output ~ 0
+RGMII_RX_CLK
 $EndSCHEMATC

Commit message: Lowering number of unique parts fix #37
Parts:
- R1, R2: value 27 -> 27R
- R4, R6: value 1k1 -> 1k
Changed lines of the file:
@@
 	1700 3200 1300 3200
-$Comp
-L Device:R_Small R1
-U 1 1 615BB539
-P 1750 3000
-F 0 "R1" V 1800 2850 50  0000 C CNN
-F 1 "27" V 1750 3000 39  0000 C CNN
-F 2 "Resistor_SMD:R_0402_1005Metric" H 1750 3000 50  0001 C CNN
-F 3 "~" H 1750 3000 50  0001 C CNN
-	1    1750 3000
-	0    -1   -1   0
-$EndComp
-$Comp
-L Device:R_Small R2
-U 1 1 615CC93A
-P 1750 3100
-F 0 "R2" V 1800 2950 50  0000 C CNN
-F 1 "27" V 1750 3100 39  0000 C CNN
-F 2 "Resistor_SMD:R_0402_1005Metric" H 1750 3100 50  0001 C CNN
-F 3 "~" H 1750 3100 50  0001 C CNN
-	1    1750 3100
-	0    -1   -1   0
-$EndComp
 $Comp
 L Device:D_Small D11
@@
 $EndComp
 $Comp
-L Device:R_Small R4
-U 1 1 616B187F
-P 2250 4700
-F 0 "R4" V 2300 4550 50  0000 C CNN
-F 1 "1k1" V 2250 4700 39  0000 C CNN
-F 2 "Resistor_SMD:R_0402_1005Metric" H 2250 4700 50  0001 C CNN
-F 3 "~" H 2250 4700 50  0001 C CNN
-	1    2250 4700
-	0    -1   -1   0
-$EndComp
-$Comp
 L Device:R_Small R5
 U 1 1 616B22AE
@@
 P 2300 5300
 F 0 "R6" V 2350 5150 50  0000 C CNN
-F 1 "1k1" V 2300 5300 39  0000 C CNN
+F 1 "1k" V 2300 5300 39  0000 C CNN
 F 2 "Resistor_SMD:R_0402_1005Metric" H 2300 5300 50  0001 C CNN
 F 3 "~" H 2300 5300 50  0001 C CNN
@@
 Text GLabel 8650 1350 0    50   Output ~ 0
 RGMII_RX_CLK
+$Comp
+L Device:R_Small R4
+U 1 1 616B187F
+P 2250 4700
+F 0 "R4" V 2300 4550 50  0000 C CNN
+F 1 "1k" V 2250 4700 39  0000 C CNN
+F 2 "Resistor_SMD:R_0402_1005Metric" H 2250 4700 50  0001 C CNN
+F 3 "~" H 2250 4700 50  0001 C CNN
+	1    2250 4700
+	0    -1   -1   0
+$EndComp
+$Comp
+L Device:R_Small R2
+U 1 1 615CC93A
+P 1750 3100
+F 0 "R2" V 1800 2950 50  0000 C CNN
+F 1 "27R" V 1750 3100 39  0000 C CNN
+F 2 "Resistor_SMD:R_0402_1005Metric" H 1750 3100 50  0001 C CNN
+F 3 "~" H 1750 3100 50  0001 C CNN
+	1    1750 3100
+	0    -1   -1   0
+$EndComp
+$Comp
+L Device:R_Small R1
+U 1 1 615BB539
+P 1750 3000
+F 0 "R1" V 1800 2850 50  0000 C CNN
+F 1 "27R" V 1750 3000 39  0000 C CNN
+F 2 "Resistor_SMD:R_0402_1005Metric" H 1750 3000 50  0001 C CNN
+F 3 "~" H 1750 3000 50  0001 C CNN
+	1    1750 3000
+	0    -1   -1   0
+$EndComp
 $EndSCHEMATC

Commit message: Removing SD-CARD sharing feature to get more GPIO pins
Changed lines of the file:
@@
 Text GLabel 10150 2250 2    60   Input ~ 0
 GPIO18
-Text GLabel 10475 800  2    60   Input ~ 0
-GPIO15
 Text GLabel 8650 2150 0    60   Input ~ 0
 GPIO23
 Text GLabel 8650 2450 0    60   Input ~ 0
 GPIO24
-Text GLabel 10475 700  2    60   Input ~ 0
-GPIO14
-Text GLabel 10475 600  2    60   Input ~ 0
-GPIO4
-Text GLabel 10475 900  2    60   Input ~ 0
-GPIO3
-Text GLabel 10475 1000 2    60   Input ~ 0
-GPIO2
 Text GLabel 1375 2025 2    60   Input ~ 0
 USB_N

Commit message: Changing Ethernet chip, connecting all gpios
Parts:
- added R64, R65, R66, R67: 0R, Resistor_SMD:R_0201_0603Metric, symbol Device:R_Small
Connections:
- net ETH_INT_N: no longer U1.M1 (PL89B)
- net GPIO12: now also U1.L2 (PL86D), R64.1; no longer J3.3 (Pin_3), U1.R5 (TDI)
- net GPIO16: now also U1.L1 (PL65C), R66.1; no longer J3.6 (Pin_6), U1.V4 (TDO)
- net GPIO20: now also U1.L3 (PL86C), R65.1; no longer J3.4 (Pin_4), U1.T5 (TCK)
- net GPIO21: now also U1.L4 (PL56C), R67.1; no longer J3.5 (Pin_5), U1.U5 (TMS)
- net RGMII_REF_CLK: now also U1.H2 (PCLKT6_0)
- net RGMII_RXD2: no longer U1.L1 (PL65C)
- net RGMII_RXD3: no longer U1.L2 (PL86D)
- net RGMII_RX_CLK: no longer U1.H2 (PCLKT6_0)
- net RGMII_TXD2: no longer U1.L4 (PL56C)
- net RGMII_TXD3: no longer U1.L3 (PL86C)
- new net JTAG_TCK: J3.4 (Pin_4), R65.2, U1.T5 (TCK)
- new net JTAG_TDI: J3.3 (Pin_3), R64.2, U1.R5 (TDI)
- new net JTAG_TDO: J3.6 (Pin_6), R66.2, U1.V4 (TDO)
- new net JTAG_TMS: J3.5 (Pin_5), R67.2, U1.U5 (TMS)
Changed lines of the file:
@@
 Sheet 6 11
 Title "ULX3S"
-Date ""
-Rev "1.0.10"
+Date "2022-09-21"
+Rev "0.0.3"
 Comp "EMARD"
 Comment1 "USB serial and JTAG"
@@
 Text Notes 1100 3600 0    60   ~ 0
 US2_ID to RTC\non "power" sheet
-Text GLabel 8650 2250 0    60   Input ~ 0
+Text GLabel 7900 2250 0    60   Input ~ 0
 USER_PROGRAMN
 NoConn ~ 8650 2950
@@
 Wire Wire Line
 	7550 5500 7600 5500
-Text GLabel 9600 5150 0    60   Input ~ 0
+Text GLabel 9125 5150 0    60   Input ~ 0
 JTAG_TDI
-Text GLabel 9600 5250 0    60   Input ~ 0
+Text GLabel 9125 5250 0    60   Input ~ 0
 JTAG_TMS
-Text GLabel 9600 5350 0    60   Input ~ 0
+Text GLabel 9125 5350 0    60   Input ~ 0
 JTAG_TCK
-Text GLabel 9600 5450 0    60   Input ~ 0
+Text GLabel 9125 5450 0    60   Input ~ 0
 JTAG_TDO
 Text GLabel 9700 5450 2    60   Input ~ 0
 GPIO16
-Wire Wire Line
-	9600 5150 9700 5150
-Wire Wire Line
-	9700 5250 9600 5250
 Text GLabel 9700 5350 2    60   Input ~ 0
 GPIO20
-Wire Wire Line
-	9600 5350 9700 5350
-Wire Wire Line
-	9700 5450 9600 5450
 Text GLabel 9700 5250 2    60   Input ~ 0
 GPIO21
@@
 Text GLabel 10150 1850 2    50   Output ~ 0
 RGMII_RX_DV
-Text GLabel 7325 1375 0    50   Output ~ 0
+Text GLabel 8650 1350 0    50   Output ~ 0
 RGMII_REF_CLK
-Text GLabel 10150 2650 2    50   Output ~ 0
+Text GLabel 6125 3475 2    50   Output ~ 0
 ETH_INT_N
-Text GLabel 8650 2550 0    50   Output ~ 0
-RGMII_RXD2
 Text GLabel 8650 1850 0    50   Output ~ 0
 RGMII_RXD1
 Text GLabel 10150 1750 2    50   Output ~ 0
 RGMII_RXD0
-Text GLabel 8650 2350 0    50   Input ~ 0
-RGMII_TXD3
-Text GLabel 8650 1950 0    50   Input ~ 0
-RGMII_TXD2
 Text GLabel 8650 1650 0    50   Input ~ 0
 RGMII_TXD1
@@
 Text GLabel 10150 1550 2    50   Input ~ 0
 RGMII_TX_EN
-Text GLabel 10150 2350 2    50   Output ~ 0
-RGMII_RXD3
 Text GLabel 8650 2050 0    60   Input ~ 0
 GPIO10
@@
 Wire Wire Line
 	2625 2225 2625 2075
-Text GLabel 8650 1350 0    50   Output ~ 0
+Text GLabel 6525 3375 0    50   Output ~ 0
 RGMII_RX_CLK
 $Comp
@@
 	0    -1   -1   0
 $EndComp
+Text GLabel 6050 3575 2    50   Output ~ 0
+RGMII_RXD3
+Text GLabel 6650 3900 0    50   Input ~ 0
+RGMII_TXD2
+Text GLabel 6575 3675 0    50   Input ~ 0
+RGMII_TXD3
+Text GLabel 6600 3775 0    50   Output ~ 0
+RGMII_RXD2
+$Comp
+L Device:R_Small R64
+U 1 1 648C922E
+P 9400 5150
+F 0 "R64" V 9450 4975 50  0000 C CNN
+F 1 "0R" V 9400 5150 50  0000 C CNN
+F 2 "Resistor_SMD:R_0201_0603Metric" H 9400 5150 50  0001 C CNN
+F 3 "~" H 9400 5150 50  0001 C CNN
+	1    9400 5150
+	0    1    1    0
+$EndComp
+$Comp
+L Device:R_Small R65
+U 1 1 64928528
+P 9400 5350
+F 0 "R65" V 9450 5175 50  0000 C CNN
+F 1 "0R" V 9400 5350 50  0000 C CNN
+F 2 "Resistor_SMD:R_0201_0603Metric" H 9400 5350 50  0001 C CNN
+F 3 "~" H 9400 5350 50  0001 C CNN
+	1    9400 5350
+	0    1    1    0
+$EndComp
+$Comp
+L Device:R_Small R66
+U 1 1 649432D8
+P 9400 5450
+F 0 "R66" V 9450 5275 50  0000 C CNN
+F 1 "0R" V 9400 5450 50  0000 C CNN
+F 2 "Resistor_SMD:R_0201_0603Metric" H 9400 5450 50  0001 C CNN
+F 3 "~" H 9400 5450 50  0001 C CNN
+	1    9400 5450
+	0    1    1    0
+$EndComp
+$Comp
+L Device:R_Small R67
+U 1 1 64976EC1
+P 9400 5250
+F 0 "R67" V 9450 5075 50  0000 C CNN
+F 1 "0R" V 9400 5250 50  0000 C CNN
+F 2 "Resistor_SMD:R_0201_0603Metric" H 9400 5250 50  0001 C CNN
+F 3 "~" H 9400 5250 50  0001 C CNN
+	1    9400 5250
+	0    1    1    0
+$EndComp
+Wire Wire Line
+	9125 5150 9300 5150
+Wire Wire Line
+	9125 5250 9300 5250
+Wire Wire Line
+	9125 5350 9300 5350
+Wire Wire Line
+	9125 5450 9300 5450
+Wire Wire Line
+	9500 5150 9700 5150
+Wire Wire Line
+	9500 5250 9700 5250
+Wire Wire Line
+	9500 5350 9700 5350
+Wire Wire Line
+	9500 5450 9700 5450
+Text GLabel 10825 2350 2    60   Input ~ 0
+GPIO12
+Text GLabel 7950 1950 0    60   Input ~ 0
+GPIO21
+Text Label 8000 1950 0    60   ~ 0
+TMS
+Text Label 10600 2350 0    60   ~ 0
+TDI
+Text GLabel 7900 2350 0    60   Input ~ 0
+GPIO20
+Text Label 7975 2350 0    60   ~ 0
+TCK
+Text GLabel 7925 2550 0    60   Input ~ 0
+GPIO16
+Text Label 8000 2550 0    60   ~ 0
+TDO
+Wire Wire Line
+	7950 1950 8650 1950
+Wire Wire Line
+	7925 2550 8650 2550
+Wire Wire Line
+	10150 2350 10825 2350
+Wire Wire Line
+	7900 2350 8650 2350
+Wire Wire Line
+	7900 2250 8650 2250
 $EndSCHEMATC

Commit message: Changing GPIO>>JTAG reseistor to connector
Parts:
- removed R64, R65, R66, R67: 0R, Resistor_SMD:R_0201_0603Metric, symbol Device:R_Small
- added J6: GPIO>>JTAG, Connector_PinHeader_1.00mm:PinHeader_2x04_P1.00mm_Vertical, symbol Connector_Generic:Conn_02x04_Odd_Even
Connections:
- net GPIO12: now also J6.3 (Pin_3)
- net GPIO16: now also J6.5 (Pin_5)
- net GPIO20: now also J6.1 (Pin_1)
- net GPIO21: now also J6.7 (Pin_7)
- net JTAG_TCK: now also J6.2 (Pin_2)
- net JTAG_TDI: now also J6.4 (Pin_4)
- net JTAG_TDO: now also J6.6 (Pin_6)
- net JTAG_TMS: now also J6.8 (Pin_8)
Changed lines of the file:
@@
 Wire Wire Line
 	7550 5500 7600 5500
-Text GLabel 9125 5150 0    60   Input ~ 0
+Text GLabel 9650 5950 2    60   Input ~ 0
 JTAG_TDI
-Text GLabel 9125 5250 0    60   Input ~ 0
+Text GLabel 9650 6150 2    60   Input ~ 0
 JTAG_TMS
-Text GLabel 9125 5350 0    60   Input ~ 0
+Text GLabel 9650 5850 2    60   Input ~ 0
 JTAG_TCK
-Text GLabel 9125 5450 0    60   Input ~ 0
+Text GLabel 9650 6050 2    60   Input ~ 0
 JTAG_TDO
-Text GLabel 9700 5450 2    60   Input ~ 0
+Text GLabel 9150 6050 0    60   Input ~ 0
 GPIO16
-Text GLabel 9700 5350 2    60   Input ~ 0
+Text GLabel 9150 5850 0    60   Input ~ 0
 GPIO20
-Text GLabel 9700 5250 2    60   Input ~ 0
+Text GLabel 9150 6150 0    60   Input ~ 0
 GPIO21
-Text GLabel 9700 5150 2    60   Input ~ 0
+Text GLabel 9150 5950 0    60   Input ~ 0
 GPIO12
 Text GLabel 5250 5100 0    60   Input ~ 0
@@
 Text GLabel 6600 3775 0    50   Output ~ 0
 RGMII_RXD2
-$Comp
-L Device:R_Small R64
-U 1 1 648C922E
-P 9400 5150
-F 0 "R64" V 9450 4975 50  0000 C CNN
-F 1 "0R" V 9400 5150 50  0000 C CNN
-F 2 "Resistor_SMD:R_0201_0603Metric" H 9400 5150 50  0001 C CNN
-F 3 "~" H 9400 5150 50  0001 C CNN
-	1    9400 5150
-	0    1    1    0
-$EndComp
-$Comp
-L Device:R_Small R65
-U 1 1 64928528
-P 9400 5350
-F 0 "R65" V 9450 5175 50  0000 C CNN
-F 1 "0R" V 9400 5350 50  0000 C CNN
-F 2 "Resistor_SMD:R_0201_0603Metric" H 9400 5350 50  0001 C CNN
-F 3 "~" H 9400 5350 50  0001 C CNN
-	1    9400 5350
-	0    1    1    0
-$EndComp
-$Comp
-L Device:R_Small R66
-U 1 1 649432D8
-P 9400 5450
-F 0 "R66" V 9450 5275 50  0000 C CNN
-F 1 "0R" V 9400 5450 50  0000 C CNN
-F 2 "Resistor_SMD:R_0201_0603Metric" H 9400 5450 50  0001 C CNN
-F 3 "~" H 9400 5450 50  0001 C CNN
-	1    9400 5450
-	0    1    1    0
-$EndComp
-$Comp
-L Device:R_Small R67
-U 1 1 64976EC1
-P 9400 5250
-F 0 "R67" V 9450 5075 50  0000 C CNN
-F 1 "0R" V 9400 5250 50  0000 C CNN
-F 2 "Resistor_SMD:R_0201_0603Metric" H 9400 5250 50  0001 C CNN
-F 3 "~" H 9400 5250 50  0001 C CNN
-	1    9400 5250
-	0    1    1    0
-$EndComp
-Wire Wire Line
-	9125 5150 9300 5150
-Wire Wire Line
-	9125 5250 9300 5250
-Wire Wire Line
-	9125 5350 9300 5350
-Wire Wire Line
-	9125 5450 9300 5450
-Wire Wire Line
-	9500 5150 9700 5150
-Wire Wire Line
-	9500 5250 9700 5250
-Wire Wire Line
-	9500 5350 9700 5350
-Wire Wire Line
-	9500 5450 9700 5450
 Text GLabel 10825 2350 2    60   Input ~ 0
 GPIO12
@@
 Wire Wire Line
 	7900 2250 8650 2250
+$Comp
+L Connector_Generic:Conn_02x04_Odd_Even J6
+U 1 1 64CCAF42
+P 9350 5950
+F 0 "J6" H 9400 6267 50  0000 C CNN
+F 1 "GPIO>>JTAG" H 9400 6176 50  0000 C CNN
+F 2 "Connector_PinHeader_1.00mm:PinHeader_2x04_P1.00mm_Vertical" H 9350 5950 50  0001 C CNN
+F 3 "~" H 9350 5950 50  0001 C CNN
+	1    9350 5950
+	1    0    0    -1
+$EndComp
 $EndSCHEMATC
