File: ram.sch (KiCad schematic (older format))
At the start: 7 parts, among them U1 LFE5U-85F-6BG381C, U9 MT48LC16M16A2TG

Commit message: Adding BGA SDRAM to schematics, removing SDRAM from PCB
Parts:
- removed U9: MT48LC16M16A2TG, TSOP54:TSOP54, symbol mt48lc16m16a2tg:MT48LC16M16A2TG
- added U2: IS42S16320D-6BLI, IS42S16320D:IS42S16320D-6BLI, symbol mt48lc16m16a2tg:IS42S16320D-6BLI

Commit message: More removal, spliting modules
Parts:
- C16: footprint Capacitor_SMD:C_0805_2012Metric -> Capacitor_SMD:C_0603_1608Metric
- C33, C34, C35: footprint Capacitor_SMD:C_0603_1608Metric -> Capacitor_SMD:C_0402_1005Metric
Changed lines of the file:
@@
 F 0 "C16" H 5375 6000 50  0000 L CNN
 F 1 "2.2uF" H 5375 5800 50  0000 L CNN
-F 2 "Capacitor_SMD:C_0805_2012Metric" H 5388 5750 50  0001 C CNN
+F 2 "Capacitor_SMD:C_0603_1608Metric" H 5388 5750 50  0001 C CNN
 F 3 "" H 5350 5900 50  0000 C CNN
 	1    5350 5900
@@
 F 0 "C33" H 5925 6000 50  0000 L CNN
 F 1 "22nF" H 5925 5800 50  0000 L CNN
-F 2 "Capacitor_SMD:C_0603_1608Metric" H 5938 5750 50  0001 C CNN
+F 2 "Capacitor_SMD:C_0402_1005Metric" H 5938 5750 50  0001 C CNN
 F 3 "" H 5900 5900 50  0000 C CNN
 F 4 "CX0603MRX7R8BB223" H 5900 5900 50  0001 C CNN "MPN"
@@
 F 0 "C34" H 6225 6000 50  0000 L CNN
 F 1 "22nF" H 6225 5800 50  0000 L CNN
-F 2 "Capacitor_SMD:C_0603_1608Metric" H 6238 5750 50  0001 C CNN
+F 2 "Capacitor_SMD:C_0402_1005Metric" H 6238 5750 50  0001 C CNN
 F 3 "" H 6200 5900 50  0000 C CNN
 F 4 "CX0603MRX7R8BB223" H 6200 5900 50  0001 C CNN "MPN"
@@
 F 0 "C35" H 6525 6000 50  0000 L CNN
 F 1 "22nF" H 6525 5800 50  0000 L CNN
-F 2 "Capacitor_SMD:C_0603_1608Metric" H 6538 5750 50  0001 C CNN
+F 2 "Capacitor_SMD:C_0402_1005Metric" H 6538 5750 50  0001 C CNN
 F 3 "" H 6500 5900 50  0000 C CNN
 F 4 "CX0603MRX7R8BB223" H 6500 5900 50  0001 C CNN "MPN"

Commit message: SDRAM routed
Connections:
- net SDRAM_A0: now also U1.L19 (PCLKT3_0); no longer U1.M20 (PCLKC3_1)
- net SDRAM_A1: now also U1.L20 (PCLKT3_1); no longer U1.M19 (PCLKC3_0)
- net SDRAM_A11: now also U1.D20 (VREF1_2); no longer U1.G20 (PR38D)
- net SDRAM_A12: now also U1.E18 (PR14C); no longer U1.G19 (GR_PCLK2_1)
- net SDRAM_A2: now also U1.M19 (PCLKC3_0); no longer U1.L20 (PCLKT3_1)
- net SDRAM_A3: now also U1.K20 (PCLKC2_0); no longer U1.L19 (PCLKT3_0)
- net SDRAM_A4: now also U1.F20 (PR38C); no longer U1.K20 (PCLKC2_0)
- net SDRAM_A5: now also U1.F18 (PR14D); no longer U1.K19 (PCLKC2_1)
- net SDRAM_A6: now also U1.E19 (PR35D); no longer U1.K18 (PR41D)
- net SDRAM_A7: now also U1.F19 (PR38B); no longer U1.J20 (PCLKT2_0)
- net SDRAM_A8: now also U1.E20 (PR38A); no longer U1.J19 (PCLKT2_1)
- net SDRAM_A9: now also U1.C20 (PR35A); no longer U1.H20 (PR41B)
- net SDRAM_BA0: now also U1.L18 (GR_PCLK3_1); no longer U1.P19 (PR83C)
- net SDRAM_BA1: now also U1.M20 (PCLKC3_1); no longer U1.N20 (PR83B)
- net SDRAM_CKE: now also U1.G20 (PR38D); no longer U1.F20 (PR38C)
- net SDRAM_CLK: now also U1.G19 (GR_PCLK2_1); no longer U1.F19 (PR38B)
- net SDRAM_D0: now also U1.U20 (PR86D); no longer U1.J16 (PR20D)
- net SDRAM_D1: now also U1.T20 (PR86C); no longer U1.L18 (GR_PCLK3_1)
- net SDRAM_D10: now also U1.K18 (PR41D); no longer U1.D19 (PR35B)
- net SDRAM_D11: now also U1.J18 (GR_PCLK2_0); no longer U1.C20 (PR35A)
- net SDRAM_D12: now also U1.J20 (PCLKT2_0); no longer U1.E18 (PR14C)
- net SDRAM_D13: now also U1.J16 (PR20D); no longer U1.F18 (PR14D)
- net SDRAM_D14: now also U1.K19 (PCLKC2_1); no longer U1.J18 (GR_PCLK2_0)
- net SDRAM_D2: now also U1.U19 (PR89C); no longer U1.M18 (PR50D)
- net SDRAM_D3: now also U1.T19 (PR89A); no longer U1.N18 (PR53C)
- net SDRAM_D4: now also U1.T18 (PR89D); no longer U1.P18 (PR83D)
- net SDRAM_D5: now also U1.T17 (GPLL0C_IN); no longer U1.T18 (PR89D)
- net SDRAM_D6: now also U1.R20 (PR86B); no longer U1.T17 (GPLL0C_IN)
- net SDRAM_D7: now also U1.P19 (PR83C); no longer U1.U20 (PR86D)
- net SDRAM_D8: now also U1.H20 (PR41B); no longer U1.E19 (PR35D)
- net SDRAM_D9: now also U1.J19 (PCLKT2_1); no longer U1.D20 (VREF1_2)
- net SDRAM_DQM0: now also U1.P20 (PR86A); no longer U1.U19 (PR89C)
- net SDRAM_DQM1: now also U1.D19 (PR35B); no longer U1.E20 (PR38A)
- net SDRAM_nCAS: now also U1.N18 (PR53C); no longer U1.T19 (PR89A)
- net SDRAM_nCS: now also U1.P18 (PR83D); no longer U1.P20 (PR86A)
- net SDRAM_nRAS: now also U1.M18 (PR50D); no longer U1.R20 (PR86B)
- net SDRAM_nWE: now also U1.N20 (PR83B); no longer U1.T20 (PR86C)
Changed lines of the file:
@@
 Text GLabel 5100 4650 0    60   Input ~ 0
 SDRAM_nCS
+Text GLabel 10050 4950 2    60   Input ~ 0
+SDRAM_D0
+Text GLabel 8550 4950 0    60   Input ~ 0
+SDRAM_D1
+Text GLabel 8550 4750 0    60   Input ~ 0
+SDRAM_D2
+Text GLabel 8550 4850 0    60   Input ~ 0
+SDRAM_D3
+Text GLabel 10050 4750 2    60   Input ~ 0
+SDRAM_D4
+Text GLabel 10050 4550 2    60   Input ~ 0
+SDRAM_D5
+Text GLabel 10050 5050 2    60   Input ~ 0
+SDRAM_D6
+Text GLabel 8550 5150 0    60   Input ~ 0
+SDRAM_D7
+Text GLabel 10050 2750 2    60   Input ~ 0
+SDRAM_D8
+Text GLabel 8550 2550 0    60   Input ~ 0
+SDRAM_D9
+Text GLabel 10050 2650 2    60   Input ~ 0
+SDRAM_D10
+Text GLabel 8550 2650 0    60   Input ~ 0
+SDRAM_D11
+Text GLabel 8550 2450 0    60   Input ~ 0
+SDRAM_D12
 Text GLabel 10050 3250 2    60   Input ~ 0
-SDRAM_D0
-Text GLabel 8550 5750 0    60   Input ~ 0
-SDRAM_D1
-Text GLabel 10050 5750 2    60   Input ~ 0
-SDRAM_D2
-Text GLabel 8550 5550 0    60   Input ~ 0
-SDRAM_D3
-Text GLabel 10050 5150 2    60   Input ~ 0
-SDRAM_D4
-Text GLabel 10050 4750 2    60   Input ~ 0
-SDRAM_D5
-Text GLabel 10050 4550 2    60   Input ~ 0
-SDRAM_D6
-Text GLabel 10050 4950 2    60   Input ~ 0
-SDRAM_D7
-Text GLabel 10050 3050 2    60   Input ~ 0
-SDRAM_D8
-Text GLabel 8550 3050 0    60   Input ~ 0
-SDRAM_D9
-Text GLabel 10050 3150 2    60   Input ~ 0
-SDRAM_D10
-Text GLabel 8550 3150 0    60   Input ~ 0
-SDRAM_D11
-Text GLabel 8550 3650 0    60   Input ~ 0
-SDRAM_D12
-Text GLabel 10050 3650 2    60   Input ~ 0
 SDRAM_D13
-Text GLabel 8550 2650 0    60   Input ~ 0
+Text GLabel 10050 2550 2    60   Input ~ 0
 SDRAM_D14
 Text GLabel 8550 3250 0    60   Input ~ 0
 SDRAM_D15
-Text GLabel 10050 6050 2    60   Input ~ 0
+Text GLabel 8550 5950 0    60   Input ~ 0
 SDRAM_A0
+Text GLabel 8550 6050 0    60   Input ~ 0
+SDRAM_A1
 Text GLabel 10050 5950 2    60   Input ~ 0
-SDRAM_A1
-Text GLabel 8550 6050 0    60   Input ~ 0
 SDRAM_A2
-Text GLabel 8550 5950 0    60   Input ~ 0
+Text GLabel 10050 2450 2    60   Input ~ 0
 SDRAM_A3
-Text GLabel 10050 2450 2    60   Input ~ 0
+Text GLabel 8550 2850 0    60   Input ~ 0
 SDRAM_A4
-Text GLabel 10050 2550 2    60   Input ~ 0
+Text GLabel 10050 3650 2    60   Input ~ 0
 SDRAM_A5
-Text GLabel 10050 2650 2    60   Input ~ 0
+Text GLabel 10050 3050 2    60   Input ~ 0
 SDRAM_A6
-Text GLabel 8550 2450 0    60   Input ~ 0
+Text GLabel 10050 2950 2    60   Input ~ 0
 SDRAM_A7
-Text GLabel 8550 2550 0    60   Input ~ 0
+Text GLabel 8550 2950 0    60   Input ~ 0
 SDRAM_A8
-Text GLabel 10050 2750 2    60   Input ~ 0
+Text GLabel 8550 3150 0    60   Input ~ 0
 SDRAM_A9
 Text GLabel 8550 5250 0    60   Input ~ 0
 SDRAM_A10
+Text GLabel 8550 3050 0    60   Input ~ 0
+SDRAM_A11
+Text GLabel 8550 5750 0    60   Input ~ 0
+SDRAM_BA0
+Text GLabel 10050 6050 2    60   Input ~ 0
+SDRAM_BA1
+Text GLabel 8550 2750 0    60   Input ~ 0
+SDRAM_CLK
 Text GLabel 10050 2850 2    60   Input ~ 0
-SDRAM_A11
-Text GLabel 8550 5150 0    60   Input ~ 0
-SDRAM_BA0
+SDRAM_CKE
+Text GLabel 8550 5050 0    60   Input ~ 0
+SDRAM_DQM0
+Text GLabel 10050 3150 2    60   Input ~ 0
+SDRAM_DQM1
+Text GLabel 10050 5750 2    60   Input ~ 0
+SDRAM_nRAS
+Text GLabel 8550 5550 0    60   Input ~ 0
+SDRAM_nCAS
 Text GLabel 10050 5250 2    60   Input ~ 0
-SDRAM_BA1
-Text GLabel 10050 2950 2    60   Input ~ 0
-SDRAM_CLK
-Text GLabel 8550 2850 0    60   Input ~ 0
-SDRAM_CKE
-Text GLabel 8550 4750 0    60   Input ~ 0
-SDRAM_DQM0
-Text GLabel 8550 2950 0    60   Input ~ 0
-SDRAM_DQM1
-Text GLabel 10050 5050 2    60   Input ~ 0
-SDRAM_nRAS
-Text GLabel 8550 4850 0    60   Input ~ 0
-SDRAM_nCAS
-Text GLabel 8550 4950 0    60   Input ~ 0
 SDRAM_nWE
-Text GLabel 8550 5050 0    60   Input ~ 0
+Text GLabel 10050 5150 2    60   Input ~ 0
 SDRAM_nCS
 Text GLabel 10050 4650 2    60   Input ~ 0
@@
 Text GLabel 5100 3750 0    60   Input ~ 0
 SDRAM_A12
-Text GLabel 8550 2750 0    60   Input ~ 0
+Text GLabel 8550 3650 0    60   Input ~ 0
 SDRAM_A12
 $Comp

Commit message: SDRAM, JTAG routed - before logo delete
Connections:
- net GP14: no longer U1.U18 (PR92A)
- new net BTN_PWRn: U1.U18 (PR92A)
Changed lines of the file:
@@
 Text GLabel 8550 5450 0    60   Input ~ 0
 GP15
-Text GLabel 8550 4650 0    60   Input ~ 0
-GP14
 Text GLabel 8550 5650 0    60   Input ~ 0
 GP16
@@
 Wire Wire Line
 	5600 4900 5600 5000
+Text GLabel 8550 4650 0    60   Input ~ 0
+BTN_PWRn
+Text GLabel 7850 4650 0    60   Input ~ 0
+GP14
 $EndSCHEMATC

Commit message: Routing cam and display differential
Connections:
- net GN18: no longer U1.H17 (PR20B)
- net GN19: no longer U1.G18 (PR17B)
- net GN20: no longer U1.E17 (PR14B)
- net GN21: no longer U1.D17 (PR11B)
- net GP18: no longer U1.H18 (PR20A)
- net GP19: no longer U1.F17 (PR17A)
- net GP20: no longer U1.D18 (PR14A)
- net GP21: no longer U1.C18 (PR11A)
- net SDRAM_A3: now also U1.H17 (PR20B); no longer U1.K20 (PCLKC2_0)
- net SDRAM_D12: now also U1.H18 (PR20A); no longer U1.J20 (PCLKT2_0)
- new net FPDI_CLK+: U1.J20 (PCLKT2_0)
- new net FPDI_CLK-: U1.K20 (PCLKC2_0)
- new net FPDI_D0+: U1.F17 (PR17A)
- new net FPDI_D0-: U1.G18 (PR17B)
- new net FPDI_D1+: U1.D18 (PR14A)
- new net FPDI_D1-: U1.E17 (PR14B)
- new net FPDI_D2+: U1.C18 (PR11A)
- new net FPDI_D2-: U1.D17 (PR11B)
Changed lines of the file:
@@
 Text GLabel 8550 2650 0    60   Input ~ 0
 SDRAM_D11
-Text GLabel 8550 2450 0    60   Input ~ 0
+Text GLabel 8550 3350 0    60   Input ~ 0
 SDRAM_D12
 Text GLabel 10050 3250 2    60   Input ~ 0
@@
 Text GLabel 10050 5950 2    60   Input ~ 0
 SDRAM_A2
-Text GLabel 10050 2450 2    60   Input ~ 0
+Text GLabel 10050 3350 2    60   Input ~ 0
 SDRAM_A3
 Text GLabel 8550 2850 0    60   Input ~ 0
@@
 Text GLabel 10050 5650 2    60   Input ~ 0
 GN16
-Text GLabel 10050 3350 2    60   Input ~ 0
-GN18
-Text GLabel 10050 3950 2    60   Input ~ 0
+Text GLabel 13200 4250 2    60   Input ~ 0
 GN21
-Text GLabel 10050 3750 2    60   Input ~ 0
+Text GLabel 13200 4100 2    60   Input ~ 0
 GN20
-Text GLabel 8550 3350 0    60   Input ~ 0
-GP18
-Text GLabel 8550 3950 0    60   Input ~ 0
+Text GLabel 13050 4250 0    60   Input ~ 0
 GP21
-Text GLabel 8550 3750 0    60   Input ~ 0
+Text GLabel 13000 4100 0    60   Input ~ 0
 GP20
-Text GLabel 10050 3550 2    60   Input ~ 0
+Text GLabel 13200 3950 2    60   Input ~ 0
 GN19
-Text GLabel 8550 3550 0    60   Input ~ 0
+Text GLabel 12950 3900 0    60   Input ~ 0
 GP19
 Text GLabel 10050 5850 2    60   Input ~ 0
@@
 Text GLabel 7850 4650 0    60   Input ~ 0
 GP14
+Text GLabel 7850 3350 0    60   Input ~ 0
+GP18
+Text GLabel 11000 3300 2    60   Input ~ 0
+GN18
+Text GLabel 8550 3950 0    60   Input ~ 0
+FPDI_D2+
+Text GLabel 10050 3950 2    60   Input ~ 0
+FPDI_D2-
+Text GLabel 8550 3750 0    60   Input ~ 0
+FPDI_D1+
+Text GLabel 10050 3750 2    60   Input ~ 0
+FPDI_D1-
+Text GLabel 8550 3550 0    60   Input ~ 0
+FPDI_D0+
+Text GLabel 10050 3550 2    60   Input ~ 0
+FPDI_D0-
+Text GLabel 8550 2450 0    60   Input ~ 0
+FPDI_CLK+
+Text GLabel 10050 2450 2    60   Input ~ 0
+FPDI_CLK-
 $EndSCHEMATC

Commit message: connecting more pins
Connections:
- net ADC_CSn: no longer U1.R17 (PR56D)
- net ADC_MISO: no longer U1.U16 (GPLL0T_IN)
- net ADC_MOSI: no longer U1.R16 (PR56C)
- net ADC_SCLK: no longer U1.P17 (PR53D)
- net BTN_PWRn: no longer U1.U18 (PR92A)
- net BTN_U: no longer U1.R18 (PR89B)
- net GN14: no longer U1.U17 (PR92B)
- net GN15: no longer U1.P16 (VREF1_3)
- new net Camera_GPIO: U1.R18 (PR89B)
- new net ID_SC: U1.R17 (PR56D)
- new net ID_SD: U1.R16 (PR56C)
- new net SCL0: U1.P16 (VREF1_3)
- new net SDA0: U1.P17 (PR53D)
- new net SD_PWR_ON: U1.U17 (PR92B)
- new net nEXTRST: U1.U16 (GPLL0T_IN)
Changed lines of the file:
@@
 Text GLabel 10050 5150 2    60   Input ~ 0
 SDRAM_nCS
-Text GLabel 10050 4650 2    60   Input ~ 0
+Text GLabel 10850 4550 2    60   Input ~ 0
 GN14
-Text GLabel 10050 5450 2    60   Input ~ 0
+Text GLabel 12100 5800 2    60   Input ~ 0
 GN15
 Text GLabel 8550 5450 0    60   Input ~ 0
@@
 	1    0    0    -1
 $EndComp
-Text GLabel 8550 4550 0    60   Input ~ 0
+Text GLabel 8500 4350 0    60   Input ~ 0
 ADC_MISO
-Text GLabel 8550 5350 0    60   Input ~ 0
+Text GLabel 7700 5350 0    60   Input ~ 0
 ADC_MOSI
-Text GLabel 10050 5350 2    60   Input ~ 0
+Text GLabel 11300 5300 2    60   Input ~ 0
 ADC_CSn
-Text GLabel 10050 5550 2    60   Input ~ 0
+Text GLabel 11950 6200 2    60   Input ~ 0
 ADC_SCLK
 Text GLabel 8550 3850 0    60   Input ~ 0
@@
 Text GLabel 8550 3450 0    60   Input ~ 0
 SHUTDOWN
-Text GLabel 10050 4850 2    60   Input ~ 0
+Text GLabel 10850 4850 2    60   Input ~ 0
 BTN_U
 Text GLabel 10050 3450 2    60   Input ~ 0
@@
 Wire Wire Line
 	5600 4900 5600 5000
-Text GLabel 8550 4650 0    60   Input ~ 0
+Text GLabel 7750 4900 0    60   Input ~ 0
 BTN_PWRn
 Text GLabel 7850 4650 0    60   Input ~ 0
@@
 Text GLabel 10050 2450 2    60   Input ~ 0
 FPDI_CLK-
+Text GLabel 10050 4650 2    60   Input ~ 0
+SD_PWR_ON
+Text GLabel 8550 4550 0    60   Input ~ 0
+nEXTRST
+Text GLabel 10050 4850 2    60   Input ~ 0
+Camera_GPIO
+Text GLabel 10050 5350 2    60   Input ~ 0
+ID_SC
+Text GLabel 8550 5350 0    60   Input ~ 0
+ID_SD
+Text GLabel 10050 5550 2    60   Input ~ 0
+SDA0
+Text GLabel 10050 5450 2    60   Input ~ 0
+SCL0
 $EndSCHEMATC

Commit message: Connecting more GPIOs, improving routing
Connections:
- net BTN_R: no longer U1.H16 (PR17D)
- net SDRAM_D14: now also U2.A2 (DQ15); no longer U2.B1 (DQ14)
- net SDRAM_D15: now also U2.B1 (DQ14); no longer U2.A2 (DQ15)
- new net GPIO5: U1.H16 (PR17D)
Changed lines of the file:
@@
 Text GLabel 6700 3850 2    60   Input ~ 0
 SDRAM_D13
+Text GLabel 6700 4050 2    60   Input ~ 0
+SDRAM_D14
 Text GLabel 6700 3950 2    60   Input ~ 0
-SDRAM_D14
-Text GLabel 6700 4050 2    60   Input ~ 0
 SDRAM_D15
 Text GLabel 6700 4300 2    60   Input ~ 0
@@
 Text GLabel 10850 4850 2    60   Input ~ 0
 BTN_U
-Text GLabel 10050 3450 2    60   Input ~ 0
+Text GLabel 10650 3450 2    60   Input ~ 0
 BTN_R
 $Comp
@@
 Text GLabel 10050 5450 2    60   Input ~ 0
 SCL0
+Text GLabel 10050 3450 2    60   Input ~ 0
+GPIO5
 $EndSCHEMATC

Commit message: Connecting all GPIOs, connecting SDCARD
Connections:
- net GP15: no longer U1.N17 (PR56A)
- net GPIO22: now reaches U1.U18 (PR92A)
- net GP17 renamed GPIO11
- net SHUTDOWN renamed GPIO9
- new net GPIO10: U1.N17 (PR56A)
Changed lines of the file:
@@
 Text GLabel 12100 5800 2    60   Input ~ 0
 GN15
-Text GLabel 8550 5450 0    60   Input ~ 0
+Text GLabel 7625 5775 0    60   Input ~ 0
 GP15
 Text GLabel 8550 5650 0    60   Input ~ 0
@@
 GN17
 Text GLabel 8550 5850 0    60   Input ~ 0
-GP17
+GPIO11
 $Comp
 L Device:C C16
@@
 $EndComp
 Text GLabel 8550 3450 0    60   Input ~ 0
-SHUTDOWN
+GPIO9
 Text GLabel 10850 4850 2    60   Input ~ 0
 BTN_U
@@
 Text GLabel 10050 3450 2    60   Input ~ 0
 GPIO5
+Text GLabel 8550 4650 0    60   Input ~ 0
+GPIO22
+Text GLabel 8550 5450 0    60   Input ~ 0
+GPIO10
 $EndSCHEMATC
