File: ram.sch (KiCad schematic (older format))
At the start: 7 parts, among them U1 LFE5U-85F-6BG381C

Commit message: Diff pair length done
Connections:
- net DDR3_A0: now also U1.F20 (PR38C); no longer U1.E16 (PR11C)
- net DDR3_A15: now also U1.P18 (PR83D); no longer U1.R20 (PR86B)
- net DDR3_A3: now also U1.E18 (PR14C); no longer U1.F16 (PR11D)
- net DDR3_A8: now also U1.E16 (PR11C); no longer U1.F20 (PR38C)
- net DDR3_CS: now also U1.H18 (PR20A); no longer U1.H17 (PR20B)
- net DDR3_DM0: now also U1.F16 (PR11D); no longer U1.E18 (PR14C)
- net DDR3_DQ10: now also U1.F19 (PR38B); no longer U1.J18 (GR_PCLK2_0)
- net DDR3_DQ12: now also U1.J18 (GR_PCLK2_0); no longer U1.F19 (PR38B)
- net DDR3_RAS: now also U1.R20 (PR86B); no longer U1.P18 (PR83D)
- net DDR3_WE: now also U1.H17 (PR20B); no longer U1.H18 (PR20A)
Changed lines of the file:
@@
 Text GLabel 8100 2400 2    50   Input ~ 0
 DDR3_A2
-Text GLabel 8100 3100 2    50   Input ~ 0
+Text GLabel 6600 2900 0    50   Input ~ 0
 DDR3_A3
 Text GLabel 8100 2700 2    50   Input ~ 0
@@
 Text GLabel 8100 3800 2    50   Input ~ 0
 DDR3_A7
-Text GLabel 6600 2100 0    50   Input ~ 0
+Text GLabel 6600 3100 0    50   Input ~ 0
 DDR3_A8
 Text GLabel 6600 4000 0    50   Input ~ 0
@@
 Text GLabel 8100 4000 2    50   Input ~ 0
 DDR3_RESET
-Text GLabel 8100 2600 2    50   Input ~ 0
+Text GLabel 6600 2600 0    50   Input ~ 0
 DDR3_CS
 Text GLabel 8100 2900 2    50   Input ~ 0
 DDR3_CAS
-Text GLabel 8100 4400 2    50   Input ~ 0
+Text GLabel 8100 4300 2    50   Input ~ 0
 DDR3_RAS
-Text GLabel 6600 2600 0    50   Input ~ 0
+Text GLabel 8100 2600 2    50   Input ~ 0
 DDR3_WE
 Text GLabel 6600 4100 0    50   Input ~ 0
@@
 Text GLabel 6600 4700 0    50   BiDi ~ 0
 DDR3_DQ7
-Text GLabel 6600 1900 0    50   BiDi ~ 0
+Text GLabel 8100 2200 2    50   BiDi ~ 0
 DDR3_DQ10
 Text GLabel 6600 2200 0    50   BiDi ~ 0
 DDR3_DQ11
-Text GLabel 8100 2200 2    50   BiDi ~ 0
+Text GLabel 6600 1900 0    50   BiDi ~ 0
 DDR3_DQ12
 Text GLabel 8100 2300 2    50   BiDi ~ 0
@@
 Text GLabel 8100 4900 2    50   BiDi ~ 0
 DDR3_DQS0-
-Text GLabel 8100 4300 2    50   Input ~ 0
+Text GLabel 8100 4400 2    50   Input ~ 0
 DDR3_A15
 Text GLabel 6600 4200 0    50   Input ~ 0
@@
 Text GLabel 8100 1800 2    50   BiDi ~ 0
 DDR3_DQ13
-Text GLabel 6600 2900 0    50   BiDi ~ 0
+Text GLabel 8100 3100 2    50   BiDi ~ 0
 DDR3_DM0
 Text GLabel 6600 2300 0    50   Input ~ 0
@@
 Text GLabel 6600 1800 0    50   BiDi ~ 0
 DDR3_DQ8
-Text GLabel 6600 3100 0    50   Input ~ 0
+Text GLabel 6600 2100 0    50   Input ~ 0
 DDR3_A0
 Text GLabel 6600 2000 0    50   BiDi ~ 0

Commit message: Almost to 10%
Connections:
- net DDR3_A0: now also U1.F18 (PR14D); no longer U1.F20 (PR38C)
- net DDR3_CAS: now also U1.F20 (PR38C); no longer U1.F18 (PR14D)
Changed lines of the file:
@@
 Text GLabel 6600 2600 0    50   Input ~ 0
 DDR3_CS
-Text GLabel 8100 2900 2    50   Input ~ 0
+Text GLabel 6600 2100 0    50   Input ~ 0
 DDR3_CAS
 Text GLabel 8100 4300 2    50   Input ~ 0
@@
 Text GLabel 6600 1800 0    50   BiDi ~ 0
 DDR3_DQ8
-Text GLabel 6600 2100 0    50   Input ~ 0
+Text GLabel 8100 2900 2    50   Input ~ 0
 DDR3_A0
 Text GLabel 6600 2000 0    50   BiDi ~ 0

Commit message: Adding SDRAM removind DDR3
Connections:
- net DDR3_A0 renamed SDRAM_A0
- net DDR3_A1 renamed SDRAM_A1
- net DDR3_A10 renamed SDRAM_A10
- net DDR3_A11 renamed SDRAM_A11
- net DDR3_A12 renamed SDRAM_A12
- net DDR3_A13: no longer names the net of U1.U20 (PR86D)
- net DDR3_A14: no longer names the net of U1.N20 (PR83B)
- net DDR3_A15: no longer names the net of U1.P18 (PR83D)
- net DDR3_A2 renamed SDRAM_A2
- net DDR3_A3 renamed SDRAM_A3
- net DDR3_A4 renamed SDRAM_A4
- net DDR3_A5 renamed SDRAM_A5
- net DDR3_A6 renamed SDRAM_A6
- net DDR3_A7 renamed SDRAM_A7
- net DDR3_A8 renamed SDRAM_A8
- net DDR3_A9 renamed SDRAM_A9
- net DDR3_BA0 renamed SDRAM_BA0
- net DDR3_BA1 renamed SDRAM_BA1
- net DDR3_BA2: no longer names the net of U1.P20 (PR86A)
- net DDR3_CAS renamed SDRAM_nCAS
- net DDR3_CKE renamed SDRAM_CKE
- net DDR3_CLK+ renamed SDRAM_CLK
- net DDR3_CLK-: no longer names the net of U1.M20 (PCLKC3_1)
- net DDR3_CS renamed SDRAM_nCS
- net DDR3_DM0 renamed SDRAM_D0
- net DDR3_DM1 renamed SDRAM_DQM1
- net DDR3_DQ0 renamed SDRAM_DQM0
- net DDR3_DQ1 renamed SDRAM_D1
- net DDR3_DQ10 renamed SDRAM_D10
- net DDR3_DQ11 renamed SDRAM_D11
- net DDR3_DQ12 renamed SDRAM_D12
- net DDR3_DQ13 renamed SDRAM_D13
- net DDR3_DQ14 renamed SDRAM_D14
- net DDR3_DQ15 renamed SDRAM_D15
- net DDR3_DQ2 renamed SDRAM_D2
- net DDR3_DQ3 renamed SDRAM_D3
- net DDR3_DQ4 renamed SDRAM_D4
- net DDR3_DQ5 renamed SDRAM_D5
- net DDR3_DQ6 renamed SDRAM_D6
- net DDR3_DQ7 renamed SDRAM_D7
- net DDR3_DQ8 renamed SDRAM_D8
- net DDR3_DQ9 renamed SDRAM_D9
- net DDR3_DQS0+: no longer names the net of U1.N16 (PR53A)
- net DDR3_DQS0-: no longer names the net of U1.M17 (PR53B)
- net DDR3_DQS1+: no longer names the net of U1.G19 (GR_PCLK2_1)
- net DDR3_DQS1-: no longer names the net of U1.H20 (PR41B)
- net DDR3_ODT: no longer names the net of U1.T19 (PR89A)
- net DDR3_RAS renamed SDRAM_nRAS
- net DDR3_RESET: no longer names the net of U1.T18 (PR89D)
- net DDR3_VREF: no longer names the net of U1.D20 (VREF1_2)
- net DDR3_VREF: no longer U1.P16 (VREF1_3)
- net DDR3_WE renamed SDRAM_nWE
Changed lines of the file:
@@
 	-1   0    0    1
 $EndComp
-Text GLabel 8100 5100 2    50   Input ~ 0
-DDR3_A1
-Text GLabel 8100 2400 2    50   Input ~ 0
-DDR3_A2
-Text GLabel 6600 2900 0    50   Input ~ 0
-DDR3_A3
-Text GLabel 8100 2700 2    50   Input ~ 0
-DDR3_A4
-Text GLabel 8100 3900 2    50   Input ~ 0
-DDR3_A6
-Text GLabel 8100 3800 2    50   Input ~ 0
-DDR3_A7
-Text GLabel 6600 3100 0    50   Input ~ 0
-DDR3_A8
-Text GLabel 6600 4000 0    50   Input ~ 0
-DDR3_A9
-Text GLabel 6600 2500 0    50   Input ~ 0
-DDR3_A10
-Text GLabel 8100 2500 2    50   Input ~ 0
-DDR3_A11
-Text GLabel 8100 4800 2    50   Input ~ 0
-DDR3_A12
-Text GLabel 8100 4500 2    50   Input ~ 0
-DDR3_A14
-Text GLabel 6600 4400 0    50   Input ~ 0
-DDR3_BA0
-Text GLabel 6600 2700 0    50   Input ~ 0
-DDR3_BA1
-Text GLabel 6600 4300 0    50   Input ~ 0
-DDR3_BA2
-Text GLabel 6600 5300 0    50   Input ~ 0
-DDR3_CLK+
-Text GLabel 8100 5300 2    50   Input ~ 0
-DDR3_CLK-
-Text GLabel 6600 4500 0    50   Input ~ 0
-DDR3_CKE
-Text GLabel 8100 4000 2    50   Input ~ 0
-DDR3_RESET
-Text GLabel 6600 2600 0    50   Input ~ 0
-DDR3_CS
-Text GLabel 6600 2100 0    50   Input ~ 0
-DDR3_CAS
-Text GLabel 8100 4300 2    50   Input ~ 0
-DDR3_RAS
-Text GLabel 8100 2600 2    50   Input ~ 0
-DDR3_WE
-Text GLabel 6600 4100 0    50   Input ~ 0
-DDR3_ODT
-Text GLabel 8100 4600 2    50   BiDi ~ 0
-DDR3_DQ0
-Text GLabel 6600 5200 0    50   BiDi ~ 0
-DDR3_DQ1
-Text GLabel 6600 4600 0    50   BiDi ~ 0
-DDR3_DQ2
-Text GLabel 6600 5100 0    50   BiDi ~ 0
-DDR3_DQ3
-Text GLabel 8100 5000 2    50   BiDi ~ 0
-DDR3_DQ4
-Text GLabel 8100 5200 2    50   BiDi ~ 0
-DDR3_DQ5
-Text GLabel 6600 4800 0    50   BiDi ~ 0
-DDR3_DQ6
-Text GLabel 6600 4700 0    50   BiDi ~ 0
-DDR3_DQ7
-Text GLabel 8100 2200 2    50   BiDi ~ 0
-DDR3_DQ10
-Text GLabel 6600 2200 0    50   BiDi ~ 0
-DDR3_DQ11
-Text GLabel 6600 1900 0    50   BiDi ~ 0
-DDR3_DQ12
-Text GLabel 8100 2300 2    50   BiDi ~ 0
-DDR3_DQ14
-Text GLabel 8100 2100 2    50   BiDi ~ 0
-DDR3_DQ15
-Text GLabel 6600 3800 0    50   BiDi ~ 0
-DDR3_DM1
-Text GLabel 6600 4900 0    50   BiDi ~ 0
-DDR3_DQS0+
-Text GLabel 8100 4900 2    50   BiDi ~ 0
-DDR3_DQS0-
-Text GLabel 8100 4400 2    50   Input ~ 0
-DDR3_A15
-Text GLabel 6600 4200 0    50   Input ~ 0
-DDR3_A5
-Text GLabel 8100 4200 2    50   Input ~ 0
-DDR3_A13
-Text GLabel 6600 2400 0    50   BiDi ~ 0
-DDR3_DQ9
-Text GLabel 8100 1800 2    50   BiDi ~ 0
-DDR3_DQ13
-Text GLabel 8100 3100 2    50   BiDi ~ 0
-DDR3_DM0
-Text GLabel 6600 2300 0    50   Input ~ 0
-DDR3_VREF
-Text GLabel 8100 4700 2    50   Input ~ 0
-DDR3_VREF
-Text GLabel 6600 1800 0    50   BiDi ~ 0
-DDR3_DQ8
-Text GLabel 8100 2900 2    50   Input ~ 0
-DDR3_A0
-Text GLabel 6600 2000 0    50   BiDi ~ 0
-DDR3_DQS1+
-Text GLabel 8100 2000 2    50   BiDi ~ 0
-DDR3_DQS1-
+Text GLabel 8100 4800 2    60   Input ~ 0
+SDRAM_A12
+Text GLabel 6600 2600 0    60   Input ~ 0
+SDRAM_nCS
+Text GLabel 8100 2600 2    60   Input ~ 0
+SDRAM_nWE
+Text GLabel 6600 2100 0    60   Input ~ 0
+SDRAM_nCAS
+Text GLabel 8100 4300 2    60   Input ~ 0
+SDRAM_nRAS
+Text GLabel 6600 4500 0    60   Input ~ 0
+SDRAM_CKE
+Text GLabel 6600 5300 0    60   Input ~ 0
+SDRAM_CLK
+Text GLabel 6600 2700 0    60   Input ~ 0
+SDRAM_BA1
+Text GLabel 6600 4400 0    60   Input ~ 0
+SDRAM_BA0
+Text GLabel 8100 2500 2    60   Input ~ 0
+SDRAM_A11
+Text GLabel 6600 2500 0    60   Input ~ 0
+SDRAM_A10
+Text GLabel 6600 4000 0    60   Input ~ 0
+SDRAM_A9
+Text GLabel 6600 3100 0    60   Input ~ 0
+SDRAM_A8
+Text GLabel 8100 3800 2    60   Input ~ 0
+SDRAM_A7
+Text GLabel 8100 3900 2    60   Input ~ 0
+SDRAM_A6
+Text GLabel 6600 4200 0    60   Input ~ 0
+SDRAM_A5
+Text GLabel 8100 2700 2    60   Input ~ 0
+SDRAM_A4
+Text GLabel 6600 2900 0    60   Input ~ 0
+SDRAM_A3
+Text GLabel 8100 2400 2    60   Input ~ 0
+SDRAM_A2
+Text GLabel 8100 5100 2    60   Input ~ 0
+SDRAM_A1
+Text GLabel 8100 2900 2    60   Input ~ 0
+SDRAM_A0
+Text GLabel 6600 3800 0    60   Input ~ 0
+SDRAM_DQM1
+Text GLabel 8100 4600 2    60   Input ~ 0
+SDRAM_DQM0
+Text GLabel 8100 2100 2    60   Input ~ 0
+SDRAM_D15
+Text GLabel 8100 2300 2    60   Input ~ 0
+SDRAM_D14
+Text GLabel 8100 1800 2    60   Input ~ 0
+SDRAM_D13
+Text GLabel 6600 1900 0    60   Input ~ 0
+SDRAM_D12
+Text GLabel 6600 2200 0    60   Input ~ 0
+SDRAM_D11
+Text GLabel 8100 2200 2    60   Input ~ 0
+SDRAM_D10
+Text GLabel 6600 2400 0    60   Input ~ 0
+SDRAM_D9
+Text GLabel 6600 1800 0    60   Input ~ 0
+SDRAM_D8
+Text GLabel 6600 4700 0    60   Input ~ 0
+SDRAM_D7
+Text GLabel 6600 4800 0    60   Input ~ 0
+SDRAM_D6
+Text GLabel 8100 5200 2    60   Input ~ 0
+SDRAM_D5
+Text GLabel 8100 5000 2    60   Input ~ 0
+SDRAM_D4
+Text GLabel 6600 5100 0    60   Input ~ 0
+SDRAM_D3
+Text GLabel 6600 4600 0    60   Input ~ 0
+SDRAM_D2
+Text GLabel 6600 5200 0    60   Input ~ 0
+SDRAM_D1
+Text GLabel 8100 3100 2    60   Input ~ 0
+SDRAM_D0
 $EndSCHEMATC

Commit message: Finshed routing SDRAM
Connections:
- net SDRAM_A0: now also U1.H16 (PR17D); no longer U1.F18 (PR14D)
- net SDRAM_A1: now also U1.D19 (PR35B); no longer U1.L17 (PR50B)
- net SDRAM_A10: now also U1.C20 (PR35A); no longer U1.J17 (PR20C)
- net SDRAM_A11: now also U1.K19 (PCLKC2_1); no longer U1.J16 (PR20D)
- net SDRAM_A12: now also U1.R20 (PR86B); no longer U1.P17 (PR53D)
- net SDRAM_A2: now also U1.F16 (PR11D); no longer U1.D19 (PR35B)
- net SDRAM_A4: now also U1.T19 (PR89A); no longer U1.H16 (PR17D)
- net SDRAM_A5: now also U1.T18 (PR89D); no longer U1.T20 (PR86C)
- net SDRAM_A6: now also U1.J16 (PR20D); no longer U1.U17 (PR92B)
- net SDRAM_A7: now also U1.P18 (PR83D); no longer U1.T17 (GPLL0C_IN)
- net SDRAM_A8: now also U1.T20 (PR86C); no longer U1.E16 (PR11C)
- net SDRAM_A9: now also U1.L19 (PCLKT3_0); no longer U1.U19 (PR89C)
- net SDRAM_BA0: now also U1.J19 (PCLKT2_1); no longer U1.P19 (PR83C)
- net SDRAM_BA1: now also U1.L16 (GR_PCLK3_0); no longer U1.G16 (PR17C)
- net SDRAM_CKE: now also U1.J17 (PR20C); no longer U1.N19 (PR83A)
- net SDRAM_D0: now also U1.J18 (GR_PCLK2_0); no longer U1.F16 (PR11D)
- net SDRAM_D1: now also U1.G20 (PR38D); no longer U1.L19 (PCLKT3_0)
- net SDRAM_D10: now also U1.M18 (PR50D); no longer U1.F19 (PR38B)
- net SDRAM_D11: now also U1.N20 (PR83B); no longer U1.E20 (PR38A)
- net SDRAM_D12: now also U1.N19 (PR83A); no longer U1.J18 (GR_PCLK2_0)
- net SDRAM_D13: now also U1.M20 (PCLKC3_1); no longer U1.K19 (PCLKC2_1)
- net SDRAM_D14: now also U1.M19 (PCLKC3_0); no longer U1.E19 (PR35D)
- net SDRAM_D15: now also U1.L17 (PR50B); no longer U1.G20 (PR38D)
- net SDRAM_D2: now also U1.G19 (GR_PCLK2_1); no longer U1.R16 (PR56C)
- net SDRAM_D3: now also U1.E16 (PR11C); no longer U1.L16 (GR_PCLK3_0)
- net SDRAM_D4: now also U1.F19 (PR38B); no longer U1.M18 (PR50D)
- net SDRAM_D5: now also U1.F20 (PR38C); no longer U1.M19 (PCLKC3_0)
- net SDRAM_D6: now also U1.H18 (PR20A); no longer U1.N18 (PR53C)
- net SDRAM_D7: now also U1.F18 (PR14D); no longer U1.N17 (PR56A)
- net SDRAM_D8: now also U1.P19 (PR83C); no longer U1.J19 (PCLKT2_1)
- net SDRAM_D9: now also U1.N17 (PR56A); no longer U1.C20 (PR35A)
- net SDRAM_DQM0: now also U1.E20 (PR38A); no longer U1.R17 (PR56D)
- net SDRAM_DQM1: now also U1.P20 (PR86A); no longer U1.U16 (GPLL0T_IN)
- net SDRAM_nCAS: now also U1.H20 (PR41B); no longer U1.F20 (PR38C)
- net SDRAM_nCS: now also U1.D20 (VREF1_2); no longer U1.H18 (PR20A)
- net SDRAM_nRAS: now also U1.G16 (PR17C); no longer U1.R20 (PR86B)
- net SDRAM_nWE: now also U1.E19 (PR35D); no longer U1.H17 (PR20B)
- new net Camera_GPIO: U1.U19 (PR89C)
- new net SCL0: U1.U17 (PR92B)
- new net SDA0: U1.T17 (GPLL0C_IN)
- new net SD_D1: U1.R16 (PR56C)
Changed lines of the file:
@@
 	-1   0    0    1
 $EndComp
-Text GLabel 8100 4800 2    60   Input ~ 0
+Text GLabel 8100 4300 2    60   Input ~ 0
 SDRAM_A12
-Text GLabel 6600 2600 0    60   Input ~ 0
+Text GLabel 6600 2300 0    60   Input ~ 0
 SDRAM_nCS
-Text GLabel 8100 2600 2    60   Input ~ 0
+Text GLabel 8100 2300 2    60   Input ~ 0
 SDRAM_nWE
-Text GLabel 6600 2100 0    60   Input ~ 0
+Text GLabel 8100 2000 2    60   Input ~ 0
 SDRAM_nCAS
-Text GLabel 8100 4300 2    60   Input ~ 0
-SDRAM_nRAS
-Text GLabel 6600 4500 0    60   Input ~ 0
+Text GLabel 6600 2500 0    60   Input ~ 0
 SDRAM_CKE
 Text GLabel 6600 5300 0    60   Input ~ 0
 SDRAM_CLK
-Text GLabel 6600 2700 0    60   Input ~ 0
+Text GLabel 6600 5100 0    60   Input ~ 0
 SDRAM_BA1
-Text GLabel 6600 4400 0    60   Input ~ 0
-SDRAM_BA0
+Text GLabel 6600 2400 0    60   Input ~ 0
+SDRAM_A10
+Text GLabel 6600 4200 0    60   Input ~ 0
+SDRAM_A8
+Text GLabel 8100 4400 2    60   Input ~ 0
+SDRAM_A7
 Text GLabel 8100 2500 2    60   Input ~ 0
-SDRAM_A11
-Text GLabel 6600 2500 0    60   Input ~ 0
-SDRAM_A10
-Text GLabel 6600 4000 0    60   Input ~ 0
-SDRAM_A9
-Text GLabel 6600 3100 0    60   Input ~ 0
-SDRAM_A8
-Text GLabel 8100 3800 2    60   Input ~ 0
-SDRAM_A7
-Text GLabel 8100 3900 2    60   Input ~ 0
 SDRAM_A6
-Text GLabel 6600 4200 0    60   Input ~ 0
+Text GLabel 8100 4000 2    60   Input ~ 0
 SDRAM_A5
-Text GLabel 8100 2700 2    60   Input ~ 0
+Text GLabel 6600 4100 0    60   Input ~ 0
 SDRAM_A4
 Text GLabel 6600 2900 0    60   Input ~ 0
 SDRAM_A3
+Text GLabel 8100 3100 2    60   Input ~ 0
+SDRAM_A2
 Text GLabel 8100 2400 2    60   Input ~ 0
-SDRAM_A2
+SDRAM_A1
+Text GLabel 8100 2700 2    60   Input ~ 0
+SDRAM_A0
+Text GLabel 6600 4300 0    60   Input ~ 0
+SDRAM_DQM1
+Text GLabel 8100 5200 2    60   Input ~ 0
+SDRAM_D14
+Text GLabel 8100 5000 2    60   Input ~ 0
+SDRAM_D10
+Text GLabel 6600 4700 0    60   Input ~ 0
+SDRAM_D9
+Text GLabel 6600 4400 0    60   Input ~ 0
+SDRAM_D8
+Text GLabel 8100 2900 2    60   Input ~ 0
+SDRAM_D7
+Text GLabel 6600 2600 0    60   Input ~ 0
+SDRAM_D6
+Text GLabel 6600 2100 0    60   Input ~ 0
+SDRAM_D5
+Text GLabel 8100 2200 2    60   Input ~ 0
+SDRAM_D4
+Text GLabel 6600 3100 0    60   Input ~ 0
+SDRAM_D3
+Text GLabel 6600 2000 0    60   Input ~ 0
+SDRAM_D2
+Text GLabel 8100 2100 2    60   Input ~ 0
+SDRAM_D1
+Text GLabel 6600 2200 0    60   Input ~ 0
+SDRAM_DQM0
+Text GLabel 8100 4500 2    60   Input ~ 0
+SDRAM_D11
+Text GLabel 6600 1900 0    60   Input ~ 0
+SDRAM_D0
+Text GLabel 6600 4500 0    60   Input ~ 0
+SDRAM_D12
+Text GLabel 6600 1800 0    60   Input ~ 0
+SDRAM_BA0
+Text GLabel 6600 2700 0    60   Input ~ 0
+SDRAM_nRAS
+Text GLabel 8100 1800 2    60   Input ~ 0
+SDRAM_A11
+Text GLabel 8100 5300 2    60   Input ~ 0
+SDRAM_D13
+Text GLabel 6600 5200 0    60   Input ~ 0
+SDRAM_A9
 Text GLabel 8100 5100 2    60   Input ~ 0
-SDRAM_A1
-Text GLabel 8100 2900 2    60   Input ~ 0
-SDRAM_A0
-Text GLabel 6600 3800 0    60   Input ~ 0
-SDRAM_DQM1
-Text GLabel 8100 4600 2    60   Input ~ 0
-SDRAM_DQM0
-Text GLabel 8100 2100 2    60   Input ~ 0
 SDRAM_D15
-Text GLabel 8100 2300 2    60   Input ~ 0
-SDRAM_D14
-Text GLabel 8100 1800 2    60   Input ~ 0
-SDRAM_D13
-Text GLabel 6600 1900 0    60   Input ~ 0
-SDRAM_D12
-Text GLabel 6600 2200 0    60   Input ~ 0
-SDRAM_D11
-Text GLabel 8100 2200 2    60   Input ~ 0
-SDRAM_D10
-Text GLabel 6600 2400 0    60   Input ~ 0
-SDRAM_D9
-Text GLabel 6600 1800 0    60   Input ~ 0
-SDRAM_D8
-Text GLabel 6600 4700 0    60   Input ~ 0
-SDRAM_D7
-Text GLabel 6600 4800 0    60   Input ~ 0
-SDRAM_D6
-Text GLabel 8100 5200 2    60   Input ~ 0
-SDRAM_D5
-Text GLabel 8100 5000 2    60   Input ~ 0
-SDRAM_D4
-Text GLabel 6600 5100 0    60   Input ~ 0
-SDRAM_D3
 Text GLabel 6600 4600 0    60   Input ~ 0
-SDRAM_D2
-Text GLabel 6600 5200 0    60   Input ~ 0
-SDRAM_D1
-Text GLabel 8100 3100 2    60   Input ~ 0
-SDRAM_D0
+SD_D1
+Text GLabel 8100 3900 2    60   Input ~ 0
+SCL0
+Text GLabel 8100 3800 2    60   Input ~ 0
+SDA0
+Text GLabel 6600 4000 0    60   Input ~ 0
+Camera_GPIO
 $EndSCHEMATC

Commit message: Adding more pins
Connections:
- net RUN_PG: now reaches U1.U16 (GPLL0T_IN)
- net GLOBAL_EN: now reaches U1.U18 (PR92A)
- net nEXTRST: now reaches U1.U20 (PR86D)
Changed lines of the file:
@@
 Text GLabel 6600 4000 0    60   Input ~ 0
 Camera_GPIO
+Text GLabel 8100 4200 2    60   Input ~ 0
+nEXTRST
+Text GLabel 6600 3900 0    60   Input ~ 0
+GLOBAL_EN
+Text GLabel 6600 3800 0    60   Input ~ 0
+RUN_PG
 $EndSCHEMATC

Commit message: Removing SD-CARD sharing feature to get more GPIO pins
Connections:
- net GPIO2: now reaches U1.M17 (PR53B)
- net GPIO15: now reaches U1.N16 (PR53A)
- net GPIO14: now reaches U1.N18 (PR53C)
- net GPIO4: now reaches U1.P16 (VREF1_3)
- net GPIO3: now reaches U1.P17 (PR53D)
Changed lines of the file:
@@
 Text GLabel 6600 3800 0    60   Input ~ 0
 RUN_PG
+Text GLabel 6600 4900 0    60   Input ~ 0
+GPIO15
+Text GLabel 6600 4800 0    60   Input ~ 0
+GPIO14
+Text GLabel 8100 4700 2    60   Input ~ 0
+GPIO4
+Text GLabel 8100 4800 2    60   Input ~ 0
+GPIO3
+Text GLabel 8100 4900 2    60   Input ~ 0
+GPIO2
 $EndSCHEMATC

Commit message: Connecting DSI1 to DSI0
Connections:
- net SW2: now reaches U1.K18 (PR41D)
- net SW1: now reaches U1.L18 (GR_PCLK3_1)
- net GPIO27: now reaches U1.R17 (PR56D)
Changed lines of the file:
@@
 Text GLabel 8100 4900 2    60   Input ~ 0
 GPIO2
+Text GLabel 8100 4600 2    60   Input ~ 0
+GPIO27
+Text GLabel 6600 5000 0    60   Input ~ 0
+SW1
+Text GLabel 8100 1900 2    60   Input ~ 0
+SW2
 $EndSCHEMATC
