File: serdes.sch (KiCad schematic (older format))
At the start: 11 parts, among them U1 LFE5U-85F-6BG381C

Commit message: More removing
Parts:
- removed C63, C64, C65, C66, C67, C68, C69, C70, C71, C72: 22nF, Capacitor_SMD:C_0603_1608Metric, symbol Device:C
Changed lines of the file:
@@
 Wire Wire Line
 	6650 3200 6650 3250
-$Comp
-L Device:C C?
-U 1 1 5F8D5462
-P 4150 1950
-AR Path="/58D686D9/5F8D5462" Ref="C?"  Part="1"
-AR Path="/58DA7327/5F8D5462" Ref="C67"  Part="1"
-F 0 "C67" V 4200 2000 50  0000 L CNN
-F 1 "22nF" V 4200 1700 50  0000 L CNN
-F 2 "Capacitor_SMD:C_0603_1608Metric" H 4188 1800 50  0001 C CNN
-F 3 "" H 4150 1950 50  0000 C CNN
-	1    4150 1950
-	0    -1   1    0
-$EndComp
-$Comp
-L Device:C C?
-U 1 1 5F8D5468
-P 7250 3600
-AR Path="/58D686D9/5F8D5468" Ref="C?"  Part="1"
-AR Path="/58DA7327/5F8D5468" Ref="C70"  Part="1"
-F 0 "C70" V 7300 3650 50  0000 L CNN
-F 1 "22nF" V 7300 3350 50  0000 L CNN
-F 2 "Capacitor_SMD:C_0603_1608Metric" H 7288 3450 50  0001 C CNN
-F 3 "" H 7250 3600 50  0000 C CNN
-	1    7250 3600
-	0    -1   1    0
-$EndComp
-$Comp
-L Device:C C?
-U 1 1 5F8D546E
-P 4150 3600
-AR Path="/58D686D9/5F8D546E" Ref="C?"  Part="1"
-AR Path="/58DA7327/5F8D546E" Ref="C69"  Part="1"
-F 0 "C69" V 4200 3650 50  0000 L CNN
-F 1 "22nF" V 4200 3350 50  0000 L CNN
-F 2 "Capacitor_SMD:C_0603_1608Metric" H 4188 3450 50  0001 C CNN
-F 3 "" H 4150 3600 50  0000 C CNN
-	1    4150 3600
-	0    -1   1    0
-$EndComp
-$Comp
-L Device:C C?
-U 1 1 5F8D5474
-P 7250 2350
-AR Path="/58D686D9/5F8D5474" Ref="C?"  Part="1"
-AR Path="/58DA7327/5F8D5474" Ref="C66"  Part="1"
-F 0 "C66" V 7300 2400 50  0000 L CNN
-F 1 "22nF" V 7300 2100 50  0000 L CNN
-F 2 "Capacitor_SMD:C_0603_1608Metric" H 7288 2200 50  0001 C CNN
-F 3 "" H 7250 2350 50  0000 C CNN
-	1    7250 2350
-	0    -1   1    0
-$EndComp
-$Comp
-L Device:C C?
-U 1 1 5F8D547D
-P 7250 1950
-AR Path="/58D686D9/5F8D547D" Ref="C?"  Part="1"
-AR Path="/58DA7327/5F8D547D" Ref="C68"  Part="1"
-F 0 "C68" V 7300 2000 50  0000 L CNN
-F 1 "22nF" V 7300 1700 50  0000 L CNN
-F 2 "Capacitor_SMD:C_0603_1608Metric" H 7288 1800 50  0001 C CNN
-F 3 "" H 7250 1950 50  0000 C CNN
-	1    7250 1950
-	0    -1   1    0
-$EndComp
-$Comp
-L Device:C C?
-U 1 1 5F8D5483
-P 4150 2350
-AR Path="/58D686D9/5F8D5483" Ref="C?"  Part="1"
-AR Path="/58DA7327/5F8D5483" Ref="C65"  Part="1"
-F 0 "C65" V 4200 2400 50  0000 L CNN
-F 1 "22nF" V 4200 2100 50  0000 L CNN
-F 2 "Capacitor_SMD:C_0603_1608Metric" H 4188 2200 50  0001 C CNN
-F 3 "" H 4150 2350 50  0000 C CNN
-	1    4150 2350
-	0    -1   1    0
-$EndComp
-$Comp
-L Device:C C?
-U 1 1 5F8D548B
-P 4150 2150
-AR Path="/58D686D9/5F8D548B" Ref="C?"  Part="1"
-AR Path="/58DA7327/5F8D548B" Ref="C63"  Part="1"
-F 0 "C63" V 4200 2200 50  0000 L CNN
-F 1 "22nF" V 4200 1900 50  0000 L CNN
-F 2 "Capacitor_SMD:C_0603_1608Metric" H 4188 2000 50  0001 C CNN
-F 3 "" H 4150 2150 50  0000 C CNN
-	1    4150 2150
-	0    -1   1    0
-$EndComp
-$Comp
-L Device:C C?
-U 1 1 5F8D5491
-P 7250 2150
-AR Path="/58D686D9/5F8D5491" Ref="C?"  Part="1"
-AR Path="/58DA7327/5F8D5491" Ref="C64"  Part="1"
-F 0 "C64" V 7300 2200 50  0000 L CNN
-F 1 "22nF" V 7300 1900 50  0000 L CNN
-F 2 "Capacitor_SMD:C_0603_1608Metric" H 7288 2000 50  0001 C CNN
-F 3 "" H 7250 2150 50  0000 C CNN
-	1    7250 2150
-	0    -1   1    0
-$EndComp
 Wire Wire Line
 	6550 2150 7100 2150
@@
 Wire Wire Line
 	6550 1950 7100 1950
-$Comp
-L Device:C C?
-U 1 1 5F8FD0D7
-P 3800 3700
-AR Path="/58D686D9/5F8FD0D7" Ref="C?"  Part="1"
-AR Path="/58DA7327/5F8FD0D7" Ref="C71"  Part="1"
-F 0 "C71" V 3850 3750 50  0000 L CNN
-F 1 "22nF" V 3850 3450 50  0000 L CNN
-F 2 "Capacitor_SMD:C_0603_1608Metric" H 3838 3550 50  0001 C CNN
-F 3 "" H 3800 3700 50  0000 C CNN
-	1    3800 3700
-	0    -1   1    0
-$EndComp
-$Comp
-L Device:C C?
-U 1 1 5F9001C5
-P 7600 3700
-AR Path="/58D686D9/5F9001C5" Ref="C?"  Part="1"
-AR Path="/58DA7327/5F9001C5" Ref="C72"  Part="1"
-F 0 "C72" V 7650 3750 50  0000 L CNN
-F 1 "22nF" V 7650 3450 50  0000 L CNN
-F 2 "Capacitor_SMD:C_0603_1608Metric" H 7638 3550 50  0001 C CNN
-F 3 "" H 7600 3700 50  0000 C CNN
-	1    7600 3700
-	0    -1   1    0
-$EndComp
 Wire Wire Line
 	6550 3700 7450 3700

Commit message: Before power placement
Parts:
- added C55, C56, C57, C58, C59, C61, C62, C63, C64, C65, C66, C67, C68, C69, C70, C71, C72, C73, C74, C75: 22n, Capacitor_SMD:C_0402_1005Metric, symbol Device:C_Small
Connections:
- net labels added: CLK_0_N, CLK_0_P, CLK_1_N, CLK_1_P, PCIe_CLK_N, PCIe_CLK_P, PCIe_CLK_nREQ, PCIe_RX_N, PCIe_RX_P, PCIe_TX_N, PCIe_TX_P, SRCLK0N, SRCLK0P, SRCLK1N, SRCLK1P, SRX00P, SRX01P, SRX10N, SRX10P, SRX11N, SRX11P, STX00P, STX01P, STX10N, STX10P, STX11N, STX11P, STXN00, STXN01, S_0_N, S_0_P, S_1_N, S_1_P, S_2_N, S_2_P, S_3_N, S_3_P, S_4_N, S_4_P, S_5_N, S_5_P, S_6_N, S_6_P, S_7_N, S_7_P
- net labels removed: OLED_BL, OLED_CLK, OLED_CS, OLED_DC, OLED_MOSI, OLED_RES, SRCLKN, SRCLKP, SRXN10, SRXP00, SRXP01, SRXP10, STXN11, STXP11
- wire segments 50 -> 80
- no-connect marks 14 -> 0

Commit message: Routing cam and display differential
Changed lines of the file:
@@
 Text Label 6650 3800 0    60   ~ 0
 S_5_N
-Text GLabel 10250 1450 2    60   Input ~ 0
-PCIe_CLK_nREQ
 Text GLabel 10250 1550 2    60   Input ~ 0
 PCIe_CLK_P

Commit message: Connecting serdes to gpio
Connections:
- net SRX01P renamed ETH_3P
- net SRX10N renamed ETH_0N
- net SRX10P renamed ETH_0P
- net SRXN01 renamed ETH_3N
- net STX01P renamed ETH_2P
- net STX10N renamed ETH_1N
- net STX10P renamed ETH_1P
- net STXN01 renamed ETH_2N
Changed lines of the file:
@@
 	4300 2150 4850 2150
 Text GLabel 7400 2150 2    60   Input ~ 0
-SRXN00
+SRX00N
 Wire Wire Line
 	6550 2350 7100 2350
@@
 Text GLabel 4050 2350 0    60   Input ~ 0
 SRX01P
-Text GLabel 7400 2350 2    60   Input ~ 0
-SRXN01
 Text Label 4450 1950 0    60   ~ 0
 CLK_0_P
@@
 Wire Wire Line
 	4050 2350 4100 2350
-Text GLabel 3400 2250 0    60   Input ~ 0
-STX01P
 Wire Wire Line
 	3400 2250 3450 2250
@@
 	0    -1   -1   0
 $EndComp
-Text GLabel 8100 2050 2    60   Input ~ 0
-STXN00
 Wire Wire Line
 	7300 1950 7400 1950
@@
 Wire Wire Line
 	8000 2250 8100 2250
-Text GLabel 8100 2250 2    60   Input ~ 0
-STXN01
 Wire Wire Line
 	6550 2050 7800 2050
@@
 	0    -1   -1   0
 $EndComp
-Text GLabel 3350 3500 0    60   Input ~ 0
-STX10P
 Text GLabel 3350 3700 0    60   Input ~ 0
 STX11P
@@
 Wire Wire Line
 	6550 3700 7800 3700
-Text GLabel 8100 3500 2    60   Input ~ 0
-STX10N
 Wire Wire Line
 	8000 3500 8100 3500
@@
 SRCLK0P
 Text GLabel 10050 1850 0    60   Input ~ 0
-SRXN00
+SRX00N
 Text GLabel 10050 1750 0    60   Input ~ 0
 SRX00P
@@
 STX00P
 Text GLabel 10050 2050 0    60   Input ~ 0
-STXN00
+STX00N
 Wire Wire Line
 	10050 1550 10250 1550
@@
 Wire Wire Line
 	10250 2050 10050 2050
+Text GLabel 3400 2250 0    60   Input ~ 0
+STX01P
+Text GLabel 3350 3500 0    60   Input ~ 0
+STX10P
+Text GLabel 8100 3500 2    60   Input ~ 0
+STX10N
+Text GLabel 7400 2350 2    60   Input ~ 0
+SRX01N
+Text GLabel 8100 2050 2    60   Input ~ 0
+STX00N
+Text GLabel 8100 2250 2    60   Input ~ 0
+STX01N
+Text GLabel 10150 2450 0    60   Input ~ 0
+SRX10N
+Text GLabel 10150 2350 0    60   Input ~ 0
+SRX10P
+Text GLabel 10150 2700 0    60   Input ~ 0
+STX10N
+Text GLabel 10150 2600 0    60   Input ~ 0
+STX10P
+Text GLabel 10150 3200 0    60   Input ~ 0
+STX01N
+Text GLabel 10150 3100 0    60   Input ~ 0
+STX01P
+Text GLabel 10150 2950 0    60   Input ~ 0
+SRX01N
+Text GLabel 10150 2850 0    60   Input ~ 0
+SRX01P
+Text GLabel 10350 2850 2    60   Input ~ 0
+ETH_3P
+Text GLabel 10350 2950 2    60   Input ~ 0
+ETH_3N
+Text GLabel 10350 3200 2    60   Input ~ 0
+ETH_2N
+Text GLabel 10350 3100 2    60   Input ~ 0
+ETH_2P
+Text GLabel 10350 2700 2    60   Input ~ 0
+ETH_1N
+Text GLabel 10350 2600 2    60   Input ~ 0
+ETH_1P
+Wire Wire Line
+	10150 2350 10350 2350
+Wire Wire Line
+	10350 2450 10150 2450
+Wire Wire Line
+	10150 2600 10350 2600
+Wire Wire Line
+	10350 2700 10150 2700
+Wire Wire Line
+	10150 2850 10350 2850
+Wire Wire Line
+	10350 2950 10150 2950
+Wire Wire Line
+	10150 3100 10350 3100
+Wire Wire Line
+	10350 3200 10150 3200
+Text GLabel 10350 2450 2    60   Input ~ 0
+ETH_0N
+Text GLabel 10350 2350 2    60   Input ~ 0
+ETH_0P
 $EndSCHEMATC

Commit message: Fixing SERDES, adding different connector as emard requested
Parts:
- added RX1, TX1: Antenna, Connector_PinHeader_2.00mm:PinHeader_1x02_P2.00mm_Vertical, symbol Device:Antenna_Dipole
Connections:
- net S_5_N: now also RX1.1
- net S_5_P: now also RX1.2
- net S_7_N: now also TX1.1
- net S_7_P: now also TX1.2
Changed lines of the file:
@@
 Text GLabel 10350 2350 2    60   Input ~ 0
 ETH_0P
+Text Label 5550 4775 3    60   ~ 0
+S_7_P
+Text Label 5450 4775 3    60   ~ 0
+S_7_N
+$Comp
+L Device:Antenna_Dipole AE?
+U 1 1 61A9CB12
+P 5450 4500
+AR Path="/58D6D447/61A9CB12" Ref="AE?"  Part="1"
+AR Path="/58DA7327/61A9CB12" Ref="TX1"  Part="1"
+F 0 "TX1" H 5530 4489 50  0000 L CNN
+F 1 "Antenna" V 5600 4075 50  0000 L CNN
+F 2 "Connector_PinHeader_2.00mm:PinHeader_1x02_P2.00mm_Vertical" H 5450 4500 50  0001 C CNN
+F 3 "~" H 5450 4500 50  0001 C CNN
+	1    5450 4500
+	1    0    0    -1
+$EndComp
+Text Label 6150 4775 3    60   ~ 0
+S_5_P
+Text Label 6050 4775 3    60   ~ 0
+S_5_N
+$Comp
+L Device:Antenna_Dipole AE?
+U 1 1 61C0795C
+P 6050 4500
+AR Path="/58D6D447/61C0795C" Ref="AE?"  Part="1"
+AR Path="/58DA7327/61C0795C" Ref="RX1"  Part="1"
+F 0 "RX1" H 6130 4489 50  0000 L CNN
+F 1 "Antenna" V 6225 4075 50  0000 L CNN
+F 2 "Connector_PinHeader_2.00mm:PinHeader_1x02_P2.00mm_Vertical" H 6050 4500 50  0001 C CNN
+F 3 "~" H 6050 4500 50  0001 C CNN
+	1    6050 4500
+	1    0    0    -1
+$EndComp
+Wire Wire Line
+	6150 4700 6150 4775
+Wire Wire Line
+	6050 4700 6050 4775
+Wire Wire Line
+	5550 4700 5550 4775
+Wire Wire Line
+	5450 4700 5450 4775
 $EndSCHEMATC
