File: serdes.sch (KiCad schematic (older format))
At the start: 23 parts, among them U1 LFE5U-85F-6BG381C

Commit message: References cleanup
Parts:
- removed RX1, TX1: Antenna, Connector_PinHeader_2.00mm:PinHeader_1x02_P2.00mm_Vertical, symbol Device:Antenna_Dipole
- added J4: Antenna, Connector_PinHeader_2.54mm:PinHeader_1x04_P2.54mm_Vertical, symbol Connector:Conn_01x04_Male
Connections:
- net S_5_N: now also J4.3 (Pin_3)
- net S_5_P: now also J4.4 (Pin_4)
- net S_7_N: now also J4.1 (Pin_1)
- net S_7_P: now also J4.2 (Pin_2)
Changed lines of the file:
@@
 $Descr A4 11693 8268
 encoding utf-8
-Sheet 11 13
+Sheet 11 11
 Title "ULX3S"
 Date ""
@@
 Text GLabel 10350 2350 2    60   Input ~ 0
 ETH_0P
-Text Label 5550 4775 3    60   ~ 0
+Text Label 7025 4625 0    60   ~ 0
 S_7_P
-Text Label 5450 4775 3    60   ~ 0
+Text Label 7025 4525 0    60   ~ 0
 S_7_N
-$Comp
-L Device:Antenna_Dipole AE?
-U 1 1 61A9CB12
-P 5450 4500
-AR Path="/58D6D447/61A9CB12" Ref="AE?"  Part="1"
-AR Path="/58DA7327/61A9CB12" Ref="TX1"  Part="1"
-F 0 "TX1" H 5530 4489 50  0000 L CNN
-F 1 "Antenna" V 5600 4075 50  0000 L CNN
-F 2 "Connector_PinHeader_2.00mm:PinHeader_1x02_P2.00mm_Vertical" H 5450 4500 50  0001 C CNN
-F 3 "~" H 5450 4500 50  0001 C CNN
-	1    5450 4500
+Text Label 7025 4825 0    60   ~ 0
+S_5_P
+Text Label 7025 4725 0    60   ~ 0
+S_5_N
+$Comp
+L Connector:Conn_01x04_Male J4
+U 1 1 651DE45E
+P 6825 4625
+F 0 "J4" H 6950 4950 50  0000 C CNN
+F 1 "Antenna" H 6950 4850 50  0000 C CNN
+F 2 "Connector_PinHeader_2.54mm:PinHeader_1x04_P2.54mm_Vertical" H 6825 4625 50  0001 C CNN
+F 3 "~" H 6825 4625 50  0001 C CNN
+	1    6825 4625
 	1    0    0    -1
 $EndComp
-Text Label 6150 4775 3    60   ~ 0
-S_5_P
-Text Label 6050 4775 3    60   ~ 0
-S_5_N
-$Comp
-L Device:Antenna_Dipole AE?
-U 1 1 61C0795C
-P 6050 4500
-AR Path="/58D6D447/61C0795C" Ref="AE?"  Part="1"
-AR Path="/58DA7327/61C0795C" Ref="RX1"  Part="1"
-F 0 "RX1" H 6130 4489 50  0000 L CNN
-F 1 "Antenna" V 6225 4075 50  0000 L CNN
-F 2 "Connector_PinHeader_2.00mm:PinHeader_1x02_P2.00mm_Vertical" H 6050 4500 50  0001 C CNN
-F 3 "~" H 6050 4500 50  0001 C CNN
-	1    6050 4500
-	1    0    0    -1
-$EndComp
-Wire Wire Line
-	6150 4700 6150 4775
-Wire Wire Line
-	6050 4700 6050 4775
-Wire Wire Line
-	5550 4700 5550 4775
-Wire Wire Line
-	5450 4700 5450 4775
 $EndSCHEMATC

Commit message: Addressing #39 on DDR3 version
Parts:
- added C125, C126, C127, C128: 22n, Capacitor_SMD:C_0201_0603Metric, symbol Device:C_Small
Connections:
- net S_5_N: now also C127.2; no longer J4.3 (Pin_3)
- net S_5_P: now also C128.2; no longer J4.4 (Pin_4)
- net S_7_N: now also C125.2; no longer J4.1 (Pin_1)
- net S_7_P: now also C126.2; no longer J4.2 (Pin_2)
- new net 1N: C125.1, J4.1 (Pin_1)
- new net 1P: C126.1, J4.2 (Pin_2)
- new net 2N: C127.1, J4.3 (Pin_3)
- new net 2P: C128.1, J4.4 (Pin_4)
Changed lines of the file:
@@
 Text GLabel 10350 2350 2    60   Input ~ 0
 ETH_0P
-Text Label 7025 4625 0    60   ~ 0
+Text Label 7900 4675 0    60   ~ 0
 S_7_P
-Text Label 7025 4525 0    60   ~ 0
+Text Label 7900 4575 0    60   ~ 0
 S_7_N
-Text Label 7025 4825 0    60   ~ 0
+Text Label 7900 4875 0    60   ~ 0
 S_5_P
-Text Label 7025 4725 0    60   ~ 0
+Text Label 7900 4775 0    60   ~ 0
 S_5_N
 $Comp
@@
 	1    0    0    -1
 $EndComp
+$Comp
+L Device:C_Small C?
+U 1 1 6350E877
+P 7450 4450
+AR Path="/58D686D9/6350E877" Ref="C?"  Part="1"
+AR Path="/58DA7327/6350E877" Ref="C125"  Part="1"
+F 0 "C125" V 7500 4350 50  0000 C CNN
+F 1 "22n" V 7400 4300 50  0000 C CNN
+F 2 "Capacitor_SMD:C_0201_0603Metric" H 7450 4450 50  0001 C CNN
+F 3 "~" H 7450 4450 50  0001 C CNN
+	1    7450 4450
+	0    -1   -1   0
+$EndComp
+$Comp
+L Device:C_Small C?
+U 1 1 6350FD45
+P 7450 4600
+AR Path="/58D686D9/6350FD45" Ref="C?"  Part="1"
+AR Path="/58DA7327/6350FD45" Ref="C126"  Part="1"
+F 0 "C126" V 7500 4500 50  0000 C CNN
+F 1 "22n" V 7400 4450 50  0000 C CNN
+F 2 "Capacitor_SMD:C_0201_0603Metric" H 7450 4600 50  0001 C CNN
+F 3 "~" H 7450 4600 50  0001 C CNN
+	1    7450 4600
+	0    -1   -1   0
+$EndComp
+$Comp
+L Device:C_Small C?
+U 1 1 63513BA5
+P 7450 4750
+AR Path="/58D686D9/63513BA5" Ref="C?"  Part="1"
+AR Path="/58DA7327/63513BA5" Ref="C127"  Part="1"
+F 0 "C127" V 7500 4650 50  0000 C CNN
+F 1 "22n" V 7400 4600 50  0000 C CNN
+F 2 "Capacitor_SMD:C_0201_0603Metric" H 7450 4750 50  0001 C CNN
+F 3 "~" H 7450 4750 50  0001 C CNN
+	1    7450 4750
+	0    -1   -1   0
+$EndComp
+$Comp
+L Device:C_Small C?
+U 1 1 63514512
+P 7450 4900
+AR Path="/58D686D9/63514512" Ref="C?"  Part="1"
+AR Path="/58DA7327/63514512" Ref="C128"  Part="1"
+F 0 "C128" V 7500 4800 50  0000 C CNN
+F 1 "22n" V 7400 4750 50  0000 C CNN
+F 2 "Capacitor_SMD:C_0201_0603Metric" H 7450 4900 50  0001 C CNN
+F 3 "~" H 7450 4900 50  0001 C CNN
+	1    7450 4900
+	0    -1   -1   0
+$EndComp
+Wire Wire Line
+	7175 4525 7175 4450
+Wire Wire Line
+	7175 4450 7350 4450
+Wire Wire Line
+	7025 4525 7175 4525
+Wire Wire Line
+	7025 4625 7175 4625
+Wire Wire Line
+	7175 4625 7175 4600
+Wire Wire Line
+	7175 4600 7350 4600
+Wire Wire Line
+	7025 4725 7350 4725
+Wire Wire Line
+	7350 4725 7350 4750
+Wire Wire Line
+	7025 4825 7350 4825
+Wire Wire Line
+	7350 4825 7350 4900
+Text Label 7175 4450 0    60   ~ 0
+1N
+Text Label 7175 4600 0    60   ~ 0
+1P
+Text Label 7175 4725 0    60   ~ 0
+2N
+Text Label 7175 4825 0    60   ~ 0
+2P
+Wire Wire Line
+	7550 4450 7900 4450
+Wire Wire Line
+	7900 4450 7900 4575
+Wire Wire Line
+	7550 4600 7775 4600
+Wire Wire Line
+	7775 4600 7775 4675
+Wire Wire Line
+	7775 4675 7900 4675
+Wire Wire Line
+	7550 4750 7775 4750
+Wire Wire Line
+	7775 4750 7775 4775
+Wire Wire Line
+	7775 4775 7900 4775
+Wire Wire Line
+	7550 4900 7775 4900
+Wire Wire Line
+	7775 4900 7775 4875
+Wire Wire Line
+	7775 4875 7900 4875
 $EndSCHEMATC
