File: wifi.sch (KiCad schematic (older format))
At the start: 0 parts

Commit message: Connecting more GPIOs, improving routing
Parts:
- added AE1: Antenna, Connector_Coaxial:CoaxialSwitch_Hirose_MS-156C3_Horizontal, symbol Device:Antenna
Changed lines of the file:
@@
 Text GLabel 8100 4250 0    60   Input ~ 0
 WIFI_GPIO0
+$Comp
+L Device:Antenna AE1
+U 1 1 61DC15E3
+P 8650 1650
+F 0 "AE1" H 8730 1639 50  0000 L CNN
+F 1 "Antenna" H 8730 1548 50  0000 L CNN
+F 2 "Connector_Coaxial:CoaxialSwitch_Hirose_MS-156C3_Horizontal" H 8650 1650 50  0001 C CNN
+F 3 "~" H 8650 1650 50  0001 C CNN
+	1    8650 1650
+	1    0    0    -1
+$EndComp
 $EndSCHEMATC

Commit message: Fixing SERDES, adding different connector as emard requested
Parts:
- removed AE1: Antenna, Connector_Coaxial:CoaxialSwitch_Hirose_MS-156C3_Horizontal, symbol Device:Antenna
Changed lines of the file:
@@
 Text GLabel 8100 4250 0    60   Input ~ 0
 WIFI_GPIO0
-$Comp
-L Device:Antenna AE1
-U 1 1 61DC15E3
-P 8650 1650
-F 0 "AE1" H 8730 1639 50  0000 L CNN
-F 1 "Antenna" H 8730 1548 50  0000 L CNN
-F 2 "Connector_Coaxial:CoaxialSwitch_Hirose_MS-156C3_Horizontal" H 8650 1650 50  0001 C CNN
-F 3 "~" H 8650 1650 50  0001 C CNN
-	1    8650 1650
-	1    0    0    -1
-$EndComp
 $EndSCHEMATC
