File: wifi.sch (KiCad schematic (older format))
At the start: 9 parts, among them J3 WIFI_OFF, U9 ESP32

Commit message: More removing
Parts:
- removed C15, C21: 22uF, Capacitor_SMD:C_0805_2012Metric, symbol Device:C
- removed J3: WIFI_OFF, Connector_PinHeader_2.54mm:PinHeader_1x02_P2.54mm_Vertical, symbol Connector_Generic:Conn_02x01
- removed R34, R56: 15k, Resistor_SMD:R_0603_1608Metric, symbol Device:R
- removed R35: 549, Resistor_SMD:R_0603_1608Metric, symbol Device:R
- removed R38: 0.47, Resistor_SMD:R_0603_1608Metric, symbol Device:R
- removed SD1: 104031-0811, micro-sd-schd3a0100-104031-811:SCHD3A100-104031-0811, symbol micro_sd_slide:104031-0811
- removed U9: ESP32, ESP32:ESP32, symbol esp32:ESP32-WROOM-WROVER
Connections:
- net labels removed: +3V3, GND, SD3V3, WIFIEN
- wire segments 31 -> 0
- no-connect marks 5 -> 0

Commit message: Before power placement
Other:
- note removed: "R56 makes ESP32 boot at power up\nno R56: FPGA should pull up GPIO0\nand pulse EN for ESP32 to boot"
Changed lines of the file:
@@
 Comment4 ""
 $EndDescr
-Text GLabel 7050 4500 3    60   Input ~ 0
-SD_D0
-Text GLabel 7550 3950 2    60   Input ~ 0
-SD_D1
-Text GLabel 6250 4500 3    60   Input ~ 0
-SD_D3
-Text GLabel 6950 4500 3    60   Input ~ 0
-SD_CMD
 Text GLabel 2000 3850 0    60   Input ~ 0
 SD_CLK
@@
 Text GLabel 2000 3650 0    60   Input ~ 0
 WIFI_GPIO26
-Text GLabel 9250 5000 0    60   Input ~ 0
-SD_D2
-Text GLabel 9250 5100 0    60   Input ~ 0
-SD_D3
-Text GLabel 9250 5200 0    60   Input ~ 0
-SD_CMD
-Text GLabel 9250 5400 0    60   Input ~ 0
-SD_CLK
-Text GLabel 9250 5600 0    60   Input ~ 0
-SD_D0
-Text GLabel 9250 5700 0    60   Input ~ 0
-SD_D1
 Text Notes 8250 6450 0    60   ~ 0
 minimum pins for compatible mode\nSD_CLK, SD_CMD, SD_D0, SD_D3
-Text Notes 8250 6100 0    60   ~ 0
+Text Notes 8250 6200 0    60   ~ 0
 SDcard connected to\nBANK6 on "usb" sheet
 Text Notes 8350 3700 0    60   ~ 0
@@
 Text GLabel 8100 4250 0    60   Input ~ 0
 WIFI_GPIO0
-Text Notes 7550 4650 0    60   ~ 0
-R56 makes ESP32 boot at power up\nno R56: FPGA should pull up GPIO0\nand pulse EN for ESP32 to boot
 $EndSCHEMATC

Commit message: Adding ethernet
Parts:
- added C1: 10u, Capacitor_Tantalum_SMD:CP_EIA-1608-08_AVX-J_Pad1.25x1.05mm_HandSolder, symbol Device:CP
- added C2, C3, C4: 100n, Capacitor_SMD:C_0603_1608Metric_Pad1.05x0.95mm_HandSolder, symbol Device:C
- added C5, C6: 18p, Capacitor_SMD:C_0603_1608Metric_Pad1.05x0.95mm_HandSolder, symbol Device:C
- added J1: RJ45_Amphenol_RJMG1BD3B8K1ANR, Connector_RJ:RJ45_Amphenol_RJMG1BD3B8K1ANR, symbol Connector:RJ45_Amphenol_RJMG1BD3B8K1ANR
- added R1, R9: 4K7, Resistor_SMD:R_0603_1608Metric_Pad1.05x0.95mm_HandSolder, symbol Device:R
- added R10: 10R, Resistor_SMD:R_0603_1608Metric_Pad1.05x0.95mm_HandSolder, symbol Device:R
- added R2: 2K7, Resistor_SMD:R_0603_1608Metric_Pad1.05x0.95mm_HandSolder, symbol Device:R
- added R3, R4, R5, R6, R7, R8: 270R, Resistor_SMD:R_0603_1608Metric_Pad1.05x0.95mm_HandSolder, symbol Device:R
- added U1: ENC28J60x-ML, Package_DFN_QFN:QFN-28-1EP_6x6mm_P0.65mm_EP4.25x4.25mm, symbol Interface_Ethernet:ENC28J60x-ML
- added Y1: Crystal, Crystal:Crystal_SMD_SeikoEpson_FA238-4Pin_3.2x2.5mm, symbol Device:Crystal
Connections:
- new net: R2.2, U1.10 (RBIAS)
- new net: C1.1, U1.25 (VCAP)
- new net: J1.L4 (LEDG_A), R3.2
- new net: J1.L1 (LEDY_A), R4.2
- new net: C4.2, R7.2, R8.2
- new net: C3.2, J1.R4 (TCT), R10.1, R5.2, R6.2
- new net: C2.1, R9.2
- new net: C6.1, U1.20 (OSC2), Y1.1
- new net +3V3: R1.1, R10.2, R9.1, U1.11 (VDDTX), U1.15 (VDDRX), U1.16 (VDDPLL), U1.21 (VDDOSC), U1.24 (VDD)
- new net CS: R1.2, U1.5 (~CS)
- new net ETH_CLKIN: C5.1, U1.19 (OSC1), Y1.2
- new net ETH_CLKOUT: U1.27 (CLKOUT)
- new net ETH_INT: U1.28 (~INT)
- new net ETH_LEDA: R3.1, U1.23 (LEDA)
- new net ETH_LEDB: R4.1, U1.22 (LEDB)
- new net ETH_RESET: U1.6 (~RESET)
- new net ETH_SCK: U1.4 (SCK)
- new net ETH_SI: U1.3 (SI)
- new net ETH_SO: U1.2 (SO)
- new net ETH_TPIN+: J1.R3 (RD+), R8.1, U1.9 (TPIN+)
- new net ETH_TPIN-: J1.R6 (RD-), R7.1, U1.8 (TPIN-)
- new net ETH_TPOUT+: J1.R1 (TD+), R6.1, U1.13 (TPOUT+)
- new net ETH_TPOUT-: J1.R2 (TD-), R5.1, U1.12 (TPOUT-)
- new net ETH_WOL: U1.1 (~WOL)
- new net GND: C1.2, C2.2, C3.1, C4.1, C5.2, C6.2, J1.13 (SHIELD), J1.L2 (LEDY_K), J1.L3 (LEDG_K), J1.R8 (GND), R2.1, U1.14 (VSSTX), U1.17 (VSSPLL), U1.18 (VSSOSC), U1.26 (VSS), U1.7 (VSSRX)
Other:
- note removed: "ESP32 ADC capable pins\nGPIO36,39,34,35,32,33,25,26,27,\nGPIO14,12,13,15 - shared with HSPI/JTAG\nConnected to BANK7 on "gpio" sheet"
- note removed: "ESP32 HSPI pins\nGPIO12: MISO\nGPIO13: MOSI\nGPIO14: SCK\nGPIO15: SS"
- note removed: "ESP32 JTAG slave interface\nEN: TRST_N\nGPIO15: TDO\nGPIO12: TDI\nGPIO13: TCK\nGPIO14: TMS\nFLASH over JTAG\nnot yet supported."
- note removed: "ESP32 VSPI pins\nGPIO5: SS\nGPIO18: SCK\nGPIO19: MISO\nGPIO23: MOSI"
- note removed: "GN10 v1.7"
- note removed: "GN11 <v3.1 GP11 <v2.0.6"
- note removed: "GN12 <v3.1 GP12 <v2.0.6"
- note removed: "GN13 <v3.1"
- note removed: "GN9 v1.7"
- note removed: "GP11 <v3.1 GN11 <v2.0.6"
- note removed: "GP12 <v3.1 GN12 <v2.0.6"
- note removed: "GP13 <v2.0.6"
- note removed: "GP13 <v3.1 GN13 <v2.0.6"
- note removed: "GP9 v1.7"
- note removed: "GPIO12 probably should be held low at reset or disconnected\nother option is to burn flash voltage efuse for 3.3V operation\nfor GPIO2 and GPIO12 bootstrapping considerations, read\nhttps://github.com/espressif/esp-idf/tree/master/examples/storage/sd_card"
- note removed: "GPIO25,26 are DAC channels that can directly replay\naudio material over i2s bus"
- note removed: "NC <v3.1 GP10 v1.7 GP10 <=v3.1.2"
- note removed: "NC >=v3.1.2"
- note removed: "NC v1.7"
- note removed: "NC v1.7, >=v3.1.2"
- note removed: "NC v1.7, WIFI_GPIO5 <v3.1 LED >=3.1.2"
- note removed: "Programming pins:\nTXD RXD EN GPIO0"
- note removed: "SD card connected according to\nArduino->Examples->ESP32->SD_MMC_Test\nhttps://github.com/espressif/esp-idf/blob/\nmaster/examples/storage/sd_card/README.md\n"
- note removed: "SDcard connected to\nBANK6 on "usb" sheet"
- note removed: "Strapping pins\n(avoid using to avoid\nboot problems)\nGPIO0,2,4,5,12,15"
- note removed: "TDO <v3.1"
- note removed: "WIFI_GPIO15 v1.7"
- note removed: "WIFI_LED v1.7"
- note removed: "WROVER GPIO16,17\nused internally for PSRAM"
- note removed: "WiFi and SDcard connected to\nBANK6 on "usb" sheet"
- note removed: "minimum pins for compatible mode\nSD_CLK, SD_CMD, SD_D0, SD_D3"

Commit message: Adding logos - adding ethernet chip as a reference
Parts:
- removed C1: 10u, Capacitor_Tantalum_SMD:CP_EIA-1608-08_AVX-J_Pad1.25x1.05mm_HandSolder, symbol Device:CP
- removed C2, C3, C4: 100n, Capacitor_SMD:C_0603_1608Metric_Pad1.05x0.95mm_HandSolder, symbol Device:C
- removed C5, C6: 18p, Capacitor_SMD:C_0603_1608Metric_Pad1.05x0.95mm_HandSolder, symbol Device:C
- removed J1: RJ45_Amphenol_RJMG1BD3B8K1ANR, Connector_RJ:RJ45_Amphenol_RJMG1BD3B8K1ANR, symbol Connector:RJ45_Amphenol_RJMG1BD3B8K1ANR
- removed R1, R9: 4K7, Resistor_SMD:R_0603_1608Metric_Pad1.05x0.95mm_HandSolder, symbol Device:R
- removed R10: 10R, Resistor_SMD:R_0603_1608Metric_Pad1.05x0.95mm_HandSolder, symbol Device:R
- removed R2: 2K7, Resistor_SMD:R_0603_1608Metric_Pad1.05x0.95mm_HandSolder, symbol Device:R
- removed R3, R4, R5, R6, R7, R8: 270R, Resistor_SMD:R_0603_1608Metric_Pad1.05x0.95mm_HandSolder, symbol Device:R
- removed U1: ENC28J60x-ML, Package_DFN_QFN:QFN-28-1EP_6x6mm_P0.65mm_EP4.25x4.25mm, symbol Interface_Ethernet:ENC28J60x-ML
- removed Y1: Crystal, Crystal:Crystal_SMD_SeikoEpson_FA238-4Pin_3.2x2.5mm, symbol Device:Crystal
- added IC1: VSC8530XMW-04, VSC8530XMW-04:QFN40P600X600X90-49N-D, symbol VSC8530XMW-04:VSC8530XMW-04
