File: wifi.sch (KiCad schematic (older format))
At the start: 1 part, among them IC1 VSC8530XMW-04

Commit message: Initial complete routing done
Parts:
- removed IC1: VSC8530XMW-04, VSC8530XMW-04:QFN40P600X600X90-49N-D, symbol VSC8530XMW-04:VSC8530XMW-04
Changed lines of the file:
@@
 $Descr A4 11693 8268
 encoding utf-8
-Sheet 7 12
+Sheet 7 13
 Title "ULX3S"
 Date ""
@@
 Comment4 ""
 $EndDescr
-$Comp
-L VSC8530XMW-04:VSC8530XMW-04 IC1
-U 1 1 61FA10AA
-P 4025 2850
-F 0 "IC1" H 5869 2446 50  0000 L CNN
-F 1 "VSC8530XMW-04" H 5869 2355 50  0000 L CNN
-F 2 "VSC8530XMW-04:QFN40P600X600X90-49N-D" H 5675 3650 50  0001 L CNN
-F 3 "" H 5675 3550 50  0001 L CNN
-F 4 "Ethernet ICs 1Port Cu GE PHY iTMP SyncE, RGMII/RMII" H 5675 3450 50  0001 L CNN "Description"
-F 5 "0.9" H 5675 3350 50  0001 L CNN "Height"
-F 6 "494-VSC8530XMW-04" H 5675 3250 50  0001 L CNN "Mouser Part Number"
-F 7 "https://www.mouser.co.uk/ProductDetail/Microchip-Microsemi/VSC8530XMW-04?qs=1mbolxNpo8eJl4Wjwwyh%252Bg%3D%3D" H 5675 3150 50  0001 L CNN "Mouser Price/Stock"
-F 8 "Microsemi Corporation" H 5675 3050 50  0001 L CNN "Manufacturer_Name"
-F 9 "VSC8530XMW-04" H 5675 2950 50  0001 L CNN "Manufacturer_Part_Number"
-	1    4025 2850
-	1    0    0    -1
-$EndComp
 $EndSCHEMATC
