File: analog.sch (KiCad schematic (older format))
At the start: 20 parts, among them U8 MAX11125

Commit message: Removind ADC and right connector
Parts:
- removed C58, C61: 22uF, Capacitor_SMD:C_0805_2012Metric, symbol Device:C
- removed C59, C62: 220nF, Capacitor_SMD:C_0603_1608Metric, symbol Device:C
- removed L4, L5: 33uH, Inductor_SMD:L_0805_2012Metric_Pad1.15x1.40mm_HandSolder, symbol Device:L_Small
- removed U8: MAX11125, max1112x-tqfn28:MAX1112x-TQFN-28-1EP_5x5mm_Pitch0.5mm, symbol max1112x:MAX1112x
Connections:
- net labels removed: +3V3, ADC3V3, ADCD3V3, ADC_CSn, ADC_MISO, ADC_MOSI, ADC_SCLK, GN14, GN15, GN16, GN17, GP14, GP15, GP16, GP17
- wire segments 59 -> 27
- no-connect marks 4 -> 2
Other:
- note removed: "ADC SPI connected to\nBANK3 of "ram" sheet"

Commit message: More removing
Parts:
- removed AUDIO1: JACK_TRS_6PINS, audio-jack:CUI_SJ-43516-SMT, symbol jack_trs_6pins_apple:JACK_TRS_6PINS_APPLE
- removed R14, R18, R57: 1.1k, Resistor_SMD:R_0603_1608Metric, symbol Device:R
- removed R15, R19, R58: 549, Resistor_SMD:R_0603_1608Metric, symbol Device:R
- removed R16, R20, R59: 270, Resistor_SMD:R_0603_1608Metric, symbol Device:R
- removed R17, R21, R60: 130, Resistor_SMD:R_0603_1608Metric, symbol Device:R
Changed lines of the file:
@@
 $EndDescr
-$Comp
-L jack_trs_6pins_apple:JACK_TRS_6PINS_APPLE AUDIO1
-U 1 1 58D82C05
-P 2300 2350
-F 0 "AUDIO1" H 2400 2750 50  0000 C CNN
-F 1 "JACK_TRS_6PINS" V 1450 2400 50  0000 C CNN
-F 2 "audio-jack:CUI_SJ-43516-SMT" H 2400 2200 50  0001 C CNN
-F 3 "http://www.cui.com/product/resource/sj-4351x-smt-series.pdf" H 2400 2200 50  0001 C CNN
-F 4 "www.cui.com" H 2300 2350 60  0001 C CNN "MNF1_URL"
-F 5 "CUI" H 2300 2350 50  0001 C CNN "MFG1"
-F 6 "SJ-43516-SMT-TR" H 2300 2350 60  0001 C CNN "MPN"
-F 7 "490-SJ43515TS-SMT-TR" H 2300 2350 50  0001 C CNN "Mouser"
-F 8 "490-SJ43515RS-SMT-TR" H 2300 2350 50  0001 C CNN "Mouse_r1"
-F 9 "490-SJ-43516-SMT-TR " H 2300 2350 60  0001 C CNN "Mouse_r2"
-F 10 "CP-43516SJCT-ND" H 2300 2350 50  0001 C CNN "Digikey"
-F 11 "SJ-43516-SMT-TR" H 2300 2350 50  0001 C CNN "Vertical"
-F 12 "0.8015$" H 2300 2350 50  0001 C CNN "price100_Vertical"
-F 13 "FAU001" H 2300 2350 50  0001 C CNN "Koncar"
-F 14 "T" H 2300 2350 50  0001 C CNN "Side"
-	1    2300 2350
-	1    0    0    -1
-$EndComp
 $Comp
 L power:GND #PWR0141
@@
 	1    1850 2750
 	1    0    0    -1
-$EndComp
-$Comp
-L Device:R R17
-U 1 1 58D90455
-P 3750 2350
-F 0 "R17" V 3830 2350 50  0000 C CNN
-F 1 "130" V 3750 2350 50  0000 C CNN
-F 2 "Resistor_SMD:R_0603_1608Metric" V 3680 2350 50  0001 C CNN
-F 3 "" H 3750 2350 50  0000 C CNN
-F 4 "www.yageo.com" V 3750 2350 50  0001 C CNN "MNF1_URL"
-F 5 "RC0603FR-07130RL" V 3750 2350 50  0001 C CNN "MPN"
-F 6 "603-RC0603FR-07130RL" V 3750 2350 50  0001 C CNN "Mouser"
-F 7 "311-130HRCT-ND" V 3750 2350 50  0001 C CNN "Digikey"
-F 8 "65T8330" V 3750 2350 50  0001 C CNN "Newark"
-F 9 "C269457" V 3750 2350 50  0001 C CNN "LCSC"
-F 10 "FR004" V 3750 2350 50  0001 C CNN "Koncar"
-	1    3750 2350
-	0    1    1    0
-$EndComp
-$Comp
-L Device:R R16
-U 1 1 58D904AE
-P 3750 2200
-F 0 "R16" V 3830 2200 50  0000 C CNN
-F 1 "270" V 3750 2200 50  0000 C CNN
-F 2 "Resistor_SMD:R_0603_1608Metric" V 3680 2200 50  0001 C CNN
-F 3 "" H 3750 2200 50  0000 C CNN
-F 4 "www.yageo.com" V 3750 2200 50  0001 C CNN "MNF1_URL"
-F 5 "RC0603FR-07270RL" V 3750 2200 50  0001 C CNN "MPN"
-F 6 "603-AC0603FR-07270RL" V 3750 2200 50  0001 C CNN "Mouser"
-F 7 "603-RC0603FR-07270RL" V 3750 2200 50  0001 C CNN "Mouse_r2"
-F 8 "311-270HRCT-ND" V 3750 2200 50  0001 C CNN "Digikey"
-F 9 "64R5333" V 3750 2200 50  0001 C CNN "Newark"
-F 10 "C325609" V 3750 2200 50  0001 C CNN "LCSC"
-F 11 "FR010" V 3750 2200 50  0001 C CNN "Koncar"
-	1    3750 2200
-	0    1    1    0
-$EndComp
-$Comp
-L Device:R R15
-U 1 1 58D904D5
-P 3750 2050
-F 0 "R15" V 3830 2050 50  0000 C CNN
-F 1 "549" V 3750 2050 50  0000 C CNN
-F 2 "Resistor_SMD:R_0603_1608Metric" V 3680 2050 50  0001 C CNN
-F 3 "" H 3750 2050 50  0000 C CNN
-F 4 "www.yageo.com" V 3750 2050 50  0001 C CNN "MNF1_URL"
-F 5 "RC0603FR-07549RL" V 3750 2050 50  0001 C CNN "MPN"
-F 6 "603-RC0603FR-07549RL" V 3750 2050 50  0001 C CNN "Mouser"
-F 7 "311-549HRCT-ND" V 3750 2050 50  0001 C CNN "Digikey"
-F 8 "65T8486" V 3750 2050 50  0001 C CNN "Newark"
-F 9 "C308281" V 3750 2050 50  0001 C CNN "LCSC"
-F 10 "FR012" V 3750 2050 50  0001 C CNN "Koncar"
-F 11 "TB" V 3750 2050 50  0001 C CNN "Side"
-	1    3750 2050
-	0    1    1    0
-$EndComp
-$Comp
-L Device:R R14
-U 1 1 58D90500
-P 3750 1900
-F 0 "R14" V 3830 1900 50  0000 C CNN
-F 1 "1.1k" V 3750 1900 50  0000 C CNN
-F 2 "Resistor_SMD:R_0603_1608Metric" V 3680 1900 50  0001 C CNN
-F 3 "" H 3750 1900 50  0000 C CNN
-F 4 "www.yageo.com" V 3750 1900 50  0001 C CNN "MNF1_URL"
-F 5 " RC0603FR-071K1L" V 3750 1900 50  0001 C CNN "MPN"
-F 6 "603-RC0603FR-071K1L" V 3750 1900 50  0001 C CNN "Mouser"
-F 7 "603-AC0603FR-071K1L" V 3750 1900 50  0001 C CNN "Mouse_r2"
-F 8 "P1.10KHCT-ND" V 3750 1900 50  0001 C CNN "Digikey"
-F 9 "65T8314" V 3750 1900 50  0001 C CNN "Newark"
-F 10 "C269415" V 3750 1900 50  0001 C CNN "LCSC"
-F 11 "FR002" V 3750 1900 50  0001 C CNN "Koncar"
-	1    3750 1900
-	0    1    1    0
 $EndComp
 Wire Wire Line
@@
 Text GLabel 3900 2350 2    60   Input ~ 0
 AUDIO_L3
-$Comp
-L Device:R R21
-U 1 1 58D907CA
-P 3750 3000
-F 0 "R21" V 3830 3000 50  0000 C CNN
-F 1 "130" V 3750 3000 50  0000 C CNN
-F 2 "Resistor_SMD:R_0603_1608Metric" V 3680 3000 50  0001 C CNN
-F 3 "" H 3750 3000 50  0000 C CNN
-	1    3750 3000
-	0    1    1    0
-$EndComp
-$Comp
-L Device:R R20
-U 1 1 58D907D0
-P 3750 2850
-F 0 "R20" V 3830 2850 50  0000 C CNN
-F 1 "270" V 3750 2850 50  0000 C CNN
-F 2 "Resistor_SMD:R_0603_1608Metric" V 3680 2850 50  0001 C CNN
-F 3 "" H 3750 2850 50  0000 C CNN
-	1    3750 2850
-	0    1    1    0
-$EndComp
-$Comp
-L Device:R R19
-U 1 1 58D907D6
-P 3750 2700
-F 0 "R19" V 3830 2700 50  0000 C CNN
-F 1 "549" V 3750 2700 50  0000 C CNN
-F 2 "Resistor_SMD:R_0603_1608Metric" V 3680 2700 50  0001 C CNN
-F 3 "" H 3750 2700 50  0000 C CNN
-	1    3750 2700
-	0    1    1    0
-$EndComp
-$Comp
-L Device:R R18
-U 1 1 58D907DC
-P 3750 2550
-F 0 "R18" V 3830 2550 50  0000 C CNN
-F 1 "1.1k" V 3750 2550 50  0000 C CNN
-F 2 "Resistor_SMD:R_0603_1608Metric" V 3680 2550 50  0001 C CNN
-F 3 "" H 3750 2550 50  0000 C CNN
-	1    3750 2550
-	0    1    1    0
-$EndComp
 Wire Wire Line
 	3500 2850 3600 2850
@@
 Text Notes 4900 2300 0    60   ~ 0
 JACK pinout for SJ-43516-SMT-TR\nhttp://www.cui.com/product/resource/sj-4351x-smt-series.pdf\npin 1 - sleeve (GND)\npin 2 - tip (left channel)\npin 3 - ring1 (right channel)\npin 4 - ring2 (video)\npin 5 - tip switch\npin 6 - ring1 switch
-$Comp
-L Device:R R60
-U 1 1 5A05BC31
-P 3750 1700
-F 0 "R60" V 3830 1700 50  0000 C CNN
-F 1 "130" V 3750 1700 50  0000 C CNN
-F 2 "Resistor_SMD:R_0603_1608Metric" V 3680 1700 50  0001 C CNN
-F 3 "" H 3750 1700 50  0000 C CNN
-	1    3750 1700
-	0    1    1    0
-$EndComp
-$Comp
-L Device:R R59
-U 1 1 5A05BC37
-P 3750 1550
-F 0 "R59" V 3830 1550 50  0000 C CNN
-F 1 "270" V 3750 1550 50  0000 C CNN
-F 2 "Resistor_SMD:R_0603_1608Metric" V 3680 1550 50  0001 C CNN
-F 3 "" H 3750 1550 50  0000 C CNN
-	1    3750 1550
-	0    1    1    0
-$EndComp
-$Comp
-L Device:R R58
-U 1 1 5A05BC3D
-P 3750 1400
-F 0 "R58" V 3830 1400 50  0000 C CNN
-F 1 "549" V 3750 1400 50  0000 C CNN
-F 2 "Resistor_SMD:R_0603_1608Metric" V 3680 1400 50  0001 C CNN
-F 3 "" H 3750 1400 50  0000 C CNN
-	1    3750 1400
-	0    1    1    0
-$EndComp
-$Comp
-L Device:R R57
-U 1 1 5A05BC43
-P 3750 1250
-F 0 "R57" V 3830 1250 50  0000 C CNN
-F 1 "1.1k" V 3750 1250 50  0000 C CNN
-F 2 "Resistor_SMD:R_0603_1608Metric" V 3680 1250 50  0001 C CNN
-F 3 "" H 3750 1250 50  0000 C CNN
-	1    3750 1250
-	0    1    1    0
-$EndComp
 Wire Wire Line
 	3500 1550 3600 1550

Commit message: Cleanup schematics
Connections:
- net labels removed: AUDIO_L, AUDIO_L0, AUDIO_L1, AUDIO_L2, AUDIO_L3, AUDIO_R, AUDIO_R0, AUDIO_R1, AUDIO_R2, AUDIO_R3, AUDIO_V, AUDIO_V0, AUDIO_V1, AUDIO_V2, AUDIO_V3, GND
- wire segments 27 -> 0
- no-connect marks 2 -> 0
Other:
- note removed: "Audio connected to\nBANK7 on "gpio" sheet"
- note removed: "JACK pinout for SJ-43516-SMT-TR\nhttp://www.cui.com/product/resource/sj-4351x-smt-series.pdf\npin 1 - sleeve (GND)\npin 2 - tip (left channel)\npin 3 - ring1 (right channel)\npin 4 - ring2 (video)\npin 5 - tip switch\npin 6 - ring1 switch"
- note removed: "Output resistance: 75 ohm\nInternal resistance of FPGA pin: 10 ohm\n1/(1/(130+10)+1/(270+10)+1/(549+10)+1/(1100+10))=74.6"
Changed lines of the file:
@@
 Comment4 ""
 $EndDescr
-$Comp
-L power:GND #PWR0141
-U 1 1 58D9043A
-P 1850 2750
-F 0 "#PWR0141" H 1850 2500 50  0001 C CNN
-F 1 "GND" H 1850 2600 50  0000 C CNN
-F 2 "" H 1850 2750 50  0000 C CNN
-F 3 "" H 1850 2750 50  0000 C CNN
-	1    1850 2750
-	1    0    0    -1
-$EndComp
-Wire Wire Line
-	2950 2350 3500 2350
-Wire Wire Line
-	3500 2200 3600 2200
-Wire Wire Line
-	3500 1900 3500 2050
-Connection ~ 3500 2350
-Wire Wire Line
-	3500 2050 3600 2050
-Connection ~ 3500 2200
-Wire Wire Line
-	3500 1900 3600 1900
-Connection ~ 3500 2050
-Text GLabel 3900 1900 2    60   Input ~ 0
-AUDIO_L0
-Text GLabel 3900 2050 2    60   Input ~ 0
-AUDIO_L1
-Text GLabel 3900 2200 2    60   Input ~ 0
-AUDIO_L2
-Text GLabel 3900 2350 2    60   Input ~ 0
-AUDIO_L3
-Wire Wire Line
-	3500 2850 3600 2850
-Wire Wire Line
-	3500 2550 3500 2700
-Wire Wire Line
-	3500 2700 3600 2700
-Connection ~ 3500 2850
-Wire Wire Line
-	2950 2550 3500 2550
-Connection ~ 3500 2700
-Text GLabel 3900 2550 2    60   Input ~ 0
-AUDIO_R0
-Text GLabel 3900 2700 2    60   Input ~ 0
-AUDIO_R1
-Text GLabel 3900 2850 2    60   Input ~ 0
-AUDIO_R2
-Text GLabel 3900 3000 2    60   Input ~ 0
-AUDIO_R3
-Wire Wire Line
-	3500 3000 3600 3000
-Connection ~ 3500 2550
-NoConn ~ 2650 2550
-Text Notes 4900 2650 0    60   ~ 0
-Audio connected to\nBANK7 on "gpio" sheet
-Text Notes 4900 2300 0    60   ~ 0
-JACK pinout for SJ-43516-SMT-TR\nhttp://www.cui.com/product/resource/sj-4351x-smt-series.pdf\npin 1 - sleeve (GND)\npin 2 - tip (left channel)\npin 3 - ring1 (right channel)\npin 4 - ring2 (video)\npin 5 - tip switch\npin 6 - ring1 switch
-Wire Wire Line
-	3500 1550 3600 1550
-Wire Wire Line
-	3500 1250 3500 1400
-Connection ~ 3500 1700
-Wire Wire Line
-	3500 1400 3600 1400
-Connection ~ 3500 1550
-Wire Wire Line
-	3500 1250 3600 1250
-Connection ~ 3500 1400
-Text GLabel 3900 1250 2    60   Input ~ 0
-AUDIO_V0
-Text GLabel 3900 1400 2    60   Input ~ 0
-AUDIO_V1
-Text GLabel 3900 1550 2    60   Input ~ 0
-AUDIO_V2
-Text GLabel 3900 1700 2    60   Input ~ 0
-AUDIO_V3
-Text Label 3050 1700 0    60   ~ 0
-AUDIO_V
-Wire Wire Line
-	3500 2350 3600 2350
-Wire Wire Line
-	3500 2200 3500 2350
-Wire Wire Line
-	3500 2050 3500 2200
-Wire Wire Line
-	3500 2850 3500 3000
-Wire Wire Line
-	3500 2700 3500 2850
-Wire Wire Line
-	3500 2550 3600 2550
-Wire Wire Line
-	3500 1700 3600 1700
-Wire Wire Line
-	3500 1550 3500 1700
-Wire Wire Line
-	3500 1400 3500 1550
-NoConn ~ 1900 1900
-Wire Wire Line
-	2050 1900 2050 1450
-Text Label 2000 2800 3    60   ~ 0
-AUDIO_V
-Wire Wire Line
-	2000 2750 2000 3200
-Wire Wire Line
-	2300 2750 2300 3200
-Wire Wire Line
-	2950 1700 3500 1700
-Text Label 2300 2800 3    60   ~ 0
-AUDIO_L
-Text Label 2050 1850 1    60   ~ 0
-AUDIO_R
-Text Label 3000 2350 0    60   ~ 0
-AUDIO_L
-Text Label 3000 2550 0    60   ~ 0
-AUDIO_R
-Text Notes 2950 3500 0    60   ~ 0
-Output resistance: 75 ohm\nInternal resistance of FPGA pin: 10 ohm\n1/(1/(130+10)+1/(270+10)+1/(549+10)+1/(1100+10))=74.6
 $EndSCHEMATC
