File: blinkey.sch (KiCad schematic (older format))
At the start: 34 parts, among them SW1 SW_DIP_x04

Commit message: More removing
Parts:
- removed B1, B2, B3, B4, B5, B6: PTS645, Button_Switch_SMD:SW_SPST_PTS645, symbol Switch:SW_Push
- removed D18: GREEN, LED_SMD:LED_0805_2012Metric, symbol Device:LED
- removed D19, D4: RED, LED_SMD:LED_0805_2012Metric, symbol Device:LED_ALT
- removed D22: BLUE, LED_SMD:LED_0805_2012Metric, symbol Device:LED
- removed D5: ORANGE, LED_SMD:LED_0805_2012Metric, symbol Device:LED_ALT
- removed D6: GREEN, LED_SMD:LED_0805_2012Metric, symbol Device:LED_ALT
- removed D7: BLUE, LED_SMD:LED_0805_2012Metric, symbol Device:LED_ALT
- removed LCD1: ST7789, st7789:st7789, symbol st7789:ST7789
- removed R36, R37, R45, R46, R47, R48, R62: 549, Resistor_SMD:R_0603_1608Metric, symbol Device:R
- removed R39, R7: 130, Resistor_SMD:R_0603_1608Metric, symbol Device:R
Connections:
- net labels removed: ALED4, ALED5, ALED6, ALED7, BTNPUL, BTNPUR
- wire segments 67 -> 39
Other:
- note removed: "DOWN"
- note removed: "FIRE1"
- note removed: "FIRE2"
- note removed: "LEFT"
- note removed: "RIGHT"
- note removed: "UP"

Commit message: Before removing USB port
Parts:
- removed SW1: SW_DIP_x04, dipswitch:SW_DIP_x4_W8.61mm_Slide_LowProfile, symbol Switch:SW_DIP_x04
Connections:
- net labels removed: SWPU
- wire segments 39 -> 31
Changed lines of the file:
@@
 	0    -1   -1   0
 $EndComp
-Wire Wire Line
-	7400 3400 7750 3400
-Wire Wire Line
-	7750 3100 7750 3200
-Wire Wire Line
-	7750 3100 7800 3100
-Connection ~ 7750 3400
-Wire Wire Line
-	7800 3200 7750 3200
-Connection ~ 7750 3200
-Wire Wire Line
-	7800 3300 7750 3300
-Connection ~ 7750 3300
 Text GLabel 8400 3100 2    60   Input ~ 0
 SW1
@@
 Wire Wire Line
 	4400 5850 4250 5850
-Text Label 7450 3400 0    60   ~ 0
-SWPU
 Text Notes 6350 5400 0    60   ~ 0
 TXLED blinks when FPGA sends data to FTDI
@@
 Wire Wire Line
 	4250 2750 4250 2950
-Wire Wire Line
-	7750 3400 7800 3400
-Wire Wire Line
-	7750 3200 7750 3300
-Wire Wire Line
-	7750 3300 7750 3400
 Text GLabel 7100 3400 0    60   Input ~ 0
 2V5_3V3
-$Comp
-L Switch:SW_DIP_x04 SW1
-U 1 1 5B1DD3B8
-P 8100 3300
-F 0 "SW1" H 8100 3767 50  0000 C CNN
-F 1 "SW_DIP_x04" H 8100 3676 50  0000 C CNN
-F 2 "dipswitch:SW_DIP_x4_W8.61mm_Slide_LowProfile" H 8100 3300 50  0001 C CNN
-F 3 "https://www.ctscorp.com/wp-content/uploads/219.pdf" H 8100 3300 50  0001 C CNN
-F 4 "www.jameco.com" H 8100 3300 50  0001 C CNN "MNF1_URL"
-F 5 "219-4MST" H 8100 3300 50  0001 C CNN "MPN"
-F 6 "https://datasheet.lcsc.com/szlcsc/1912111437_XKB-Enterprise-DSHP04TS-S_C319050.pdf" H 8100 3300 50  0001 C CNN "MNF2_URL"
-F 7 "DSHP04TS-S" H 8100 3300 50  0001 C CNN "MPN2"
-F 8 "774-2194MST" H 8100 3300 50  0001 C CNN "Mouser"
-F 9 "CT2194MST-ND" H 8100 3300 50  0001 C CNN "Digikey"
-F 10 "29P1768" H 8100 3300 50  0001 C CNN "Newark"
-F 11 "C319050" H 8100 3300 50  0001 C CNN "LCSC"
-F 12 "FSW002" H 8100 3300 50  0001 C CNN "Koncar"
-F 13 "T" H 8100 3300 50  0001 C CNN "Side"
-	1    8100 3300
-	1    0    0    -1
-$EndComp
 Text GLabel 4850 1950 2    60   Input ~ 0
 OLED_BL

Commit message: More removal, spliting modules
Parts:
- removed R51: 130, Resistor_SMD:R_0603_1608Metric, symbol Device:R
- C46: footprint Capacitor_SMD:C_0805_2012Metric -> Capacitor_SMD:C_0603_1608Metric
- D0, D1, D2, D3: footprint LED_SMD:LED_0805_2012Metric -> LED_SMD:LED_0603_1608Metric
- R41, R42, R43, R44: footprint Resistor_SMD:R_0603_1608Metric -> Capacitor_SMD:C_0402_1005Metric
Changed lines of the file:
@@
 F 0 "R41" V 5330 2550 50  0000 C CNN
 F 1 "549" V 5250 2550 50  0000 C CNN
-F 2 "Resistor_SMD:R_0603_1608Metric" V 5180 2550 50  0001 C CNN
+F 2 "Capacitor_SMD:C_0402_1005Metric" V 5180 2550 50  0001 C CNN
 F 3 "" H 5250 2550 50  0000 C CNN
 	1    5250 2550
@@
 F 0 "R42" V 5330 2750 50  0000 C CNN
 F 1 "549" V 5250 2750 50  0000 C CNN
-F 2 "Resistor_SMD:R_0603_1608Metric" V 5180 2750 50  0001 C CNN
+F 2 "Capacitor_SMD:C_0402_1005Metric" V 5180 2750 50  0001 C CNN
 F 3 "" H 5250 2750 50  0000 C CNN
 	1    5250 2750
@@
 F 0 "R43" V 5330 2950 50  0000 C CNN
 F 1 "549" V 5250 2950 50  0000 C CNN
-F 2 "Resistor_SMD:R_0603_1608Metric" V 5180 2950 50  0001 C CNN
+F 2 "Capacitor_SMD:C_0402_1005Metric" V 5180 2950 50  0001 C CNN
 F 3 "" H 5250 2950 50  0000 C CNN
 	1    5250 2950
@@
 F 0 "R44" V 5330 3150 50  0000 C CNN
 F 1 "549" V 5250 3150 50  0000 C CNN
-F 2 "Resistor_SMD:R_0603_1608Metric" V 5180 3150 50  0001 C CNN
+F 2 "Capacitor_SMD:C_0402_1005Metric" V 5180 3150 50  0001 C CNN
 F 3 "" H 5250 3150 50  0000 C CNN
 	1    5250 3150
@@
 Text Notes 2100 4400 0    60   ~ 0
 BTN_R,U to BANK2,3 on "ram" sheet\nBTN_F1,F2,D,L to BANK8 on "flash" sheet
-$Comp
-L Device:R R51
-U 1 1 595B9C2F
-P 7250 3400
-F 0 "R51" V 7330 3400 50  0000 C CNN
-F 1 "130" V 7250 3400 50  0000 C CNN
-F 2 "Resistor_SMD:R_0603_1608Metric" V 7180 3400 50  0001 C CNN
-F 3 "" H 7250 3400 50  0000 C CNN
-	1    7250 3400
-	0    -1   -1   0
-$EndComp
 Text GLabel 8400 3100 2    60   Input ~ 0
 SW1
@@
 F 0 "D3" H 4550 3250 50  0000 C CNN
 F 1 "BLUE" H 4200 3150 50  0000 R CNN
-F 2 "LED_SMD:LED_0805_2012Metric" H 4550 3150 50  0001 C CNN
+F 2 "LED_SMD:LED_0603_1608Metric" H 4550 3150 50  0001 C CNN
 F 3 "http://optoelectronics.liteon.com/upload/download/DS-22-99-0226/LTST-C170TBKT.pdf" H 4550 3150 50  0001 C CNN
 F 4 "www.liteon.com" H 4550 3150 60  0001 C CNN "MNF1_URL"
@@
 F 0 "D2" H 4550 3050 50  0000 C CNN
 F 1 "GREEN" H 4200 2950 50  0000 R CNN
-F 2 "LED_SMD:LED_0805_2012Metric" H 4550 2950 50  0001 C CNN
+F 2 "LED_SMD:LED_0603_1608Metric" H 4550 2950 50  0001 C CNN
 F 3 "http://optoelectronics.liteon.com/upload/download/DS22-2000-073/LTST-C170KGKT.pdf" H 4550 2950 50  0001 C CNN
 F 4 "www.liteon.com" H 4550 2950 60  0001 C CNN "MNF1_URL"
@@
 F 0 "D0" H 4550 2650 50  0000 C CNN
 F 1 "RED" H 4200 2550 50  0000 R CNN
-F 2 "LED_SMD:LED_0805_2012Metric" H 4550 2550 50  0001 C CNN
+F 2 "LED_SMD:LED_0603_1608Metric" H 4550 2550 50  0001 C CNN
 F 3 "https://optoelectronics.liteon.com/upload/download/DS-22-99-0150/LTST-C170KRKT.pdf" H 4550 2550 50  0001 C CNN
 F 4 "www.liteon.com" H 4550 2550 60  0001 C CNN "MNF1_URL"
@@
 F 0 "D1" H 4550 2850 50  0000 C CNN
 F 1 "ORANGE" H 4200 2750 50  0000 R CNN
-F 2 "LED_SMD:LED_0805_2012Metric" H 4550 2750 50  0001 C CNN
+F 2 "LED_SMD:LED_0603_1608Metric" H 4550 2750 50  0001 C CNN
 F 3 "https://optoelectronics.liteon.com/upload/download/DS-22-99-0185/LTST-C170KFKT.pdf" H 4550 2750 50  0001 C CNN
 F 4 "www.liteon.com" H 4550 2750 60  0001 C CNN "MNF1_URL"
@@
 F 0 "C46" H 6675 1450 50  0000 L CNN
 F 1 "2.2uF" H 6675 1250 50  0000 L CNN
-F 2 "Capacitor_SMD:C_0805_2012Metric" H 6688 1200 50  0001 C CNN
+F 2 "Capacitor_SMD:C_0603_1608Metric" H 6688 1200 50  0001 C CNN
 F 3 "" H 6650 1350 50  0001 C CNN
 F 4 "www.yageo.com" H 6650 1350 50  0001 C CNN "MNF1_URL"

Commit message: Adding buttons
Parts:
- added R18: 130, Capacitor_SMD:C_0402_1005Metric, symbol Device:R
- added SW1, SW2: SW_Push, Switch_EVPAA:Switch_EVPAA, symbol Switch:SW_Push
Connections:
- net labels added: BTN1, BTN2
- net labels removed: BTN_F1, BTN_F2
- wire segments 31 -> 36
Changed lines of the file:
@@
 OLED_CS
-Wire Wire Line
-	3250 2950 3350 2950
-Wire Wire Line
-	3250 3150 3350 3150
 Wire Wire Line
 	3250 3350 3350 3350
@@
 	3250 3950 3350 3950
 Text GLabel 3350 2950 2    60   Input ~ 0
-BTN_F1
+BTN1
 Text GLabel 3350 3150 2    60   Input ~ 0
-BTN_F2
+BTN2
 Text GLabel 3350 3350 2    60   Input ~ 0
 BTN_U
@@
 	1    0    0    -1
 $EndComp
+$Comp
+L Switch:SW_Push SW1
+U 1 1 6256B27F
+P 2900 2950
+F 0 "SW1" H 3100 3000 50  0000 C CNN
+F 1 "SW_Push" H 2600 3000 50  0000 C CNN
+F 2 "Switch_EVPAA:Switch_EVPAA" H 2900 3150 50  0001 C CNN
+F 3 "https://www.mouser.in/datasheet/2/315/PANA_S_A0001791376_1-2560543.pdf" H 2900 3150 50  0001 C CNN
+F 4 "https://www.mouser.in/ProductDetail/Panasonic/EVP-AA302K?qs=qvwOHSmaRMmnf4H35tvzww==" H 2900 2950 50  0001 C CNN "Mouser"
+F 5 "https://www.digikey.com/en/products/detail/panasonic-electronic-components/EVP-AA302K/2810555" H 2900 2950 50  0001 C CNN "DigiKey"
+	1    2900 2950
+	1    0    0    -1
+$EndComp
+Wire Wire Line
+	3100 2950 3350 2950
+Wire Wire Line
+	3100 3150 3350 3150
+$Comp
+L Device:R R18
+U 1 1 625797F0
+P 2150 2950
+F 0 "R18" V 2230 2950 50  0000 C CNN
+F 1 "130" V 2150 2950 50  0000 C CNN
+F 2 "Capacitor_SMD:C_0402_1005Metric" V 2080 2950 50  0001 C CNN
+F 3 "" H 2150 2950 50  0000 C CNN
+	1    2150 2950
+	0    1    1    0
+$EndComp
+Wire Wire Line
+	2300 2950 2400 2950
+Wire Wire Line
+	2400 2950 2400 3150
+Wire Wire Line
+	2400 3150 2700 3150
+Connection ~ 2400 2950
+Wire Wire Line
+	2400 2950 2700 2950
+$Comp
+L power:+3V3 #PWR0112
+U 1 1 6257D2AA
+P 1850 2950
+F 0 "#PWR0112" H 1850 2800 50  0001 C CNN
+F 1 "+3V3" H 1850 3090 50  0000 C CNN
+F 2 "" H 1850 2950 50  0000 C CNN
+F 3 "" H 1850 2950 50  0000 C CNN
+	1    1850 2950
+	0    -1   -1   0
+$EndComp
+Wire Wire Line
+	1850 2950 2000 2950
+$Comp
+L Switch:SW_Push SW2
+U 1 1 6258110E
+P 2900 3150
+F 0 "SW2" H 3100 3200 50  0000 C CNN
+F 1 "SW_Push" H 2600 3200 50  0000 C CNN
+F 2 "Switch_EVPAA:Switch_EVPAA" H 2900 3350 50  0001 C CNN
+F 3 "https://www.mouser.in/datasheet/2/315/PANA_S_A0001791376_1-2560543.pdf" H 2900 3350 50  0001 C CNN
+F 4 "https://www.mouser.in/ProductDetail/Panasonic/EVP-AA302K?qs=qvwOHSmaRMmnf4H35tvzww==" H 2900 3150 50  0001 C CNN "Mouser"
+F 5 "https://www.digikey.com/en/products/detail/panasonic-electronic-components/EVP-AA302K/2810555" H 2900 3150 50  0001 C CNN "DigiKey"
+	1    2900 3150
+	1    0    0    -1
+$EndComp

Commit message: Cleanup schematics
Connections:
- net labels removed: 2V5_3V3, BTN_D, BTN_L, BTN_R, BTN_U, FT2V5, FTDI_nSLEEP, FTDI_nTXLED, JTAG_TMS, LED4, LED5, LED6, LED7, LED_PWREN, LED_TXLED, LED_WIFI, OLED_BL, OLED_CLK, OLED_CS, OLED_DC, OLED_MOSI, OLED_RES, SW1, SW2, SW3, SW4
- wire segments 36 -> 19
Other:
- note removed: "BTN_R,U to BANK2,3 on "ram" sheet\nBTN_F1,F2,D,L to BANK8 on "flash" sheet"
- note removed: "DIP switch connected to\nBANK0 on 'gpio' sheet"
- note removed: "LEDs connected to\nBANK7 on "gpio" sheet"
- note removed: "OLED connected to\nBANK6 on "usb" sheet"
- note removed: "TXLED blinks when FPGA sends data to FTDI"
- note removed: "To fix issues with FT231XS rev A,B,C\nShort-circuit D18 LED, but then\nboard cannot keep awake by USB.\nchip rev D works properly\nSee TN140_FT231X Errata\n"
- note removed: "WIFI_GPIO2 v1.7, WIFI_GPIO5 <v3.1"
Changed lines of the file:
@@
 Comment4 ""
 $EndDescr
-Wire Wire Line
-	4750 1450 4850 1450
-Wire Wire Line
-	4750 1550 4850 1550
-Wire Wire Line
-	4750 1650 4850 1650
-Wire Wire Line
-	4750 1750 4850 1750
-Wire Wire Line
-	4750 1850 4850 1850
-Text GLabel 4850 1450 2    60   Input ~ 0
-OLED_CLK
-Text GLabel 4850 1550 2    60   Input ~ 0
-OLED_MOSI
-Text GLabel 4850 1650 2    60   Input ~ 0
-OLED_RES
-Text GLabel 4850 1750 2    60   Input ~ 0
-OLED_DC
-Text GLabel 4850 1850 2    60   Input ~ 0
-OLED_CS
-Wire Wire Line
-	3250 3350 3350 3350
-Wire Wire Line
-	3250 3550 3350 3550
-Wire Wire Line
-	3250 3750 3350 3750
-Wire Wire Line
-	3250 3950 3350 3950
 Text GLabel 3350 2950 2    60   Input ~ 0
 BTN1
 Text GLabel 3350 3150 2    60   Input ~ 0
 BTN2
-Text GLabel 3350 3350 2    60   Input ~ 0
-BTN_U
-Text GLabel 3350 3550 2    60   Input ~ 0
-BTN_D
-Text GLabel 3350 3750 2    60   Input ~ 0
-BTN_L
-Text GLabel 3350 3950 2    60   Input ~ 0
-BTN_R
 Text Notes 4450 1050 0    60   ~ 0
 ST7789/SSD1331/SSD1351/SSD1306\ncompatible LCD/OLED 0.96/1.3/1.54" PCB \n14x14 units\n1 unit = 2.54 mm
@@
 Text GLabel 5400 3150 2    60   Input ~ 0
 LED3
-Text GLabel 5400 3350 2    60   Input ~ 0
-LED4
-Text GLabel 5400 3550 2    60   Input ~ 0
-LED5
-Text GLabel 5400 3750 2    60   Input ~ 0
-LED6
-Text GLabel 5400 3950 2    60   Input ~ 0
-LED7
-Text GLabel 5650 4600 2    60   Input ~ 0
-FTDI_nSLEEP
-Wire Wire Line
-	4700 4600 5350 4600
-Text Label 4750 4600 0    60   ~ 0
-LED_PWREN
-Wire Wire Line
-	4400 4600 4250 4600
-Wire Wire Line
-	4250 4600 4250 4950
-$Comp
-L power:GND #PWR084
-U 1 1 590B5B6D
-P 4250 4950
-F 0 "#PWR084" H 4250 4700 50  0001 C CNN
-F 1 "GND" H 4250 4800 50  0000 C CNN
-F 2 "" H 4250 4950 50  0000 C CNN
-F 3 "" H 4250 4950 50  0000 C CNN
-	1    4250 4950
-	1    0    0    -1
-$EndComp
-Text GLabel 5650 5350 2    60   Input ~ 0
-FTDI_nTXLED
-Wire Wire Line
-	4700 5350 5350 5350
-Text Label 4750 5350 0    60   ~ 0
-LED_TXLED
-Text GLabel 4300 5350 0    60   Input ~ 0
-FT2V5
-Wire Wire Line
-	4300 5350 4400 5350
 $Comp
 L Device:R R41
@@
 Text Label 4750 3150 0    60   ~ 0
 ALED3
-Text Notes 4600 4300 0    60   ~ 0
-LEDs connected to\nBANK7 on "gpio" sheet
-Text Notes 2100 4400 0    60   ~ 0
-BTN_R,U to BANK2,3 on "ram" sheet\nBTN_F1,F2,D,L to BANK8 on "flash" sheet
-Text GLabel 8400 3100 2    60   Input ~ 0
-SW1
-Text GLabel 8400 3200 2    60   Input ~ 0
-SW2
-Text GLabel 8400 3300 2    60   Input ~ 0
-SW3
-Text GLabel 8400 3400 2    60   Input ~ 0
-SW4
-Text Notes 7700 3750 0    60   ~ 0
-DIP switch connected to\nBANK0 on 'gpio' sheet
-Text Notes 8000 4550 0    60   ~ 0
-To fix issues with FT231XS rev A,B,C\nShort-circuit D18 LED, but then\nboard cannot keep awake by USB.\nchip rev D works properly\nSee TN140_FT231X Errata\n
-Text GLabel 5650 5850 2    60   Input ~ 0
-JTAG_TMS
-Wire Wire Line
-	4700 5850 5350 5850
-Text Label 4750 5850 0    60   ~ 0
-LED_WIFI
-Wire Wire Line
-	4400 5850 4250 5850
-Text Notes 6350 5400 0    60   ~ 0
-TXLED blinks when FPGA sends data to FTDI
-Text Notes 4450 2300 0    60   ~ 0
-OLED connected to\nBANK6 on "usb" sheet
 $Comp
 L Device:LED_ALT D3
@@
 	1    0    0    -1
 $EndComp
-Text Notes 6400 5900 0    60   ~ 0
-WIFI_GPIO2 v1.7, WIFI_GPIO5 <v3.1
 $Comp
 L Device:C C46
@@
 Wire Wire Line
 	4250 2750 4250 2950
-Text GLabel 7100 3400 0    60   Input ~ 0
-2V5_3V3
-Text GLabel 4850 1950 2    60   Input ~ 0
-OLED_BL
-Wire Wire Line
-	4750 1950 4850 1950
-$Comp
-L power:+3V3 #PWR0122
-U 1 1 5F0C55F7
-P 4250 5850
-F 0 "#PWR0122" H 4250 5700 50  0001 C CNN
-F 1 "+3V3" H 4250 5990 50  0000 C CNN
-F 2 "" H 4250 5850 50  0000 C CNN
-F 3 "" H 4250 5850 50  0000 C CNN
-	1    4250 5850
-	0    -1   -1   0
-$EndComp
 Wire Wire Line
 	4250 3150 4250 3300
