File: blinkey.sch (KiCad schematic (older format))
At the start: 12 parts, among them SW1 SW_Push, SW2 SW_Push

Commit message: Adding 4 more LEDs - moving button
Parts:
- added D4: RED, LED_SMD:LED_0603_1608Metric, symbol Device:LED_ALT
- added D5: ORANGE, LED_SMD:LED_0603_1608Metric, symbol Device:LED_ALT
- added D6: GREEN, LED_SMD:LED_0603_1608Metric, symbol Device:LED_ALT
- added D7: BLUE, LED_SMD:LED_0603_1608Metric, symbol Device:LED_ALT
- added R49, R50, R51, R52: 549, Capacitor_SMD:C_0402_1005Metric, symbol Device:R
Connections:
- net GND: now also D4.1 (K), D5.1 (K), D6.1 (K), D7.1 (K)
- new net ALED4: D4.2 (A), R49.2
- new net ALED5: D5.2 (A), R50.2
- new net ALED6: D6.2 (A), R51.2
- new net ALED7: D7.2 (A), R52.2
- new net LED4: R49.1
- new net LED5: R50.1
- new net LED6: R51.1
- new net LED7: R52.1
Changed lines of the file:
@@
+	1    0    0    -1
+$EndComp
+Wire Wire Line
+	4350 3675 4200 3675
+Wire Wire Line
+	4200 3675 4200 3875
+Wire Wire Line
+	4350 4275 4200 4275
+Connection ~ 4200 4275
+Wire Wire Line
+	4350 4075 4200 4075
+Connection ~ 4200 4075
+Wire Wire Line
+	4350 3875 4200 3875
+Connection ~ 4200 3875
+Wire Wire Line
+	4650 3675 5050 3675
+Wire Wire Line
+	4650 3875 5050 3875
+Wire Wire Line
+	4650 4075 5050 4075
+Wire Wire Line
+	4650 4275 5050 4275
+Text GLabel 5350 3675 2    60   Input ~ 0
+LED4
+Text GLabel 5350 3875 2    60   Input ~ 0
+LED5
+Text GLabel 5350 4075 2    60   Input ~ 0
+LED6
+Text GLabel 5350 4275 2    60   Input ~ 0
+LED7
+$Comp
+L Device:R R49
+U 1 1 627AFA63
+P 5200 3675
+F 0 "R49" V 5280 3675 50  0000 C CNN
+F 1 "549" V 5200 3675 50  0000 C CNN
+F 2 "Capacitor_SMD:C_0402_1005Metric" V 5130 3675 50  0001 C CNN
+F 3 "" H 5200 3675 50  0000 C CNN
+	1    5200 3675
+	0    1    1    0
+$EndComp
+$Comp
+L Device:R R50
+U 1 1 627AFA6D
+P 5200 3875
+F 0 "R50" V 5280 3875 50  0000 C CNN
+F 1 "549" V 5200 3875 50  0000 C CNN
+F 2 "Capacitor_SMD:C_0402_1005Metric" V 5130 3875 50  0001 C CNN
+F 3 "" H 5200 3875 50  0000 C CNN
+	1    5200 3875
+	0    1    1    0
+$EndComp
+$Comp
+L Device:R R51
+U 1 1 627AFA77
+P 5200 4075
+F 0 "R51" V 5280 4075 50  0000 C CNN
+F 1 "549" V 5200 4075 50  0000 C CNN
+F 2 "Capacitor_SMD:C_0402_1005Metric" V 5130 4075 50  0001 C CNN
+F 3 "" H 5200 4075 50  0000 C CNN
+	1    5200 4075
+	0    1    1    0
+$EndComp
+$Comp
+L Device:R R52
+U 1 1 627AFA81
+P 5200 4275
+F 0 "R52" V 5280 4275 50  0000 C CNN
+F 1 "549" V 5200 4275 50  0000 C CNN
+F 2 "Capacitor_SMD:C_0402_1005Metric" V 5130 4275 50  0001 C CNN
+F 3 "" H 5200 4275 50  0000 C CNN
+	1    5200 4275
+	0    1    1    0
+$EndComp
+Text Label 4700 3675 0    60   ~ 0
+ALED4
+Text Label 4700 3875 0    60   ~ 0
+ALED5
+Text Label 4700 4075 0    60   ~ 0
+ALED6
+Text Label 4700 4275 0    60   ~ 0
+ALED7
+$Comp
+L Device:LED_ALT D7
+U 1 1 627AFAA1
+P 4500 4275
+F 0 "D7" H 4500 4375 50  0000 C CNN
+F 1 "BLUE" H 4150 4275 50  0000 R CNN
+F 2 "LED_SMD:LED_0603_1608Metric" H 4500 4275 50  0001 C CNN
+F 3 "http://optoelectronics.liteon.com/upload/download/DS-22-99-0226/LTST-C170TBKT.pdf" H 4500 4275 50  0001 C CNN
+F 4 "www.liteon.com" H 4500 4275 60  0001 C CNN "MNF1_URL"
+F 5 "LTST-C170TBKT" H 4500 4275 60  0001 C CNN "MPN"
+F 6 "http://optoelectronics.liteon.com/upload/download/ds22-2000-233/ltst-c171tbkt(0630).pdf" H 4500 4275 50  0001 C CNN "Datasheet2"
+F 7 "LTST-C171TBKT" H 4500 4275 50  0001 C CNN "MP_N2"
+F 8 "https://www.rohm.com/datasheet/SML-M13UT" H 4500 4275 50  0001 C CNN "Datasheet3"
+F 9 "SMLMN2BCTT86C" H 4500 4275 50  0001 C CNN "MP_N3"
+F 10 "859-LTST-C170TBKT" H 4500 4275 60  0001 C CNN "Mouser"
+F 11 "593-LSM0805463V" H 4500 4275 50  0001 C CNN "Mouse_r1"
+F 12 "755-SMLMN2BCTT86C" H 4500 4275 50  0001 C CNN "Mouse_r2"
+F 13 "859-LTST-C171TBKT" H 4500 4275 50  0001 C CNN "Mouse_r3"
+F 14 "160-1579-1-ND" H 4500 4275 50  0001 C CNN "Digikey"
+F 15 "94T2911" H 4500 4275 50  0001 C CNN "Newark"
+F 16 "19J8850" H 4500 4275 50  0001 C CNN "Newar_k2"
+F 17 "C375453" H 4500 4275 50  0001 C CNN "LCSC"
+F 18 "0.02930$" H 4500 4275 50  0001 C CNN "price300_LCSC"
+F 19 "LTST-C170KRKT" H 4500 4275 50  0001 C CNN "LowCost"
+F 20 "FV004" H 4500 4275 50  0001 C CNN "Koncar"
+F 21 "T" H 4500 4275 50  0001 C CNN "Side"
+	1    4500 4275
+	1    0    0    -1
+$EndComp
+$Comp
+L Device:LED_ALT D6
+U 1 1 627AFAB6
+P 4500 4075
+F 0 "D6" H 4500 4175 50  0000 C CNN
+F 1 "GREEN" H 4150 4075 50  0000 R CNN
+F 2 "LED_SMD:LED_0603_1608Metric" H 4500 4075 50  0001 C CNN
+F 3 "http://optoelectronics.liteon.com/upload/download/DS22-2000-073/LTST-C170KGKT.pdf" H 4500 4075 50  0001 C CNN
+F 4 "www.liteon.com" H 4500 4075 60  0001 C CNN "MNF1_URL"
+F 5 "LTST-C170TGKT" H 4500 4075 50  0001 C CNN "MPN"
+F 6 "859-LTST-C170TGKT" H 4500 4075 50  0001 C CNN "Mouser"
+F 7 "160-1887-1-ND" H 4500 4075 50  0001 C CNN "Digikey"
+F 8 "75R0588" H 4500 4075 50  0001 C CNN "Newark"
+F 9 "C364562" H 4500 4075 50  0001 C CNN "LCSC"
+F 10 "LTST-C170TGKT" H 4500 4075 50  0001 C CNN "TME"
+F 11 "0.0789$" H 4500 4075 50  0001 C CNN "price300_TME"
+F 12 "LTST-C170KRKT" H 4500 4075 50  0001 C CNN "LowCost"
+F 13 "FV005" H 4500 4075 50  0001 C CNN "Koncar"
+F 14 "T" H 4500 4075 50  0001 C CNN "Side"
+	1    4500 4075
+	1    0    0    -1
+$EndComp
+$Comp
+L Device:LED_ALT D4
+U 1 1 627AFACD
+P 4500 3675
+F 0 "D4" H 4500 3775 50  0000 C CNN
+F 1 "RED" H 4150 3675 50  0000 R CNN
+F 2 "LED_SMD:LED_0603_1608Metric" H 4500 3675 50  0001 C CNN
+F 3 "https://optoelectronics.liteon.com/upload/download/DS-22-99-0150/LTST-C170KRKT.pdf" H 4500 3675 50  0001 C CNN
+F 4 "www.liteon.com" H 4500 3675 60  0001 C CNN "MNF1_URL"
+F 5 "LTST-C170KRKT" H 4500 3675 60  0001 C CNN "MPN"
+F 6 "859-LTST-C170KRKT" H 4500 3675 60  0001 C CNN "Mouser"
+F 7 "859-LTST-C171KRKT" H 4500 3675 50  0001 C CNN "Mouse_r1"
+F 8 "743-IN-S85ATR" H 4500 3675 50  0001 C CNN "Mouse_r2"
+F 9 "645-598-8110-107F" H 4500 3675 50  0001 C CNN "Mouse_r3"
+F 10 "160-1415-1-ND" H 4500 3675 50  0001 C CNN "Digikey"
+F 11 "75R0581" H 4500 3675 50  0001 C CNN "Newark"
+F 12 "61AC0090" H 4500 3675 50  0001 C CNN "Newar_k2"
+F 13 "C94868" H 4500 3675 50  0001 C CNN "LCSC"
+F 14 "0.0195$" H 4500 3675 50  0001 C CNN "price400_LCSC"
+F 15 "FV007" H 4500 3675 50  0001 C CNN "Koncar"
+F 16 "TB" H 4500 3675 50  0001 C CNN "Side"
+	1    4500 3675
+	1    0    0    -1
+$EndComp
+$Comp
+L Device:LED_ALT D5
+U 1 1 627AFAE4
+P 4500 3875
+F 0 "D5" H 4500 3975 50  0000 C CNN
+F 1 "ORANGE" H 4150 3875 50  0000 R CNN
+F 2 "LED_SMD:LED_0603_1608Metric" H 4500 3875 50  0001 C CNN
+F 3 "https://optoelectronics.liteon.com/upload/download/DS-22-99-0185/LTST-C170KFKT.pdf" H 4500 3875 50  0001 C CNN
+F 4 "www.liteon.com" H 4500 3875 60  0001 C CNN "MNF1_URL"
+F 5 "LTST-C170KFKT" H 4500 3875 60  0001 C CNN "MPN"
+F 6 "859-LTST-C170KFKT" H 4500 3875 60  0001 C CNN "Mouser"
+F 7 "859-LTST-C171KFKT" H 4500 3875 50  0001 C CNN "Mouse_r1"
+F 8 "645-598-8130-107F" H 4500 3875 50  0001 C CNN "Mouse_r3"
+F 9 "160-1413-1-ND" H 4500 3875 50  0001 C CNN "Digikey"
+F 10 "75R0583" H 4500 3875 50  0001 C CNN "Newark"
+F 11 "61AC0088" H 4500 3875 50  0001 C CNN "Newar_k2"
+F 12 "C284931" H 4500 3875 50  0001 C CNN "LCSC"
+F 13 "0.02075$" H 4500 3875 50  0001 C CNN "price200_LCSC"
+F 14 "LTST-C170KRKT" H 4500 3875 50  0001 C CNN "LowCost"
+F 15 "FV006" H 4500 3875 50  0001 C CNN "Koncar"
+F 16 "T" H 4500 3875 50  0001 C CNN "Side"
+	1    4500 3875
+	1    0    0    -1
+$EndComp
+Wire Wire Line
+	4200 4075 4200 4275
+Wire Wire Line
+	4200 3875 4200 4075
+Wire Wire Line
+	4200 4275 4200 4425
+$Comp
+L power:GND #PWR019
+U 1 1 627AFAF1
+P 4200 4425
+F 0 "#PWR019" H 4200 4175 50  0001 C CNN
+F 1 "GND" H 4200 4275 50  0000 C CNN
+F 2 "" H 4200 4425 50  0000 C CNN
+F 3 "" H 4200 4425 50  0000 C CNN
+	1    4200 4425
 	1    0    0    -1
 $EndComp

Commit message: Removing termination chip
Parts:
- added SW3: SW_Push, Switch_EVPAA:Switch_EVPAA, symbol Switch:SW_Push
Connections:
- net at R18.1, SW1.1, SW2.1: now also SW3.1
- new net BTN3: SW3.2
Changed lines of the file:
@@
 	1    0    0    -1
 $EndComp
+$Comp
+L Switch:SW_Push SW3
+U 1 1 628C84D7
+P 2900 3375
+F 0 "SW3" H 3100 3425 50  0000 C CNN
+F 1 "SW_Push" H 2600 3425 50  0000 C CNN
+F 2 "Switch_EVPAA:Switch_EVPAA" H 2900 3575 50  0001 C CNN
+F 3 "https://www.mouser.in/datasheet/2/315/PANA_S_A0001791376_1-2560543.pdf" H 2900 3575 50  0001 C CNN
+F 4 "https://www.mouser.in/ProductDetail/Panasonic/EVP-AA302K?qs=qvwOHSmaRMmnf4H35tvzww==" H 2900 3375 50  0001 C CNN "Mouser"
+F 5 "https://www.digikey.com/en/products/detail/panasonic-electronic-components/EVP-AA302K/2810555" H 2900 3375 50  0001 C CNN "DigiKey"
+	1    2900 3375
+	1    0    0    -1
+$EndComp
+Text GLabel 3350 3375 2    60   Input ~ 0
+BTN3
+Wire Wire Line
+	3100 3375 3350 3375
+Wire Wire Line
+	2700 3375 2400 3375
+Wire Wire Line
+	2400 3375 2400 3150
+Connection ~ 2400 3150
 $EndSCHEMATC

Commit message: DDR3 lines are now around 10% - all GPIOs should be connected
Parts:
- renumbered SW1 to BTN1, SW2 to BTN2, SW3 to BTN3, R41 to R40, R42 to R41, R43 to R42, R44 to R43, R49 to R44, R50 to R45, R51 to R46, R52 to R47
Changed lines of the file:
@@
 LED3
 $Comp
-L Device:R R41
+L Device:R R40
 U 1 1 591E1845
 P 5250 2550
-F 0 "R41" V 5330 2550 50  0000 C CNN
+F 0 "R40" V 5330 2550 50  0000 C CNN
 F 1 "549" V 5250 2550 50  0000 C CNN
 F 2 "Capacitor_SMD:C_0402_1005Metric" V 5180 2550 50  0001 C CNN
@@
 $EndComp
 $Comp
-L Device:R R42
+L Device:R R41
 U 1 1 591E199B
 P 5250 2750
-F 0 "R42" V 5330 2750 50  0000 C CNN
+F 0 "R41" V 5330 2750 50  0000 C CNN
 F 1 "549" V 5250 2750 50  0000 C CNN
 F 2 "Capacitor_SMD:C_0402_1005Metric" V 5180 2750 50  0001 C CNN
@@
 $EndComp
 $Comp
-L Device:R R43
+L Device:R R42
 U 1 1 591E1A9D
 P 5250 2950
-F 0 "R43" V 5330 2950 50  0000 C CNN
+F 0 "R42" V 5330 2950 50  0000 C CNN
 F 1 "549" V 5250 2950 50  0000 C CNN
 F 2 "Capacitor_SMD:C_0402_1005Metric" V 5180 2950 50  0001 C CNN
@@
 $EndComp
 $Comp
-L Device:R R44
+L Device:R R43
 U 1 1 591E1AA3
 P 5250 3150
-F 0 "R44" V 5330 3150 50  0000 C CNN
+F 0 "R43" V 5330 3150 50  0000 C CNN
 F 1 "549" V 5250 3150 50  0000 C CNN
 F 2 "Capacitor_SMD:C_0402_1005Metric" V 5180 3150 50  0001 C CNN
@@
 $EndComp
 $Comp
-L Switch:SW_Push SW1
+L Switch:SW_Push BTN1
 U 1 1 6256B27F
 P 2900 2950
-F 0 "SW1" H 3100 3000 50  0000 C CNN
+F 0 "BTN1" H 3100 3000 50  0000 C CNN
 F 1 "SW_Push" H 2600 3000 50  0000 C CNN
 F 2 "Switch_EVPAA:Switch_EVPAA" H 2900 3150 50  0001 C CNN
@@
 	1850 2950 2000 2950
 $Comp
-L Switch:SW_Push SW2
+L Switch:SW_Push BTN2
 U 1 1 6258110E
 P 2900 3150
-F 0 "SW2" H 3100 3200 50  0000 C CNN
+F 0 "BTN2" H 3100 3200 50  0000 C CNN
 F 1 "SW_Push" H 2600 3200 50  0000 C CNN
 F 2 "Switch_EVPAA:Switch_EVPAA" H 2900 3350 50  0001 C CNN
@@
 Wire Wire Line
 	4650 4275 5050 4275
-Text GLabel 5350 3675 2    60   Input ~ 0
-LED4
-Text GLabel 5350 3875 2    60   Input ~ 0
-LED5
-Text GLabel 5350 4075 2    60   Input ~ 0
-LED6
-Text GLabel 5350 4275 2    60   Input ~ 0
-LED7
-$Comp
-L Device:R R49
+$Comp
+L Device:R R44
 U 1 1 627AFA63
 P 5200 3675
-F 0 "R49" V 5280 3675 50  0000 C CNN
+F 0 "R44" V 5280 3675 50  0000 C CNN
 F 1 "549" V 5200 3675 50  0000 C CNN
 F 2 "Capacitor_SMD:C_0402_1005Metric" V 5130 3675 50  0001 C CNN
@@
 $EndComp
 $Comp
-L Device:R R50
+L Device:R R45
 U 1 1 627AFA6D
 P 5200 3875
-F 0 "R50" V 5280 3875 50  0000 C CNN
+F 0 "R45" V 5280 3875 50  0000 C CNN
 F 1 "549" V 5200 3875 50  0000 C CNN
 F 2 "Capacitor_SMD:C_0402_1005Metric" V 5130 3875 50  0001 C CNN
@@
 $EndComp
 $Comp
-L Device:R R51
+L Device:R R46
 U 1 1 627AFA77
 P 5200 4075
-F 0 "R51" V 5280 4075 50  0000 C CNN
+F 0 "R46" V 5280 4075 50  0000 C CNN
 F 1 "549" V 5200 4075 50  0000 C CNN
 F 2 "Capacitor_SMD:C_0402_1005Metric" V 5130 4075 50  0001 C CNN
@@
 $EndComp
 $Comp
-L Device:R R52
+L Device:R R47
 U 1 1 627AFA81
 P 5200 4275
-F 0 "R52" V 5280 4275 50  0000 C CNN
+F 0 "R47" V 5280 4275 50  0000 C CNN
 F 1 "549" V 5200 4275 50  0000 C CNN
 F 2 "Capacitor_SMD:C_0402_1005Metric" V 5130 4275 50  0001 C CNN
@@
 $EndComp
 $Comp
-L Switch:SW_Push SW3
+L Switch:SW_Push BTN3
 U 1 1 628C84D7
 P 2900 3375
-F 0 "SW3" H 3100 3425 50  0000 C CNN
+F 0 "BTN3" H 3100 3425 50  0000 C CNN
 F 1 "SW_Push" H 2600 3425 50  0000 C CNN
 F 2 "Switch_EVPAA:Switch_EVPAA" H 2900 3575 50  0001 C CNN
@@
 	2400 3375 2400 3150
 Connection ~ 2400 3150
+Text GLabel 5350 4275 2    60   Input ~ 0
+LED7
+Text GLabel 5350 4075 2    60   Input ~ 0
+LED6
+Text GLabel 5350 3875 2    60   Input ~ 0
+LED5
+Text GLabel 5350 3675 2    60   Input ~ 0
+LED4
 $EndSCHEMATC

Commit message: References cleanup
Parts:
- renumbered C46 to C54
Changed lines of the file:
@@
 $Descr A4 11693 8268
 encoding utf-8
-Sheet 4 13
+Sheet 4 11
 Title "ULX3S"
 Date ""
@@
 $EndComp
 $Comp
-L Device:C C46
+L Device:C C54
 U 1 1 5A881E8B
 P 6650 1350
-F 0 "C46" H 6675 1450 50  0000 L CNN
+F 0 "C54" H 6675 1450 50  0000 L CNN
 F 1 "2.2uF" H 6675 1250 50  0000 L CNN
 F 2 "Capacitor_SMD:C_0603_1608Metric" H 6688 1200 50  0001 C CNN

Commit message: Lowering number of unique parts fix #37
Parts:
- R18: value 130 -> 300; footprint Capacitor_SMD:C_0402_1005Metric -> Resistor_SMD:R_0402_1005Metric
- R40, R41, R42, R43, R44, R45, R46, R47: value 549 -> 300; footprint Capacitor_SMD:C_0402_1005Metric -> Resistor_SMD:R_0402_1005Metric
Changed lines of the file:
@@
 P 5250 2550
 F 0 "R40" V 5330 2550 50  0000 C CNN
-F 1 "549" V 5250 2550 50  0000 C CNN
-F 2 "Capacitor_SMD:C_0402_1005Metric" V 5180 2550 50  0001 C CNN
+F 1 "300" V 5250 2550 50  0000 C CNN
+F 2 "Resistor_SMD:R_0402_1005Metric" V 5180 2550 50  0001 C CNN
 F 3 "" H 5250 2550 50  0000 C CNN
 	1    5250 2550
@@
 P 5250 2750
 F 0 "R41" V 5330 2750 50  0000 C CNN
-F 1 "549" V 5250 2750 50  0000 C CNN
-F 2 "Capacitor_SMD:C_0402_1005Metric" V 5180 2750 50  0001 C CNN
+F 1 "300" V 5250 2750 50  0000 C CNN
+F 2 "Resistor_SMD:R_0402_1005Metric" V 5180 2750 50  0001 C CNN
 F 3 "" H 5250 2750 50  0000 C CNN
 	1    5250 2750
@@
 P 5250 2950
 F 0 "R42" V 5330 2950 50  0000 C CNN
-F 1 "549" V 5250 2950 50  0000 C CNN
-F 2 "Capacitor_SMD:C_0402_1005Metric" V 5180 2950 50  0001 C CNN
+F 1 "300" V 5250 2950 50  0000 C CNN
+F 2 "Resistor_SMD:R_0402_1005Metric" V 5180 2950 50  0001 C CNN
 F 3 "" H 5250 2950 50  0000 C CNN
 	1    5250 2950
@@
 P 5250 3150
 F 0 "R43" V 5330 3150 50  0000 C CNN
-F 1 "549" V 5250 3150 50  0000 C CNN
-F 2 "Capacitor_SMD:C_0402_1005Metric" V 5180 3150 50  0001 C CNN
+F 1 "300" V 5250 3150 50  0000 C CNN
+F 2 "Resistor_SMD:R_0402_1005Metric" V 5180 3150 50  0001 C CNN
 F 3 "" H 5250 3150 50  0000 C CNN
 	1    5250 3150
@@
 P 2150 2950
 F 0 "R18" V 2230 2950 50  0000 C CNN
-F 1 "130" V 2150 2950 50  0000 C CNN
-F 2 "Capacitor_SMD:C_0402_1005Metric" V 2080 2950 50  0001 C CNN
+F 1 "300" V 2150 2950 50  0000 C CNN
+F 2 "Resistor_SMD:R_0402_1005Metric" V 2080 2950 50  0001 C CNN
 F 3 "" H 2150 2950 50  0000 C CNN
 	1    2150 2950
@@
 P 5200 3675
 F 0 "R44" V 5280 3675 50  0000 C CNN
-F 1 "549" V 5200 3675 50  0000 C CNN
-F 2 "Capacitor_SMD:C_0402_1005Metric" V 5130 3675 50  0001 C CNN
+F 1 "300" V 5200 3675 50  0000 C CNN
+F 2 "Resistor_SMD:R_0402_1005Metric" V 5130 3675 50  0001 C CNN
 F 3 "" H 5200 3675 50  0000 C CNN
 	1    5200 3675
@@
 P 5200 3875
 F 0 "R45" V 5280 3875 50  0000 C CNN
-F 1 "549" V 5200 3875 50  0000 C CNN
-F 2 "Capacitor_SMD:C_0402_1005Metric" V 5130 3875 50  0001 C CNN
+F 1 "300" V 5200 3875 50  0000 C CNN
+F 2 "Resistor_SMD:R_0402_1005Metric" V 5130 3875 50  0001 C CNN
 F 3 "" H 5200 3875 50  0000 C CNN
 	1    5200 3875
@@
 P 5200 4075
 F 0 "R46" V 5280 4075 50  0000 C CNN
-F 1 "549" V 5200 4075 50  0000 C CNN
-F 2 "Capacitor_SMD:C_0402_1005Metric" V 5130 4075 50  0001 C CNN
+F 1 "300" V 5200 4075 50  0000 C CNN
+F 2 "Resistor_SMD:R_0402_1005Metric" V 5130 4075 50  0001 C CNN
 F 3 "" H 5200 4075 50  0000 C CNN
 	1    5200 4075
@@
 P 5200 4275
 F 0 "R47" V 5280 4275 50  0000 C CNN
-F 1 "549" V 5200 4275 50  0000 C CNN
-F 2 "Capacitor_SMD:C_0402_1005Metric" V 5130 4275 50  0001 C CNN
+F 1 "300" V 5200 4275 50  0000 C CNN
+F 2 "Resistor_SMD:R_0402_1005Metric" V 5130 4275 50  0001 C CNN
 F 3 "" H 5200 4275 50  0000 C CNN
 	1    5200 4275
