File: flash.sch (KiCad schematic (older format))
At the start: 13 parts, among them U1 LFE5U-85F-6BG381C, U10 IS25LP128F-JBLE

Commit message: More removal, spliting modules
Parts:
- R11, R12, R27, R28, R29, R30, R31, R32, R33: footprint Resistor_SMD:R_0603_1608Metric -> Capacitor_SMD:C_0402_1005Metric
Changed lines of the file:
@@
 F 0 "R27" V 3530 2350 50  0000 C CNN
 F 1 "10k" V 3450 2350 50  0000 C CNN
-F 2 "Resistor_SMD:R_0603_1608Metric" V 3380 2350 50  0001 C CNN
+F 2 "Capacitor_SMD:C_0402_1005Metric" V 3380 2350 50  0001 C CNN
 F 3 "" H 3450 2350 50  0000 C CNN
 	1    3450 2350
@@
 F 0 "R28" V 3730 2350 50  0000 C CNN
 F 1 "10k" V 3650 2350 50  0000 C CNN
-F 2 "Resistor_SMD:R_0603_1608Metric" V 3580 2350 50  0001 C CNN
+F 2 "Capacitor_SMD:C_0402_1005Metric" V 3580 2350 50  0001 C CNN
 F 3 "" H 3650 2350 50  0000 C CNN
 	1    3650 2350
@@
 F 0 "R29" V 3930 2350 50  0000 C CNN
 F 1 "1.1k" V 3850 2350 50  0000 C CNN
-F 2 "Resistor_SMD:R_0603_1608Metric" V 3780 2350 50  0001 C CNN
+F 2 "Capacitor_SMD:C_0402_1005Metric" V 3780 2350 50  0001 C CNN
 F 3 "" H 3850 2350 50  0000 C CNN
 	1    3850 2350
@@
 F 0 "R30" V 4130 2350 50  0000 C CNN
 F 1 "4.7k" V 4050 2350 50  0000 C CNN
-F 2 "Resistor_SMD:R_0603_1608Metric" V 3980 2350 50  0001 C CNN
+F 2 "Capacitor_SMD:C_0402_1005Metric" V 3980 2350 50  0001 C CNN
 F 3 "" H 4050 2350 50  0000 C CNN
 F 4 "www.yageo.com" V 4050 2350 50  0001 C CNN "MNF1_URL"
@@
 F 0 "R11" V 3130 2350 50  0000 C CNN
 F 1 "10k" V 3050 2350 50  0000 C CNN
-F 2 "Resistor_SMD:R_0603_1608Metric" V 2980 2350 50  0001 C CNN
+F 2 "Capacitor_SMD:C_0402_1005Metric" V 2980 2350 50  0001 C CNN
 F 3 "" H 3050 2350 50  0000 C CNN
 F 4 "www.yageo.com" V 3050 2350 50  0001 C CNN "MNF1_URL"
@@
 F 0 "R12" V 3330 2350 50  0000 C CNN
 F 1 "10k" V 3250 2350 50  0000 C CNN
-F 2 "Resistor_SMD:R_0603_1608Metric" V 3180 2350 50  0001 C CNN
+F 2 "Capacitor_SMD:C_0402_1005Metric" V 3180 2350 50  0001 C CNN
 F 3 "" H 3250 2350 50  0000 C CNN
 	1    3250 2350
@@
 F 0 "R31" V 5280 2350 50  0000 C CNN
 F 1 "15k" V 5200 2350 50  0000 C CNN
-F 2 "Resistor_SMD:R_0603_1608Metric" V 5130 2350 50  0001 C CNN
+F 2 "Capacitor_SMD:C_0402_1005Metric" V 5130 2350 50  0001 C CNN
 F 3 "" H 5200 2350 50  0000 C CNN
 	1    5200 2350
@@
 F 0 "R32" V 5480 2350 50  0000 C CNN
 F 1 "15k" V 5400 2350 50  0000 C CNN
-F 2 "Resistor_SMD:R_0603_1608Metric" V 5330 2350 50  0001 C CNN
+F 2 "Capacitor_SMD:C_0402_1005Metric" V 5330 2350 50  0001 C CNN
 F 3 "" H 5400 2350 50  0000 C CNN
 	1    5400 2350
@@
 F 0 "R33" V 5680 2350 50  0000 C CNN
 F 1 "15k" V 5600 2350 50  0000 C CNN
-F 2 "Resistor_SMD:R_0603_1608Metric" V 5530 2350 50  0001 C CNN
+F 2 "Capacitor_SMD:C_0402_1005Metric" V 5530 2350 50  0001 C CNN
 F 3 "" H 5600 2350 50  0000 C CNN
 	1    5600 2350

Commit message: Before power placement
Parts:
- D28, D29: footprint Diode_SMD:D_SOD-323_HandSoldering -> Diode_SMD:D_SOD-323
Changed lines of the file:
@@
 F 0 "D28" H 5000 3500 50  0000 C CNN
 F 1 "1N914" H 5400 3400 50  0000 C CNN
-F 2 "Diode_SMD:D_SOD-323_HandSoldering" H 5000 3400 50  0001 C CNN
+F 2 "Diode_SMD:D_SOD-323" H 5000 3400 50  0001 C CNN
 F 3 "~" H 5000 3400 50  0001 C CNN
 F 4 "Leave empty" H 5000 3400 50  0001 C CNN "Note"
@@
 F 0 "D29" H 5000 3450 50  0000 C CNN
 F 1 "1N914" H 5400 3550 50  0000 C CNN
-F 2 "Diode_SMD:D_SOD-323_HandSoldering" H 5000 3550 50  0001 C CNN
+F 2 "Diode_SMD:D_SOD-323" H 5000 3550 50  0001 C CNN
 F 3 "~" H 5000 3550 50  0001 C CNN
 	1    5000 3550

Commit message: Connecting more GPIOs, improving routing
Connections:
- net labels added: GPIO13, GPIO19, GPIO26, GPIO6
Changed lines of the file:
@@
 	0    1    1    0
 $EndComp
-Text GLabel 6500 3800 0    60   Input ~ 0
+Text GLabel 8400 3300 0    60   Input ~ 0
 BTN_F1
-Text GLabel 8000 3800 2    60   Input ~ 0
+Text GLabel 9000 3650 2    60   Input ~ 0
 BTN_F2
-Text GLabel 8000 3900 2    60   Input ~ 0
+Text GLabel 9050 3500 2    60   Input ~ 0
 BTN_D
-Text GLabel 6500 3900 0    60   Input ~ 0
+Text GLabel 8650 3450 0    60   Input ~ 0
 BTN_L
 Text Notes 4700 1950 0    60   ~ 0
@@
 	1    0    0    -1
 $EndComp
+Text GLabel 8000 3900 2    60   Input ~ 0
+GPIO26
+Text GLabel 6500 3900 0    60   Input ~ 0
+GPIO19
+Text GLabel 8000 3800 2    60   Input ~ 0
+GPIO13
+Text GLabel 6500 3800 0    60   Input ~ 0
+GPIO6
 $EndSCHEMATC

Commit message: Cleanup schematics
Connections:
- net labels removed: BTN_D, BTN_F1, BTN_F2, BTN_L
Changed lines of the file:
@@
 	0    1    1    0
 $EndComp
-Text GLabel 8400 3300 0    60   Input ~ 0
-BTN_F1
-Text GLabel 9000 3650 2    60   Input ~ 0
-BTN_F2
-Text GLabel 9050 3500 2    60   Input ~ 0
-BTN_D
-Text GLabel 8650 3450 0    60   Input ~ 0
-BTN_L
 Text Notes 4700 1950 0    60   ~ 0
 pullups to allow entering USER mode\nTN1260: lattice ECP5 sysCONFIG guide p.6, p.8, p.13
