File: flash.sch (KiCad schematic (older format))
At the start: 13 parts, among them U1 LFE5U-85F-6BG381C, U10 IS25LP128F-JBLE

Commit message: Fix #12 If RC1 and RC2 are placed voltahe will be 1.2V
Parts:
- R29: value 1.1k -> 1k1
- R30: value 4.7k -> 4k7
Changed lines of the file:
@@
 P 3850 2350
 F 0 "R29" V 3930 2350 50  0000 C CNN
-F 1 "1.1k" V 3850 2350 50  0000 C CNN
+F 1 "1k1" V 3850 2350 50  0000 C CNN
 F 2 "Capacitor_SMD:C_0402_1005Metric" V 3780 2350 50  0001 C CNN
 F 3 "" H 3850 2350 50  0000 C CNN
@@
 P 4050 2350
 F 0 "R30" V 4130 2350 50  0000 C CNN
-F 1 "4.7k" V 4050 2350 50  0000 C CNN
+F 1 "4k7" V 4050 2350 50  0000 C CNN
 F 2 "Capacitor_SMD:C_0402_1005Metric" V 3980 2350 50  0001 C CNN
 F 3 "" H 4050 2350 50  0000 C CNN

Commit message: Removing termination chip
Parts:
- D28, D29: footprint Diode_SMD:D_SOD-323 -> (none)
Changed lines of the file:
@@
 F 0 "D28" H 5000 3500 50  0000 C CNN
 F 1 "1N914" H 5400 3400 50  0000 C CNN
-F 2 "Diode_SMD:D_SOD-323" H 5000 3400 50  0001 C CNN
+F 2 "" H 5000 3400 50  0001 C CNN
 F 3 "~" H 5000 3400 50  0001 C CNN
 F 4 "Leave empty" H 5000 3400 50  0001 C CNN "Note"
@@
 F 0 "D29" H 5000 3450 50  0000 C CNN
 F 1 "1N914" H 5400 3550 50  0000 C CNN
-F 2 "Diode_SMD:D_SOD-323" H 5000 3550 50  0001 C CNN
+F 2 "" H 5000 3550 50  0001 C CNN
 F 3 "~" H 5000 3550 50  0001 C CNN
 	1    5000 3550

Commit message: fix #19 fix #18
Parts:
- renumbered U10 to U3
Changed lines of the file:
@@
 $EndDescr
 $Comp
-L Memory_EEPROM:25LCxxx U10
+L Memory_EEPROM:25LCxxx U3
 U 1 1 58D913F5
 P 3650 4350
-F 0 "U10" H 3350 4600 50  0000 L CNN
+F 0 "U3" H 3350 4600 50  0000 L CNN
 F 1 "IS25LP128F-JBLE" H 3700 4600 50  0000 L CNN
 F 2 "SOA008-150mil:SOA008-150-208mil" H 3300 4300 50  0001 C CNN

Commit message: Lowering number of unique parts fix #37
Parts:
- R11, R12, R27, R28: value 10k -> 15k; footprint Capacitor_SMD:C_0402_1005Metric -> Resistor_SMD:R_0402_1005Metric
- R29: value 1k1 -> 1k; footprint Capacitor_SMD:C_0402_1005Metric -> Resistor_SMD:R_0402_1005Metric
- R30, R31, R32, R33: footprint Capacitor_SMD:C_0402_1005Metric -> Resistor_SMD:R_0402_1005Metric
Changed lines of the file:
@@
 P 3450 2350
 F 0 "R27" V 3530 2350 50  0000 C CNN
-F 1 "10k" V 3450 2350 50  0000 C CNN
-F 2 "Capacitor_SMD:C_0402_1005Metric" V 3380 2350 50  0001 C CNN
+F 1 "15k" V 3450 2350 50  0000 C CNN
+F 2 "Resistor_SMD:R_0402_1005Metric" V 3380 2350 50  0001 C CNN
 F 3 "" H 3450 2350 50  0000 C CNN
 	1    3450 2350
@@
 P 3650 2350
 F 0 "R28" V 3730 2350 50  0000 C CNN
-F 1 "10k" V 3650 2350 50  0000 C CNN
-F 2 "Capacitor_SMD:C_0402_1005Metric" V 3580 2350 50  0001 C CNN
+F 1 "15k" V 3650 2350 50  0000 C CNN
+F 2 "Resistor_SMD:R_0402_1005Metric" V 3580 2350 50  0001 C CNN
 F 3 "" H 3650 2350 50  0000 C CNN
 	1    3650 2350
@@
 P 3850 2350
 F 0 "R29" V 3930 2350 50  0000 C CNN
-F 1 "1k1" V 3850 2350 50  0000 C CNN
-F 2 "Capacitor_SMD:C_0402_1005Metric" V 3780 2350 50  0001 C CNN
+F 1 "1k" V 3850 2350 50  0000 C CNN
+F 2 "Resistor_SMD:R_0402_1005Metric" V 3780 2350 50  0001 C CNN
 F 3 "" H 3850 2350 50  0000 C CNN
 	1    3850 2350
@@
 F 0 "R30" V 4130 2350 50  0000 C CNN
 F 1 "4k7" V 4050 2350 50  0000 C CNN
-F 2 "Capacitor_SMD:C_0402_1005Metric" V 3980 2350 50  0001 C CNN
+F 2 "Resistor_SMD:R_0402_1005Metric" V 3980 2350 50  0001 C CNN
 F 3 "" H 4050 2350 50  0000 C CNN
 F 4 "www.yageo.com" V 4050 2350 50  0001 C CNN "MNF1_URL"
@@
 P 3050 2350
 F 0 "R11" V 3130 2350 50  0000 C CNN
-F 1 "10k" V 3050 2350 50  0000 C CNN
-F 2 "Capacitor_SMD:C_0402_1005Metric" V 2980 2350 50  0001 C CNN
+F 1 "15k" V 3050 2350 50  0000 C CNN
+F 2 "Resistor_SMD:R_0402_1005Metric" V 2980 2350 50  0001 C CNN
 F 3 "" H 3050 2350 50  0000 C CNN
 F 4 "www.yageo.com" V 3050 2350 50  0001 C CNN "MNF1_URL"
@@
 P 3250 2350
 F 0 "R12" V 3330 2350 50  0000 C CNN
-F 1 "10k" V 3250 2350 50  0000 C CNN
-F 2 "Capacitor_SMD:C_0402_1005Metric" V 3180 2350 50  0001 C CNN
+F 1 "15k" V 3250 2350 50  0000 C CNN
+F 2 "Resistor_SMD:R_0402_1005Metric" V 3180 2350 50  0001 C CNN
 F 3 "" H 3250 2350 50  0000 C CNN
 	1    3250 2350
@@
 F 0 "R31" V 5280 2350 50  0000 C CNN
 F 1 "15k" V 5200 2350 50  0000 C CNN
-F 2 "Capacitor_SMD:C_0402_1005Metric" V 5130 2350 50  0001 C CNN
+F 2 "Resistor_SMD:R_0402_1005Metric" V 5130 2350 50  0001 C CNN
 F 3 "" H 5200 2350 50  0000 C CNN
 	1    5200 2350
@@
 F 0 "R32" V 5480 2350 50  0000 C CNN
 F 1 "15k" V 5400 2350 50  0000 C CNN
-F 2 "Capacitor_SMD:C_0402_1005Metric" V 5330 2350 50  0001 C CNN
+F 2 "Resistor_SMD:R_0402_1005Metric" V 5330 2350 50  0001 C CNN
 F 3 "" H 5400 2350 50  0000 C CNN
 	1    5400 2350
@@
 F 0 "R33" V 5680 2350 50  0000 C CNN
 F 1 "15k" V 5600 2350 50  0000 C CNN
-F 2 "Capacitor_SMD:C_0402_1005Metric" V 5530 2350 50  0001 C CNN
+F 2 "Resistor_SMD:R_0402_1005Metric" V 5530 2350 50  0001 C CNN
 F 3 "" H 5600 2350 50  0000 C CNN
 	1    5600 2350
