File: gpdi.sch (KiCad schematic (older format))
At the start: 21 parts, among them U1 LFE5U-85F-6BG381C, U11 PCA9306D

Commit message: More removing
Parts:
- removed C18: 100pF, Capacitor_SMD:C_0603_1608Metric, symbol Device:C
- removed C38, C39, C40, C41, C42, C43, C44, C45: 22nF, Capacitor_SMD:C_0603_1608Metric, symbol Device:C
- removed D30: 3.6V, Diode_SMD:D_SOD-323_HandSoldering, symbol Device:D_Zener_Small_ALT
- removed GPDI1: GPDI-D, conn-fci:CONN-10029449-111RLF, symbol hdmi-d:HDMI-D
- removed R22, R23: 3.3k, Resistor_SMD:R_0603_1608Metric, symbol Device:R
- removed R24: 100k, Resistor_SMD:R_0603_1608Metric, symbol Device:R
- removed R25, R26: 4.7k, Resistor_SMD:R_0603_1608Metric, symbol Device:R
- removed R55: 10k, Resistor_SMD:R_0603_1608Metric, symbol Device:R
- removed R61: 549, Resistor_SMD:R_0603_1608Metric, symbol Device:R
- removed U11: PCA9306D, SM8:SM8, symbol pca9306d:PCA9306D

Commit message: Sync sch and pcb
Parts:
- removed R67: 549, Resistor_SMD:R_0603_1608Metric, symbol Device:R
Connections:
- net labels removed: +3V3, +5V, GND, GPDI_CEC, GPDI_CLK+, GPDI_CLK-, GPDI_D0+, GPDI_D0-, GPDI_D1+, GPDI_D1-, GPDI_D2+, GPDI_D2-, GPDI_HPD, GPDI_UTIL, VREF2
- wire segments 63 -> 0

Commit message: Before power placement
Parts:
- added C13, C14, C15, C18, C21, C36, C37, C38, C39, C40, C41, C42, C43, C44, C45, C54: 100n, Capacitor_SMD:C_0402_1005Metric, symbol Device:C_Small
- added R10, R13, R14, R15: 4K7, Resistor_SMD:R_0402_1005Metric, symbol Device:R_Small
- added R16, R17, R8, R9: 100K, Resistor_SMD:R_0402_1005Metric, symbol Device:R_Small
Connections:
- net FPDI_CLK+: now also C37.1
- net FPDI_CLK-: now also C38.1
- net FPDI_D0+: now also C21.1
- net FPDI_D0-: now also C36.1
- net FPDI_D1+: now also C15.1
- net FPDI_D1-: now also C18.1
- net FPDI_D2+: now also C13.1
- net FPDI_D2-: now also C14.1
- new net +3V3: R16.1, R8.1
- new net +5V: R10.1, R13.1, R14.1, R15.1
- new net GN0: C54.1
- new net GN3: C44.1
- new net GN4: C42.1
- new net GN5: C40.1
- new net GND: R17.1, R9.1
- new net GP0: C45.1
- new net GP3: C43.1
- new net GP4: C41.1
- new net GP5: C39.1
- new net HDMI0_CEC: R8.2
- new net HDMI0_CLK_N: C38.2
- new net HDMI0_CLK_P: C37.2
- new net HDMI0_HOTPLUG: R9.2
- new net HDMI0_SCL: R14.2
- new net HDMI0_SDA: R15.2
- new net HDMI0_TX0_N: C36.2
- new net HDMI0_TX0_P: C21.2
- new net HDMI0_TX1_N: C18.2
- new net HDMI0_TX1_P: C15.2
- new net HDMI0_TX2_N: C14.2
- new net HDMI0_TX2_P: C13.2
- new net HDMI1_CEC: R16.2
- new net HDMI1_CLK_N: C54.2
- new net HDMI1_CLK_P: C45.2
- new net HDMI1_HOTPLUG: R17.2
- new net HDMI1_SCL: R10.2
- new net HDMI1_SDA: R13.2
- new net HDMI1_TX0_N: C44.2
- new net HDMI1_TX0_P: C43.2
- new net HDMI1_TX1_N: C42.2
- new net HDMI1_TX1_P: C41.2
- new net HDMI1_TX2_N: C40.2
- new net HDMI1_TX2_P: C39.2
Other:
- note added: "0"
- note added: "1"
- note added: "2"
- note added: "3"
- note added: "4"
- note added: "5"
- note added: "6"
- note added: "DAC WIFI_GPIO25"
- note added: "GR_PCLK0_0"
- note added: "GR_PCLK0_1"
- note added: "PCLKC0_0"
- note added: "PCLKC0_1"
- note added: "PCLKT0_0"
- note added: "PCLKT0_1"
- note removed: "i2c shared with RTC\non "power" sheet"
- note removed: "v1.9: VCC1=3.3V EN=5V"

Commit message: SDRAM, JTAG routed - before logo delete
Connections:
- net USB_FPGA_PULL_D+: no longer names the net of U1.B12 (PCLKT1_0)
- net USB_FPGA_PULL_D-: no longer names the net of U1.C12 (PCLKC1_0)
Changed lines of the file:
@@
 Text Notes 5400 3650 0    60   ~ 0
 FPDI SCL v1.7
-Text GLabel 2850 3600 0    60   Input ~ 0
-USB_FPGA_PULL_D+
-Text GLabel 4350 3600 2    60   Input ~ 0
-USB_FPGA_PULL_D-
 Text Notes 7550 6200 0    60   ~ 0
 PCB v1.8.1 and higher accept FCI 10029449-111RLF\nwww.amphenol-icc.com\nmouser PN: 649-10029449-111RLF\nhttp://portal.fciconnect.com/Comergent/fci/drawing/10029449.pdf\n\nPCB v1.7 and v1.8 accept\nmouser PN: 538-47151-1001 (Molex)\nhttps://www.molex.com/pdm_docs/sd/471511001_sd.pdf\nmouser PN: 710-685119134923 (Wurth)\nhttps://katalog.we-online.com/em/datasheet/685119134923.pdf

Commit message: Routing cam and display differential
Connections:
- net FPDI_CLK+: no longer U1.A17 (PT116A)
- net FPDI_CLK-: no longer U1.B18 (PT116B)
- net FPDI_D0+: no longer U1.A16 (PT110A)
- net FPDI_D0-: no longer U1.B16 (PT110B)
- net FPDI_D1+: no longer U1.A14 (PT83A)
- net FPDI_D1-: no longer U1.C14 (PT83B)
- net FPDI_D2+: no longer U1.A12 (PT76A)
- net FPDI_D2-: no longer U1.A13 (PT76B)
- net FPDI_SCL: no longer U1.E12 (GR_PCLK1_1)
- net GN26: no longer U1.C13 (PT78B)
- net GN27: no longer U1.E13 (PT80B)
- net GP26: no longer U1.B13 (PT78A)
- net GP27: no longer U1.D13 (PT80A)
- net CAM0_C_P: now reaches U1.B12 (PCLKT1_0)
- net CAM0_C_N: now reaches U1.C12 (PCLKC1_0)
- net DSI0_C_P: now reaches U1.D12 (GR_PCLK1_0)
- new net CAM0_D0_N: U1.A13 (PT76B)
- new net CAM0_D0_P: U1.A12 (PT76A)
- new net CAM0_D1_N: U1.C13 (PT78B)
- new net CAM0_D1_P: U1.B13 (PT78A)
- new net DSI0_C_N: U1.E12 (GR_PCLK1_1)
- new net DSI0_D0_N: U1.E13 (PT80B)
- new net DSI0_D0_P: U1.D13 (PT80A)
- new net DSI0_D1_N: U1.C14 (PT83B)
- new net DSI0_D1_P: U1.A14 (PT83A)
Changed lines of the file:
@@
 Text GLabel 3250 5950 0    60   Input ~ 0
 FPDI_SDA
-Text GLabel 2850 2700 0    60   Input ~ 0
-FPDI_D0+
-Text GLabel 4350 2700 2    60   Input ~ 0
-FPDI_D0-
-Text GLabel 4350 3100 2    60   Input ~ 0
-FPDI_D1-
-Text GLabel 4350 3400 2    60   Input ~ 0
-FPDI_D2-
-Text GLabel 4350 2400 2    60   Input ~ 0
-FPDI_CLK-
 Text GLabel 4350 2200 2    60   Input ~ 0
 FPDI_HPD
-Text GLabel 2850 3100 0    60   Input ~ 0
-FPDI_D1+
-Text GLabel 2850 3400 0    60   Input ~ 0
-FPDI_D2+
-Text GLabel 2850 2400 0    60   Input ~ 0
-FPDI_CLK+
 Text GLabel 2850 2200 0    60   Input ~ 0
 FPDI_UTIL
-Text GLabel 4350 3500 2    60   Input ~ 0
+Text GLabel 4550 4050 2    60   Input ~ 0
 FPDI_SCL
 Text GLabel 4350 2300 2    60   Input ~ 0
@@
 Text GLabel 4350 3000 2    60   Input ~ 0
 GN25
-Text GLabel 4350 3300 2    60   Input ~ 0
+Text GLabel 1050 3500 2    60   Input ~ 0
 GN26
-Text GLabel 4350 3200 2    60   Input ~ 0
+Text GLabel 1600 3600 2    60   Input ~ 0
 GN27
-Text GLabel 2850 3200 0    60   Input ~ 0
+Text GLabel 1800 3200 0    60   Input ~ 0
 GP27
 Text GLabel 2850 2600 0    60   Input ~ 0
@@
 Text GLabel 2850 2500 0    60   Input ~ 0
 GP23
-Text GLabel 2850 3300 0    60   Input ~ 0
+Text GLabel 1350 3350 0    60   Input ~ 0
 GP26
 Text GLabel 2850 2900 0    60   Input ~ 0
@@
 	0    -1   -1   0
 $EndComp
+Text GLabel 4350 3400 2    60   Input ~ 0
+CAM0_D0_N
+Text GLabel 2850 3400 0    60   Input ~ 0
+CAM0_D0_P
+Text GLabel 4350 3300 2    60   Input ~ 0
+CAM0_D1_N
+Text GLabel 2850 3300 0    60   Input ~ 0
+CAM0_D1_P
+Text GLabel 4350 3600 2    60   Input ~ 0
+CAM0_C_N
+Text GLabel 2850 3600 0    60   Input ~ 0
+CAM0_C_P
+Text GLabel 2850 3500 0    60   Input ~ 0
+DSI0_C_P
+Text GLabel 4350 3500 2    60   Input ~ 0
+DSI0_C_N
+Text GLabel 2850 3100 0    60   Input ~ 0
+DSI0_D1_P
+Text GLabel 4350 3100 2    60   Input ~ 0
+DSI0_D1_N
+Text GLabel 2850 3200 0    60   Input ~ 0
+DSI0_D0_P
+Text GLabel 4350 3200 2    60   Input ~ 0
+DSI0_D0_N
 $EndSCHEMATC

Commit message: Connecting all GPIOs, connecting SDCARD
Connections:
- net FPDI_CEC: no longer U1.A18 (PT119A)
- net FPDI_HPD: no longer U1.B20 (PT121B)
- net FPDI_SDA: no longer U1.B19 (PT119B)
- net FPDI_UTIL: no longer U1.A19 (PT121A)
- new net DSI1_D2_N: U1.B20 (PT121B)
- new net DSI1_D2_P: U1.A19 (PT121A)
- new net DSI1_D3_N: U1.B19 (PT119B)
- new net DSI1_D3_P: U1.A18 (PT119A)
Changed lines of the file:
@@
 Text GLabel 3250 5950 0    60   Input ~ 0
 FPDI_SDA
-Text GLabel 4350 2200 2    60   Input ~ 0
+Text GLabel 5000 1750 2    60   Input ~ 0
 FPDI_HPD
-Text GLabel 2850 2200 0    60   Input ~ 0
+Text GLabel 1900 2150 0    60   Input ~ 0
 FPDI_UTIL
 Text GLabel 4550 4050 2    60   Input ~ 0
 FPDI_SCL
-Text GLabel 4350 2300 2    60   Input ~ 0
+Text GLabel 5050 1875 2    60   Input ~ 0
 FPDI_SDA
-Text GLabel 2850 2300 0    60   Input ~ 0
+Text GLabel 1900 2250 0    60   Input ~ 0
 FPDI_CEC
 Text GLabel 4350 2900 2    60   Input ~ 0
@@
 Text GLabel 4350 3200 2    60   Input ~ 0
 DSI0_D0_N
+Text GLabel 4350 2200 2    60   Input ~ 0
+DSI1_D2_N
+Text GLabel 2850 2200 0    60   Input ~ 0
+DSI1_D2_P
+Text GLabel 4350 2300 2    60   Input ~ 0
+DSI1_D3_N
+Text GLabel 2850 2300 0    60   Input ~ 0
+DSI1_D3_P
 $EndSCHEMATC

Commit message: Cleanup schematics
Connections:
- net GN22: no longer names the net of U1.C15 (PT105B)
- net GN23: no longer names the net of U1.C17 (PT114B)
- net GN24: no longer names the net of U1.D16 (PT112B)
- net GN25: no longer names the net of U1.E14 (PT85B)
- net GP22: no longer names the net of U1.B15 (PT105A)
- net GP23: no longer names the net of U1.B17 (PT114A)
- net GP24: no longer names the net of U1.C16 (PT112A)
- net GP25: no longer names the net of U1.D14 (PT85A)
Other:
- note removed: "0"
- note removed: "1"
- note removed: "2"
- note removed: "3"
- note removed: "4"
- note removed: "5"
- note removed: "6"
- note removed: "DAC WIFI_GPIO25"
- note removed: "FPDI SCL v1.7"
- note removed: "GN22 v1.7"
- note removed: "GN25 v1.7"
- note removed: "GP22 v1.7"
- note removed: "GP25 v1.7"
- note removed: "GR_PCLK0_0"
- note removed: "GR_PCLK0_1"
- note removed: "PCB v1.8.1 and higher accept FCI 10029449-111RLF\nwww.amphenol-icc.com\nmouser PN: 649-10029449-111RLF\nhttp://portal.fciconnect.com/Comergent/fci/drawing/10029449.pdf\n\nPCB v1.7 and v1.8 accept\nmouser PN: 538-47151-1001 (Molex)\nhttps://www.molex.com/pdm_docs/sd/471511001_sd.pdf\nmouser PN: 710-685119134923 (Wurth)\nhttps://katalog.we-online.com/em/datasheet/685119134923.pdf"
- note removed: "PCLKC0_0"
- note removed: "PCLKC0_1"
- note removed: "PCLKT0_0"
- note removed: "PCLKT0_1"
Changed lines of the file:
@@
 Comment4 ""
 $EndDescr
-Text GLabel 2600 6000 0    60   Input ~ 0
-FPDI_HPD
-Text GLabel 3250 6100 0    60   Input ~ 0
-FPDI_UTIL
 Text GLabel 6950 2100 0    60   Input ~ 0
 FPDI_D2+
@@
 Text GLabel 6950 3500 0    60   Input ~ 0
 FPDI_CLK-
-Text GLabel 2600 6100 0    60   Input ~ 0
-FPDI_CEC
-Text GLabel 2850 6450 2    60   Input ~ 0
-GPDI_SDA
-Text GLabel 2850 6300 2    60   Input ~ 0
-GPDI_SCL
-Text GLabel 3250 5800 0    60   Input ~ 0
-FPDI_SCL
-Text GLabel 3250 5950 0    60   Input ~ 0
-FPDI_SDA
-Text GLabel 5000 1750 2    60   Input ~ 0
-FPDI_HPD
-Text GLabel 1900 2150 0    60   Input ~ 0
-FPDI_UTIL
-Text GLabel 4550 4050 2    60   Input ~ 0
-FPDI_SCL
-Text GLabel 5050 1875 2    60   Input ~ 0
-FPDI_SDA
-Text GLabel 1900 2250 0    60   Input ~ 0
-FPDI_CEC
-Text GLabel 4350 2900 2    60   Input ~ 0
-GN22
-Text GLabel 4350 2500 2    60   Input ~ 0
-GN23
-Text GLabel 4350 2600 2    60   Input ~ 0
-GN24
-Text GLabel 4350 3000 2    60   Input ~ 0
-GN25
-Text GLabel 1050 3500 2    60   Input ~ 0
-GN26
-Text GLabel 1600 3600 2    60   Input ~ 0
-GN27
-Text GLabel 1800 3200 0    60   Input ~ 0
-GP27
-Text GLabel 2850 2600 0    60   Input ~ 0
-GP24
-Text GLabel 2850 2500 0    60   Input ~ 0
-GP23
-Text GLabel 1350 3350 0    60   Input ~ 0
-GP26
-Text GLabel 2850 2900 0    60   Input ~ 0
-GP22
-Text GLabel 2850 3000 0    60   Input ~ 0
-GP25
 $Comp
 L lfe5bg381:LFE5UM-85F-6BG381C U1
@@
 	1    0    0    -1
 $EndComp
-Text Notes 1600 2850 0    60   ~ 0
-GP22 v1.7
-Text Notes 5100 2850 0    60   ~ 0
-GN22 v1.7
-Text Notes 1600 2950 0    60   ~ 0
-GP25 v1.7
-Text Notes 5100 2950 0    60   ~ 0
-GN25 v1.7
 Text GLabel 2850 2800 0    60   Input ~ 0
 USB_FPGA_D+
 Text GLabel 4350 2800 2    60   Input ~ 0
 USB_FPGA_D-
-Text Notes 5400 3650 0    60   ~ 0
-FPDI SCL v1.7
-Text Notes 7550 6200 0    60   ~ 0
-PCB v1.8.1 and higher accept FCI 10029449-111RLF\nwww.amphenol-icc.com\nmouser PN: 649-10029449-111RLF\nhttp://portal.fciconnect.com/Comergent/fci/drawing/10029449.pdf\n\nPCB v1.7 and v1.8 accept\nmouser PN: 538-47151-1001 (Molex)\nhttps://www.molex.com/pdm_docs/sd/471511001_sd.pdf\nmouser PN: 710-685119134923 (Wurth)\nhttps://katalog.we-online.com/em/datasheet/685119134923.pdf
 NoConn ~ 2850 3700
 NoConn ~ 2850 3800
@@
 Text GLabel 8550 4600 2    60   Input ~ 0
 HDMI0_SCL
-Text GLabel 3150 5600 0    60   Input ~ 0
-GND
 Text GLabel 7500 3500 2    60   Input ~ 0
 HDMI0_CLK_N
@@
 Text GLabel 8900 3300 0    60   Input ~ 0
 GP0
-Text GLabel 3500 7000 2    60   Input ~ 0
-GN1
-Text GLabel 3000 7000 0    60   Input ~ 0
-GP1
-Text GLabel 3500 7100 2    60   Input ~ 0
-GN2
-Text GLabel 3000 7100 0    60   Input ~ 0
-GP2
 Text GLabel 8900 2900 0    60   Input ~ 0
 GP3
@@
 Text GLabel 8900 2300 0    60   Input ~ 0
 GN5
-Text Notes 3300 6950 2    60   ~ 0
-0
-Text Notes 3300 7050 2    60   ~ 0
-1
-Text Notes 3300 7150 2    60   ~ 0
-2
-Text Notes 3300 7250 2    60   ~ 0
-3
-Text Notes 3300 7350 2    60   ~ 0
-4
-Text Notes 3300 7450 2    60   ~ 0
-5
-Text Notes 3300 7550 2    60   ~ 0
-6
-Text Notes 2700 6950 2    60   ~ 0
-PCLKT0_0
-Text Notes 4250 6950 2    60   ~ 0
-PCLKC0_0
-Text Notes 2700 7050 2    60   ~ 0
-PCLKT0_1
-Text Notes 4250 7050 2    60   ~ 0
-PCLKC0_1
-Text Notes 2700 7150 2    60   ~ 0
-GR_PCLK0_1
-Text Notes 4350 7150 2    60   ~ 0
-GR_PCLK0_0
-Text Notes 2450 6850 2    60   ~ 0
-DAC WIFI_GPIO25
-Text GLabel 3000 7500 0    60   Input ~ 0
-GP6
-Text GLabel 3500 7500 2    60   Input ~ 0
-GN6
 $Comp
 L Device:R_Small R?
