File: gpdi.sch (KiCad schematic (older format))
At the start: 25 parts, among them U1 LFE5U-85F-6BG381C

Commit message: Fix #9 Cam0 and Cam1 are now true diff #6
Connections:
- net CAM0_C_N: no longer names the net of U1.C12 (PCLKC1_0)
- net CAM0_C_P: no longer names the net of U1.B12 (PCLKT1_0)
- net CAM0_D0_N: no longer names the net of U1.A13 (PT76B)
- net CAM0_D0_P: no longer names the net of U1.A12 (PT76A)
- net CAM0_D1_N: no longer names the net of U1.C13 (PT78B)
- net CAM0_D1_P: no longer names the net of U1.B13 (PT78A)
- net USB_FPGA_D+: no longer names the net of U1.D15 (PT107A)
- net USB_FPGA_D-: no longer names the net of U1.E15 (PT107B)
Other:
- note added: "SINGLE ENDED - NOT DIFFERENTIAL"
Changed lines of the file:
@@
 	1    0    0    -1
 $EndComp
-Text GLabel 2850 2800 0    60   Input ~ 0
-USB_FPGA_D+
-Text GLabel 4350 2800 2    60   Input ~ 0
-USB_FPGA_D-
 NoConn ~ 2850 3700
 NoConn ~ 2850 3800
@@
 	0    -1   -1   0
 $EndComp
-Text GLabel 4350 3400 2    60   Input ~ 0
-CAM0_D0_N
-Text GLabel 2850 3400 0    60   Input ~ 0
-CAM0_D0_P
-Text GLabel 4350 3300 2    60   Input ~ 0
-CAM0_D1_N
-Text GLabel 2850 3300 0    60   Input ~ 0
-CAM0_D1_P
-Text GLabel 4350 3600 2    60   Input ~ 0
-CAM0_C_N
-Text GLabel 2850 3600 0    60   Input ~ 0
-CAM0_C_P
+Text Notes 2850 4100 0    60   ~ 0
+SINGLE ENDED - NOT DIFFERENTIAL
 Text GLabel 2850 3500 0    60   Input ~ 0
 DSI0_C_P

Commit message: initial v003
Parts:
- added R22, R23, R24, R25, R26, R34, R35, R36, R37, R38: 300, Resistor_SMD:R_0402_1005Metric, symbol Device:R_Small
- added R39, R40, R45, R46, R47, R48: 70, Resistor_SMD:R_0402_1005Metric, symbol Device:R_Small
Connections:
- net DSI0_C_N: now also R38.2, R39.1; no longer U1.E12 (GR_PCLK1_1)
- net DSI0_C_P: now also R26.1, R40.1; no longer U1.D12 (GR_PCLK1_0)
- net DSI0_D0_N: now also R37.2, R46.1; no longer U1.E13 (PT80B)
- net DSI0_D0_P: now also R25.1, R45.1; no longer U1.D13 (PT80A)
- net DSI0_D1_N: now also R36.2, R48.1; no longer U1.C14 (PT83B)
- net DSI0_D1_P: now also R24.1, R47.1; no longer U1.A14 (PT83A)
- net DSI1_D2_N: now also R34.2; no longer U1.B20 (PT121B)
- net DSI1_D2_P: now also R22.1; no longer U1.A19 (PT121A)
- net DSI1_D3_N: now also R35.2; no longer U1.B19 (PT119B)
- net DSI1_D3_P: now also R23.1; no longer U1.A18 (PT119A)
- net GND: now also R39.2, R40.2, R45.2, R46.2, R47.2, R48.2
- new net: R24.2, U1.A14 (PT83A)
- new net: R23.2, U1.A18 (PT119A)
- new net: R22.2, U1.A19 (PT121A)
- new net: R35.1, U1.B19 (PT119B)
- new net: R34.1, U1.B20 (PT121B)
- new net: R36.1, U1.C14 (PT83B)
- new net: R26.2, U1.D12 (GR_PCLK1_0)
- new net: R25.2, U1.D13 (PT80A)
- new net: R38.1, U1.E12 (GR_PCLK1_1)
- new net: R37.1, U1.E13 (PT80B)

Commit message: Fix #12 If RC1 and RC2 are placed voltahe will be 1.2V
Parts:
- R10, R13, R14, R15: value 4K7 -> 4k7
- R16, R17, R8, R9: value 100K -> 100k
Changed lines of the file:
@@
 AR Path="/58D686D9/617A8D23" Ref="R8"  Part="1"
 F 0 "R8" V 7250 3550 50  0000 C CNN
-F 1 "100K" V 7200 3700 39  0000 C CNN
+F 1 "100k" V 7200 3700 39  0000 C CNN
 F 2 "Resistor_SMD:R_0402_1005Metric" H 7200 3700 50  0001 C CNN
 F 3 "~" H 7200 3700 50  0001 C CNN
@@
 AR Path="/58D686D9/617AC694" Ref="R9"  Part="1"
 F 0 "R9" V 7350 3700 50  0000 C CNN
-F 1 "100K" V 7300 3850 39  0000 C CNN
+F 1 "100k" V 7300 3850 39  0000 C CNN
 F 2 "Resistor_SMD:R_0402_1005Metric" H 7300 3850 50  0001 C CNN
 F 3 "~" H 7300 3850 50  0001 C CNN
@@
 AR Path="/58D686D9/6184415B" Ref="R16"  Part="1"
 F 0 "R16" V 9250 3550 50  0000 C CNN
-F 1 "100K" V 9200 3700 39  0000 C CNN
+F 1 "100k" V 9200 3700 39  0000 C CNN
 F 2 "Resistor_SMD:R_0402_1005Metric" H 9200 3700 50  0001 C CNN
 F 3 "~" H 9200 3700 50  0001 C CNN
@@
 AR Path="/58D686D9/61844EFE" Ref="R17"  Part="1"
 F 0 "R17" V 9300 3700 50  0000 C CNN
-F 1 "100K" V 9250 3850 39  0000 C CNN
+F 1 "100k" V 9250 3850 39  0000 C CNN
 F 2 "Resistor_SMD:R_0402_1005Metric" H 9250 3850 50  0001 C CNN
 F 3 "~" H 9250 3850 50  0001 C CNN
@@
 AR Path="/58D686D9/618C8B2E" Ref="R10"  Part="1"
 F 0 "R10" V 8400 4250 50  0000 C CNN
-F 1 "4K7" V 8350 4400 39  0000 C CNN
+F 1 "4k7" V 8350 4400 39  0000 C CNN
 F 2 "Resistor_SMD:R_0402_1005Metric" H 8350 4400 50  0001 C CNN
 F 3 "~" H 8350 4400 50  0001 C CNN
@@
 AR Path="/58D686D9/618D3240" Ref="R13"  Part="1"
 F 0 "R13" V 8400 4350 50  0000 C CNN
-F 1 "4K7" V 8350 4500 39  0000 C CNN
+F 1 "4k7" V 8350 4500 39  0000 C CNN
 F 2 "Resistor_SMD:R_0402_1005Metric" H 8350 4500 50  0001 C CNN
 F 3 "~" H 8350 4500 50  0001 C CNN
@@
 AR Path="/58D686D9/618DA045" Ref="R14"  Part="1"
 F 0 "R14" V 8400 4450 50  0000 C CNN
-F 1 "4K7" V 8350 4600 39  0000 C CNN
+F 1 "4k7" V 8350 4600 39  0000 C CNN
 F 2 "Resistor_SMD:R_0402_1005Metric" H 8350 4600 50  0001 C CNN
 F 3 "~" H 8350 4600 50  0001 C CNN
@@
 AR Path="/58D686D9/618E1A8E" Ref="R15"  Part="1"
 F 0 "R15" V 8400 4550 50  0000 C CNN
-F 1 "4K7" V 8350 4700 39  0000 C CNN
+F 1 "4k7" V 8350 4700 39  0000 C CNN
 F 2 "Resistor_SMD:R_0402_1005Metric" H 8350 4700 50  0001 C CNN
 F 3 "~" H 8350 4700 50  0001 C CNN

Commit message: DDR3 lines are now around 10% - all GPIOs should be connected
Parts:
- renumbered R40 to R49, R45 to R50, R46 to R51, R47 to R52
Connections:
- net SCL0: now reaches U1.A12 (PT76A)
- net SDA0: now reaches U1.A13 (PT76B)
- net Camera_GPIO: now reaches U1.A17 (PT116A)
- net SD_D0: now reaches U1.B15 (PT105A)
- net SD_D1: now reaches U1.B18 (PT116B)
- net SD_D2: now reaches U1.E14 (PT85B)
Changed lines of the file:
@@
 P 3375 4825
 AR Path="/58D6BF46/634A9BEB" Ref="R?"  Part="1"
-AR Path="/58D686D9/634A9BEB" Ref="R40"  Part="1"
-F 0 "R40" V 3450 4825 50  0000 C CNN
+AR Path="/58D686D9/634A9BEB" Ref="R49"  Part="1"
+F 0 "R49" V 3450 4825 50  0000 C CNN
 F 1 "70" V 3375 4825 39  0000 C CNN
 F 2 "Resistor_SMD:R_0402_1005Metric" H 3375 4825 50  0001 C CNN
@@
 P 3950 4825
 AR Path="/58D6BF46/634E7C26" Ref="R?"  Part="1"
-AR Path="/58D686D9/634E7C26" Ref="R47"  Part="1"
-F 0 "R47" V 3875 4825 50  0000 C CNN
+AR Path="/58D686D9/634E7C26" Ref="R52"  Part="1"
+F 0 "R52" V 3875 4825 50  0000 C CNN
 F 1 "70" V 3950 4825 39  0000 C CNN
 F 2 "Resistor_SMD:R_0402_1005Metric" H 3950 4825 50  0001 C CNN
@@
 P 3725 4825
 AR Path="/58D6BF46/634E1082" Ref="R?"  Part="1"
-AR Path="/58D686D9/634E1082" Ref="R46"  Part="1"
-F 0 "R46" V 3800 4825 50  0000 C CNN
+AR Path="/58D686D9/634E1082" Ref="R51"  Part="1"
+F 0 "R51" V 3800 4825 50  0000 C CNN
 F 1 "70" V 3725 4825 39  0000 C CNN
 F 2 "Resistor_SMD:R_0402_1005Metric" H 3725 4825 50  0001 C CNN
@@
 P 3600 4825
 AR Path="/58D6BF46/634E0FA0" Ref="R?"  Part="1"
-AR Path="/58D686D9/634E0FA0" Ref="R45"  Part="1"
-F 0 "R45" V 3525 4825 50  0000 C CNN
+AR Path="/58D686D9/634E0FA0" Ref="R50"  Part="1"
+F 0 "R50" V 3525 4825 50  0000 C CNN
 F 1 "70" V 3600 4825 39  0000 C CNN
 F 2 "Resistor_SMD:R_0402_1005Metric" H 3600 4825 50  0001 C CNN
@@
 Wire Wire Line
 	3600 4650 3600 4725
+Text GLabel 4350 2400 2    60   Input ~ 0
+SD_D1
+Text GLabel 5400 2750 2    60   Input ~ 0
+SD_PWR_ON
+Text GLabel 2400 5450 0    60   Input ~ 0
+nEXTRST
+Text GLabel 2850 3400 0    60   Input ~ 0
+SCL0
+Text GLabel 4350 3400 2    60   Input ~ 0
+SDA0
+Text GLabel 4350 3000 2    60   Input ~ 0
+SD_D2
+Text GLabel 2850 2400 0    60   Input ~ 0
+Camera_GPIO
+Text GLabel 2850 2900 0    60   Input ~ 0
+SD_D0
 $EndSCHEMATC

Commit message: References cleanup
Parts:
- added R70: 130, Resistor_SMD:R_0402_1005Metric, symbol Device:R_Small
- added SW1: SW_DIP_x02, Button_Switch_SMD:SW_DIP_SPSTx02_Slide_Copal_CVS-02xB_W5.9mm_P1mm, symbol Switch:SW_DIP_x02
- renumbered C38 to C30, C37 to C31, C36 to C32, C21 to C33, C18 to C34, C15 to C35, C14 to C36, C13 to C37, C54 to C40, C45 to C41, C44 to C42, C42 to C44, C41 to C45, C40 to C46, C39 to C47
Connections:
- net +3V3: now also R70.1
- net SW2: now reaches U1.B13 (PT78A)
- net SW2: now also SW1.3
- net SW1: now reaches U1.C13 (PT78B)
- net SW1: now also SW1.4
- new net: R70.2, SW1.1, SW1.2
Changed lines of the file:
@@
 $Descr A4 11693 8268
 encoding utf-8
-Sheet 5 13
+Sheet 5 11
 Title "ULX3S"
 Date ""
@@
 HDMI0_CEC
 $Comp
-L Device:C_Small C13
+L Device:C_Small C37
 U 1 1 612E1A2D
 P 7200 2100
-F 0 "C13" V 7250 2000 50  0000 C CNN
+F 0 "C37" V 7250 2000 50  0000 C CNN
 F 1 "100n" V 7150 1950 50  0000 C CNN
 F 2 "Capacitor_SMD:C_0402_1005Metric" H 7200 2100 50  0001 C CNN
@@
 $EndComp
 $Comp
-L Device:C_Small C14
+L Device:C_Small C36
 U 1 1 612E4477
 P 7200 2300
-F 0 "C14" V 7250 2200 50  0000 C CNN
+F 0 "C36" V 7250 2200 50  0000 C CNN
 F 1 "100n" V 7150 2150 50  0000 C CNN
 F 2 "Capacitor_SMD:C_0402_1005Metric" H 7200 2300 50  0001 C CNN
@@
 	7500 2300 7300 2300
 $Comp
-L Device:C_Small C15
+L Device:C_Small C35
 U 1 1 613050D7
 P 7200 2500
-F 0 "C15" V 7250 2400 50  0000 C CNN
+F 0 "C35" V 7250 2400 50  0000 C CNN
 F 1 "100n" V 7150 2350 50  0000 C CNN
 F 2 "Capacitor_SMD:C_0402_1005Metric" H 7200 2500 50  0001 C CNN
@@
 $EndComp
 $Comp
-L Device:C_Small C18
+L Device:C_Small C34
 U 1 1 61305963
 P 7200 2700
-F 0 "C18" V 7250 2600 50  0000 C CNN
+F 0 "C34" V 7250 2600 50  0000 C CNN
 F 1 "100n" V 7150 2550 50  0000 C CNN
 F 2 "Capacitor_SMD:C_0402_1005Metric" H 7200 2700 50  0001 C CNN
@@
 	7100 2700 6950 2700
 $Comp
-L Device:C_Small C21
+L Device:C_Small C33
 U 1 1 6133C604
 P 7200 2900
-F 0 "C21" V 7250 2800 50  0000 C CNN
+F 0 "C33" V 7250 2800 50  0000 C CNN
 F 1 "100n" V 7150 2750 50  0000 C CNN
 F 2 "Capacitor_SMD:C_0402_1005Metric" H 7200 2900 50  0001 C CNN
@@
 $EndComp
 $Comp
-L Device:C_Small C36
+L Device:C_Small C32
 U 1 1 6133D002
 P 7200 3100
-F 0 "C36" V 7250 3000 50  0000 C CNN
+F 0 "C32" V 7250 3000 50  0000 C CNN
 F 1 "100n" V 7150 2950 50  0000 C CNN
 F 2 "Capacitor_SMD:C_0402_1005Metric" H 7200 3100 50  0001 C CNN
@@
 	7100 3100 6950 3100
 $Comp
-L Device:C_Small C37
+L Device:C_Small C31
 U 1 1 6136976F
 P 7200 3300
-F 0 "C37" V 7250 3200 50  0000 C CNN
+F 0 "C31" V 7250 3200 50  0000 C CNN
 F 1 "100n" V 7150 3150 50  0000 C CNN
 F 2 "Capacitor_SMD:C_0402_1005Metric" H 7200 3300 50  0001 C CNN
@@
 $EndComp
 $Comp
-L Device:C_Small C38
+L Device:C_Small C30
 U 1 1 6136A15F
 P 7200 3500
-F 0 "C38" V 7250 3400 50  0000 C CNN
+F 0 "C30" V 7250 3400 50  0000 C CNN
 F 1 "100n" V 7150 3350 50  0000 C CNN
 F 2 "Capacitor_SMD:C_0402_1005Metric" H 7200 3500 50  0001 C CNN
@@
 	6950 3500 7100 3500
 $Comp
-L Device:C_Small C39
+L Device:C_Small C47
 U 1 1 61412C70
 P 9150 2100
-F 0 "C39" V 9200 2000 50  0000 C CNN
+F 0 "C47" V 9200 2000 50  0000 C CNN
 F 1 "100n" V 9100 1950 50  0000 C CNN
 F 2 "Capacitor_SMD:C_0402_1005Metric" H 9150 2100 50  0001 C CNN
@@
 $EndComp
 $Comp
-L Device:C_Small C40
+L Device:C_Small C46
 U 1 1 61413054
 P 9150 2300
-F 0 "C40" V 9200 2200 50  0000 C CNN
+F 0 "C46" V 9200 2200 50  0000 C CNN
 F 1 "100n" V 9100 2150 50  0000 C CNN
 F 2 "Capacitor_SMD:C_0402_1005Metric" H 9150 2300 50  0001 C CNN
@@
 	9450 2300 9250 2300
 $Comp
-L Device:C_Small C41
+L Device:C_Small C45
 U 1 1 61413062
 P 9150 2500
-F 0 "C41" V 9200 2400 50  0000 C CNN
+F 0 "C45" V 9200 2400 50  0000 C CNN
 F 1 "100n" V 9100 2350 50  0000 C CNN
 F 2 "Capacitor_SMD:C_0402_1005Metric" H 9150 2500 50  0001 C CNN
@@
 $EndComp
 $Comp
-L Device:C_Small C42
+L Device:C_Small C44
 U 1 1 6141306C
 P 9150 2700
-F 0 "C42" V 9200 2600 50  0000 C CNN
+F 0 "C44" V 9200 2600 50  0000 C CNN
 F 1 "100n" V 9100 2550 50  0000 C CNN
 F 2 "Capacitor_SMD:C_0402_1005Metric" H 9150 2700 50  0001 C CNN
@@
 $EndComp
 $Comp
-L Device:C_Small C44
+L Device:C_Small C42
 U 1 1 61413084
 P 9150 3100
-F 0 "C44" V 9200 3000 50  0000 C CNN
+F 0 "C42" V 9200 3000 50  0000 C CNN
 F 1 "100n" V 9100 2950 50  0000 C CNN
 F 2 "Capacitor_SMD:C_0402_1005Metric" H 9150 3100 50  0001 C CNN
@@
 	9050 3100 8900 3100
 $Comp
-L Device:C_Small C45
+L Device:C_Small C41
 U 1 1 61413092
 P 9150 3300
-F 0 "C45" V 9200 3200 50  0000 C CNN
+F 0 "C41" V 9200 3200 50  0000 C CNN
 F 1 "100n" V 9100 3150 50  0000 C CNN
 F 2 "Capacitor_SMD:C_0402_1005Metric" H 9150 3300 50  0001 C CNN
@@
 $EndComp
 $Comp
-L Device:C_Small C54
+L Device:C_Small C40
 U 1 1 6141309C
 P 9150 3500
-F 0 "C54" V 9200 3400 50  0000 C CNN
+F 0 "C40" V 9200 3400 50  0000 C CNN
 F 1 "100n" V 9100 3350 50  0000 C CNN
 F 2 "Capacitor_SMD:C_0402_1005Metric" H 9150 3500 50  0001 C CNN
@@
 Text GLabel 2850 2900 0    60   Input ~ 0
 SD_D0
+Text GLabel 4350 3300 2    60   Input ~ 0
+SW1
+Text GLabel 2850 3300 0    60   Input ~ 0
+SW2
+$Comp
+L Switch:SW_DIP_x02 SW1
+U 1 1 6519BDE2
+P 5700 4775
+F 0 "SW1" H 5700 5142 50  0000 C CNN
+F 1 "SW_DIP_x02" H 5700 5051 50  0000 C CNN
+F 2 "Button_Switch_SMD:SW_DIP_SPSTx02_Slide_Copal_CVS-02xB_W5.9mm_P1mm" H 5700 4775 50  0001 C CNN
+F 3 "~" H 5700 4775 50  0001 C CNN
+	1    5700 4775
+	1    0    0    -1
+$EndComp
+$Comp
+L power:+3V3 #PWR?
+U 1 1 651A4B65
+P 4950 4775
+AR Path="/58D51CAD/651A4B65" Ref="#PWR?"  Part="1"
+AR Path="/58D686D9/651A4B65" Ref="#PWR0145"  Part="1"
+F 0 "#PWR0145" H 4950 4625 50  0001 C CNN
+F 1 "+3V3" H 4950 4915 50  0000 C CNN
+F 2 "" H 4950 4775 50  0000 C CNN
+F 3 "" H 4950 4775 50  0000 C CNN
+	1    4950 4775
+	0    -1   -1   0
+$EndComp
+$Comp
+L Device:R_Small R?
+U 1 1 651A6533
+P 5150 4775
+AR Path="/58D6BF46/651A6533" Ref="R?"  Part="1"
+AR Path="/58D686D9/651A6533" Ref="R70"  Part="1"
+F 0 "R70" V 5225 4775 50  0000 C CNN
+F 1 "130" V 5150 4775 39  0000 C CNN
+F 2 "Resistor_SMD:R_0402_1005Metric" H 5150 4775 50  0001 C CNN
+F 3 "~" H 5150 4775 50  0001 C CNN
+	1    5150 4775
+	0    -1   -1   0
+$EndComp
+Wire Wire Line
+	4950 4775 5050 4775
+Wire Wire Line
+	5250 4775 5325 4775
+Wire Wire Line
+	5400 4675 5325 4675
+Wire Wire Line
+	5325 4675 5325 4775
+Connection ~ 5325 4775
+Wire Wire Line
+	5325 4775 5400 4775
+Text GLabel 6075 4675 2    60   Input ~ 0
+SW1
+Text GLabel 6075 4775 2    60   Input ~ 0
+SW2
+Wire Wire Line
+	6000 4675 6075 4675
+Wire Wire Line
+	6075 4775 6000 4775
 $EndSCHEMATC

Commit message: Connecting SD-POWER pin
Connections:
- net SD_PWR_ON: now also U1.E15 (PT107B)
Changed lines of the file:
@@
 Text GLabel 4350 2400 2    60   Input ~ 0
 SD_D1
-Text GLabel 5400 2750 2    60   Input ~ 0
+Text GLabel 4350 2800 2    60   Input ~ 0
 SD_PWR_ON
 Text GLabel 2400 5450 0    60   Input ~ 0
