File: gpdi.sch (KiCad schematic (older format))
At the start: 43 parts, among them SW1 SW_DIP_x02, U1 LFE5U-85F-6BG381C

Commit message: Adding few test pads #24
Parts:
- added TP_C16: C16, ecp5-dc-scm:Testpoint_smd_1mm, symbol Connector:TestPoint_Small
- added TP_D16: D16, ecp5-dc-scm:Testpoint_smd_1mm, symbol Connector:TestPoint_Small
Connections:
- net at U1.C16 (PT112A): now also TP_C16.1
- net at U1.D16 (PT112B): now also TP_D16.1
Changed lines of the file:
@@
 Wire Wire Line
 	6075 4775 6000 4775
+$Comp
+L Connector:TestPoint_Small TP_D?
+U 1 1 6226F065
+P 2650 2600
+AR Path="/56AC389C/6226F065" Ref="TP_D?"  Part="1"
+AR Path="/58D686D9/6226F065" Ref="TP_C16"  Part="1"
+F 0 "TP_C16" H 2875 2600 50  0000 L CNN
+F 1 "C16" H 2698 2555 50  0000 L CNN
+F 2 "ecp5-dc-scm:Testpoint_smd_1mm" H 2850 2600 50  0001 C CNN
+F 3 "~" H 2850 2600 50  0001 C CNN
+	1    2650 2600
+	-1   0    0    1
+$EndComp
+Wire Wire Line
+	2650 2600 2850 2600
+$Comp
+L Connector:TestPoint_Small TP_C?
+U 1 1 62286908
+P 4550 2600
+AR Path="/56AC389C/62286908" Ref="TP_C?"  Part="1"
+AR Path="/58D686D9/62286908" Ref="TP_D16"  Part="1"
+F 0 "TP_D16" H 4775 2600 50  0000 L CNN
+F 1 "D16" H 4598 2555 50  0000 L CNN
+F 2 "ecp5-dc-scm:Testpoint_smd_1mm" H 4750 2600 50  0001 C CNN
+F 3 "~" H 4750 2600 50  0001 C CNN
+	1    4550 2600
+	1    0    0    -1
+$EndComp
+Wire Wire Line
+	4550 2600 4350 2600
 $EndSCHEMATC

Commit message: Lowering number of unique parts fix #37
Parts:
- R16, R17, R8, R9: value 100k -> 15k
- R70: value 130 -> 300
Changed lines of the file:
@@
 AR Path="/58D686D9/617A8D23" Ref="R8"  Part="1"
 F 0 "R8" V 7250 3550 50  0000 C CNN
-F 1 "100k" V 7200 3700 39  0000 C CNN
+F 1 "15k" V 7200 3700 39  0000 C CNN
 F 2 "Resistor_SMD:R_0402_1005Metric" H 7200 3700 50  0001 C CNN
 F 3 "~" H 7200 3700 50  0001 C CNN
@@
 AR Path="/58D686D9/617AC694" Ref="R9"  Part="1"
 F 0 "R9" V 7350 3700 50  0000 C CNN
-F 1 "100k" V 7300 3850 39  0000 C CNN
+F 1 "15k" V 7300 3850 39  0000 C CNN
 F 2 "Resistor_SMD:R_0402_1005Metric" H 7300 3850 50  0001 C CNN
 F 3 "~" H 7300 3850 50  0001 C CNN
@@
 AR Path="/58D686D9/6184415B" Ref="R16"  Part="1"
 F 0 "R16" V 9250 3550 50  0000 C CNN
-F 1 "100k" V 9200 3700 39  0000 C CNN
+F 1 "15k" V 9200 3700 39  0000 C CNN
 F 2 "Resistor_SMD:R_0402_1005Metric" H 9200 3700 50  0001 C CNN
 F 3 "~" H 9200 3700 50  0001 C CNN
@@
 AR Path="/58D686D9/61844EFE" Ref="R17"  Part="1"
 F 0 "R17" V 9300 3700 50  0000 C CNN
-F 1 "100k" V 9250 3850 39  0000 C CNN
+F 1 "15k" V 9250 3850 39  0000 C CNN
 F 2 "Resistor_SMD:R_0402_1005Metric" H 9250 3850 50  0001 C CNN
 F 3 "~" H 9250 3850 50  0001 C CNN
@@
 AR Path="/58D686D9/651A6533" Ref="R70"  Part="1"
 F 0 "R70" V 5225 4775 50  0000 C CNN
-F 1 "130" V 5150 4775 39  0000 C CNN
+F 1 "300" V 5150 4775 39  0000 C CNN
 F 2 "Resistor_SMD:R_0402_1005Metric" H 5150 4775 50  0001 C CNN
 F 3 "~" H 5150 4775 50  0001 C CNN

Commit message: Finshed routing SDRAM
Connections:
- net Camera_GPIO: no longer names the net of U1.A17 (PT116A)
- net SCL0: no longer names the net of U1.A12 (PT76A)
- net SDA0: no longer names the net of U1.A13 (PT76B)
- net SD_D1: no longer names the net of U1.B18 (PT116B)
Changed lines of the file:
@@
 Wire Wire Line
 	3600 4650 3600 4725
-Text GLabel 4350 2400 2    60   Input ~ 0
-SD_D1
 Text GLabel 4350 2800 2    60   Input ~ 0
 SD_PWR_ON
 Text GLabel 2400 5450 0    60   Input ~ 0
 nEXTRST
-Text GLabel 2850 3400 0    60   Input ~ 0
-SCL0
-Text GLabel 4350 3400 2    60   Input ~ 0
-SDA0
 Text GLabel 4350 3000 2    60   Input ~ 0
 SD_D2
-Text GLabel 2850 2400 0    60   Input ~ 0
-Camera_GPIO
 Text GLabel 2850 2900 0    60   Input ~ 0
 SD_D0

Commit message: Connecting DSI1 to DSI0
Connections:
- net SW1: no longer U1.C13 (PT78B)
- net SW2: no longer U1.B13 (PT78A)
Changed lines of the file:
@@
 Text GLabel 2850 2900 0    60   Input ~ 0
 SD_D0
-Text GLabel 4350 3300 2    60   Input ~ 0
-SW1
-Text GLabel 2850 3300 0    60   Input ~ 0
-SW2
 $Comp
 L Switch:SW_DIP_x02 SW1
