File: power.sch (KiCad schematic (older format))
At the start: 84 parts, among them J5 VJ1, Q1 BC857, Q2 2N7002, U1 LFE5U-85F-6BG381C, U3 TLV62569DBV, U4 TLV62569DBV, U5 TLV62569DBV, U7 MCP7940NT, Y2 32768Hz

Commit message: More removing
Parts:
- removed BAT1: CR1225, Keystone_3000_1x12mm-CoinCell:Keystone_3000_1x12mm-CoinCell, symbol Device:Battery_Cell
- removed C13: 2.2uF, Capacitor_SMD:C_0805_2012Metric, symbol Device:C
- removed C14: 220nF, Capacitor_SMD:C_0603_1608Metric, symbol Device:C
- removed C54, C55: 22uF, Capacitor_SMD:C_0805_2012Metric, symbol Device:C
- removed C56, C57: 4.7pF, Capacitor_SMD:C_0603_1608Metric, symbol Device:C
- removed D10, D13, D14: 1N914, Diode_SMD:D_SOD-323_HandSoldering, symbol Device:D
- removed D11: RED, LED_SMD:LED_0805_2012Metric, symbol Device:LED_ALT
- removed D15: BAT54W, Diode_SMD:D_SOD-323_HandSoldering, symbol Device:D_Schottky
- removed Q1: BC857, Package_TO_SOT_SMD:SOT-23, symbol Device:Q_PNP_BEC
- removed Q2: 2N7002, Package_TO_SOT_SMD:SOT-23, symbol Device:Q_NMOS_GSD
- removed R1: 4.7k, Resistor_SMD:R_0603_1608Metric, symbol Device:R
- removed R10: 130, Resistor_SMD:R_0603_1608Metric, symbol Device:R
- removed R13: 15k, Resistor_SMD:R_0603_1608Metric, symbol Device:R
- removed R2: 18k, Resistor_SMD:R_0603_1608Metric, symbol Device:R
- removed R5: 2.2M, Resistor_SMD:R_0603_1608Metric, symbol Device:R
- removed R6, R8: 1.1k, Resistor_SMD:R_0603_1608Metric, symbol Device:R
- removed R65: 549, Resistor_SMD:R_0603_1608Metric, symbol Device:R
- removed U7: MCP7940NT, SOT96-1:SOT96-1, symbol Timer_RTC:PCF8563T
- removed Y2: 32768Hz, abs25:Crystal_SMD_ABS25, symbol Device:Crystal_GND23
Connections:
- net labels removed: OSCI_32k, OSCO_32k, RTCVDD, SHD, SHUT, VBAT, WAKE, WAKEUPn, WKUP, WKn
- wire segments 450 -> 395
- no-connect marks 2 -> 0

Commit message: Sync sch and pcb
Parts:
- removed D12: BAT54W, Diode_SMD:D_SOD-323_HandSoldering, symbol Device:D_Schottky
Connections:
- net labels removed: FTDI_nSUSPEND
- wire segments 395 -> 391
Changed lines of the file:
@@
 	7450 4700 6950 4700
 Wire Wire Line
-	3950 4950 4100 4950
-Wire Wire Line
 	4100 1050 4200 1050
 Wire Wire Line
@@
 Wire Wire Line
 	4850 4950 4850 4850
-Wire Wire Line
-	4100 4950 4100 5050
-Connection ~ 4100 4950
-Wire Wire Line
-	2850 4950 3650 4950
 Wire Wire Line
 	7750 1050 7750 1150
@@
 Wire Wire Line
 	2500 4950 2550 4950
-Text Label 2900 4950 0    60   ~ 0
-FTDI_nSUSPEND
 $Comp
 L Device:C C17
@@
 	1    0    0    -1
 $EndComp
-$Comp
-L Device:D_Schottky D12
-U 1 1 5AF673FF
-P 3800 4950
-F 0 "D12" H 3800 5050 50  0000 C CNN
-F 1 "BAT54W" H 3800 4850 50  0000 C CNN
-F 2 "Diode_SMD:D_SOD-323_HandSoldering" H 3800 4950 50  0001 C CNN
-F 3 "" H 3800 4950 50  0001 C CNN
-	1    3800 4950
-	-1   0    0    1
-$EndComp
 Text Notes 850  5050 0    60   ~ 0
 FTDI_nSLEEP is 2.5V\nD12 must be schottky
@@
 Wire Wire Line
 	2900 3700 2900 3800
-Wire Wire Line
-	4100 4950 4850 4950
 $EndSCHEMATC

Commit message: Before removing USB port
Parts:
- removed B0: PTS645, Button_Switch_SMD:SW_SPST_PTS645, symbol Switch:SW_Push
Changed lines of the file:
@@
 Text GLabel 3300 4150 2    60   Input ~ 0
 BTN_PWRn
-$Comp
-L Switch:SW_Push B0
-U 1 1 58E83FE0
-P 2200 4600
-F 0 "B0" H 2100 4700 50  0000 C CNN
-F 1 "PTS645" H 2350 4700 50  0000 C CNN
-F 2 "Button_Switch_SMD:SW_SPST_PTS645" H 2200 3400 50  0001 C CNN
-F 3 "http://www.ckswitches.com/media/1471/pts645.pdf" H 2200 3400 50  0001 C CNN
-F 4 "www.ckswitches.com" H 2200 4600 60  0001 C CNN "MNF1_URL"
-F 5 "PTS645SL50SMTR92 LFS" H 2200 4600 60  0001 C CNN "MPN"
-F 6 "611-PTS645SL50SMTR92" H 2200 4600 50  0001 C CNN "Mouser"
-F 7 "CKN9088CT-ND" H 2200 4600 50  0001 C CNN "Digikey"
-F 8 "15N4500" H 2200 4600 50  0001 C CNN "Newark"
-F 9 "79AH5908" H 2200 4600 50  0001 C CNN "Newar_k2"
-F 10 "C285463" H 2200 4600 50  0001 C CNN "LCSC"
-F 11 "0.09966$" H 2200 4600 50  0001 C CNN "price700_LCSC"
-F 12 "FSW001" H 2200 4600 50  0001 C CNN "Koncar"
-F 13 "T" H 2200 4600 50  0001 C CNN "Side"
-	1    2200 4600
-	-1   0    0    -1
-$EndComp
 Wire Wire Line
 	2350 2600 2450 2600

Commit message: More removal, spliting modules
Parts:
- removed D16, D27: 1N914, Diode_SMD:D_SOD-323_HandSoldering, symbol Device:D
- removed R4: 4.7k, Resistor_SMD:R_0603_1608Metric, symbol Device:R
- removed R66: 1.1k, Resistor_SMD:R_0603_1608Metric, symbol Device:R
- C1, C11, C12, C17, C19, C20, C22, C23, C24, C3, C4, C47, C5, C7, C8, C9: footprint Capacitor_SMD:C_0805_2012Metric -> Capacitor_SMD:C_0603_1608Metric
- C10, C2, C25, C26, C27, C28, C29, C30, C31, C32, C6, C60: footprint Capacitor_SMD:C_0603_1608Metric -> Capacitor_SMD:C_0402_1005Metric
- R3, RA1, RA2, RA3, RB1, RB2, RB3: footprint Resistor_SMD:R_0603_1608Metric -> Capacitor_SMD:C_0402_1005Metric
Connections:
- net labels removed: HOLD, US2_ID
- wire segments 391 -> 384

Commit message: Before power placement
Parts:
- removed J5: VJ1, Connector_PinHeader_2.54mm:PinHeader_1x03_P2.54mm_Vertical, symbol Connector_Generic:Conn_01x03
- D17: footprint Diode_SMD:D_SOD-323_HandSoldering -> Diode_SMD:D_SOD-323
Connections:
- wire segments 384 -> 379
Changed lines of the file:
@@
 F 0 "D17" H 3150 4050 50  0000 C CNN
 F 1 "1N914" H 3200 4250 50  0000 C CNN
-F 2 "Diode_SMD:D_SOD-323_HandSoldering" H 3150 4150 50  0001 C CNN
+F 2 "Diode_SMD:D_SOD-323" H 3150 4150 50  0001 C CNN
 F 3 "" H 3150 4150 50  0000 C CNN
 	1    3150 4150
@@
 Text Notes 4400 5300 0    60   ~ 0
 D11 (2V), R2, R4 hold PWREN on 1V\nin the middle of 0.4-1.5V hysteresis
-Wire Wire Line
-	1350 1850 1350 1800
-$Comp
-L power:+2V5 #PWR023
-U 1 1 5AA2ABFC
-P 1350 1850
-F 0 "#PWR023" H 1350 1700 50  0001 C CNN
-F 1 "+2V5" H 1400 2000 50  0000 C CNN
-F 2 "" H 1350 1850 50  0001 C CNN
-F 3 "" H 1350 1850 50  0001 C CNN
-	1    1350 1850
-	1    0    0    1
-$EndComp
-Wire Wire Line
-	1350 1800 1400 1800
-Wire Wire Line
-	1100 1700 1400 1700
-$Comp
-L power:+3V3 #PWR024
-U 1 1 5AA2AD24
-P 1350 1550
-F 0 "#PWR024" H 1350 1400 50  0001 C CNN
-F 1 "+3V3" H 1300 1700 50  0000 C CNN
-F 2 "" H 1350 1550 50  0001 C CNN
-F 3 "" H 1350 1550 50  0001 C CNN
-	1    1350 1550
-	-1   0    0    -1
-$EndComp
-Wire Wire Line
-	1350 1550 1350 1600
-Wire Wire Line
-	1350 1600 1400 1600
-$Comp
-L Connector_Generic:Conn_01x03 J5
-U 1 1 5AA2A24D
-P 1600 1700
-AR Path="/5AA2A24D" Ref="J5"  Part="1"
-AR Path="/58D51CAD/5AA2A24D" Ref="J5"  Part="1"
-F 0 "J5" H 1600 1900 50  0000 C CNN
-F 1 "VJ1" H 1600 1500 50  0000 C CNN
-F 2 "Connector_PinHeader_2.54mm:PinHeader_1x03_P2.54mm_Vertical" H 1600 1700 50  0001 C CNN
-F 3 "" H 1600 1700 50  0001 C CNN
-F 4 "Leave empty" H 1600 1700 60  0001 C CNN "Note"
-F 5 "T" H 1600 1700 50  0001 C CNN "Side"
-	1    1600 1700
-	1    0    0    1
-$EndComp
 $EndSCHEMATC

Commit message: Cleaning DRC errors
Connections:
- net PWREN is gone; now on net +5V: U3.1 (EN), U4.1 (EN), U5.1 (EN)
Changed lines of the file:
@@
 Text Notes 4400 5300 0    60   ~ 0
 D11 (2V), R2, R4 hold PWREN on 1V\nin the middle of 0.4-1.5V hysteresis
+$Comp
+L power:+5V #PWR0106
+U 1 1 61F07160
+P 6900 3500
+F 0 "#PWR0106" H 6900 3350 50  0001 C CNN
+F 1 "+5V" H 6900 3640 50  0000 C CNN
+F 2 "" H 6900 3500 50  0000 C CNN
+F 3 "" H 6900 3500 50  0000 C CNN
+	1    6900 3500
+	0    -1   -1   0
+$EndComp
+$Comp
+L power:+5V #PWR0107
+U 1 1 61F0B598
+P 6950 4700
+F 0 "#PWR0107" H 6950 4550 50  0001 C CNN
+F 1 "+5V" H 6950 4840 50  0000 C CNN
+F 2 "" H 6950 4700 50  0000 C CNN
+F 3 "" H 6950 4700 50  0000 C CNN
+	1    6950 4700
+	0    -1   -1   0
+$EndComp
+$Comp
+L power:+5V #PWR0108
+U 1 1 61F0BEE7
+P 6950 5900
+F 0 "#PWR0108" H 6950 5750 50  0001 C CNN
+F 1 "+5V" H 6950 6040 50  0000 C CNN
+F 2 "" H 6950 5900 50  0000 C CNN
+F 3 "" H 6950 5900 50  0000 C CNN
+	1    6950 5900
+	0    -1   -1   0
+$EndComp
 $EndSCHEMATC

Commit message: Cleanup schematics
Other:
- note removed: "D14 discharges\nC14 at shutdown"
- note removed: "FTDI_nSLEEP is 2.5V\nD12 must be schottky"
- note removed: "SHUTDOWN connected to\nBANK2 on "ram" sheet"
Changed lines of the file:
@@
 	1    0    0    -1
 $EndComp
-Text GLabel 1250 3950 2    60   Input ~ 0
-FPDI_SCL
-Text GLabel 1250 4100 2    60   Input ~ 0
-FPDI_SDA
 Text Notes 6250 3350 0    60   ~ 0
 PWREN\nabove +1.5V turns ON\nbelow +0.4V turns OFF
@@
 Text Notes 3450 4750 0    60   ~ 0
 D13 discharges\nC13 at shutdown
-Text Notes 2450 5400 0    60   ~ 0
-D14 discharges\nC14 at shutdown
-Text GLabel 2700 5600 0    60   Input ~ 0
-SHUTDOWN
 $Comp
 L Device:R R3
@@
 Text Notes 2100 3200 0    60   ~ 0
 RC network for proper switchover\nto battery at fast fall of VDD.\nSee page 54 NXP PCF8523T datasheet.\nRTC can also be powered from 2.5V\nbut it is easier to route 3.3V
-Text GLabel 1750 4300 0    60   Input ~ 0
-FTDI_nSLEEP
 $Comp
 L Device:C C17
@@
 Text Notes 8000 7050 0    60   ~ 0
 Switching regulators 2A SOT23-5\nTexas instruments TLV62569DBV (2A) (best)\nDioo microcircuits DIO6015B (1.5A) (osc. acceptable)\nMicrosemi LX7172 (1.2A) (osc. unacceptable)\nDiodes AP3429/A (2A) - (will damage board)\n
-Text Notes 950  5700 0    60   ~ 0
-SHUTDOWN connected to\nBANK2 on "ram" sheet
 Text Notes 2750 6350 0    60   ~ 0
 Works without R5
@@
 	1    0    0    -1
 $EndComp
-Text Notes 850  5050 0    60   ~ 0
-FTDI_nSLEEP is 2.5V\nD12 must be schottky
 Wire Wire Line
 	1100 1600 1100 1700
