File: power.sch (KiCad schematic (older format))
At the start: 53 parts, among them U1 LFE5U-85F-6BG381C, U3 TLV62569DBV, U4 TLV62569DBV, U5 TLV62569DBV

Commit message: Adding 1.1/1.2V to bank 7 voltage selection
Parts:
- added 1.1V_1: 1.1V, TestPoint:TestPoint_Pad_1.0x1.0mm, symbol Connector:TestPoint_Small
Connections:
- net +1V1: now also 1.1V_1.1
Changed lines of the file:
@@
 	0    -1   -1   0
 $EndComp
+$Comp
+L Connector:TestPoint_Small 1.1V_1
+U 1 1 638D858E
+P 1250 3750
+F 0 "1.1V_1" H 1298 3796 50  0000 L CNN
+F 1 "1.1V" H 1298 3705 50  0000 L CNN
+F 2 "TestPoint:TestPoint_Pad_1.0x1.0mm" H 1450 3750 50  0001 C CNN
+F 3 "~" H 1450 3750 50  0001 C CNN
+	1    1250 3750
+	1    0    0    -1
+$EndComp
+$Comp
+L power:+1V1 #PWR012
+U 1 1 638DDA16
+P 1250 3925
+F 0 "#PWR012" H 1250 3775 50  0001 C CNN
+F 1 "+1V1" H 1250 4065 50  0000 C CNN
+F 2 "" H 1250 3925 50  0001 C CNN
+F 3 "" H 1250 3925 50  0001 C CNN
+	1    1250 3925
+	-1   0    0    1
+$EndComp
+Wire Wire Line
+	1250 3750 1250 3925
 $EndSCHEMATC

Commit message: Fix #12 If RC1 and RC2 are placed voltahe will be 1.2V
Parts:
- added RC1: *DNP, Capacitor_SMD:C_0402_1005Metric, symbol Device:R
- added RC2: 91k, Capacitor_SMD:C_0402_1005Metric, symbol Device:R
- R3, RB2: value 4.7k -> 4k7
- RB3: value 3.3k -> 3k3
Connections:
- net FB1: now also RC1.2
- net GND: now also RC2.1
- new net: RC1.1, RC2.2
Other:
- note added: "0R"
Changed lines of the file:
@@
 AR Path="/58D5A1E5" Ref="RB1"  Part="1"
 AR Path="/58D51CAD/58D5A1E5" Ref="RB1"  Part="1"
-F 0 "RB1" V 9680 3500 50  0000 C CNN
+F 0 "RB1" V 9525 3500 50  0000 C CNN
 F 1 "18k" V 9600 3500 50  0000 C CNN
 F 2 "Capacitor_SMD:C_0402_1005Metric" V 9530 3500 50  0001 C CNN
@@
 L power:GND #PWR075
 U 1 1 58D5AE5E
-P 9800 3600
-F 0 "#PWR075" H 9800 3350 50  0001 C CNN
-F 1 "GND" H 9800 3450 50  0000 C CNN
-F 2 "" H 9800 3600 50  0000 C CNN
-F 3 "" H 9800 3600 50  0000 C CNN
-	1    9800 3600
+P 9800 3950
+F 0 "#PWR075" H 9800 3700 50  0001 C CNN
+F 1 "GND" H 9800 3800 50  0000 C CNN
+F 2 "" H 9800 3950 50  0000 C CNN
+F 3 "" H 9800 3950 50  0000 C CNN
+	1    9800 3950
 	1    0    0    -1
 $EndComp
@@
 AR Path="/58D51CAD/58D62976" Ref="RB3"  Part="1"
 F 0 "RB3" V 9680 5900 50  0000 C CNN
-F 1 "3.3k" V 9600 5900 50  0000 C CNN
+F 1 "3k3" V 9600 5900 50  0000 C CNN
 F 2 "Capacitor_SMD:C_0402_1005Metric" V 9530 5900 50  0001 C CNN
 F 3 "" H 9600 5900 50  0000 C CNN
@@
 AR Path="/58D51CAD/58D67BEA" Ref="RB2"  Part="1"
 F 0 "RB2" V 9680 4700 50  0000 C CNN
-F 1 "4.7k" V 9600 4700 50  0000 C CNN
+F 1 "4k7" V 9600 4700 50  0000 C CNN
 F 2 "Capacitor_SMD:C_0402_1005Metric" V 9530 4700 50  0001 C CNN
 F 3 "" H 9600 4700 50  0000 C CNN
@@
 Text Label 8800 3500 0    60   ~ 0
 FB1
-Text Notes 8700 4150 0    60   ~ 0
+Text Notes 8175 4175 0    60   ~ 0
 (15k/4.7k+1)*0.6V = 2.51V\n
 Text Notes 8700 5350 0    60   ~ 0
@@
 AR Path="/58D51CAD/58E810CC" Ref="R3"  Part="1"
 F 0 "R3" V 3250 4400 50  0000 C CNN
-F 1 "4.7k" V 3150 4400 50  0000 C CNN
+F 1 "4k7" V 3150 4400 50  0000 C CNN
 F 2 "Capacitor_SMD:C_0402_1005Metric" V 3080 4400 50  0001 C CNN
 F 3 "" H 3150 4400 50  0000 C CNN
@@
 	2600 1050 2700 1050
 Wire Wire Line
-	9800 3500 9800 3600
-Wire Wire Line
 	9800 3500 10150 3500
 Wire Wire Line
@@
 Wire Wire Line
 	1250 3750 1250 3925
+$Comp
+L Device:R RB?
+U 1 1 61DA59CF
+P 9575 3900
+AR Path="/61DA59CF" Ref="RB?"  Part="1"
+AR Path="/58D51CAD/61DA59CF" Ref="RC2"  Part="1"
+F 0 "RC2" V 9655 3900 50  0000 C CNN
+F 1 "91k" V 9575 3900 50  0000 C CNN
+F 2 "Capacitor_SMD:C_0402_1005Metric" V 9505 3900 50  0001 C CNN
+F 3 "" H 9575 3900 50  0000 C CNN
+F 4 "www.yageo.com" V 9575 3900 50  0001 C CNN "MNF1_URL"
+F 5 "RC0603FR-1018KL" V 9575 3900 50  0001 C CNN "MPN"
+F 6 "71-CRCW060318K0FKEAC" V 9575 3900 50  0001 C CNN "Mouser"
+F 7 " 311-18.0KHRCT-ND" V 9575 3900 50  0001 C CNN "Digikey"
+F 8 "94X1474" V 9575 3900 50  0001 C CNN "Newark"
+F 9 "C425614" V 9575 3900 50  0001 C CNN "LCSC"
+F 10 "FR006" V 9575 3900 50  0001 C CNN "Koncar"
+	1    9575 3900
+	0    1    1    0
+$EndComp
+$Comp
+L Device:R RC?
+U 1 1 61E2F041
+P 9400 3700
+AR Path="/61E2F041" Ref="RC?"  Part="1"
+AR Path="/58D51CAD/61E2F041" Ref="RC1"  Part="1"
+F 0 "RC1" V 9480 3700 50  0000 C CNN
+F 1 "*DNP" V 9300 3700 50  0000 C CNN
+F 2 "Capacitor_SMD:C_0402_1005Metric" V 9330 3700 50  0001 C CNN
+F 3 "" H 9400 3700 50  0000 C CNN
+F 4 "www.yageo.com" V 9400 3700 50  0001 C CNN "MNF1_URL"
+F 5 "RC0603FR-1018KL" V 9400 3700 50  0001 C CNN "MPN"
+F 6 "71-CRCW060318K0FKEAC" V 9400 3700 50  0001 C CNN "Mouser"
+F 7 " 311-18.0KHRCT-ND" V 9400 3700 50  0001 C CNN "Digikey"
+F 8 "94X1474" V 9400 3700 50  0001 C CNN "Newark"
+F 9 "C425614" V 9400 3700 50  0001 C CNN "LCSC"
+F 10 "FR006" V 9400 3700 50  0001 C CNN "Koncar"
+	1    9400 3700
+	-1   0    0    1
+$EndComp
+Wire Wire Line
+	9400 3550 9400 3500
+Wire Wire Line
+	9400 3850 9400 3900
+Wire Wire Line
+	9400 3900 9425 3900
+Wire Wire Line
+	9800 3500 9800 3900
+Wire Wire Line
+	9725 3900 9800 3900
+Wire Wire Line
+	9800 3950 9800 3900
+Connection ~ 9800 3900
+Text Notes 9425 3750 1    39   ~ 0
+0R
 $EndSCHEMATC

Commit message: DDR3 GND and VCC
Parts:
- added C76, C95, C96: 22uF, Capacitor_SMD:C_0603_1608Metric, symbol Device:C
- added C77: 100pF, Capacitor_SMD:C_0402_1005Metric, symbol Device:C
- added C97, C98: 2.2uF, Capacitor_SMD:C_0603_1608Metric, symbol Device:C
- added L4: 2.2uH, L_1008_1210:L_1008_1210, symbol Device:L
- added RA4: 15k, Capacitor_SMD:C_0402_1005Metric, symbol Device:R
- added RB4: 12k, Capacitor_SMD:C_0402_1005Metric, symbol Device:R
- added RP4: 0, jumper:R_0805_2012Metric_Pad1.29x1.40mm_HandSolder_Jumper_NC, symbol Device:Jumper_NC_Small
- added U6: TLV62569DBV, TSOT-25:TSOT-25, symbol dcdc:DCDC
Connections:
- net +5V: now also C76.1, U6.1 (EN), U6.4 (VIN)
- net GND: now also C76.2, C95.2, C96.2, C97.2, C98.2, RB4.1, U6.2 (GND)
- new net +1V35: C98.1, RP4.2
- new net FB4: C77.2, RA4.2, RB4.2, U6.5 (FB)
- new net L4: L4.1, U6.3 (LX)
- new net P1V35: C77.1, C95.1, C96.1, C97.1, L4.2, RA4.1, RP4.1
Other:
- note added: "(15k/12k+1)*0.6V = 1.35V\n"

Commit message: Removing termination chip
Parts:
- C60, R3: footprint Capacitor_SMD:C_0402_1005Metric -> (none)
- D17: footprint Diode_SMD:D_SOD-323 -> (none)
Changed lines of the file:
@@
 F 0 "R3" V 3250 4400 50  0000 C CNN
 F 1 "4k7" V 3150 4400 50  0000 C CNN
-F 2 "Capacitor_SMD:C_0402_1005Metric" V 3080 4400 50  0001 C CNN
+F 2 "" V 3080 4400 50  0001 C CNN
 F 3 "" H 3150 4400 50  0000 C CNN
 F 4 "AC0603FR-104K7L" V 3150 4400 50  0001 C CNN "MPN"
@@
 F 0 "D17" H 3150 4050 50  0000 C CNN
 F 1 "1N914" H 3200 4250 50  0000 C CNN
-F 2 "Diode_SMD:D_SOD-323" H 3150 4150 50  0001 C CNN
+F 2 "" H 3150 4150 50  0001 C CNN
 F 3 "" H 3150 4150 50  0000 C CNN
 	1    3150 4150
@@
 F 0 "C60" V 2150 4800 50  0000 L CNN
 F 1 "220nF" V 2250 4800 50  0000 L CNN
-F 2 "Capacitor_SMD:C_0402_1005Metric" H 2238 4600 50  0001 C CNN
+F 2 "" H 2238 4600 50  0001 C CNN
 F 3 "" H 2200 4750 50  0000 C CNN
 	1    2200 4750

Commit message: fix #19 fix #18
Parts:
- renumbered U3 to U5, U4 to U6, U5 to U7, U6 to U8
Connections:
- net +1V35: now also C25.1, C32.1, U1.H14 (VCCio2), U1.H15 (VCCio2), U1.J15 (VCCio2), U1.L14 (VCCio3), U1.L15 (VCCio3), U1.M15 (VCCio3)
- net +3V3: no longer C25.1, C32.1, U1.H14 (VCCio2), U1.H15 (VCCio2), U1.J15 (VCCio2), U1.L14 (VCCio3), U1.L15 (VCCio3), U1.M15 (VCCio3)
Other:
- moved on the sheet: 1.1V_1, C25, C32, C47, C48, C49, C50, C51, C60, C76, C77, C95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

Commit message: fix #20 Adding USB connector - fix diff lengths
Parts:
- RV2, RV3: footprint Resistor_SMD:R_0805_2012Metric_Pad1.29x1.40mm_HandSolder -> Resistor_SMD:R_0603_1608Metric_Pad0.98x0.95mm_HandSolder
Changed lines of the file:
@@
 F 0 "RV2" H 875 1400 50  0000 C CNN
 F 1 "0" H 875 1250 50  0000 C CNN
-F 2 "Resistor_SMD:R_0805_2012Metric_Pad1.29x1.40mm_HandSolder" H 875 1300 50  0001 C CNN
+F 2 "Resistor_SMD:R_0603_1608Metric_Pad0.98x0.95mm_HandSolder" H 875 1300 50  0001 C CNN
 F 3 "" H 875 1300 50  0001 C CNN
 F 4 "www.yageo.com" H 875 1300 50  0001 C CNN "MNF1_URL"
@@
 F 0 "RV3" H 875 1100 50  0000 C CNN
 F 1 "0" H 875 950 50  0000 C CNN
-F 2 "Resistor_SMD:R_0805_2012Metric_Pad1.29x1.40mm_HandSolder" H 875 1000 50  0001 C CNN
+F 2 "Resistor_SMD:R_0603_1608Metric_Pad0.98x0.95mm_HandSolder" H 875 1000 50  0001 C CNN
 F 3 "" H 875 1000 50  0001 C CNN
 F 4 "www.yageo.com" H 875 1000 50  0001 C CNN "MNF1_URL"
