File: power.sch (KiCad schematic (older format))
At the start: 67 parts, among them U1 LFE5U-85F-6BG381C, U5 TLV62569DBV, U6 TLV62569DBV, U7 TLV62569DBV, U8 TLV62569DBV

Commit message: References cleanup
Changed lines of the file:
@@
 $Descr A4 11693 8268
 encoding utf-8
-Sheet 3 13
+Sheet 3 11
 Title "ULX3S"
 Date ""
@@
 P 5750 4000
 AR Path="/5A5FC402" Ref="C30"  Part="1"
-AR Path="/58D51CAD/5A5FC402" Ref="C30"  Part="1"
-F 0 "C30" H 5775 4100 50  0000 L CNN
+AR Path="/58D51CAD/5A5FC402" Ref="C39"  Part="1"
+F 0 "C39" H 5775 4100 50  0000 L CNN
 F 1 "22nF" H 5775 3900 50  0000 L CNN
 F 2 "Capacitor_SMD:C_0402_1005Metric" H 5788 3850 50  0001 C CNN
@@
 P 5750 4750
 AR Path="/5A5FEEA6" Ref="C31"  Part="1"
-AR Path="/58D51CAD/5A5FEEA6" Ref="C31"  Part="1"
-F 0 "C31" H 5775 4850 50  0000 L CNN
+AR Path="/58D51CAD/5A5FEEA6" Ref="C14"  Part="1"
+F 0 "C14" H 5775 4850 50  0000 L CNN
 F 1 "22nF" H 5775 4650 50  0000 L CNN
 F 2 "Capacitor_SMD:C_0402_1005Metric" H 5788 4600 50  0001 C CNN
@@
 P 3925 5375
 AR Path="/5A6007F1" Ref="C32"  Part="1"
-AR Path="/58D51CAD/5A6007F1" Ref="C32"  Part="1"
-F 0 "C32" H 3950 5475 50  0000 L CNN
+AR Path="/58D51CAD/5A6007F1" Ref="C13"  Part="1"
+F 0 "C13" H 3950 5475 50  0000 L CNN
 F 1 "22nF" H 3950 5275 50  0000 L CNN
 F 2 "Capacitor_SMD:C_0402_1005Metric" H 3963 5225 50  0001 C CNN
@@
 P 1075 1400
 AR Path="/5AB6B7B8" Ref="C47"  Part="1"
-AR Path="/58D51CAD/5AB6B7B8" Ref="C47"  Part="1"
-F 0 "C47" H 1075 1300 50  0000 L CNN
+AR Path="/58D51CAD/5AB6B7B8" Ref="C38"  Part="1"
+F 0 "C38" H 1075 1300 50  0000 L CNN
 F 1 "2.2uF" H 1075 1500 50  0000 L CNN
 F 2 "Capacitor_SMD:C_0603_1608Metric" H 1113 1250 50  0001 C CNN

Commit message: Adding few test pads #24
Parts:
- added TP_1V35: 1V35, ecp5-dc-scm:Testpoint_smd_1mm, symbol Connector:TestPoint_Small
Connections:
- net +1V35: now also TP_1V35.1
Changed lines of the file:
@@
 	1    0    0    -1
 $EndComp
+$Comp
+L power:+1V35 #PWR?
+U 1 1 622C7816
+P 6025 5725
+F 0 "#PWR?" H 6025 5575 50  0001 C CNN
+F 1 "+1V35" H 6040 5898 50  0000 C CNN
+F 2 "" H 6025 5725 50  0001 C CNN
+F 3 "" H 6025 5725 50  0001 C CNN
+	1    6025 5725
+	1    0    0    -1
+$EndComp
+$Comp
+L Connector:TestPoint_Small TP_D?
+U 1 1 622D7422
+P 6025 5875
+AR Path="/56AC389C/622D7422" Ref="TP_D?"  Part="1"
+AR Path="/58D686D9/622D7422" Ref="TP_D?"  Part="1"
+AR Path="/58D51CAD/622D7422" Ref="TP_1V35"  Part="1"
+F 0 "TP_1V35" V 5925 5775 50  0000 L CNN
+F 1 "1V35" V 6125 5750 50  0000 L CNN
+F 2 "ecp5-dc-scm:Testpoint_smd_1mm" H 6225 5875 50  0001 C CNN
+F 3 "~" H 6225 5875 50  0001 C CNN
+	1    6025 5875
+	1    0    0    -1
+$EndComp
+Wire Wire Line
+	6025 5875 6025 5725
 $EndSCHEMATC

Commit message: Lowering number of unique parts fix #37
Parts:
- RA1, RA2, RA3, RA4, RB1, RB2, RB3, RB4, RC1, RC2: footprint Capacitor_SMD:C_0402_1005Metric -> Resistor_SMD:R_0402_1005Metric
Changed lines of the file:
@@
 F 0 "RA1" V 9480 3300 50  0000 C CNN
 F 1 "15k" V 9400 3300 50  0000 C CNN
-F 2 "Capacitor_SMD:C_0402_1005Metric" V 9330 3300 50  0001 C CNN
+F 2 "Resistor_SMD:R_0402_1005Metric" V 9330 3300 50  0001 C CNN
 F 3 "" H 9400 3300 50  0000 C CNN
 F 4 "www.yageo.com" V 9400 3300 50  0001 C CNN "MNF1_URL"
@@
 F 0 "RB1" V 9525 3500 50  0000 C CNN
 F 1 "18k" V 9600 3500 50  0000 C CNN
-F 2 "Capacitor_SMD:C_0402_1005Metric" V 9530 3500 50  0001 C CNN
+F 2 "Resistor_SMD:R_0402_1005Metric" V 9530 3500 50  0001 C CNN
 F 3 "" H 9600 3500 50  0000 C CNN
 F 4 "www.yageo.com" V 9600 3500 50  0001 C CNN "MNF1_URL"
@@
 F 0 "RA3" V 9480 5700 50  0000 C CNN
 F 1 "15k" V 9400 5700 50  0000 C CNN
-F 2 "Capacitor_SMD:C_0402_1005Metric" V 9330 5700 50  0001 C CNN
+F 2 "Resistor_SMD:R_0402_1005Metric" V 9330 5700 50  0001 C CNN
 F 3 "" H 9400 5700 50  0000 C CNN
 	1    9400 5700
@@
 F 0 "RB3" V 9680 5900 50  0000 C CNN
 F 1 "3k3" V 9600 5900 50  0000 C CNN
-F 2 "Capacitor_SMD:C_0402_1005Metric" V 9530 5900 50  0001 C CNN
+F 2 "Resistor_SMD:R_0402_1005Metric" V 9530 5900 50  0001 C CNN
 F 3 "" H 9600 5900 50  0000 C CNN
 F 4 "www.yageo.com" V 9600 5900 50  0001 C CNN "MNF1_URL"
@@
 F 0 "RA2" V 9480 4500 50  0000 C CNN
 F 1 "15k" V 9400 4500 50  0000 C CNN
-F 2 "Capacitor_SMD:C_0402_1005Metric" V 9330 4500 50  0001 C CNN
+F 2 "Resistor_SMD:R_0402_1005Metric" V 9330 4500 50  0001 C CNN
 F 3 "" H 9400 4500 50  0000 C CNN
 	1    9400 4500
@@
 F 0 "RB2" V 9680 4700 50  0000 C CNN
 F 1 "4k7" V 9600 4700 50  0000 C CNN
-F 2 "Capacitor_SMD:C_0402_1005Metric" V 9530 4700 50  0001 C CNN
+F 2 "Resistor_SMD:R_0402_1005Metric" V 9530 4700 50  0001 C CNN
 F 3 "" H 9600 4700 50  0000 C CNN
 F 4 "AC0603FR-104K7L" V 9600 4700 50  0001 C CNN "MPN"
@@
 F 0 "RC2" V 9655 3900 50  0000 C CNN
 F 1 "91k" V 9575 3900 50  0000 C CNN
-F 2 "Capacitor_SMD:C_0402_1005Metric" V 9505 3900 50  0001 C CNN
+F 2 "Resistor_SMD:R_0402_1005Metric" V 9505 3900 50  0001 C CNN
 F 3 "" H 9575 3900 50  0000 C CNN
 F 4 "www.yageo.com" V 9575 3900 50  0001 C CNN "MNF1_URL"
@@
 F 0 "RC1" V 9480 3700 50  0000 C CNN
 F 1 "*DNP" V 9300 3700 50  0000 C CNN
-F 2 "Capacitor_SMD:C_0402_1005Metric" V 9330 3700 50  0001 C CNN
+F 2 "Resistor_SMD:R_0402_1005Metric" V 9330 3700 50  0001 C CNN
 F 3 "" H 9400 3700 50  0000 C CNN
 F 4 "www.yageo.com" V 9400 3700 50  0001 C CNN "MNF1_URL"
@@
 F 0 "RA4" V 5230 6725 50  0000 C CNN
 F 1 "15k" V 5150 6725 50  0000 C CNN
-F 2 "Capacitor_SMD:C_0402_1005Metric" V 5080 6725 50  0001 C CNN
+F 2 "Resistor_SMD:R_0402_1005Metric" V 5080 6725 50  0001 C CNN
 F 3 "" H 5150 6725 50  0000 C CNN
 	1    5150 6725
@@
 F 0 "RB4" V 5430 6925 50  0000 C CNN
 F 1 "12k" V 5350 6925 50  0000 C CNN
-F 2 "Capacitor_SMD:C_0402_1005Metric" V 5280 6925 50  0001 C CNN
+F 2 "Resistor_SMD:R_0402_1005Metric" V 5280 6925 50  0001 C CNN
 F 3 "" H 5350 6925 50  0000 C CNN
 F 4 "www.yageo.com" V 5350 6925 50  0001 C CNN "MNF1_URL"

Commit message: Connecting DSI1 to DSI0
Connections:
- net +1V35: no longer C25.1, C32.1, U1.H14 (VCCio2), U1.H15 (VCCio2), U1.J15 (VCCio2), U1.L14 (VCCio3), U1.L15 (VCCio3), U1.M15 (VCCio3)
- net +3V3: now also C25.1, C32.1, U1.H14 (VCCio2), U1.H15 (VCCio2), U1.J15 (VCCio2), U1.L14 (VCCio3), U1.L15 (VCCio3), U1.M15 (VCCio3)
Changed lines of the file:
@@
 L power:+3V3 #PWR053
 U 1 1 5A5F7519
-P 3100 4875
-F 0 "#PWR053" H 3100 4725 50  0001 C CNN
-F 1 "+3V3" H 3100 5015 50  0000 C CNN
-F 2 "" H 3100 4875 50  0000 C CNN
-F 3 "" H 3100 4875 50  0000 C CNN
-	1    3100 4875
+P 3675 5225
+F 0 "#PWR053" H 3675 5075 50  0001 C CNN
+F 1 "+3V3" H 3675 5365 50  0000 C CNN
+F 2 "" H 3675 5225 50  0000 C CNN
+F 3 "" H 3675 5225 50  0000 C CNN
+	1    3675 5225
 	1    0    0    -1
 $EndComp
@@
 L power:+3V3 #PWR046
 U 1 1 5A6007FD
-P 3100 5150
-F 0 "#PWR046" H 3100 5000 50  0001 C CNN
-F 1 "+3V3" H 3100 5290 50  0000 C CNN
-F 2 "" H 3100 5150 50  0000 C CNN
-F 3 "" H 3100 5150 50  0000 C CNN
-	1    3100 5150
+P 3925 5225
+F 0 "#PWR046" H 3925 5075 50  0001 C CNN
+F 1 "+3V3" H 3925 5365 50  0000 C CNN
+F 2 "" H 3925 5225 50  0000 C CNN
+F 3 "" H 3925 5225 50  0000 C CNN
+	1    3925 5225
 	1    0    0    -1
 $EndComp
@@
 Wire Wire Line
 	5000 1050 5000 925
-$Comp
-L power:+1V35 #PWR0142
-U 1 1 649E2281
-P 5300 925
-F 0 "#PWR0142" H 5300 775 50  0001 C CNN
-F 1 "+1V35" H 5315 1098 50  0000 C CNN
-F 2 "" H 5300 925 50  0001 C CNN
-F 3 "" H 5300 925 50  0001 C CNN
-	1    5300 925
-	1    0    0    -1
-$EndComp
 Wire Wire Line
 	5300 925  5300 1050
@@
 L power:+1V35 #PWR0143
 U 1 1 64D9D79E
-P 3925 5225
-F 0 "#PWR0143" H 3925 5075 50  0001 C CNN
-F 1 "+1V35" H 3940 5398 50  0000 C CNN
-F 2 "" H 3925 5225 50  0001 C CNN
-F 3 "" H 3925 5225 50  0001 C CNN
-	1    3925 5225
+P 3125 5750
+F 0 "#PWR0143" H 3125 5600 50  0001 C CNN
+F 1 "+1V35" H 3140 5923 50  0000 C CNN
+F 2 "" H 3125 5750 50  0001 C CNN
+F 3 "" H 3125 5750 50  0001 C CNN
+	1    3125 5750
 	1    0    0    -1
 $EndComp
@@
 L power:+1V35 #PWR0144
 U 1 1 64D9EB5E
-P 3675 5225
-F 0 "#PWR0144" H 3675 5075 50  0001 C CNN
-F 1 "+1V35" H 3690 5398 50  0000 C CNN
-F 2 "" H 3675 5225 50  0001 C CNN
-F 3 "" H 3675 5225 50  0001 C CNN
-	1    3675 5225
+P 2975 5575
+F 0 "#PWR0144" H 2975 5425 50  0001 C CNN
+F 1 "+1V35" H 2990 5748 50  0000 C CNN
+F 2 "" H 2975 5575 50  0001 C CNN
+F 3 "" H 2975 5575 50  0001 C CNN
+	1    2975 5575
 	1    0    0    -1
 $EndComp
@@
 Wire Wire Line
 	6025 5875 6025 5725
+$Comp
+L power:+3V3 #PWR0116
+U 1 1 63AE3AA8
+P 5300 925
+F 0 "#PWR0116" H 5300 775 50  0001 C CNN
+F 1 "+3V3" H 5300 1065 50  0000 C CNN
+F 2 "" H 5300 925 50  0000 C CNN
+F 3 "" H 5300 925 50  0000 C CNN
+	1    5300 925
+	1    0    0    -1
+$EndComp
 $EndSCHEMATC
