File: ulx4m.kicad_pcb (KiCad board)
At the start: 6 copper layers, 55.1 x 40 mm, 176 parts, among them IC1 VSC8530XMW-04, J1 DF40C-100DP-0.4V(51), J2 DF40C-100DP-0.4V(51), J3 JTAG, SW1 SW_Push, SW2 SW_Push, U1 LFE5U-85F-6BG381C, U10 IS25LP128F-JBLE, U2 IS42S16320D-6BLI, U3 TLV62569DBV, U4 TLV62569DBV, U5 TLV62569DBV, Y1 FNETHE025

Commit message: Routing SerDes lines near eth chip
Routing:
- net /serdes/S_4_P: track 3.74 -> 29.2 mm
- net /serdes/S_4_N: track 3.61 -> 28.6 mm
- net /serdes/S_3_N: track 5.17 -> 26.8 mm
- net /serdes/S_6_P: track 4.57 -> 25.7 mm
- net /serdes/S_3_P: track 4.10 -> 25.2 mm
- net /serdes/S_6_N: track 4.45 -> 25.1 mm
- net /serdes/S_1_N: track 3.33 -> 18.8 mm
- net /serdes/S_1_P: track 3.58 -> 18.4 mm
- net GPIO5: track 24.0 -> 23.1 mm
- net +1V1: track 132.4 -> 131.7 mm
- net /flash/FPGA_PROGRAMN: track 53.2 -> 53.9 mm
- net GPIO19: track 22.2 -> 22.9 mm
- net /flash/FLASH_MOSI: track 29.1 -> 29.8 mm
- net GPIO26: track 19.9 -> 20.6 mm
- net GPIO13: track 22.1 -> 22.8 mm
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
Commit message: Before DDR3 branch
Routing:
- net GND: vias 212 -> 233

Commit message: Adding DDR3 symbol and footprint
Parts:
- U2: value IS42S16320D-6BLI -> MT41K256M16TW-107_P; footprint IS42S16320D:IS42S16320D-6BLI -> MT41K256M16TW-107_P:BGA96C80P9X16_800X1400X120
- moved U2 2.14 mm to (138.9, 93.3), turned to 90 degrees
- moved radiona 0.82 mm to (136.7, 99.6)
Connections:
- U1 pad C20: SDRAM_A9 -> (no net)
- U1 pad D19: SDRAM_DQM1 -> (no net)
- U1 pad D20: SDRAM_A11 -> (no net)
- U1 pad E18: SDRAM_A12 -> (no net)
- U1 pad E19: SDRAM_A6 -> (no net)
- U1 pad E20: SDRAM_A8 -> (no net)
- U1 pad F18: SDRAM_A5 -> (no net)
- U1 pad F19: SDRAM_A7 -> (no net)
- U1 pad F20: SDRAM_A4 -> (no net)
- U1 pad G19: SDRAM_CLK -> (no net)
- U1 pad G20: SDRAM_CKE -> (no net)
- U1 pad H17: SDRAM_A3 -> (no net)
- U1 pad H18: SDRAM_D12 -> (no net)
- U1 pad H20: SDRAM_D8 -> (no net)
- U1 pad J16: SDRAM_D13 -> (no net)
- U1 pad J17: SDRAM_D15 -> (no net)
- U1 pad J18: SDRAM_D11 -> (no net)
- U1 pad J19: SDRAM_D9 -> (no net)
- U1 pad K18: SDRAM_D10 -> (no net)
- U1 pad K19: SDRAM_D14 -> (no net)
- U1 pad L18: SDRAM_BA0 -> (no net)
- U1 pad L19: SDRAM_A0 -> (no net)
- U1 pad L20: SDRAM_A1 -> (no net)
- U1 pad M18: SDRAM_nRAS -> (no net)
- U1 pad M19: SDRAM_A2 -> (no net)
- U1 pad M20: SDRAM_BA1 -> (no net)
- U1 pad N18: SDRAM_nCAS -> (no net)
- U1 pad N19: SDRAM_A10 -> (no net)
- U1 pad N20: SDRAM_nWE -> (no net)
- U1 pad P18: SDRAM_nCS -> (no net)
- U1 pad P19: SDRAM_D7 -> (no net)
- U1 pad P20: SDRAM_DQM0 -> (no net)
- U1 pad R20: SDRAM_D6 -> (no net)
- U1 pad T17: SDRAM_D5 -> (no net)
- U1 pad T18: SDRAM_D4 -> (no net)
- U1 pad T19: SDRAM_D3 -> (no net)
- U1 pad T20: SDRAM_D1 -> (no net)
- U1 pad U19: SDRAM_D2 -> (no net)
- U1 pad U20: SDRAM_D0 -> (no net)
- U2 pad A1: GND -> (no net)
- U2 pad A2: SDRAM_D14 -> (no net)
- U2 pad A3: GND -> (no net)
- U2 pad A7: CM4_3.3V -> (no net)
- U2 pad A8: SDRAM_D0 -> (no net)
- U2 pad A9: CM4_3.3V -> (no net)
- U2 pad B1: SDRAM_D15 -> (no net)
- U2 pad B2: SDRAM_D13 -> (no net)
- U2 pad B3: CM4_3.3V -> (no net)
- U2 pad B7: GND -> (no net)
- U2 pad B8: SDRAM_D2 -> (no net)
- U2 pad B9: SDRAM_D1 -> (no net)
- U2 pad C1: SDRAM_D12 -> (no net)
- U2 pad C2: SDRAM_D11 -> (no net)
- U2 pad C3: GND -> (no net)
- U2 pad C7: CM4_3.3V -> (no net)
- U2 pad C8: SDRAM_D4 -> (no net)
- U2 pad C9: SDRAM_D3 -> (no net)
- U2 pad D1: SDRAM_D10 -> (no net)
- U2 pad D2: SDRAM_D9 -> (no net)
- U2 pad D3: CM4_3.3V -> (no net)
- U2 pad D7: GND -> (no net)
- U2 pad D8: SDRAM_D6 -> (no net)
- U2 pad D9: SDRAM_D5 -> (no net)
- U2 pad E1: SDRAM_D8 -> (no net)
- U2 pad E3: GND -> (no net)
- U2 pad E7: CM4_3.3V -> (no net)
- U2 pad E8: SDRAM_DQM0 -> (no net)
- U2 pad E9: SDRAM_D7 -> (no net)
- U2 pad F1: SDRAM_DQM1 -> (no net)
- U2 pad F2: SDRAM_CLK -> (no net)
- U2 pad F3: SDRAM_CKE -> (no net)
- U2 pad F7: SDRAM_nCAS -> (no net)
- U2 pad F8: SDRAM_nRAS -> (no net)
- U2 pad F9: SDRAM_nWE -> (no net)
- U2 pad G1: SDRAM_A12 -> (no net)
- U2 pad G2: SDRAM_A11 -> (no net)
- U2 pad G3: SDRAM_A9 -> (no net)
- U2 pad G7: SDRAM_BA0 -> (no net)
- U2 pad G8: SDRAM_BA1 -> (no net)
- U2 pad G9: SDRAM_nCS -> (no net)
- U2 pad H1: SDRAM_A8 -> (no net)
- U2 pad H2: SDRAM_A7 -> (no net)
- U2 pad H3: SDRAM_A6 -> (no net)
- U2 pad H7: SDRAM_A0 -> (no net)
- U2 pad H8: SDRAM_A1 -> (no net)
- U2 pad H9: SDRAM_A10 -> (no net)
- U2 pad J1: GND -> (no net)
- U2 pad J2: SDRAM_A5 -> (no net)
- U2 pad J3: SDRAM_A4 -> (no net)
- U2 pad J7: SDRAM_A3 -> (no net)
- U2 pad J8: SDRAM_A2 -> (no net)
- U2 pad J9: CM4_3.3V -> (no net)
Routing:
- net (no net): track 0.00 -> 252.7 mm, vias 0 -> 26
- net SDRAM_D15: track 21.5 -> 0.00 mm, vias 3 -> 0
- net SDRAM_D5: track 21.4 -> 0.00 mm
- net SDRAM_nCAS: track 20.8 -> 0.00 mm, vias 2 -> 0
- net SDRAM_D2: track 20.7 -> 0.00 mm, vias 2 -> 0
- net SDRAM_D11: track 20.4 -> 0.00 mm, vias 2 -> 0
- net SDRAM_nRAS: track 20.3 -> 0.00 mm, vias 2 -> 0
- net SDRAM_A2: track 20.1 -> 0.00 mm
- net SDRAM_D9: track 20.1 -> 0.00 mm, vias 2 -> 0
- net SDRAM_D14: track 20.1 -> 0.00 mm
- net SDRAM_D13: track 20.1 -> 0.00 mm, vias 3 -> 0
- net SDRAM_CLK: track 20.1 -> 0.00 mm
- net SDRAM_A0: track 20.1 -> 0.00 mm, vias 3 -> 0
- net SDRAM_BA1: track 20.0 -> 0.00 mm
- net SDRAM_A12: track 20.0 -> 0.00 mm, vias 2 -> 0
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Other:
- board text added: "04.01.2022. v0.0.4"
- board text added: "CAM0"
- board text added: "CAM1"
- board text added: "DDR3"
- board text added: "DISP0"
- board text added: "DISP1"
- board text added: "ULX4M-LD"
- board text added: "USB"
- board text removed: "01.01.2022. v0.0.3"
- board text removed: "SDRAM"
- board text removed: "ULX4M-LS"

Commit message: Adding ecp5-dc-scm ddr3 schematics and footprint
Routing:
- net GND: track 265.5 -> 264.7 mm

Commit message: DDR3 GND and VCC
Parts:
- added C196: C_1n_0402, ecp5-dc-scm:0402-cap, F.Cu at (175.0, 113.7)
- added C197: C_10u_0402, ecp5-dc-scm:0402-cap, F.Cu at (240.8, 68.9)
- added C198: C_10u_0402, ecp5-dc-scm:0402-cap, F.Cu at (240.3, 85.9)
- added C199: C_10u_0402, ecp5-dc-scm:0402-cap, F.Cu at (242.8, 79.6)
- added C200: C_100n_0402, ecp5-dc-scm:0402-cap, F.Cu at (232.0, 98.5)
- added C201: C_100n_0402, ecp5-dc-scm:0402-cap, F.Cu at (177.9, 113.7)
- added C202: C_100n_0402, ecp5-dc-scm:0402-cap, F.Cu at (237.4, 85.9)
- added C240: C_100n_0402, ecp5-dc-scm:0402-cap, F.Cu at (243.2, 85.9)
- added C76: 22uF, Capacitor_SMD:C_0603_1608Metric, B.Cu at (136.8, 95.4)
- added C77: 100pF, Capacitor_SMD:C_0402_1005Metric, B.Cu at (136.9, 91.5)
- added C78: C_10u_0402, ecp5-dc-scm:0402-cap, F.Cu at (167.6, 50.5)
- added C79: C_4u7_0402, ecp5-dc-scm:0402-cap, F.Cu at (231.5, 86.5)
- added C80: C_470n_0402, ecp5-dc-scm:0402-cap, F.Cu at (234.1, 78.6)
- added C81: C_470n_0402, ecp5-dc-scm:0402-cap, F.Cu at (209.1, 106.8)
- added C82: C_470n_0402, ecp5-dc-scm:0402-cap, F.Cu at (180.4, 100.5)
- added C83: C_470n_0402, ecp5-dc-scm:0402-cap, F.Cu at (177.5, 100.5)
- added C84: C_470n_0402, ecp5-dc-scm:0402-cap, F.Cu at (179.2, 50.9)
- added C85: C_470n_0402, ecp5-dc-scm:0402-cap, F.Cu at (234.5, 86.5)
- added C86: C_470n_0402, ecp5-dc-scm:0402-cap, F.Cu at (237.0, 79.6)
- added C87: C_470n_0402, ecp5-dc-scm:0402-cap, F.Cu at (226.2, 98.5)
- added C88: C_100n_0402, ecp5-dc-scm:0402-cap, F.Cu at (212.0, 106.8)
- added C89: C_470n_0402, ecp5-dc-scm:0402-cap, F.Cu at (183.3, 99.9)
- added C90: C_470n_0402, ecp5-dc-scm:0402-cap, F.Cu at (237.9, 68.9)
- added C91: C_470n_0402, ecp5-dc-scm:0402-cap, F.Cu at (235.0, 68.9)
- added C92: C_470n_0402, ecp5-dc-scm:0402-cap, F.Cu at (239.9, 79.6)
- added C93: C_100n_0402, ecp5-dc-scm:0402-cap, F.Cu at (229.1, 98.5)
- added C94: C_100n_0402, ecp5-dc-scm:0402-cap, F.Cu at (214.9, 106.8)
- added C95: 22uF, Capacitor_SMD:C_0603_1608Metric, B.Cu at (139.3, 91.5)
- added C96: 22uF, Capacitor_SMD:C_0603_1608Metric, B.Cu at (141.0, 91.5)
- added C97: 2.2uF, Capacitor_SMD:C_0603_1608Metric, B.Cu at (146.1, 93.7)
- added C98: 2.2uF, Capacitor_SMD:C_0603_1608Metric, B.Cu at (138.0, 127.3)
- added L4: 2.2uH, L_1008_1210:L_1008_1210, B.Cu at (143.6, 94.1)
- added R78: R_10k_0402, ecp5-dc-scm:0402-res, F.Cu at (245.8, 79.0)
- added R79: R_10k_0402, ecp5-dc-scm:0402-res, F.Cu at (180.9, 113.7)
- added R80: R_10k_0402, ecp5-dc-scm:0402-res, F.Cu at (182.1, 50.9)
- added R81: R_240R_0402, ecp5-dc-scm:0402-res, F.Cu at (248.7, 79.0)
- added R82: R_51R_0402, ecp5-dc-scm:0402-res, F.Cu at (183.8, 113.1)
- added R83: R_51R_0402, ecp5-dc-scm:0402-res, F.Cu at (186.7, 113.1)
- added RA4: 15k, Capacitor_SMD:C_0402_1005Metric, B.Cu at (138.0, 91.5)
- added RB4: 12k, Capacitor_SMD:C_0402_1005Metric, B.Cu at (137.5, 93.0)
- added RP4: 0, jumper:R_0805_2012Metric_Pad1.29x1.40mm_HandSolder_Jumper_NC, B.Cu at (143.0, 89.8)
- added U6: TLV62569DBV, TSOT-25:TSOT-25, B.Cu at (139.8, 95.4)
- U2: value MT41K256M16TW-107_P -> AS4C256M16D3; footprint MT41K256M16TW-107_P:BGA96C80P9X16_800X1400X120 -> AS4C256M16D3:BGA-96_9.0x13.0mm_Layout2x3x16_P0.8mm
- moved D17 67.0 mm to (75.2, 98.4)
- moved C60 67.0 mm to (77.2, 100.5)
- moved R3 67.0 mm to (75.3, 100.5)
- moved D28 67.0 mm to (77.2, 98.4)
- moved D29 67.0 mm to (79.2, 98.4)
- moved R31 57.8 mm to (81.7, 101.2)
- moved C34 30.9 mm to (164.1, 97.3)
- moved C16 30.7 mm to (164.4, 99.7)
- moved C33 30.1 mm to (170.4, 102.5)
- moved C35 29.1 mm to (163.9, 104.5)
- moved C52 29.1 mm to (166.4, 104.8)
- moved REF** 22.7 mm to (137.1, 60.7)
- moved C24 8.62 mm to (135.2, 83.1), turned to 90 degrees
- moved C9 6.85 mm to (144.5, 81.3), turned to 270 degrees
- moved L3 5.70 mm to (137.6, 82.6), turned to 270 degrees
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Connections:
- J1 pad 100: nEXTRST -> (no net)
- J1 pad 34: GPIO5 -> (no net)
- J1 pad 35: ID_SC -> (no net)
- J1 pad 36: ID_SD -> (no net)
- J1 pad 38: GPIO11 -> (no net)
- J1 pad 44: GPIO10 -> (no net)
- J1 pad 46: GPIO22 -> (no net)
- J1 pad 50: GPIO17 -> (no net)
- J1 pad 80: SCL0 -> (no net)
- J1 pad 82: SDA0 -> (no net)
- J1 pad 97: Camera_GPIO -> (no net)
- U1 pad C20: (no net) -> DDR3_DQ12
- U1 pad D19: (no net) -> DDR3_DQ13
- U1 pad D20: (no net) -> DDR3_A4
- U1 pad E16: GPIO4 -> DDR3_A15
- U1 pad E18: (no net) -> DDR3_A8
- U1 pad E19: (no net) -> DDR3_A3
- U1 pad F16: GPIO3 -> DDR3_A0
- U1 pad F18: (no net) -> DDR3_A7
- U1 pad F19: (no net) -> DDR3_DQ15
- U1 pad F20: (no net) -> DDR3_A2
- U1 pad G16: GPIO2 -> DDR3_A13
- U1 pad G19: (no net) -> DDR3_DM0
- U1 pad G20: (no net) -> DDR3_A1
- U1 pad H16: GPIO5 -> DDR3_A14
- U1 pad H17: (no net) -> DDR3_DQ11
- U1 pad H18: (no net) -> DDR3_DQ10
- U1 pad H20: (no net) -> DDR3_DM1
- U1 pad J16: (no net) -> DDR3_A5
- U1 pad J17: (no net) -> DDR3_A6
- U1 pad L16: GPIO11 -> DDR3_DQS1+
- U1 pad L17: GPIO17 -> DDR3_DQS1-
- U1 pad L18: (no net) -> DDR3_CKE
- U1 pad L20: (no net) -> DDR3_CLK+
- U1 pad M17: (no net) -> DDR3_DQ1
- U1 pad M18: (no net) -> DDR3_RESET
- U1 pad M20: (no net) -> DDR3_CLK-
- U1 pad N16: (no net) -> DDR3_DQ0
- U1 pad N17: GPIO10 -> DDR3_DQS0+
- U1 pad N18: (no net) -> DDR3_CS
- U1 pad N19: (no net) -> DDR3_DQ2
- U1 pad N20: (no net) -> DDR3_DQ3
- U1 pad P16: SCL0 -> DDR3_DQS0-
- U1 pad P17: SDA0 -> DDR3_RAS
- U1 pad P18: (no net) -> DDR3_BA0
- U1 pad P19: (no net) -> DDR3_ODT
- U1 pad P20: (no net) -> DDR3_DQ4
- U1 pad R16: ID_SD -> DDR3_CAS
- U1 pad R17: ID_SC -> DDR3_WE
- U1 pad R18: Camera_GPIO -> DDR3_DQ7
- U1 pad R20: (no net) -> DDR3_DQ5
- U1 pad T17: (no net) -> DDR3_A9
- U1 pad T18: (no net) -> DDR3_A11
- U1 pad T19: (no net) -> DDR3_DQ6
- U1 pad T20: (no net) -> DDR3_BA1
- U1 pad U16: nEXTRST -> DDR3_A10
- U1 pad U17: SD_PWR_ON -> DDR3_DQ9
- U1 pad U18: GPIO22 -> DDR3_DQ8
- U1 pad U19: (no net) -> DDR3_A12
- U1 pad U20: (no net) -> DDR3_BA2
- U2 pad A1: (no net) -> VCC1V35
- U2 pad A2: (no net) -> DDR3_DQ13
- U2 pad A3: (no net) -> DDR3_DQ15
- U2 pad A7: (no net) -> DDR3_DQ12
- U2 pad A8: (no net) -> VCC1V35
- U2 pad A9: (no net) -> GND
- U2 pad B1: (no net) -> GND
- U2 pad B2: (no net) -> VCC1V35
- U2 pad B3: (no net) -> GND
- U2 pad B7: (no net) -> DDR3_DQS1-
- U2 pad B9: (no net) -> GND
- U2 pad C1: (no net) -> VCC1V35
- U2 pad C2: (no net) -> DDR3_DQ11
- U2 pad C3: (no net) -> DDR3_DQ9
- U2 pad C7: (no net) -> DDR3_DQS1+
- U2 pad C8: (no net) -> DDR3_DQ10
- U2 pad C9: (no net) -> VCC1V35
- U2 pad D1: (no net) -> GND
- U2 pad D2: (no net) -> VCC1V35
- U2 pad D3: (no net) -> DDR3_DM1
- U2 pad D7: (no net) -> DDR3_DQ8
- U2 pad D8: (no net) -> GND
- U2 pad D9: (no net) -> VCC1V35
- U2 pad E1: (no net) -> GND
- U2 pad E2: (no net) -> GND
- U2 pad E3: (no net) -> DDR3_DQ0
- U2 pad E7: (no net) -> DDR3_DM0
- U2 pad E8: (no net) -> GND
- U2 pad E9: (no net) -> VCC1V35
- U2 pad F1: (no net) -> VCC1V35
- U2 pad F2: (no net) -> DDR3_DQ2
- U2 pad F3: (no net) -> DDR3_DQS0+
- U2 pad F7: (no net) -> DDR3_DQ1
- U2 pad F8: (no net) -> DDR3_DQ3
- U2 pad F9: (no net) -> GND
- U2 pad G1: (no net) -> GND
- U2 pad G2: (no net) -> DDR3_DQ6
- U2 pad G3: (no net) -> DDR3_DQS0-
- U2 pad G7: (no net) -> VCC1V35
- U2 pad G8: (no net) -> GND
- U2 pad G9: (no net) -> GND
- U2 pad H1: (no net) -> DDR3_VREF
- U2 pad H2: (no net) -> VCC1V35
- U2 pad H3: (no net) -> DDR3_DQ4
- U2 pad H7: (no net) -> DDR3_DQ7
- U2 pad H8: (no net) -> DDR3_DQ5
- U2 pad H9: (no net) -> VCC1V35
- U2 pad J2: (no net) -> GND
- U2 pad J3: (no net) -> DDR3_RAS
- U2 pad J7: (no net) -> DDR3_CLK+
- U2 pad J8: (no net) -> GND
- U2 pad K1: (no net) -> DDR3_ODT
- U2 pad K2: (no net) -> VCC1V35
- U2 pad K3: (no net) -> DDR3_CAS
- U2 pad K7: (no net) -> DDR3_CLK-
- U2 pad K8: (no net) -> VCC1V35
- U2 pad K9: (no net) -> DDR3_CKE
- U2 pad L2: (no net) -> DDR3_CS
- U2 pad L3: (no net) -> DDR3_WE
- U2 pad L7: (no net) -> DDR3_A10
- U2 pad L8: (no net) -> Net-(R81-Pad1)
- U2 pad M1: (no net) -> GND
- U2 pad M2: (no net) -> DDR3_BA0
- U2 pad M3: (no net) -> DDR3_BA2
- U2 pad M7: (no net) -> DDR3_A15
- U2 pad M8: (no net) -> DDR3_VREF
- U2 pad M9: (no net) -> GND
- U2 pad N1: (no net) -> VCC1V35
- U2 pad N2: (no net) -> DDR3_A3
- U2 pad N3: (no net) -> DDR3_A0
- U2 pad N7: (no net) -> DDR3_A12
- U2 pad N8: (no net) -> DDR3_BA1
- U2 pad N9: (no net) -> VCC1V35
- U2 pad P1: (no net) -> GND
- U2 pad P2: (no net) -> DDR3_A5
- U2 pad P3: (no net) -> DDR3_A2
- U2 pad P7: (no net) -> DDR3_A1
- U2 pad P8: (no net) -> DDR3_A4
- U2 pad P9: (no net) -> GND
- U2 pad R1: (no net) -> VCC1V35
- U2 pad R2: (no net) -> DDR3_A7
- U2 pad R3: (no net) -> DDR3_A9
- U2 pad R7: (no net) -> DDR3_A11
- U2 pad R8: (no net) -> DDR3_A6
- U2 pad R9: (no net) -> VCC1V35
- U2 pad T1: (no net) -> GND
- U2 pad T2: (no net) -> DDR3_RESET
- U2 pad T3: (no net) -> DDR3_A13
- U2 pad T7: (no net) -> DDR3_A14
- U2 pad T8: (no net) -> DDR3_A8
- U2 pad T9: (no net) -> GND
Routing:
- net (no net): track 252.7 -> 42.1 mm, vias 26 -> 6
- net /flash/FPGA_PROGRAMN: track 53.9 -> 0.00 mm, vias 1 -> 0
- net USER_PROGRAMN: track 50.1 -> 0.00 mm, vias 3 -> 0
- net GPIO10: track 30.5 -> 0.00 mm, vias 4 -> 0
- net Camera_GPIO: track 24.1 -> 0.00 mm, vias 5 -> 0
- net GPIO17: track 24.0 -> 0.00 mm, vias 3 -> 0
- net GPIO5: track 23.1 -> 0.00 mm, vias 3 -> 0
- net GPIO4: track 26.8 -> 3.93 mm, vias 3 -> 2
- net GPIO3: track 27.8 -> 5.64 mm, vias 2 -> 0
- net GPIO2: track 26.9 -> 7.39 mm, vias 3 -> 2
- net nEXTRST: track 19.1 -> 0.00 mm, vias 3 -> 0
- net GND: track 264.7 -> 283.6 mm, vias 212 -> 231
- net DSI1_D2_P: track 25.3 -> 8.20 mm, vias 2 -> 1
- net SDA0: track 17.0 -> 0.00 mm, vias 3 -> 0
- net DSI1_D2_N: track 28.2 -> 11.4 mm, vias 1 -> 0
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Other:
- board text added: "1.35V"
