File: ulx4m.kicad_pcb (KiCad board)
At the start: 6 copper layers, 55.1 x 40 mm, 218 parts, among them IC1 VSC8530XMW-04, J1 DF40C-100DP-0.4V(51), J2 DF40C-100DP-0.4V(51), J3 JTAG, SW1 SW_Push, SW2 SW_Push, U1 LFE5U-85F-6BG381C, U10 IS25LP128F-JBLE, U2 AS4C256M16D3, U3 TLV62569DBV, U4 TLV62569DBV, U5 TLV62569DBV, U6 TLV62569DBV, Y1 FNETHE025

Commit message: Routing out all FPGA needed pins
Routing:
- net DDR3_CAS: track 0.00 -> 8.83 mm, vias 0 -> 1
- net DDR3_A10: track 0.00 -> 8.37 mm, vias 0 -> 1
- net DDR3_DQS1+: track 4.54 -> 12.1 mm, vias 0 -> 1
- net DDR3_WE: track 0.00 -> 7.50 mm, vias 0 -> 1
- net DDR3_RAS: track 0.00 -> 7.35 mm, vias 0 -> 1
- net DDR3_A14: track 0.00 -> 7.27 mm, vias 0 -> 1
- net DDR3_DQ7: track 0.00 -> 7.24 mm, vias 0 -> 1
- net DDR3_DQS0-: track 7.93 -> 14.9 mm, vias 0 -> 1
- net DDR3_DQ9: track 0.00 -> 6.98 mm, vias 0 -> 1
- net DDR3_DQS1-: track 4.09 -> 11.1 mm, vias 0 -> 1
- net DDR3_DQ0: track 0.00 -> 6.91 mm, vias 0 -> 1
- net DDR3_DQ1: track 0.00 -> 6.80 mm, vias 0 -> 1
- net DDR3_DQS0+: track 7.29 -> 13.9 mm, vias 0 -> 1
- net DDR3_DQ11: track 9.21 -> 15.4 mm, vias 2 -> 4
- net DDR3_A12: track 11.6 -> 5.45 mm, vias 1 -> 0
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
Commit message: Rounting out DDR3
Routing:
- net DDR3_DQ4: track 5.09 -> 14.3 mm
- net DDR3_DQ7: track 7.24 -> 15.9 mm, vias 1 -> 2
- net DDR3_CAS: track 8.83 -> 16.2 mm
- net DDR3_DQ0: track 6.91 -> 14.2 mm
- net DDR3_CS: track 7.82 -> 14.8 mm
- net DDR3_WE: track 7.50 -> 14.2 mm
- net DDR3_RAS: track 7.35 -> 13.5 mm
- net DDR3_A3: track 1.76 -> 7.70 mm
- net DDR3_DM1: track 0.40 -> 6.13 mm
- net DDR3_BA2: track 3.58 -> 8.90 mm
- net DDR3_DQ11: track 15.4 -> 20.6 mm
- net DDR3_DQ8: track 5.83 -> 10.9 mm
- net DDR3_A0: track 5.55 -> 9.63 mm
- net DDR3_DQ10: track 9.23 -> 13.3 mm
- net DDR3_BA0: track 8.38 -> 12.2 mm
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
Commit message: More DDR3 routing
Parts:
- added AR1: 8x51R_0602_array, ecp5-dc-scm:R_Array_Convex_8x0602, F.Cu at (179.5, 84.8)
- added AR2: 8x51R_0602_array, ecp5-dc-scm:R_Array_Convex_8x0602, F.Cu at (183.6, 84.8)
- added AR3: 8x51R_0602_array, ecp5-dc-scm:R_Array_Convex_8x0602, F.Cu at (187.8, 84.8)
- added U7: TPS51200DRC, ecp5-dc-scm:VSON-10-1EP_3x3mm, F.Cu at (179.8, 90.0)
Connections:
- U1 pad G16: DDR3_A13 -> DDR3_BA2
- U1 pad T17: DDR3_A9 -> DDR3_A12
- U1 pad U19: DDR3_A12 -> DDR3_A9
- U1 pad U20: DDR3_BA2 -> DDR3_A13
Routing:
- net DDR3_A13: track 6.30 -> 28.6 mm, vias 2 -> 0
- net DDR3_A2: track 5.63 -> 27.8 mm
- net DDR3_A9: track 10.5 -> 32.4 mm
- net DDR3_A10: track 8.91 -> 30.7 mm
- net DDR3_VREF: track 1.79 -> 23.2 mm
- net DDR3_A0: track 9.63 -> 30.3 mm
- net DDR3_BA2: track 8.90 -> 29.2 mm, vias 0 -> 2
- net DDR3_A3: track 7.70 -> 27.4 mm
- net DDR3_CS: track 14.8 -> 32.4 mm
- net DDR3_WE: track 14.2 -> 31.0 mm
- net DDR3_CAS: track 16.2 -> 32.1 mm
- net DDR3_DQ4: track 14.3 -> 29.8 mm
- net DDR3_A14: track 7.90 -> 23.4 mm
- net DDR3_A11: track 8.64 -> 23.9 mm
- net DDR3_A7: track 8.15 -> 23.2 mm
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
Commit message: Initial DDR3 signals routing
Connections:
- U1 pad C20: DDR3_DQ12 -> DDR3_DQ4
- U1 pad D19: DDR3_DQ13 -> DDR3_DQ8
- U1 pad D20: DDR3_A4 -> DDR3_A2
- U1 pad E16: DDR3_A15 -> DDR3_A3
- U1 pad E18: DDR3_A8 -> DDR3_A0
- U1 pad E19: DDR3_A3 -> DDR3_BA2
- U1 pad E20: (no net) -> DDR3_DM0
- U1 pad F16: DDR3_A0 -> DDR3_CAS
- U1 pad F18: DDR3_A7 -> DDR3_CS
- U1 pad F19: DDR3_DQ15 -> DDR3_DQ14
- U1 pad F20: DDR3_A2 -> DDR3_A8
- U1 pad G16: DDR3_BA2 -> DDR3_BA1
- U1 pad G19: DDR3_DM0 -> DDR3_DQ12
- U1 pad G20: DDR3_A1 -> DDR3_CKE
- U1 pad H16: DDR3_A14 -> DDR3_WE
- U1 pad H17: DDR3_DQ11 -> DDR3_DQ3
- U1 pad H20: DDR3_DM1 -> DDR3_A4
- U1 pad J16: DDR3_A5 -> DDR3_A11
- U1 pad J17: DDR3_A6 -> DDR3_A10
- U1 pad L18: DDR3_CKE -> DDR3_A1
- U1 pad M18: DDR3_RESET -> DDR3_RAS
- U1 pad N16: DDR3_DQ0 -> DDR3_DQ7
- U1 pad N18: DDR3_CS -> DDR3_ODT
- U1 pad N19: DDR3_DQ2 -> DDR3_DQ5
- U1 pad N20: DDR3_DQ3 -> DDR3_DQ11
- U1 pad P17: DDR3_RAS -> DDR3_A12
- U1 pad P18: DDR3_BA0 -> DDR3_A14
- U1 pad P19: DDR3_ODT -> DDR3_BA0
- U1 pad P20: DDR3_DQ4 -> DDR3_DQ9
- U1 pad R16: DDR3_CAS -> DDR3_A6
- U1 pad R17: DDR3_WE -> DDR3_A15
- U1 pad R18: DDR3_DQ7 -> DDR3_DQ0
- U1 pad R20: DDR3_DQ5 -> DDR3_DQ2
- U1 pad T17: DDR3_A12 -> DDR3_A7
- U1 pad T18: DDR3_A11 -> DDR3_A5
- U1 pad T20: DDR3_BA1 -> DDR3_RESET
- U1 pad U16: DDR3_A10 -> DDR3_DM1
- U1 pad U17: DDR3_DQ9 -> DDR3_DQ15
- U1 pad U18: DDR3_DQ8 -> DDR3_DQ13
- U2 pad B8: (no net) -> DDR3_DQ14
Routing:
- net (no net): track 42.0 -> 0.00 mm, vias 6 -> 0
- net DDR3_DM1: track 5.31 -> 22.9 mm, vias 0 -> 2
- net DDR3_A4: track 6.77 -> 24.1 mm, vias 1 -> 2
- net DDR3_A5: track 14.3 -> 31.4 mm, vias 2 -> 0
- net DDR3_DQ15: track 5.40 -> 20.5 mm, vias 0 -> 2
- net DDR3_DQ13: track 4.80 -> 18.4 mm, vias 0 -> 2
- net DDR3_A8: track 10.8 -> 24.2 mm, vias 3 -> 2
- net DDR3_VREF: track 23.2 -> 10.1 mm, vias 1 -> 2
- net DDR3_A3: track 27.4 -> 40.1 mm, vias 0 -> 4
- net DDR3_DQ7: track 14.9 -> 26.7 mm
- net DDR3_A1: track 14.9 -> 26.3 mm, vias 1 -> 3
- net DDR3_DQS1-: track 8.40 -> 19.4 mm, vias 1 -> 2
- net DDR3_DQ14: track 0.00 -> 10.8 mm
- net DDR3_DQ1: track 12.7 -> 23.5 mm
- net DDR3_A11: track 23.9 -> 34.4 mm, vias 1 -> 3
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
Commit message: Improved routing
Parts:
- C200, C201, C79, C80, C81, C82, C83, C84, C85, C86, C87, C89, C90, C91, C93, C94, R81, R82, R83: moved to B.Cu
- C33: moved to F.Cu
- C78: footprint ecp5-dc-scm:0402-cap -> Capacitor_SMD:C_0402_1005Metric
- C92: footprint ecp5-dc-scm:0402-cap -> Capacitor_SMD:C_0402_1005Metric; moved to B.Cu
- moved C86 103.6 mm to (134.2, 92.2)
- moved R81 103.2 mm to (145.6, 84.5), turned to 90 degrees
- moved C200 98.0 mm to (134.0, 98.0), turned to 180 degrees
- moved C90 97.8 mm to (144.2, 97.0)
- moved C85 96.8 mm to (137.7, 87.3), turned to 90 degrees
- moved C79 96.3 mm to (135.3, 85.3), turned to 90 degrees
- moved C92 93.7 mm to (146.9, 90.5)
- moved C93 93.7 mm to (135.5, 98.5), turned to 270 degrees
- moved C87 92.2 mm to (134.1, 95.3)
- moved C91 90.9 mm to (146.9, 91.5)
- moved C80 88.6 mm to (145.8, 86.4)
- moved C81 77.9 mm to (134.3, 85.3), turned to 90 degrees
- moved C94 74.5 mm to (143.0, 87.5), turned to 180 degrees
- moved C88 74.2 mm to (138.3, 98.0), turned to 225 degrees
- moved C33 68.4 mm to (103.0, 90.9), turned to 270 degrees
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Connections:
- U1 pad D19: DDR3_DQ8 -> DDR3_A2
- U1 pad D20: DDR3_A2 -> DDR3_A0
- U1 pad E16: DDR3_A3 -> DDR3_DQ8
- U1 pad E18: DDR3_A0 -> DDR3_DM0
- U1 pad E19: DDR3_BA2 -> DDR3_A3
- U1 pad E20: DDR3_DM0 -> DDR3_BA2
- U1 pad F16: DDR3_CAS -> DDR3_DQ14
- U1 pad F18: DDR3_CS -> DDR3_DQ12
- U1 pad F19: DDR3_DQ14 -> DDR3_CAS
- U1 pad G19: DDR3_DQ12 -> DDR3_CS
- U1 pad H16: DDR3_WE -> DDR3_DQ10
- U1 pad H18: DDR3_DQ10 -> DDR3_WE
- U1 pad R16: DDR3_A6 -> DDR3_DQ15
- U1 pad T18: DDR3_A5 -> DDR3_RESET
- U1 pad T20: DDR3_RESET -> DDR3_A5
- U1 pad U17: DDR3_DQ15 -> DDR3_A6
Routing:
- net VCC1V35: track 15.0 -> 85.7 mm
- net GND: track 284.5 -> 321.3 mm, vias 229 -> 236
- net +5V: track 147.9 -> 169.6 mm, vias 13 -> 14
- net CM4_3.3V: track 134.9 -> 153.6 mm, vias 22 -> 26
- net DDR3_DQ12: track 9.74 -> 26.7 mm, vias 0 -> 4
- net DDR3_DQ14: track 10.8 -> 26.2 mm, vias 0 -> 4
- net DDR3_VREF: track 10.1 -> 21.9 mm, vias 2 -> 4
- net /flash/FLASH_SCK: track 17.1 -> 28.1 mm
- net /power/P1V35: track 0.55 -> 11.5 mm
- net DSI1_D2_P: track 10.1 -> 20.7 mm, vias 1 -> 2
- net DSI1_D3_N: track 20.6 -> 31.0 mm
- net FPDI_D1-: track 10.4 -> 20.4 mm
- net DDR3_DM0: track 12.5 -> 22.3 mm, vias 2 -> 3
- net DSI1_D3_P: track 20.2 -> 29.8 mm
- net /serdes/CLK_1_N: track 71.4 -> 61.9 mm
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