File: ulx4m.kicad_pcb (KiCad board)
At the start: 6 copper layers, 55.1 x 40 mm, 213 parts, among them IC1 VSC8530XMW-04, J1 DF40C-100DP-0.4V(51), J2 DF40C-100DP-0.4V(51), J3 JTAG, U1 LFE5U-85F-6BG381C, U10 IS25LP128F-JBLE, U2 AS4C256M16D3, U3 TLV62569DBV, U4 TLV62569DBV, U5 TLV62569DBV, U6 TLV62569DBV, Y1 FNETHE025

Commit message: Initial complete routing done
Parts:
- removed IC1: VSC8530XMW-04, VSC8530XMW-04:QFN40P600X600X90-49N-D
- added C100: C_470n_0402, Capacitor_SMD:C_0402_1005Metric, B.Cu at (98.3, 95.9)
- added C101: C_100n_0402, Capacitor_SMD:C_0402_1005Metric, F.Cu at (95.2, 101.2)
- added C102: C_470n_0402, Capacitor_SMD:C_0402_1005Metric, B.Cu at (97.3, 95.9)
- added C103: C_470n_0402, Capacitor_SMD:C_0402_1005Metric, B.Cu at (99.3, 95.9)
- added C104: C_10n_0402, Capacitor_SMD:C_0402_1005Metric, B.Cu at (100.3, 96.0)
- added C105: C_4u7_0402, Capacitor_SMD:C_0402_1005Metric, B.Cu at (102.0, 101.2)
- added C106: C_10n_0402, Capacitor_SMD:C_0402_1005Metric, B.Cu at (101.3, 95.8)
- added C107: C_470n_0402, Capacitor_SMD:C_0402_1005Metric, B.Cu at (102.0, 100.2)
- added C108: C_10n_0402, Capacitor_SMD:C_0402_1005Metric, B.Cu at (102.3, 95.3)
- added C109: C_4u7_0402, Capacitor_SMD:C_0402_1005Metric, B.Cu at (97.2, 104.3)
- added C110: C_10n_0402, Capacitor_SMD:C_0402_1005Metric, B.Cu at (102.0, 99.2)
- added C111: C_10n_0402, Capacitor_SMD:C_0402_1005Metric, B.Cu at (103.3, 95.3)
- added C112: C_10n_0402, Capacitor_SMD:C_0402_1005Metric, B.Cu at (98.2, 104.3)
- added C113: C_10n_0402, Capacitor_SMD:C_0402_1005Metric, B.Cu at (102.0, 98.2)
- added C114: C_10n_0402, Capacitor_SMD:C_0402_1005Metric, B.Cu at (104.2, 95.0)
- added C115: C_10n_0402, Capacitor_SMD:C_0402_1005Metric, B.Cu at (99.2, 104.5)
- added C116: C_10n_0402, Capacitor_SMD:C_0402_1005Metric, B.Cu at (102.0, 97.2)
- added C117: C_4u7_0402, Capacitor_SMD:C_0402_1005Metric, B.Cu at (101.4, 103.7)
- added C118: C_470n_0402, Capacitor_SMD:C_0402_1005Metric, B.Cu at (100.4, 103.7)
- added C119: C_10n_0402, Capacitor_SMD:C_0402_1005Metric, B.Cu at (102.3, 103.7)
- added C120: C_4u7_0402, Capacitor_SMD:C_0402_1005Metric, B.Cu at (97.9, 99.0)
- added C121: C_10n_0402, Capacitor_SMD:C_0402_1005Metric, B.Cu at (103.3, 103.7)
- added C122: C_100n_0402, Capacitor_SMD:C_0402_1005Metric, B.Cu at (99.6, 97.5)
- added C123: C_10n_0402, Capacitor_SMD:C_0402_1005Metric, B.Cu at (96.0, 99.0)
- added C124: C_10n_0402, Capacitor_SMD:C_0402_1005Metric, B.Cu at (99.7, 101.5)
- added C99: C_4u7_0402, Capacitor_SMD:C_0402_1005Metric, B.Cu at (96.4, 95.9)
- added FB1: BLM18PG121SN1D, Inductor_SMD:L_0603_1608Metric, B.Cu at (96.0, 104.8)
- added FB2: BLM18PG121SN1D, Inductor_SMD:L_0603_1608Metric, B.Cu at (105.3, 103.9)
- added FB3: BLM18PG121SN1D, Inductor_SMD:L_0603_1608Metric, B.Cu at (97.1, 97.7)
- added R58: R_4k7_0402, Resistor_SMD:R_0402_1005Metric, F.Cu at (95.2, 99.2)
- added R61: R_2k2_0402, Resistor_SMD:R_0402_1005Metric, F.Cu at (105.8, 93.8)
- added R65: R_12k1_0402, Resistor_SMD:R_0402_1005Metric, F.Cu at (95.2, 103.1)
- added R66: R_1k_0402, Resistor_SMD:R_0402_1005Metric, F.Cu at (107.5, 108.9)
- added R67: R_1k_0402, Resistor_SMD:R_0402_1005Metric, F.Cu at (106.2, 109.0)
- added U8: KSZ9031RNXCA, ecp5-dc-scm:QFN-48-Microchip-QFN77-48LD-PL-2, F.Cu at (100.0, 99.2)
- added U9: ASEMB-25.000MHZ-LC-T, ecp5-dc-scm:OSC_ASEM1-16.000MHZ-LC-T, B.Cu at (97.1, 101.4)
- J3: footprint Connector_PinSocket_2.54mm:PinSocket_2x03_P2.54mm_Vertical -> Connector_PinHeader_1.00mm:PinHeader_2x03_P1.00mm_Vertical_SMD
- moved R33 7.15 mm to (105.4, 100.4), turned to 270 degrees
- moved R32 7.08 mm to (104.4, 100.4), turned to 270 degrees
- moved C35 4.00 mm to (100.6, 105.2), turned to 180 degrees
- moved J3 3.66 mm to (102.0, 107.7), turned to 135 degrees
- moved TX1 0.74 mm to (147.9, 98.2)
- moved RX1 0.73 mm to (147.9, 103.3)
- moved R30 0.23 mm to (107.2, 101.9)
Connections:
- net +1V1 renamed VCC1V2
- J1 pad 17: (no net) -> ETH_nLED2
- J1 pad 19: (no net) -> ETH_nLED1
- U1 pad E6: (no net) -> ETH_MDIO
- U1 pad G5: GPIO10 -> ETH_~RESET
- U1 pad H2: ID_SC -> RGMII_REF_CLK
- U1 pad H4: (no net) -> RGMII_TX_CLK
- U1 pad H5: (no net) -> RGMII_RX_CLK
- U1 pad J1: (no net) -> RGMII_RX_DV
- U1 pad J3: (no net) -> ID_SC
- U1 pad J4: (no net) -> RGMII_TXD1
- U1 pad J5: (no net) -> ETH_MDC
- U1 pad K1: (no net) -> RGMII_RXD0
- U1 pad K2: (no net) -> RGMII_RXD1
- U1 pad K3: (no net) -> RGMII_TX_EN
- U1 pad K4: (no net) -> GPIO10
- U1 pad K5: (no net) -> RGMII_TXD0
- U1 pad L1: (no net) -> RGMII_RXD2
- U1 pad L2: (no net) -> RGMII_RXD3
- U1 pad L3: (no net) -> RGMII_TXD3
- U1 pad L4: (no net) -> RGMII_TXD2
- U1 pad L5: (no net) -> GPIO9
- U1 pad M1: GPIO9 -> ETH_INT_N
Routing:
- net VCC1V2: track 131.5 -> 180.2 mm, vias 11 -> 15
- net ETH_~RESET: track 0.00 -> 39.1 mm, vias 0 -> 2
- net GND: track 326.7 -> 361.7 mm, vias 241 -> 243
- net CM4_3.3V: track 155.9 -> 190.9 mm, vias 27 -> 33
- net RGMII_REF_CLK: track 0.00 -> 28.8 mm, vias 0 -> 2
- net ETH_0P: track 5.68 -> 32.0 mm, vias 0 -> 2
- net ETH_MDIO: track 0.00 -> 26.3 mm, vias 0 -> 2
- net /serdes/S_4_N: track 28.6 -> 3.61 mm
- net ETH_0N: track 5.01 -> 29.9 mm, vias 0 -> 2
- net RGMII_RX_CLK: track 0.00 -> 24.6 mm, vias 0 -> 4
- net /serdes/S_4_P: track 29.2 -> 5.02 mm
- net ETH_INT_N: track 0.00 -> 23.6 mm, vias 0 -> 3
- net ETH_1N: track 4.60 -> 27.7 mm, vias 0 -> 2
- net ETH_1P: track 3.65 -> 25.8 mm, vias 0 -> 2
- net /serdes/S_3_N: track 26.8 -> 5.17 mm
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Other:
- board text added: "26.01.2022. v0.0.1"
- board text removed: "25.01.2022. v0.0.1"

Commit message: fix #16
Parts:
- added R68: R_10k_0402, Resistor_SMD:R_0402_1005Metric, B.Cu at (143.9, 98.5)
- added R69: R_10k_0402, Resistor_SMD:R_0402_1005Metric, B.Cu at (145.0, 98.5)
Connections:
- U1 pad D20: DDR3_A0 -> DDR3_VREF
- U1 pad E16: DDR3_DQ8 -> DDR3_A0
- U1 pad K18: (no net) -> DDR3_DQ8
- U1 pad L19: (no net) -> DDR3_DQ1
- U1 pad M17: DDR3_DQ1 -> DDR3_DQS0-
- U1 pad N16: DDR3_DQ7 -> DDR3_DQS0+
- U1 pad N17: DDR3_DQS0+ -> DDR3_DQ7
- U1 pad P16: DDR3_DQS0- -> DDR3_VREF
Routing:
- net DDR3_VREF: track 21.8 -> 53.8 mm, vias 4 -> 7
- net DDR3_DQS0+: track 32.7 -> 36.2 mm
- net DDR3_CKE: track 32.0 -> 35.0 mm
- net DDR3_A0: track 32.9 -> 35.9 mm, vias 2 -> 3
- net DDR3_DQ12: track 32.0 -> 35.0 mm
- net DDR3_A14: track 32.2 -> 35.1 mm
- net DDR3_DQ15: track 32.2 -> 35.0 mm
- net DDR3_A15: track 32.3 -> 34.9 mm
- net DDR3_DQ8: track 32.0 -> 34.0 mm
- net DDR3_DQ1: track 32.0 -> 34.0 mm
- net DDR3_RAS: track 32.2 -> 34.0 mm
- net DDR3_DQ14: track 32.5 -> 34.1 mm
- net DDR3_A11: track 34.1 -> 35.6 mm
- net GND: track 361.7 -> 363.1 mm
- net DDR3_DQS1-: track 32.6 -> 31.4 mm
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
Commit message: Fix #17 DDR3 length matched - we should now be inside +-0.75mm
Routing:
- net DDR3_DQS1-: track 31.4 -> 35.0 mm
- net DDR3_DQ3: track 32.5 -> 35.5 mm
- net DDR3_DQ5: track 32.3 -> 35.1 mm
- net DDR3_DQ7: track 32.3 -> 35.0 mm
- net DDR3_ODT: track 32.8 -> 35.3 mm
- net DDR3_DQS1+: track 32.7 -> 35.0 mm
- net DDR3_DQ9: track 32.7 -> 35.0 mm
- net DDR3_DQ11: track 32.8 -> 35.0 mm
- net DDR3_DQ13: track 32.8 -> 35.0 mm
- net DDR3_A12: track 32.8 -> 35.0 mm
- net DDR3_DQ2: track 32.8 -> 35.0 mm
- net DDR3_DQ10: track 32.8 -> 34.9 mm
- net DDR3_A5: track 32.9 -> 35.0 mm
- net DDR3_A13: track 33.0 -> 35.0 mm
- net DDR3_A9: track 33.6 -> 35.6 mm
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
Commit message: fix #19 fix #18
Parts:
- renumbered U10 to U3, U8 to U4, U3 to U5, U4 to U6, U5 to U7, U6 to U8, U9 to Y2
Connections:
- C25 pad 1: CM4_3.3V -> VCC1V35
- C32 pad 1: CM4_3.3V -> VCC1V35
- U1 pad H14: CM4_3.3V -> VCC1V35
- U1 pad H15: CM4_3.3V -> VCC1V35
- U1 pad J15: CM4_3.3V -> VCC1V35
- U1 pad L14: CM4_3.3V -> VCC1V35
- U1 pad L15: CM4_3.3V -> VCC1V35
- U1 pad M15: CM4_3.3V -> VCC1V35
Routing:
- net VCC1V35: track 86.4 -> 117.4 mm, vias 16 -> 19
- net CM4_3.3V: track 190.9 -> 219.1 mm, vias 33 -> 31
- net DDR3_VREF: track 53.8 -> 71.1 mm
- net /serdes/S_0_P: track 29.1 -> 21.3 mm
- net /serdes/S_0_N: track 30.1 -> 22.8 mm
- net GND: track 363.1 -> 366.1 mm, vias 243 -> 240
- net GPIO16: track 42.8 -> 40.6 mm
- net +2V5: track 108.7 -> 107.6 mm
- net /flash/FPGA_DONE: track 10.3 -> 9.22 mm
- net GPIO9: track 29.5 -> 28.6 mm
- net /flash/FLASH_nCS: track 13.4 -> 13.9 mm
- net VCC1V2: track 180.2 -> 179.6 mm
Other:
- board text added: "<< Place for 1.2V"
- board text added: "Ethernet"
- board text added: "Length of lines --------- DDR3 - 34mm GPDI0 - 100mm GPDI1 - 100mm DSI0 - 100mm DSI1 - 100mm CSI0 - 100mm CSI1 - 100mm SerDes0 - 100mm SerDes1 - 100mm"
