File: ulx4m.kicad_pcb (KiCad board)
At the start: 6 copper layers, 55.5 x 40.5 mm, 239 parts, among them J1 DF40C-100DP-0.4V(51), J2 DF40C-100DP-0.4V(51), J3 JTAG, J4 Antenna, J5 SerDes, J6 GPIO>>JTAG, P1 USB_OTG, SW1 SW_DIP_x02, U1 LFE5U-85F-6BG381C, U2 IS42S16320D-6BLI, U3 IS25LP128F-JBLE, U4 LAN8720A, U5 TLV62569DBV, U6 TLV62569DBV, U7 TLV62569DBV, U8 TLV62569DBV, Y1 FNETHE025

Commit message: Updating project
Parts:
- added C57: 22n, Capacitor_SMD:C_0402_1005Metric, F.Cu at (159.1, 93.3)
- added C60: 220nF, Capacitor_SMD:C_0402_1005Metric, F.Cu at (166.8, 96.2)
- added C64: 22n, Capacitor_SMD:C_0402_1005Metric, F.Cu at (159.1, 95.3)
- added C70: 22n, Capacitor_SMD:C_0402_1005Metric, F.Cu at (159.1, 97.2)
- added C74: 22n, Capacitor_SMD:C_0402_1005Metric, F.Cu at (159.1, 99.2)
- added D14: 1N914, Diode_SMD:D_SOD-323, F.Cu at (164.7, 93.8)
- added D15: 1N914, Diode_SMD:D_SOD-323, F.Cu at (164.7, 100.7)
- added R3: 4k7, Resistor_SMD:R_0402_1005Metric, F.Cu at (164.0, 96.2)
Connections:
- BTN1 pad 1: unconnected-(BTN1-Pad1) -> Net-(BTN1-Pad1)
- BTN2 pad 1: unconnected-(BTN1-Pad1) -> Net-(BTN1-Pad1)
- BTN3 pad 1: unconnected-(BTN1-Pad1) -> Net-(BTN1-Pad1)
- J1 pad 76: (no net) -> unconnected-(J1-Pad76)
- J2 pad 4: (no net) -> unconnected-(J2-Pad4)
- J2 pad 6: (no net) -> unconnected-(J2-Pad6)
- R18 pad 1: unconnected-(BTN1-Pad1) -> Net-(BTN1-Pad1)
- R70 pad 2: unconnected-(R70-Pad2) -> Net-(R70-Pad2)
- SW1 pad 1: unconnected-(R70-Pad2) -> Net-(R70-Pad2)
- SW1 pad 2: unconnected-(R70-Pad2) -> Net-(R70-Pad2)
- TP_D8 pad 1: unconnected-(U1A-PT13B-PadD8) -> Net-(U1A-PT13B)
- TP_E9 pad 1: unconnected-(U1A-PT20B-PadE9) -> Net-(U1A-PT20B)
- U1 pad D8: unconnected-(U1A-PT13B-PadD8) -> Net-(U1A-PT13B)
- U1 pad E9: unconnected-(U1A-PT20B-PadE9) -> Net-(U1A-PT20B)
- U4 pad 4: (no net) -> unconnected-(U4-XTAL2-Pad4)
Routing:
- net unconnected-(BTN1-Pad1): track 25.6 -> 0.00 mm, vias 1 -> 0
- net Net-(BTN1-Pad1): track 0.00 -> 25.6 mm, vias 0 -> 1
- net unconnected-(R70-Pad2): track 3.23 -> 0.00 mm
- net Net-(R70-Pad2): track 0.00 -> 3.23 mm
- net unconnected-(U1A-PT20B-PadE9): track 1.67 -> 0.00 mm, vias 1 -> 0
- net Net-(U1A-PT20B): track 0.00 -> 1.67 mm, vias 0 -> 1
- net unconnected-(U1A-PT13B-PadD8): track 1.52 -> 0.00 mm, vias 1 -> 0
- net Net-(U1A-PT13B): track 0.00 -> 1.52 mm, vias 0 -> 1

Commit message: Errors cleanup
Parts:
- removed C57, C64, C70, C74: 22n, Capacitor_SMD:C_0402_1005Metric
- removed C60: 220nF, Capacitor_SMD:C_0402_1005Metric
- removed D14: 1N914, Diode_SMD:D_SOD-323
- removed R3: 4k7, Resistor_SMD:R_0402_1005Metric
- D15: moved to B.Cu
- moved D15 55.7 mm to (109.0, 99.7), turned to -90 degrees
- moved 1.1V_1 0.25 mm to (101.5, 77.3)
Connections:
- C10 pad 1: /power/P2V5 -> +2V5
- C11 pad 1: /power/P2V5 -> +2V5
- C12 pad 1: /power/P2V5 -> +2V5
- C23 pad 1: /power/P2V5 -> +2V5
- C24 pad 1: /power/P3V3 -> CM4_3.3V
- C6 pad 1: /power/P3V3 -> CM4_3.3V
- C7 pad 1: /power/P3V3 -> CM4_3.3V
- C77 pad 1: /power/P1V35 -> +1V35
- C8 pad 1: /power/P3V3 -> CM4_3.3V
- C95 pad 1: /power/P1V35 -> +1V35
- C96 pad 1: /power/P1V35 -> +1V35
- C97 pad 1: /power/P1V35 -> +1V35
- L2 pad 2: /power/P2V5 -> +2V5
- L3 pad 2: /power/P3V3 -> CM4_3.3V
- L4 pad 2: /power/P1V35 -> +1V35
- RA2 pad 1: /power/P2V5 -> +2V5
- RA3 pad 1: /power/P3V3 -> CM4_3.3V
- RA4 pad 1: /power/P1V35 -> +1V35
- RP2 pad 1: /power/P2V5 -> +2V5
- RP3 pad 1: /power/P3V3 -> CM4_3.3V
- RP4 pad 1: /power/P1V35 -> +1V35
Routing:
- net CM4_3.3V: track 234.6 -> 246.7 mm
- net +2V5: track 107.0 -> 118.6 mm
- net /power/P1V35: track 11.5 -> 0.00 mm
- net +1V35: track 20.4 -> 31.8 mm, vias 2 -> 3
- net /power/P3V3: track 11.2 -> 0.00 mm
- net /power/P2V5: track 11.0 -> 0.00 mm
- net USER_PROGRAMN: track 0.00 -> 6.90 mm, vias 0 -> 2
- net /flash/FPGA_INITN: track 6.51 -> 12.1 mm
- net /flash/FLASH_MOSI: track 28.0 -> 33.1 mm
- net /flash/FLASH_SCK: track 25.2 -> 29.8 mm
- net GPIO9: track 28.6 -> 29.9 mm
- net /flash/FPGA_PROGRAMN: track 8.22 -> 9.38 mm
- net RGMII_TX_CLK: track 14.5 -> 15.2 mm
- net PWRBTn: track 21.3 -> 20.8 mm
