File: ulx4m.kicad_pcb (KiCad board)
At the start: 6 copper layers, 55.1 x 40 mm, 271 parts, among them J1 DF40C-100DP-0.4V(51), J2 DF40C-100DP-0.4V(51), J3 JTAG, J4 Antenna, P1 USB_OTG, SW1 SW_DIP_x02, U1 LFE5U-85F-6BG381C, U2 AS4C256M16D3, U3 IS25LP128F-JBLE, U4 KSZ9031RNXCA, U5 TLV62569DBV, U6 TLV62569DBV, U7 TLV62569DBV, U8 TLV62569DBV, Y1 FNETHE025, Y2 ASEMB-25.000MHZ-LC-T

Commit message: Changing ethernet resistor value to 0R fix #54
Parts:
- R66: value 300 -> 0R
Changed lines of the file:
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@@
 			)
 		)
-		(property "Val" "300"
+		(property "Val" "0R"
 			(at 0 0 135)
 			(unlocked yes)
@@
 			)
 		)
-		(property "Value" "300"
+		(property "Value" "0R"
 			(at 0 0.374999 -45)
 			(layer "F.Fab")
@@
 			)
 		)
-		(property "Val" "300"
+		(property "Val" "0R"
 			(at 0 0 135)
 			(unlocked yes)
