File: ulx4m.kicad_pcb (KiCad board)
At the start: 6 copper layers, 55.6 x 40.6 mm, 279 parts, among them J1 DF40C-100DP-0.4V(51), J2 DF40C-100DP-0.4V(51), J3 JTAG, J4 Antenna, P1 USB_OTG, SW1 SW_DIP_x02, U1 LFE5U-85F-6BG381C, U2 AS4C256M16D3, U3 IS25LP128F-JBLE, U4 KSZ9031RNXCA, U5 TLV62569DBV, U6 TLV62569DBV, U7 TLV62569DBV, U8 TLV62569DBV, Y1 FNETHE025, Y2 ASEMB-25.000MHZ-LC-T

Commit message: Cleanup
Parts:
- removed C200, C201: 100n, Capacitor_SMD:C_0402_1005Metric
- removed C78: 4u7, Capacitor_SMD:C_0402_1005Metric
- removed R61: 2k2, Resistor_SMD:R_0402_1005Metric
Connections:
- TP_D8 pad 1: Net-(U1A-PT13B) -> PCIe_nRST
- U1 pad A9: PCIe_nRST -> unconnected-(U1A-GR_PCLK0_1-PadA9)
- U1 pad D8: Net-(U1A-PT13B) -> PCIe_nRST
Routing:
- net PCIe_nRST: track 10.3 -> 13.9 mm
- net Net-(U1A-PT13B): track 1.52 -> 0.00 mm, vias 1 -> 0
- net BTN1: track 25.5 -> 27.0 mm
- net /serdes/S_2_P: track 30.3 -> 29.7 mm
- net GND: track 409.0 -> 409.1 mm, vias 240 -> 241
