File: ddr3.sch (KiCad schematic (older format))
At the start: 36 parts, among them U10 AS4C256M16D3, U11 TPS51200DRC

Commit message: DDR3 GND and VCC
Parts:
- AR1: renamed from R124; footprint ecp5-dc-scm-footprints:R_Array_Convex_8x0602 -> ecp5-dc-scm:R_Array_Convex_8x0602
- AR2: renamed from R125; footprint ecp5-dc-scm-footprints:R_Array_Convex_8x0602 -> ecp5-dc-scm:R_Array_Convex_8x0602
- AR3: renamed from R136; footprint ecp5-dc-scm-footprints:R_Array_Convex_8x0602 -> ecp5-dc-scm:R_Array_Convex_8x0602
- C196: footprint ecp5-dc-scm-footprints:0402-res -> ecp5-dc-scm:0402-cap
- C197, C198, C199, C200, C201, C202, C240, C78, C79, C80, C81, C82, C83, C84, C85, C86, C87, C88, C89, C90, C91, C92, C93, C94: footprint ecp5-dc-scm-footprints:0402-cap -> ecp5-dc-scm:0402-cap
- R78, R79, R80, R81, R82, R83: footprint ecp5-dc-scm-footprints:0402-res -> ecp5-dc-scm:0402-res
- U2: renamed from U10; footprint ecp5-dc-scm-footprints:BGA-96_9.0x13.0mm_Layout2x3x16_P0.8mm -> AS4C256M16D3:BGA-96_9.0x13.0mm_Layout2x3x16_P0.8mm
- U7: renamed from U11; footprint ecp5-dc-scm-footprints:VSON-10-1EP_3x3mm -> ecp5-dc-scm:VSON-10-1EP_3x3mm
Connections:
- net VCC1V35 renamed +1V35
- net VCC3V3 renamed +3V3

Commit message: Improved routing
Parts:
- C78, C92: footprint ecp5-dc-scm:0402-cap -> Capacitor_SMD:C_0402_1005Metric
Changed lines of the file:
@@
 F 0 "C92" H 11350 4000 60  0000 L CNN
 F 1 "C_470n_0402" H 11325 3750 60  0001 C CNN
-F 2 "ecp5-dc-scm:0402-cap" H 11525 4100 60  0001 L CNN
+F 2 "Capacitor_SMD:C_0402_1005Metric" H 11525 4100 60  0001 L CNN
 F 3 "" H 11325 3900 50  0001 C CNN
 F 4 "TDK" H 11525 4300 60  0001 L CNN "Manufacturer"
@@
 F 0 "C78" H 9275 8900 60  0000 L CNN
 F 1 "C_10u_0402" H 9250 8650 60  0001 C CNN
-F 2 "ecp5-dc-scm:0402-cap" H 9450 9000 60  0001 L CNN
+F 2 "Capacitor_SMD:C_0402_1005Metric" H 9450 9000 60  0001 L CNN
 F 3 "" H 9250 8800 50  0001 C CNN
 F 4 "MURATA" H 9450 9200 60  0001 L CNN "Manufacturer"

Commit message: Adding 4 more LEDs - moving button
Parts:
- C196, C197, C198, C199, C200, C201, C202, C240, C79, C80, C81, C82, C83, C84, C85, C86, C87, C88, C89, C90, C91, C93, C94: footprint ecp5-dc-scm:0402-cap -> Capacitor_SMD:C_0402_1005Metric
- R78, R79, R80, R81, R82, R83: footprint ecp5-dc-scm:0402-res -> Resistor_SMD:R_0402_1005Metric
Changed lines of the file:
@@
 F 0 "C79" H 9500 3100 60  0000 L CNN
 F 1 "C_4u7_0402" H 9475 2850 60  0001 C CNN
-F 2 "ecp5-dc-scm:0402-cap" H 9675 3200 60  0001 L CNN
+F 2 "Capacitor_SMD:C_0402_1005Metric" H 9675 3200 60  0001 L CNN
 F 3 "" H 9475 3000 50  0001 C CNN
 F 4 "MURATA" H 9675 3400 60  0001 L CNN "Manufacturer"
@@
 F 0 "C80" H 9850 3100 60  0000 L CNN
 F 1 "C_470n_0402" H 9825 2850 60  0001 C CNN
-F 2 "ecp5-dc-scm:0402-cap" H 10025 3200 60  0001 L CNN
+F 2 "Capacitor_SMD:C_0402_1005Metric" H 10025 3200 60  0001 L CNN
 F 3 "" H 9825 3000 50  0001 C CNN
 F 4 "TDK" H 10025 3400 60  0001 L CNN "Manufacturer"
@@
 F 0 "C82" H 10150 3100 60  0000 L CNN
 F 1 "C_470n_0402" H 10125 2850 60  0001 C CNN
-F 2 "ecp5-dc-scm:0402-cap" H 10325 3200 60  0001 L CNN
+F 2 "Capacitor_SMD:C_0402_1005Metric" H 10325 3200 60  0001 L CNN
 F 3 "" H 10125 3000 50  0001 C CNN
 F 4 "TDK" H 10325 3400 60  0001 L CNN "Manufacturer"
@@
 F 0 "C84" H 10450 3100 60  0000 L CNN
 F 1 "C_470n_0402" H 10425 2850 60  0001 C CNN
-F 2 "ecp5-dc-scm:0402-cap" H 10625 3200 60  0001 L CNN
+F 2 "Capacitor_SMD:C_0402_1005Metric" H 10625 3200 60  0001 L CNN
 F 3 "" H 10425 3000 50  0001 C CNN
 F 4 "TDK" H 10625 3400 60  0001 L CNN "Manufacturer"
@@
 F 0 "C86" H 10750 3100 60  0000 L CNN
 F 1 "C_470n_0402" H 10725 2850 60  0001 C CNN
-F 2 "ecp5-dc-scm:0402-cap" H 10925 3200 60  0001 L CNN
+F 2 "Capacitor_SMD:C_0402_1005Metric" H 10925 3200 60  0001 L CNN
 F 3 "" H 10725 3000 50  0001 C CNN
 F 4 "TDK" H 10925 3400 60  0001 L CNN "Manufacturer"
@@
 F 0 "C89" H 11050 3100 60  0000 L CNN
 F 1 "C_470n_0402" H 11025 2850 60  0001 C CNN
-F 2 "ecp5-dc-scm:0402-cap" H 11225 3200 60  0001 L CNN
+F 2 "Capacitor_SMD:C_0402_1005Metric" H 11225 3200 60  0001 L CNN
 F 3 "" H 11025 3000 50  0001 C CNN
 F 4 "TDK" H 11225 3400 60  0001 L CNN "Manufacturer"
@@
 F 0 "C91" H 11350 3100 60  0000 L CNN
 F 1 "C_470n_0402" H 11325 2850 60  0001 C CNN
-F 2 "ecp5-dc-scm:0402-cap" H 11525 3200 60  0001 L CNN
+F 2 "Capacitor_SMD:C_0402_1005Metric" H 11525 3200 60  0001 L CNN
 F 3 "" H 11325 3000 50  0001 C CNN
 F 4 "TDK" H 11525 3400 60  0001 L CNN "Manufacturer"
@@
 F 0 "C81" H 9850 4000 60  0000 L CNN
 F 1 "C_470n_0402" H 9825 3750 60  0001 C CNN
-F 2 "ecp5-dc-scm:0402-cap" H 10025 4100 60  0001 L CNN
+F 2 "Capacitor_SMD:C_0402_1005Metric" H 10025 4100 60  0001 L CNN
 F 3 "" H 9825 3900 50  0001 C CNN
 F 4 "TDK" H 10025 4300 60  0001 L CNN "Manufacturer"
@@
 F 0 "C83" H 10150 4000 60  0000 L CNN
 F 1 "C_470n_0402" H 10125 3750 60  0001 C CNN
-F 2 "ecp5-dc-scm:0402-cap" H 10325 4100 60  0001 L CNN
+F 2 "Capacitor_SMD:C_0402_1005Metric" H 10325 4100 60  0001 L CNN
 F 3 "" H 10125 3900 50  0001 C CNN
 F 4 "TDK" H 10325 4300 60  0001 L CNN "Manufacturer"
@@
 F 0 "C85" H 10450 4000 60  0000 L CNN
 F 1 "C_470n_0402" H 10425 3750 60  0001 C CNN
-F 2 "ecp5-dc-scm:0402-cap" H 10625 4100 60  0001 L CNN
+F 2 "Capacitor_SMD:C_0402_1005Metric" H 10625 4100 60  0001 L CNN
 F 3 "" H 10425 3900 50  0001 C CNN
 F 4 "TDK" H 10625 4300 60  0001 L CNN "Manufacturer"
@@
 F 0 "C87" H 10750 4000 60  0000 L CNN
 F 1 "C_470n_0402" H 10725 3750 60  0001 C CNN
-F 2 "ecp5-dc-scm:0402-cap" H 10925 4100 60  0001 L CNN
+F 2 "Capacitor_SMD:C_0402_1005Metric" H 10925 4100 60  0001 L CNN
 F 3 "" H 10725 3900 50  0001 C CNN
 F 4 "TDK" H 10925 4300 60  0001 L CNN "Manufacturer"
@@
 F 0 "C90" H 11050 4000 60  0000 L CNN
 F 1 "C_470n_0402" H 11025 3750 60  0001 C CNN
-F 2 "ecp5-dc-scm:0402-cap" H 11225 4100 60  0001 L CNN
+F 2 "Capacitor_SMD:C_0402_1005Metric" H 11225 4100 60  0001 L CNN
 F 3 "" H 11025 3900 50  0001 C CNN
 F 4 "TDK" H 11225 4300 60  0001 L CNN "Manufacturer"
@@
 F 0 "C88" H 11000 5200 60  0000 L CNN
 F 1 "C_100n_0402" H 10975 4950 60  0001 C CNN
-F 2 "ecp5-dc-scm:0402-cap" H 11175 5300 60  0001 L CNN
+F 2 "Capacitor_SMD:C_0402_1005Metric" H 11175 5300 60  0001 L CNN
 F 3 "" H 10975 5100 50  0001 C CNN
 F 4 "Walsin" H 11175 5500 60  0001 L CNN "Manufacturer"
@@
 F 0 "C93" H 11350 5200 60  0000 L CNN
 F 1 "C_100n_0402" H 11325 4950 60  0001 C CNN
-F 2 "ecp5-dc-scm:0402-cap" H 11525 5300 60  0001 L CNN
+F 2 "Capacitor_SMD:C_0402_1005Metric" H 11525 5300 60  0001 L CNN
 F 3 "" H 11325 5100 50  0001 C CNN
 F 4 "Walsin" H 11525 5500 60  0001 L CNN "Manufacturer"
@@
 F 0 "R81" V 11630 5270 60  0000 L CNN
 F 1 "R_240R_0402" H 11675 5050 60  0001 C CNN
-F 2 "ecp5-dc-scm:0402-res" H 11875 5400 60  0001 L CNN
+F 2 "Resistor_SMD:R_0402_1005Metric" H 11875 5400 60  0001 L CNN
 F 3 "" H 11675 5200 50  0001 C CNN
 F 4 "PANASONIC" H 11875 5600 60  0001 L CNN "Manufacturer"
@@
 F 0 "C197" H 6425 7400 60  0000 L CNN
 F 1 "C_10u_0402" H 6400 7150 60  0001 C CNN
-F 2 "ecp5-dc-scm:0402-cap" H 6600 7500 60  0001 L CNN
+F 2 "Capacitor_SMD:C_0402_1005Metric" H 6600 7500 60  0001 L CNN
 F 3 "" H 6400 7300 50  0001 C CNN
 F 4 "MURATA" H 6600 7700 60  0001 L CNN "Manufacturer"
@@
 F 0 "R78" H 6050 8775 60  0000 L CNN
 F 1 "R_10k_0402" H 6000 8700 60  0001 C CNN
-F 2 "ecp5-dc-scm:0402-res" H 6200 9050 60  0001 L CNN
+F 2 "Resistor_SMD:R_0402_1005Metric" H 6200 9050 60  0001 L CNN
 F 3 "" H 6000 8850 50  0001 C CNN
 F 4 "VISHAY" H 6200 9250 60  0001 L CNN "Manufacturer"
@@
 F 0 "C198" H 6725 7400 60  0000 L CNN
 F 1 "C_10u_0402" H 6700 7150 60  0001 C CNN
-F 2 "ecp5-dc-scm:0402-cap" H 6900 7500 60  0001 L CNN
+F 2 "Capacitor_SMD:C_0402_1005Metric" H 6900 7500 60  0001 L CNN
 F 3 "" H 6700 7300 50  0001 C CNN
 F 4 "MURATA" H 6900 7700 60  0001 L CNN "Manufacturer"
@@
 F 0 "C199" H 7025 7400 60  0000 L CNN
 F 1 "C_10u_0402" H 7000 7150 60  0001 C CNN
-F 2 "ecp5-dc-scm:0402-cap" H 7200 7500 60  0001 L CNN
+F 2 "Capacitor_SMD:C_0402_1005Metric" H 7200 7500 60  0001 L CNN
 F 3 "" H 7000 7300 50  0001 C CNN
 F 4 "MURATA" H 7200 7700 60  0001 L CNN "Manufacturer"
@@
 F 0 "C202" H 8125 7400 60  0000 L CNN
 F 1 "C_100n_0402" H 8100 7150 60  0001 C CNN
-F 2 "ecp5-dc-scm:0402-cap" H 8300 7500 60  0001 L CNN
+F 2 "Capacitor_SMD:C_0402_1005Metric" H 8300 7500 60  0001 L CNN
 F 3 "" H 8100 7300 50  0001 C CNN
 F 4 "Walsin" H 8300 7700 60  0001 L CNN "Manufacturer"
@@
 F 0 "R79" V 6230 8320 60  0000 L CNN
 F 1 "R_10k_0402" H 6275 8100 60  0001 C CNN
-F 2 "ecp5-dc-scm:0402-res" H 6475 8450 60  0001 L CNN
+F 2 "Resistor_SMD:R_0402_1005Metric" H 6475 8450 60  0001 L CNN
 F 3 "" H 6275 8250 50  0001 C CNN
 F 4 "VISHAY" H 6475 8650 60  0001 L CNN "Manufacturer"
@@
 F 0 "R80" V 6880 8445 60  0000 L CNN
 F 1 "R_10k_0402" H 6925 8225 60  0001 C CNN
-F 2 "ecp5-dc-scm:0402-res" H 7125 8575 60  0001 L CNN
+F 2 "Resistor_SMD:R_0402_1005Metric" H 7125 8575 60  0001 L CNN
 F 3 "" H 6925 8375 50  0001 C CNN
 F 4 "VISHAY" H 7125 8775 60  0001 L CNN "Manufacturer"
@@
 F 0 "C240" H 8425 7400 60  0000 L CNN
 F 1 "C_100n_0402" H 8400 7150 60  0001 C CNN
-F 2 "ecp5-dc-scm:0402-cap" H 8600 7500 60  0001 L CNN
+F 2 "Capacitor_SMD:C_0402_1005Metric" H 8600 7500 60  0001 L CNN
 F 3 "" H 8400 7300 50  0001 C CNN
 F 4 "Walsin" H 8600 7700 60  0001 L CNN "Manufacturer"
@@
 F 0 "C200" H 6975 9275 60  0000 L CNN
 F 1 "C_100n_0402" H 6950 9025 60  0001 C CNN
-F 2 "ecp5-dc-scm:0402-cap" H 7150 9375 60  0001 L CNN
+F 2 "Capacitor_SMD:C_0402_1005Metric" H 7150 9375 60  0001 L CNN
 F 3 "" H 6950 9175 50  0001 C CNN
 F 4 "Walsin" H 7150 9575 60  0001 L CNN "Manufacturer"
@@
 F 0 "C201" H 7275 9275 60  0000 L CNN
 F 1 "C_100n_0402" H 7250 9025 60  0001 C CNN
-F 2 "ecp5-dc-scm:0402-cap" H 7450 9375 60  0001 L CNN
+F 2 "Capacitor_SMD:C_0402_1005Metric" H 7450 9375 60  0001 L CNN
 F 3 "" H 7250 9175 50  0001 C CNN
 F 4 "Walsin" H 7450 9575 60  0001 L CNN "Manufacturer"
@@
 F 0 "C94" V 13700 7675 60  0000 L CNN
 F 1 "C_100n_0402" H 13800 7675 60  0001 C CNN
-F 2 "ecp5-dc-scm:0402-cap" H 14000 8025 60  0001 L CNN
+F 2 "Capacitor_SMD:C_0402_1005Metric" H 14000 8025 60  0001 L CNN
 F 3 "" H 13800 7825 50  0001 C CNN
 F 4 "Walsin" H 14000 8225 60  0001 L CNN "Manufacturer"
@@
 F 0 "R82" V 13280 7695 60  0000 L CNN
 F 1 "R_51R_0402" H 13325 7475 60  0001 C CNN
-F 2 "ecp5-dc-scm:0402-res" H 13525 7825 60  0001 L CNN
+F 2 "Resistor_SMD:R_0402_1005Metric" H 13525 7825 60  0001 L CNN
 F 3 "" H 13325 7625 50  0001 C CNN
 F 4 "YAGEO" H 13525 8025 60  0001 L CNN "Manufacturer"
@@
 F 0 "R83" V 13280 8095 60  0000 L CNN
 F 1 "R_51R_0402" H 13325 7875 60  0001 C CNN
-F 2 "ecp5-dc-scm:0402-res" H 13525 8225 60  0001 L CNN
+F 2 "Resistor_SMD:R_0402_1005Metric" H 13525 8225 60  0001 L CNN
 F 3 "" H 13325 8025 50  0001 C CNN
 F 4 "YAGEO" H 13525 8425 60  0001 L CNN "Manufacturer"
@@
 F 0 "C196" H 6300 9150 60  0000 L CNN
 F 1 "C_1n_0402" H 6275 8900 60  0001 C CNN
-F 2 "ecp5-dc-scm:0402-cap" H 6475 9250 60  0001 L CNN
+F 2 "Capacitor_SMD:C_0402_1005Metric" H 6475 9250 60  0001 L CNN
 F 3 "" H 6275 9050 50  0001 C CNN
 F 4 "YAGEO" H 6475 9450 60  0001 L CNN "Manufacturer"

Commit message: Removing termination chip
Parts:
- AR1, AR2, AR3: footprint ecp5-dc-scm:R_Array_Convex_8x0602 -> (none)
- C196, C197, C198, C199, C200, C201, C202, C240: footprint Capacitor_SMD:C_0402_1005Metric -> (none)
- R78, R79, R80: footprint Resistor_SMD:R_0402_1005Metric -> (none)
- U7: footprint ecp5-dc-scm:VSON-10-1EP_3x3mm -> (none)
Changed lines of the file:
@@
 F 0 "AR1" H 4800 8422 60  0000 C CNN
 F 1 "8x51R_0602_array" H 4800 8316 60  0000 C CNN
-F 2 "ecp5-dc-scm:R_Array_Convex_8x0602" H 4625 8425 60  0001 L CNN
+F 2 "" H 4625 8425 60  0001 L CNN
 F 3 "http://industrial.panasonic.com/cdbs/www-data/pdf/AOC0000/AOC0000C14.pdf" H 4625 8525 60  0001 L CNN
 F 4 "EXB2HV510JV" H 4625 8725 60  0001 L CNN "MPN"
@@
 F 0 "AR2" H 4800 9822 60  0000 C CNN
 F 1 "8x51R_0602_array" H 4800 9716 60  0000 C CNN
-F 2 "ecp5-dc-scm:R_Array_Convex_8x0602" H 4625 9825 60  0001 L CNN
+F 2 "" H 4625 9825 60  0001 L CNN
 F 3 "http://industrial.panasonic.com/cdbs/www-data/pdf/AOC0000/AOC0000C14.pdf" H 4625 9925 60  0001 L CNN
 F 4 "EXB2HV510JV" H 4625 10125 60  0001 L CNN "MPN"
@@
 F 0 "AR3" H 4800 11222 60  0000 C CNN
 F 1 "8x51R_0602_array" H 4800 11116 60  0000 C CNN
-F 2 "ecp5-dc-scm:R_Array_Convex_8x0602" H 4625 11225 60  0001 L CNN
+F 2 "" H 4625 11225 60  0001 L CNN
 F 3 "http://industrial.panasonic.com/cdbs/www-data/pdf/AOC0000/AOC0000C14.pdf" H 4625 11325 60  0001 L CNN
 F 4 "EXB2HV510JV" H 4625 11525 60  0001 L CNN "MPN"
@@
 F 0 "C197" H 6425 7400 60  0000 L CNN
 F 1 "C_10u_0402" H 6400 7150 60  0001 C CNN
-F 2 "Capacitor_SMD:C_0402_1005Metric" H 6600 7500 60  0001 L CNN
+F 2 "" H 6600 7500 60  0001 L CNN
 F 3 "" H 6400 7300 50  0001 C CNN
 F 4 "MURATA" H 6600 7700 60  0001 L CNN "Manufacturer"
@@
 F 0 "R78" H 6050 8775 60  0000 L CNN
 F 1 "R_10k_0402" H 6000 8700 60  0001 C CNN
-F 2 "Resistor_SMD:R_0402_1005Metric" H 6200 9050 60  0001 L CNN
+F 2 "" H 6200 9050 60  0001 L CNN
 F 3 "" H 6000 8850 50  0001 C CNN
 F 4 "VISHAY" H 6200 9250 60  0001 L CNN "Manufacturer"
@@
 F 0 "C198" H 6725 7400 60  0000 L CNN
 F 1 "C_10u_0402" H 6700 7150 60  0001 C CNN
-F 2 "Capacitor_SMD:C_0402_1005Metric" H 6900 7500 60  0001 L CNN
+F 2 "" H 6900 7500 60  0001 L CNN
 F 3 "" H 6700 7300 50  0001 C CNN
 F 4 "MURATA" H 6900 7700 60  0001 L CNN "Manufacturer"
@@
 F 0 "C199" H 7025 7400 60  0000 L CNN
 F 1 "C_10u_0402" H 7000 7150 60  0001 C CNN
-F 2 "Capacitor_SMD:C_0402_1005Metric" H 7200 7500 60  0001 L CNN
+F 2 "" H 7200 7500 60  0001 L CNN
 F 3 "" H 7000 7300 50  0001 C CNN
 F 4 "MURATA" H 7200 7700 60  0001 L CNN "Manufacturer"
@@
 F 0 "C202" H 8125 7400 60  0000 L CNN
 F 1 "C_100n_0402" H 8100 7150 60  0001 C CNN
-F 2 "Capacitor_SMD:C_0402_1005Metric" H 8300 7500 60  0001 L CNN
+F 2 "" H 8300 7500 60  0001 L CNN
 F 3 "" H 8100 7300 50  0001 C CNN
 F 4 "Walsin" H 8300 7700 60  0001 L CNN "Manufacturer"
@@
 F 0 "R79" V 6230 8320 60  0000 L CNN
 F 1 "R_10k_0402" H 6275 8100 60  0001 C CNN
-F 2 "Resistor_SMD:R_0402_1005Metric" H 6475 8450 60  0001 L CNN
+F 2 "" H 6475 8450 60  0001 L CNN
 F 3 "" H 6275 8250 50  0001 C CNN
 F 4 "VISHAY" H 6475 8650 60  0001 L CNN "Manufacturer"
@@
 F 0 "R80" V 6880 8445 60  0000 L CNN
 F 1 "R_10k_0402" H 6925 8225 60  0001 C CNN
-F 2 "Resistor_SMD:R_0402_1005Metric" H 7125 8575 60  0001 L CNN
+F 2 "" H 7125 8575 60  0001 L CNN
 F 3 "" H 6925 8375 50  0001 C CNN
 F 4 "VISHAY" H 7125 8775 60  0001 L CNN "Manufacturer"
@@
 F 0 "C240" H 8425 7400 60  0000 L CNN
 F 1 "C_100n_0402" H 8400 7150 60  0001 C CNN
-F 2 "Capacitor_SMD:C_0402_1005Metric" H 8600 7500 60  0001 L CNN
+F 2 "" H 8600 7500 60  0001 L CNN
 F 3 "" H 8400 7300 50  0001 C CNN
 F 4 "Walsin" H 8600 7700 60  0001 L CNN "Manufacturer"
@@
 F 0 "C200" H 6975 9275 60  0000 L CNN
 F 1 "C_100n_0402" H 6950 9025 60  0001 C CNN
-F 2 "Capacitor_SMD:C_0402_1005Metric" H 7150 9375 60  0001 L CNN
+F 2 "" H 7150 9375 60  0001 L CNN
 F 3 "" H 6950 9175 50  0001 C CNN
 F 4 "Walsin" H 7150 9575 60  0001 L CNN "Manufacturer"
@@
 F 0 "C201" H 7275 9275 60  0000 L CNN
 F 1 "C_100n_0402" H 7250 9025 60  0001 C CNN
-F 2 "Capacitor_SMD:C_0402_1005Metric" H 7450 9375 60  0001 L CNN
+F 2 "" H 7450 9375 60  0001 L CNN
 F 3 "" H 7250 9175 50  0001 C CNN
 F 4 "Walsin" H 7450 9575 60  0001 L CNN "Manufacturer"
@@
 F 0 "U7" H 7850 9431 50  0000 C CNN
 F 1 "TPS51200DRC" H 7850 9340 50  0000 C CNN
-F 2 "ecp5-dc-scm:VSON-10-1EP_3x3mm" H 7850 9600 50  0001 C CNN
+F 2 "" H 7850 9600 50  0001 C CNN
 F 3 "" H 7850 9600 50  0001 C CNN
 	1    7850 8750
@@
 F 0 "C196" H 6300 9150 60  0000 L CNN
 F 1 "C_1n_0402" H 6275 8900 60  0001 C CNN
-F 2 "Capacitor_SMD:C_0402_1005Metric" H 6475 9250 60  0001 L CNN
+F 2 "" H 6475 9250 60  0001 L CNN
 F 3 "" H 6275 9050 50  0001 C CNN
 F 4 "YAGEO" H 6475 9450 60  0001 L CNN "Manufacturer"

Commit message: DDR3 lines are now around 10% - all GPIOs should be connected
Other:
- note added: "Not used on v001 - footprints are removed"
Changed lines of the file:
@@
 Wire Wire Line
 	8700 5475 8700 5575
+Wire Notes Line
+	3600 6525 9850 6525
+Wire Notes Line
+	9850 6525 9850 11000
+Wire Notes Line
+	9850 11000 3600 11000
+Wire Notes Line
+	3600 11000 3600 6525
+Text Notes 3600 6500 0    60   ~ 0
+Not used on v001 - footprints are removed
 $EndSCHEMATC

Commit message: fix #16
Parts:
- added R68, R69: R_10k_0402, Resistor_SMD:R_0402_1005Metric, symbol ecp5-dc-scm:R_10k_0402
Connections:
- net +1V35: now also R68.1
- net DDR3_VREF: now also R68.2, R69.1
- net GND: now also R69.2
Changed lines of the file:
@@
 Text Notes 3600 6500 0    60   ~ 0
 Not used on v001 - footprints are removed
+$Comp
+L ecp5-dc-scm:R_10k_0402 R69
+U 1 1 6443B8E5
+P 10750 6800
+F 0 "R69" V 10705 6870 60  0000 L CNN
+F 1 "R_10k_0402" H 10750 6650 60  0001 C CNN
+F 2 "Resistor_SMD:R_0402_1005Metric" H 10950 7000 60  0001 L CNN
+F 3 "" H 10750 6800 50  0001 C CNN
+F 4 "VISHAY" H 10950 7200 60  0001 L CNN "Manufacturer"
+F 5 "CRCW040210K0FKEDHP" H 10950 7100 60  0001 L CNN "MPN"
+F 6 "1k" V 10803 6870 50  0000 L CNN "Val"
+	1    10750 6800
+	0    1    1    0
+$EndComp
+$Comp
+L ecp5-dc-scm:R_10k_0402 R68
+U 1 1 6443A58A
+P 10750 6400
+F 0 "R68" V 10705 6470 60  0000 L CNN
+F 1 "R_10k_0402" H 10750 6250 60  0001 C CNN
+F 2 "Resistor_SMD:R_0402_1005Metric" H 10950 6600 60  0001 L CNN
+F 3 "" H 10750 6400 50  0001 C CNN
+F 4 "VISHAY" H 10950 6800 60  0001 L CNN "Manufacturer"
+F 5 "CRCW040210K0FKEDHP" H 10950 6700 60  0001 L CNN "MPN"
+F 6 "1k" V 10803 6470 50  0000 L CNN "Val"
+	1    10750 6400
+	0    1    1    0
+$EndComp
+Text GLabel 10625 6600 0    50   Input ~ 0
+DDR3_VREF
+Text GLabel 10750 6150 1    50   Input ~ 0
+VCC1V35
+$Comp
+L ecp5-dc-scm:GND #PWR033
+U 1 1 64471E09
+P 10750 7050
+F 0 "#PWR033" H 10750 6800 50  0001 C CNN
+F 1 "GND" H 10755 6877 50  0000 C CNN
+F 2 "" H 10750 7050 50  0001 C CNN
+F 3 "" H 10750 7050 50  0001 C CNN
+	1    10750 7050
+	1    0    0    -1
+$EndComp
+Wire Wire Line
+	10750 6150 10750 6250
+Wire Wire Line
+	10750 6550 10750 6600
+Wire Wire Line
+	10750 6950 10750 7050
+Wire Wire Line
+	10625 6600 10750 6600
+Connection ~ 10750 6600
+Wire Wire Line
+	10750 6600 10750 6650
 $EndSCHEMATC
