File: ddr3.sch (KiCad schematic (older format))
At the start: 38 parts, among them U2 AS4C256M16D3, U7 TPS51200DRC

Commit message: fix #19 fix #18
Parts:
- renumbered U7 to U10
Changed lines of the file:
@@
 	13325 7475 13175 7475
 $Comp
-L ecp5-dc-scm:TPS51200DRC U7
+L ecp5-dc-scm:TPS51200DRC U10
 U 1 1 63F37552
 P 7850 8750
-F 0 "U7" H 7850 9431 50  0000 C CNN
+F 0 "U10" H 7850 9431 50  0000 C CNN
 F 1 "TPS51200DRC" H 7850 9340 50  0000 C CNN
 F 2 "" H 7850 9600 50  0001 C CNN

Commit message: Fixing names
Parts:
- C196: value C_1n_0402 -> 1n
- C197, C198, C199, C78: value C_10u_0402 -> 10u
- C200, C201, C202, C240, C88, C93, C94: value C_100n_0402 -> 100n
- C79: value C_4u7_0402 -> 470n
- C80, C81, C82, C83, C84, C85, C86, C87, C89, C90, C91, C92: value C_470n_0402 -> 470n
- R68, R69: value R_10k_0402 -> 1K
- R78, R79, R80: value R_10k_0402 -> 10K
- R81: value R_240R_0402 -> 240R
- R82, R83: value R_51R_0402 -> 51R
Changed lines of the file:
@@
 P 9475 3000
 F 0 "C79" H 9500 3100 60  0000 L CNN
-F 1 "C_4u7_0402" H 9475 2850 60  0001 C CNN
+F 1 "470n" H 9475 2850 60  0001 C CNN
 F 2 "Capacitor_SMD:C_0402_1005Metric" H 9675 3200 60  0001 L CNN
 F 3 "" H 9475 3000 50  0001 C CNN
@@
 P 9825 3000
 F 0 "C80" H 9850 3100 60  0000 L CNN
-F 1 "C_470n_0402" H 9825 2850 60  0001 C CNN
+F 1 "470n" H 9825 2850 60  0001 C CNN
 F 2 "Capacitor_SMD:C_0402_1005Metric" H 10025 3200 60  0001 L CNN
 F 3 "" H 9825 3000 50  0001 C CNN
@@
 P 10125 3000
 F 0 "C82" H 10150 3100 60  0000 L CNN
-F 1 "C_470n_0402" H 10125 2850 60  0001 C CNN
+F 1 "470n" H 10125 2850 60  0001 C CNN
 F 2 "Capacitor_SMD:C_0402_1005Metric" H 10325 3200 60  0001 L CNN
 F 3 "" H 10125 3000 50  0001 C CNN
@@
 P 10425 3000
 F 0 "C84" H 10450 3100 60  0000 L CNN
-F 1 "C_470n_0402" H 10425 2850 60  0001 C CNN
+F 1 "470n" H 10425 2850 60  0001 C CNN
 F 2 "Capacitor_SMD:C_0402_1005Metric" H 10625 3200 60  0001 L CNN
 F 3 "" H 10425 3000 50  0001 C CNN
@@
 P 10725 3000
 F 0 "C86" H 10750 3100 60  0000 L CNN
-F 1 "C_470n_0402" H 10725 2850 60  0001 C CNN
+F 1 "470n" H 10725 2850 60  0001 C CNN
 F 2 "Capacitor_SMD:C_0402_1005Metric" H 10925 3200 60  0001 L CNN
 F 3 "" H 10725 3000 50  0001 C CNN
@@
 P 11025 3000
 F 0 "C89" H 11050 3100 60  0000 L CNN
-F 1 "C_470n_0402" H 11025 2850 60  0001 C CNN
+F 1 "470n" H 11025 2850 60  0001 C CNN
 F 2 "Capacitor_SMD:C_0402_1005Metric" H 11225 3200 60  0001 L CNN
 F 3 "" H 11025 3000 50  0001 C CNN
@@
 P 11325 3000
 F 0 "C91" H 11350 3100 60  0000 L CNN
-F 1 "C_470n_0402" H 11325 2850 60  0001 C CNN
+F 1 "470n" H 11325 2850 60  0001 C CNN
 F 2 "Capacitor_SMD:C_0402_1005Metric" H 11525 3200 60  0001 L CNN
 F 3 "" H 11325 3000 50  0001 C CNN
@@
 P 9825 3900
 F 0 "C81" H 9850 4000 60  0000 L CNN
-F 1 "C_470n_0402" H 9825 3750 60  0001 C CNN
+F 1 "470n" H 9825 3750 60  0001 C CNN
 F 2 "Capacitor_SMD:C_0402_1005Metric" H 10025 4100 60  0001 L CNN
 F 3 "" H 9825 3900 50  0001 C CNN
@@
 P 10125 3900
 F 0 "C83" H 10150 4000 60  0000 L CNN
-F 1 "C_470n_0402" H 10125 3750 60  0001 C CNN
+F 1 "470n" H 10125 3750 60  0001 C CNN
 F 2 "Capacitor_SMD:C_0402_1005Metric" H 10325 4100 60  0001 L CNN
 F 3 "" H 10125 3900 50  0001 C CNN
@@
 P 10425 3900
 F 0 "C85" H 10450 4000 60  0000 L CNN
-F 1 "C_470n_0402" H 10425 3750 60  0001 C CNN
+F 1 "470n" H 10425 3750 60  0001 C CNN
 F 2 "Capacitor_SMD:C_0402_1005Metric" H 10625 4100 60  0001 L CNN
 F 3 "" H 10425 3900 50  0001 C CNN
@@
 P 10725 3900
 F 0 "C87" H 10750 4000 60  0000 L CNN
-F 1 "C_470n_0402" H 10725 3750 60  0001 C CNN
+F 1 "470n" H 10725 3750 60  0001 C CNN
 F 2 "Capacitor_SMD:C_0402_1005Metric" H 10925 4100 60  0001 L CNN
 F 3 "" H 10725 3900 50  0001 C CNN
@@
 P 11025 3900
 F 0 "C90" H 11050 4000 60  0000 L CNN
-F 1 "C_470n_0402" H 11025 3750 60  0001 C CNN
+F 1 "470n" H 11025 3750 60  0001 C CNN
 F 2 "Capacitor_SMD:C_0402_1005Metric" H 11225 4100 60  0001 L CNN
 F 3 "" H 11025 3900 50  0001 C CNN
@@
 P 11325 3900
 F 0 "C92" H 11350 4000 60  0000 L CNN
-F 1 "C_470n_0402" H 11325 3750 60  0001 C CNN
+F 1 "470n" H 11325 3750 60  0001 C CNN
 F 2 "Capacitor_SMD:C_0402_1005Metric" H 11525 4100 60  0001 L CNN
 F 3 "" H 11325 3900 50  0001 C CNN
@@
 AR Path="/61E7DB84/6053AE48" Ref="C88"  Part="1"
 F 0 "C88" H 11000 5200 60  0000 L CNN
-F 1 "C_100n_0402" H 10975 4950 60  0001 C CNN
+F 1 "100n" H 10975 4950 60  0001 C CNN
 F 2 "Capacitor_SMD:C_0402_1005Metric" H 11175 5300 60  0001 L CNN
 F 3 "" H 10975 5100 50  0001 C CNN
@@
 AR Path="/61E7DB84/605C067B" Ref="C93"  Part="1"
 F 0 "C93" H 11350 5200 60  0000 L CNN
-F 1 "C_100n_0402" H 11325 4950 60  0001 C CNN
+F 1 "100n" H 11325 4950 60  0001 C CNN
 F 2 "Capacitor_SMD:C_0402_1005Metric" H 11525 5300 60  0001 L CNN
 F 3 "" H 11325 5100 50  0001 C CNN
@@
 P 11675 5200
 F 0 "R81" V 11630 5270 60  0000 L CNN
-F 1 "R_240R_0402" H 11675 5050 60  0001 C CNN
+F 1 "240R" H 11675 5050 60  0001 C CNN
 F 2 "Resistor_SMD:R_0402_1005Metric" H 11875 5400 60  0001 L CNN
 F 3 "" H 11675 5200 50  0001 C CNN
@@
 P 6400 7300
 F 0 "C197" H 6425 7400 60  0000 L CNN
-F 1 "C_10u_0402" H 6400 7150 60  0001 C CNN
+F 1 "10u" H 6400 7150 60  0001 C CNN
 F 2 "" H 6600 7500 60  0001 L CNN
 F 3 "" H 6400 7300 50  0001 C CNN
@@
 P 6000 8850
 F 0 "R78" H 6050 8775 60  0000 L CNN
-F 1 "R_10k_0402" H 6000 8700 60  0001 C CNN
+F 1 "10K" H 6000 8700 60  0001 C CNN
 F 2 "" H 6200 9050 60  0001 L CNN
 F 3 "" H 6000 8850 50  0001 C CNN
@@
 P 6700 7300
 F 0 "C198" H 6725 7400 60  0000 L CNN
-F 1 "C_10u_0402" H 6700 7150 60  0001 C CNN
+F 1 "10u" H 6700 7150 60  0001 C CNN
 F 2 "" H 6900 7500 60  0001 L CNN
 F 3 "" H 6700 7300 50  0001 C CNN
@@
 P 7000 7300
 F 0 "C199" H 7025 7400 60  0000 L CNN
-F 1 "C_10u_0402" H 7000 7150 60  0001 C CNN
+F 1 "10u" H 7000 7150 60  0001 C CNN
 F 2 "" H 7200 7500 60  0001 L CNN
 F 3 "" H 7000 7300 50  0001 C CNN
@@
 AR Path="/61E7DB84/60AEFC4F" Ref="C202"  Part="1"
 F 0 "C202" H 8125 7400 60  0000 L CNN
-F 1 "C_100n_0402" H 8100 7150 60  0001 C CNN
+F 1 "100n" H 8100 7150 60  0001 C CNN
 F 2 "" H 8300 7500 60  0001 L CNN
 F 3 "" H 8100 7300 50  0001 C CNN
@@
 P 6275 8250
 F 0 "R79" V 6230 8320 60  0000 L CNN
-F 1 "R_10k_0402" H 6275 8100 60  0001 C CNN
+F 1 "10K" H 6275 8100 60  0001 C CNN
 F 2 "" H 6475 8450 60  0001 L CNN
 F 3 "" H 6275 8250 50  0001 C CNN
@@
 P 6925 8375
 F 0 "R80" V 6880 8445 60  0000 L CNN
-F 1 "R_10k_0402" H 6925 8225 60  0001 C CNN
+F 1 "10K" H 6925 8225 60  0001 C CNN
 F 2 "" H 7125 8575 60  0001 L CNN
 F 3 "" H 6925 8375 50  0001 C CNN
@@
 P 9250 8800
 F 0 "C78" H 9275 8900 60  0000 L CNN
-F 1 "C_10u_0402" H 9250 8650 60  0001 C CNN
+F 1 "10u" H 9250 8650 60  0001 C CNN
 F 2 "Capacitor_SMD:C_0402_1005Metric" H 9450 9000 60  0001 L CNN
 F 3 "" H 9250 8800 50  0001 C CNN
@@
 AR Path="/61E7DB84/628665BB" Ref="C240"  Part="1"
 F 0 "C240" H 8425 7400 60  0000 L CNN
-F 1 "C_100n_0402" H 8400 7150 60  0001 C CNN
+F 1 "100n" H 8400 7150 60  0001 C CNN
 F 2 "" H 8600 7500 60  0001 L CNN
 F 3 "" H 8400 7300 50  0001 C CNN
@@
 AR Path="/61E7DB84/62867A2A" Ref="C200"  Part="1"
 F 0 "C200" H 6975 9275 60  0000 L CNN
-F 1 "C_100n_0402" H 6950 9025 60  0001 C CNN
+F 1 "100n" H 6950 9025 60  0001 C CNN
 F 2 "" H 7150 9375 60  0001 L CNN
 F 3 "" H 6950 9175 50  0001 C CNN
@@
 AR Path="/61E7DB84/62867ED9" Ref="C201"  Part="1"
 F 0 "C201" H 7275 9275 60  0000 L CNN
-F 1 "C_100n_0402" H 7250 9025 60  0001 C CNN
+F 1 "100n" H 7250 9025 60  0001 C CNN
 F 2 "" H 7450 9375 60  0001 L CNN
 F 3 "" H 7250 9175 50  0001 C CNN
@@
 AR Path="/61E7DB84/6286E330" Ref="C94"  Part="1"
 F 0 "C94" V 13700 7675 60  0000 L CNN
-F 1 "C_100n_0402" H 13800 7675 60  0001 C CNN
+F 1 "100n" H 13800 7675 60  0001 C CNN
 F 2 "Capacitor_SMD:C_0402_1005Metric" H 14000 8025 60  0001 L CNN
 F 3 "" H 13800 7825 50  0001 C CNN
@@
 P 13325 7625
 F 0 "R82" V 13280 7695 60  0000 L CNN
-F 1 "R_51R_0402" H 13325 7475 60  0001 C CNN
+F 1 "51R" H 13325 7475 60  0001 C CNN
 F 2 "Resistor_SMD:R_0402_1005Metric" H 13525 7825 60  0001 L CNN
 F 3 "" H 13325 7625 50  0001 C CNN
@@
 P 13325 8025
 F 0 "R83" V 13280 8095 60  0000 L CNN
-F 1 "R_51R_0402" H 13325 7875 60  0001 C CNN
+F 1 "51R" H 13325 7875 60  0001 C CNN
 F 2 "Resistor_SMD:R_0402_1005Metric" H 13525 8225 60  0001 L CNN
 F 3 "" H 13325 8025 50  0001 C CNN
@@
 AR Path="/61E7DB84/6FB36477" Ref="C196"  Part="1"
 F 0 "C196" H 6300 9150 60  0000 L CNN
-F 1 "C_1n_0402" H 6275 8900 60  0001 C CNN
+F 1 "1n" H 6275 8900 60  0001 C CNN
 F 2 "" H 6475 9250 60  0001 L CNN
 F 3 "" H 6275 9050 50  0001 C CNN
@@
 P 10750 6800
 F 0 "R69" V 10705 6870 60  0000 L CNN
-F 1 "R_10k_0402" H 10750 6650 60  0001 C CNN
+F 1 "1K" H 10750 6650 60  0001 C CNN
 F 2 "Resistor_SMD:R_0402_1005Metric" H 10950 7000 60  0001 L CNN
 F 3 "" H 10750 6800 50  0001 C CNN
@@
 P 10750 6400
 F 0 "R68" V 10705 6470 60  0000 L CNN
-F 1 "R_10k_0402" H 10750 6250 60  0001 C CNN
+F 1 "1K" H 10750 6250 60  0001 C CNN
 F 2 "Resistor_SMD:R_0402_1005Metric" H 10950 6600 60  0001 L CNN
 F 3 "" H 10750 6400 50  0001 C CNN

Commit message: Lowering number of unique parts fix #37
Parts:
- C78: value 10u -> 4u7; Val 10u -> 4u7
- R68, R69: value 1K -> 1k
- R78, R79, R80: value 10K -> 15k; Val 10k -> 15k
- R82, R83: value 51R -> 70; Val 51R -> 70
Changed lines of the file:
@@
 P 6000 8850
 F 0 "R78" H 6050 8775 60  0000 L CNN
-F 1 "10K" H 6000 8700 60  0001 C CNN
+F 1 "15k" H 6000 8700 60  0001 C CNN
 F 2 "" H 6200 9050 60  0001 L CNN
 F 3 "" H 6000 8850 50  0001 C CNN
 F 4 "VISHAY" H 6200 9250 60  0001 L CNN "Manufacturer"
 F 5 "CRCW040210K0FKEDHP" H 6200 9150 60  0001 L CNN "MPN"
-F 6 "10k" H 5750 8900 50  0000 L CNN "Val"
+F 6 "15k" H 5750 8900 50  0000 L CNN "Val"
 	1    6000 8850
 	-1   0    0    1
@@
 P 6275 8250
 F 0 "R79" V 6230 8320 60  0000 L CNN
-F 1 "10K" H 6275 8100 60  0001 C CNN
+F 1 "15k" H 6275 8100 60  0001 C CNN
 F 2 "" H 6475 8450 60  0001 L CNN
 F 3 "" H 6275 8250 50  0001 C CNN
 F 4 "VISHAY" H 6475 8650 60  0001 L CNN "Manufacturer"
 F 5 "CRCW040210K0FKEDHP" H 6475 8550 60  0001 L CNN "MPN"
-F 6 "10k" V 6328 8320 50  0000 L CNN "Val"
+F 6 "15k" V 6328 8320 50  0000 L CNN "Val"
 	1    6275 8250
 	0    1    1    0
@@
 P 6925 8375
 F 0 "R80" V 6880 8445 60  0000 L CNN
-F 1 "10K" H 6925 8225 60  0001 C CNN
+F 1 "15k" H 6925 8225 60  0001 C CNN
 F 2 "" H 7125 8575 60  0001 L CNN
 F 3 "" H 6925 8375 50  0001 C CNN
 F 4 "VISHAY" H 7125 8775 60  0001 L CNN "Manufacturer"
 F 5 "CRCW040210K0FKEDHP" H 7125 8675 60  0001 L CNN "MPN"
-F 6 "10k" V 6978 8445 50  0000 L CNN "Val"
+F 6 "15k" V 6978 8445 50  0000 L CNN "Val"
 	1    6925 8375
 	0    1    1    0
@@
 P 9250 8800
 F 0 "C78" H 9275 8900 60  0000 L CNN
-F 1 "10u" H 9250 8650 60  0001 C CNN
+F 1 "4u7" H 9250 8650 60  0001 C CNN
 F 2 "Capacitor_SMD:C_0402_1005Metric" H 9450 9000 60  0001 L CNN
 F 3 "" H 9250 8800 50  0001 C CNN
 F 4 "MURATA" H 9450 9200 60  0001 L CNN "Manufacturer"
 F 5 "GRM155R60J106ME44D" H 9450 9100 60  0001 L CNN "MPN"
-F 6 "10u" H 9275 8700 50  0000 L CNN "Val"
+F 6 "4u7" H 9275 8700 50  0000 L CNN "Val"
 	1    9250 8800
 	1    0    0    -1
@@
 P 13325 7625
 F 0 "R82" V 13280 7695 60  0000 L CNN
-F 1 "51R" H 13325 7475 60  0001 C CNN
+F 1 "70" H 13325 7475 60  0001 C CNN
 F 2 "Resistor_SMD:R_0402_1005Metric" H 13525 7825 60  0001 L CNN
 F 3 "" H 13325 7625 50  0001 C CNN
 F 4 "YAGEO" H 13525 8025 60  0001 L CNN "Manufacturer"
 F 5 "RC0402FR-0751RL" H 13525 7925 60  0001 L CNN "MPN"
-F 6 "51R" V 13378 7695 50  0000 L CNN "Val"
+F 6 "70" V 13378 7695 50  0000 L CNN "Val"
 	1    13325 7625
 	0    1    1    0
@@
 P 13325 8025
 F 0 "R83" V 13280 8095 60  0000 L CNN
-F 1 "51R" H 13325 7875 60  0001 C CNN
+F 1 "70" H 13325 7875 60  0001 C CNN
 F 2 "Resistor_SMD:R_0402_1005Metric" H 13525 8225 60  0001 L CNN
 F 3 "" H 13325 8025 50  0001 C CNN
 F 4 "YAGEO" H 13525 8425 60  0001 L CNN "Manufacturer"
 F 5 "RC0402FR-0751RL" H 13525 8325 60  0001 L CNN "MPN"
-F 6 "51R" V 13378 8095 50  0000 L CNN "Val"
+F 6 "70" V 13378 8095 50  0000 L CNN "Val"
 	1    13325 8025
 	0    1    1    0
@@
 P 10750 6800
 F 0 "R69" V 10705 6870 60  0000 L CNN
-F 1 "1K" H 10750 6650 60  0001 C CNN
+F 1 "1k" H 10750 6650 60  0001 C CNN
 F 2 "Resistor_SMD:R_0402_1005Metric" H 10950 7000 60  0001 L CNN
 F 3 "" H 10750 6800 50  0001 C CNN
@@
 P 10750 6400
 F 0 "R68" V 10705 6470 60  0000 L CNN
-F 1 "1K" H 10750 6250 60  0001 C CNN
+F 1 "1k" H 10750 6250 60  0001 C CNN
 F 2 "Resistor_SMD:R_0402_1005Metric" H 10950 6600 60  0001 L CNN
 F 3 "" H 10750 6400 50  0001 C CNN

Commit message: Adding SDRAM removind DDR3
Parts:
- removed AR1, AR2, AR3: 8x51R_0602_array, symbol ecp5-dc-scm:8x51R_0602_array
- removed C196: 1n, symbol ecp5-dc-scm:C_1n_0402
- removed C197, C198, C199: 10u, symbol ecp5-dc-scm:C_10u_0402
- removed C200, C201, C202, C240: 100n, symbol ecp5-dc-scm:C_100n_0402
- removed C78: 4u7, Capacitor_SMD:C_0402_1005Metric, symbol ecp5-dc-scm:C_10u_0402
- removed C79: 470n, Capacitor_SMD:C_0402_1005Metric, symbol ecp5-dc-scm:C_4u7_0402
- removed C80, C81, C82, C83, C84, C85, C86, C87, C89, C90, C91, C92: 470n, Capacitor_SMD:C_0402_1005Metric, symbol ecp5-dc-scm:C_470n_0402
- removed C88, C93, C94: 100n, Capacitor_SMD:C_0402_1005Metric, symbol ecp5-dc-scm:C_100n_0402
- removed R68, R69: 1k, Resistor_SMD:R_0402_1005Metric, symbol ecp5-dc-scm:R_10k_0402
- removed R78, R79, R80: 15k, symbol ecp5-dc-scm:R_10k_0402
- removed R81: 240R, Resistor_SMD:R_0402_1005Metric, symbol ecp5-dc-scm:R_240R_0402
- removed R82, R83: 70, Resistor_SMD:R_0402_1005Metric, symbol ecp5-dc-scm:R_51R_0402
- removed U10: TPS51200DRC, symbol ecp5-dc-scm:TPS51200DRC
- removed U2: AS4C256M16D3, AS4C256M16D3:BGA-96_9.0x13.0mm_Layout2x3x16_P0.8mm, symbol ecp5-dc-scm:AS4C256M16D3
- added C78: 2.2uF, Capacitor_SMD:C_0603_1608Metric, symbol Device:C
- added C79, C80, C81: 22nF, Capacitor_SMD:C_0402_1005Metric, symbol Device:C
- added C82: 22nF, Capacitor_SMD:C_0603_1608Metric, symbol Device:C
- added U2: IS42S16320D-6BLI, IS42S16320D:IS42S16320D-6BLI, symbol mt48lc16m16a2tg:IS42S16320D-6BLI
Connections:
- net +3V3: now also C78.1, C79.1, C80.1, C81.1, C82.1, U2.A7 (VDDQ), U2.A9 (VDD), U2.B3 (VDDQ), U2.C7 (VDDQ), U2.D3 (VDDQ), U2.E7 (VDD), U2.J9 (VDD)
- net GND: now also C78.2, C79.2, C80.2, C81.2, C82.2, U2.A1 (VSS), U2.A3 (VSSQ), U2.B7 (VSSQ), U2.C3 (VSSQ), U2.D7 (VSSQ), U2.E3 (VSS), U2.J1 (VSS)
- new net SDRAM_A0: U2.H7 (A0)
- new net SDRAM_A1: U2.H8 (A1)
- new net SDRAM_A10: U2.H9 (A10)
- new net SDRAM_A11: U2.G2 (A11)
- new net SDRAM_A12: U2.G1 (A12)
- new net SDRAM_A2: U2.J8 (A2)
- new net SDRAM_A3: U2.J7 (A3)
- new net SDRAM_A4: U2.J3 (A4)
- new net SDRAM_A5: U2.J2 (A5)
- new net SDRAM_A6: U2.H3 (A6)
- new net SDRAM_A7: U2.H2 (A7)
- new net SDRAM_A8: U2.H1 (A8)
- new net SDRAM_A9: U2.G3 (A9)
- new net SDRAM_BA0: U2.G7 (BA0)
- new net SDRAM_BA1: U2.G8 (BA1)
- new net SDRAM_CKE: U2.F3 (CKE)
- new net SDRAM_CLK: U2.F2 (CLK)
- new net SDRAM_D0: U2.A8 (DQ0)
- new net SDRAM_D1: U2.B9 (DQ1)
- new net SDRAM_D10: U2.D1 (DQ10)
- new net SDRAM_D11: U2.C2 (DQ11)
- new net SDRAM_D12: U2.C1 (DQ12)
- new net SDRAM_D13: U2.B2 (DQ13)
- new net SDRAM_D14: U2.A2 (DQ15)
- new net SDRAM_D15: U2.B1 (DQ14)
- new net SDRAM_D2: U2.B8 (DQ2)
- new net SDRAM_D3: U2.C9 (DQ3)
- new net SDRAM_D4: U2.C8 (DQ4)
- new net SDRAM_D5: U2.D9 (DQ5)
- new net SDRAM_D6: U2.D8 (DQ6)
- new net SDRAM_D7: U2.E9 (DQ7)
- new net SDRAM_D8: U2.E1 (DQ8)
- new net SDRAM_D9: U2.D2 (DQ9)
- new net SDRAM_DQM0: U2.E8 (DQML)
- new net SDRAM_DQM1: U2.F1 (DQMH)
- new net SDRAM_nCAS: U2.F7 (~CAS~)
- new net SDRAM_nCS: U2.G9 (~CS~)
- new net SDRAM_nRAS: U2.F8 (~RAS~)
- new net SDRAM_nWE: U2.F9 (~WE~)
- no-connect marks 4 -> 0
Other:
- note removed: "Not used on v001 - footprints are removed"
- note removed: "Source:Trellis board"
