File: ethernet.sch (KiCad schematic (older format))
At the start: 46 parts, among them U8 KSZ9031RNXCA, U9 ASEMB-25.000MHZ-LC-T

Commit message: fix #19 fix #18
Parts:
- renumbered U8 to U4, U9 to Y2
Changed lines of the file:
@@
 RGMII_RX_DV
 $Comp
-L ecp5-dc-scm:KSZ9031RNXCA U8
+L ecp5-dc-scm:KSZ9031RNXCA U4
 U 1 1 619D6509
 P 5400 3750
-F 0 "U8" H 5450 3825 50  0000 C CNN
+F 0 "U4" H 5450 3825 50  0000 C CNN
 F 1 "KSZ9031RNXCA" H 5800 850 50  0000 C CNN
 F 2 "ecp5-dc-scm:QFN-48-Microchip-QFN77-48LD-PL-2" H 5400 4250 50  0001 L CNN
@@
 $EndComp
 $Comp
-L ecp5-dc-scm:ASEMB-25.000MHZ-LC-T U9
+L ecp5-dc-scm:ASEMB-25.000MHZ-LC-T Y2
 U 1 1 6074CE5C
 P 8250 7225
-F 0 "U9" H 8875 7512 60  0000 C CNN
+F 0 "Y2" H 8875 7512 60  0000 C CNN
 F 1 "ASEMB-25.000MHZ-LC-T" H 8875 7406 60  0000 C CNN
 F 2 "ecp5-dc-scm:OSC_ASEM1-16.000MHZ-LC-T" H 9050 7465 60  0001 C CNN

Commit message: Chaning RGMII_RX_CLK to H2, removing H5, adding pulldown to pin 33 fix #35
Parts:
- added R?: R_4k7_0402, Resistor_SMD:R_0402_1005Metric, symbol ecp5-dc-scm:R_4k7_0402
Connections:
- net GND: now also R?.2
- net RGMII_RX_DV: now also R?.1
Changed lines of the file:
@@
 Text GLabel 13350 4225 2    60   Input ~ 0
 ETH_nLED1
+Text GLabel 2800 4725 1    50   Output ~ 0
+RGMII_RX_DV
+$Comp
+L ecp5-dc-scm:R_4k7_0402 R?
+U 1 1 62BEA1F3
+P 2800 5025
+AR Path="/5FCFE2A8/62BEA1F3" Ref="R?"  Part="1"
+AR Path="/5FC6B687/62BEA1F3" Ref="R?"  Part="1"
+AR Path="/624C566F/62BEA1F3" Ref="R?"  Part="1"
+AR Path="/60570C04/62BEA1F3" Ref="R?"  Part="1"
+AR Path="/633E0B89/62BEA1F3" Ref="R?"  Part="1"
+F 0 "R?" V 2755 5095 60  0000 L CNN
+F 1 "R_4k7_0402" H 2800 4875 60  0001 C CNN
+F 2 "Resistor_SMD:R_0402_1005Metric" H 3000 5225 60  0001 L CNN
+F 3 "" H 2800 5025 50  0001 C CNN
+F 4 "PANASONIC_ELECTRONIC_COMPONENTS" H 3000 5425 60  0001 L CNN "Manufacturer"
+F 5 "ERJ2GEJ472X" H 3000 5325 60  0001 L CNN "MPN"
+F 6 "4k7" V 2853 5095 50  0000 L CNN "Val"
+	1    2800 5025
+	0    1    1    0
+$EndComp
+$Comp
+L ecp5-dc-scm:GND #PWR?
+U 1 1 62BEA67D
+P 2800 5275
+F 0 "#PWR?" H 2800 5025 50  0001 C CNN
+F 1 "GND" H 2805 5102 50  0000 C CNN
+F 2 "" H 2800 5275 50  0001 C CNN
+F 3 "" H 2800 5275 50  0001 C CNN
+	1    2800 5275
+	1    0    0    -1
+$EndComp
+Wire Wire Line
+	2800 4725 2800 4875
+Wire Wire Line
+	2800 5175 2800 5275
 $EndSCHEMATC

Commit message: Fixing names
Parts:
- C1, C10, C18, C22, C6: value C_4u7_0402 -> 4u7
- C11, C12, C124, C13, C14, C15, C16, C17, C21, C23, C25, C5, C7, C9: value C_10n_0402 -> 10n
- C19, C2, C3, C4, C8: value C_470n_0402 -> 470n
- C24, C47: value C_100n_0402 -> 100n
- R48: value R_4k7_0402 -> 4k7
- R53, R54, R55, R56, R57, R59, R60, R62, R63, R64: value R_10k2_0402 -> 10k2
- R61: value R_2k2_0402 -> 2k2
- R65: value R_12k1_0402 -> 12k1
- R66, R67: value R_1k_0402 -> 1k
- R71: renamed from R?; value R_4k7_0402 -> 4k7

Commit message: Lowering number of unique parts fix #37
Parts:
- R66, R67: value 1k -> 300; Val 1k -> 300
Changed lines of the file:
@@
 P 13025 3875
 F 0 "R66" H 12850 3925 60  0000 C CNN
-F 1 "1k" H 13025 3725 60  0001 C CNN
+F 1 "300" H 13025 3725 60  0001 C CNN
 F 2 "Resistor_SMD:R_0402_1005Metric" H 13225 4075 60  0001 L CNN
 F 3 "" H 13025 3875 50  0001 C CNN
 F 4 "BOURNS" H 13225 4275 60  0001 L CNN "Manufacturer"
 F 5 "CR0402-FX-1001GLF" H 13225 4175 60  0001 L CNN "MPN"
-F 6 "1k" H 13175 3825 50  0000 C CNN "Val"
+F 6 "300" H 13025 3875 50  0000 C CNN "Val"
 	1    13025 3875
 	-1   0    0    -1
@@
 P 13025 4225
 F 0 "R67" H 12850 4275 60  0000 C CNN
-F 1 "1k" H 13025 4075 60  0001 C CNN
+F 1 "300" H 13025 4075 60  0001 C CNN
 F 2 "Resistor_SMD:R_0402_1005Metric" H 13225 4425 60  0001 L CNN
 F 3 "" H 13025 4225 50  0001 C CNN
 F 4 "BOURNS" H 13225 4625 60  0001 L CNN "Manufacturer"
 F 5 "CR0402-FX-1001GLF" H 13225 4525 60  0001 L CNN "MPN"
-F 6 "1k" H 13175 4175 50  0000 C CNN "Val"
+F 6 "300" H 13025 4225 50  0000 C CNN "Val"
 	1    13025 4225
 	-1   0    0    -1

Commit message: Changing Ethernet chip, connecting all gpios
Parts:
- removed C1, C10, C18, C22, C6: 4u7, Capacitor_SMD:C_0402_1005Metric, symbol ecp5-dc-scm:C_4u7_0402
- removed C11, C12, C124, C13, C14, C15, C16, C17, C21, C23, C25, C5, C7, C9: 10n, Capacitor_SMD:C_0402_1005Metric, symbol ecp5-dc-scm:C_10n_0402
- removed C19, C2, C3, C4, C8: 470n, Capacitor_SMD:C_0402_1005Metric, symbol ecp5-dc-scm:C_470n_0402
- removed C24, C47: 100n, Capacitor_SMD:C_0402_1005Metric, symbol ecp5-dc-scm:C_100n_0402
- removed FB1, FB2, FB3: BLM18PG121SN1D, Inductor_SMD:L_0603_1608Metric, symbol ecp5-dc-scm:BLM18PG121SN1D
- removed R48, R71: 4k7, Resistor_SMD:R_0402_1005Metric, symbol ecp5-dc-scm:R_4k7_0402
- removed R53, R54, R55, R56, R57, R59, R60, R62, R63, R64: 10k2, symbol ecp5-dc-scm:R_10k2_0402
- removed R61: 2k2, symbol ecp5-dc-scm:R_2k2_0402
- removed R65: 12k1, Resistor_SMD:R_0402_1005Metric, symbol ecp5-dc-scm:R_12k1_0402
- removed U4: KSZ9031RNXCA, ecp5-dc-scm:QFN-48-Microchip-QFN77-48LD-PL-2, symbol ecp5-dc-scm:KSZ9031RNXCA
- removed Y2: ASEMB-25.000MHZ-LC-T, ecp5-dc-scm:OSC_ASEM1-16.000MHZ-LC-T, symbol ecp5-dc-scm:ASEMB-25.000MHZ-LC-T
- added C83, C84, C90: 100n, Capacitor_SMD:C_0402_1005Metric, symbol Device:C_Small
- added C85: 1u1R, Capacitor_SMD:C_0603_1608Metric, symbol Device:C_Small
- added C86, C89: 10n, Capacitor_SMD:C_0402_1005Metric, symbol Device:C_Small
- added C87: 470p, Capacitor_SMD:C_0402_1005Metric, symbol Device:C_Small
- added C88: 22n, Capacitor_SMD:C_0402_1005Metric, symbol Device:C_Small
- added FB1: 30R, Inductor_SMD:L_0603_1608Metric, symbol Device:Ferrite_Bead_Small
- added R53: 10K, Resistor_SMD:R_0402_1005Metric, symbol Device:R_Small
- added R54, R56, R58, R60: 10R, Resistor_SMD:R_0402_1005Metric, symbol Device:R_Small
- added R55, R57: 1K5, Resistor_SMD:R_0402_1005Metric, symbol Device:R_Small
- added R59: 33R, Resistor_SMD:R_0402_1005Metric, symbol Device:R_Small
- added R63: 12K1, Resistor_SMD:R_0402_1005Metric, symbol Device:R_Small
- added U4: LAN8720A, Package_DFN_QFN:QFN-24-1EP_4x4mm_P0.5mm_EP2.6x2.6mm, symbol Interface_Ethernet:LAN8720A
- renumbered R66 to R61, R67 to R62
Connections:
- net +3V3: now also C84.1, FB1.1, R53.1, R54.2, R55.1, R57.1, U4.9 (VDDIO)
- net ETH_0N: now also U4.20 (TXN)
- net ETH_0P: now also U4.21 (TXP)
- net ETH_1N: now also U4.22 (RXN)
- net ETH_1P: now also U4.23 (RXP)
- net ETH_MDC: now also U4.13 (MDC)
- net ETH_MDIO: now also R57.2, U4.12 (MDIO)
- net ETH_~RESET: now also C83.2, R53.2, U4.15 (RST)
- net GND: now also C83.1, C84.2, C85.2, C86.2, C87.2, C88.2, C89.2, C90.2, R63.2, U4.25 (VSS)
- net RGMII_REF_CLK: now also U4.14 (INT/REFCLKO)
- net RGMII_RXD0: now also R60.2
- net RGMII_RXD1: now also R56.2
- net RGMII_RX_DV: now also R55.2, R58.1
- net RGMII_TXD0: now also U4.17 (TXD0)
- net RGMII_TXD1: now also U4.18 (TXD1)
- net RGMII_TX_CLK: now also R59.2
- net RGMII_TX_EN: now also U4.16 (TXEN)
- net ETH_LED1 renamed ACTLED
- net ACTLED: now also U4.3 (LED1/REGOFF)
- net ETH_LED2 renamed LINKLED
- net LINKLED: now also U4.2 (LED2/nINTSEL)
- new net: R54.1, U4.10 (RXER/PHYAD0)
- new net: R58.2, U4.11 (CRS_DV/MODE2)
- new net: R56.1, U4.7 (RXD1/MODE1)
- new net: R60.1, U4.8 (RXD0/MODE0)
- new net +3.3VA: C86.1, C88.1, C90.1, FB1.2, U4.1 (VDD2A), U4.19 (VDD1A)
- new net RBIAS: R63.1, U4.24 (RBIAS)
- new net VDDCR: C85.1, C87.1, C89.1, U4.6 (VDDCR)
- new net XTAL: R59.1, U4.5 (XTAL1/CLKIN)
- no-connect marks 2 -> 1
Other:
- note removed: "Pull up resistors - we will try internal"
- moved on the sheet: R61, R62
