File: flash.kicad_sch (KiCad schematic)
At the start: 13 parts, among them U1 LFE5U-85F-6BG381C, U3 IS25LP128F-JBLE

Commit message: Before graphical cleanup
Parts:
- added C99: 100n, Capacitor_SMD:C_0402_1005Metric, symbol Device:C_Small
- D28: footprint (none) -> Diode_SMD:D_SOD-323
Connections:
- net +3V3: now also C99.2
- net FPGA_PROGRAMN: now also C99.1
