File: flash.kicad_sch (KiCad schematic)
At the start: 14 parts, among them U1 LFE5U-85F-6BG381C, U3 IS25LP128F-JBLE

Commit message: Updating schematics
Parts:
- D15: renamed from D29; footprint (none) -> Diode_SMD:D_SOD-323
- U1: Digike_y2 (none) -> 220-2071-ND; Digikey (none) -> 220-2177-ND; Koncar (none) -> FU004; LCSC (none) -> C446029; LowCost (none) -> 842-LFE5U12F6BG381C; MFG1 (none) -> Lattice; MFG2 (none) -> Lattice; MNF1_URL (none) -> www.latticesemi.com; MNF2_URL (none) -> www.latticesemi.com; MP_N2 (none) -> LFE5U-12F-6BG381C; Mouser (none) -> 842-LFE5U85F6BG381C; Mouser_URL (none) -> www.mouser.com; Side (none) -> T; price100_Mouse (none) -> 22.82$

Commit message: initial ULX4M-Ls v004
Parts:
- D28: footprint Diode_SMD:D_SOD-323 -> (none)
Changed lines of the file:
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@@
 			)
 		)
-		(property "Footprint" "Diode_SMD:D_SOD-323"
+		(property "Footprint" ""
 			(at 127 86.36 0)
 			(effects

Commit message: Cleanup
Parts:
- D28: footprint (none) -> Diode_SMD:D_SOD-323
Changed lines of the file:
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@@
 			)
 		)
-		(property "Footprint" ""
+		(property "Footprint" "Diode_SMD:D_SOD-323"
 			(at 127 86.36 0)
 			(effects
