File: gpdi.kicad_sch (KiCad schematic)
At the start: 45 parts, among them SW1 SW_DIP_x02, U1 LFE5U-85F-6BG381C

Commit message: Before graphical cleanup
Parts:
- renumbered TP_D16 to TP_C?, TP_C16 to TP_D?
Changed lines of the file:
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@@
 		(pin "1"
+		)
+		(instances
+			(project ""
+				(path "/1876dd7c-56e8-4d11-a76e-0d3f3f8be70a/00000000-0000-0000-0000-000058d686d9"
+					(reference "#PWR0101")
+					(unit 1)
+				)
+			)
 		)
 	)
@@
 		(pin "1"
 		)
+		(instances
+			(project ""
+				(path "/1876dd7c-56e8-4d11-a76e-0d3f3f8be70a/00000000-0000-0000-0000-000058d686d9"
+					(reference "#PWR0102")
+					(unit 1)
+				)
+			)
+		)
 	)
 	(symbol
@@
 		(on_board yes)
 		(dnp no)
-		(property "Reference" "#PWR0103"
+		(property "Reference" "#PWR?"
 			(at 180.34 93.98 0)
 			(effects
@@
 		(on_board yes)
 		(dnp no)
-		(property "Reference" "#PWR0104"
+		(property "Reference" "#PWR?"
 			(at 229.87 93.98 0)
 			(effects
@@
 		(on_board yes)
 		(dnp no)
-		(property "Reference" "#PWR0105"
+		(property "Reference" "#PWR?"
 			(at 210.82 114.3 0)
 			(effects
@@
 		(on_board yes)
 		(dnp no)
-		(property "Reference" "TP_C16"
+		(property "Reference" "TP_D?"
 			(at 61.595 66.04 0)
 			(effects
@@
 		(on_board yes)
 		(dnp no)
-		(property "Reference" "TP_D16"
+		(property "Reference" "TP_C?"
 			(at 121.285 66.04 0)
 			(effects
@@
 		(pin "1"
 		)
+		(instances
+			(project ""
+				(path "/1876dd7c-56e8-4d11-a76e-0d3f3f8be70a/00000000-0000-0000-0000-000058d686d9"
+					(reference "#PWR010")
+					(unit 1)
+				)
+			)
+		)
 	)
 	(symbol
@@
 		(on_board yes)
 		(dnp no)
-		(property "Reference" "#PWR0145"
+		(property "Reference" "#PWR?"
 			(at 129.54 121.285 0)
 			(effects
