File: gpdi.kicad_sch (KiCad schematic)
At the start: 45 parts, among them SW1 SW_DIP_x02, U1 LFE5U-85F-6BG381C

Commit message: Updating schematics
Parts:
- U1: Digike_y2 (none) -> 220-2071-ND; Digikey (none) -> 220-2177-ND; Koncar (none) -> FU004; LCSC (none) -> C446029; LowCost (none) -> 842-LFE5U12F6BG381C; MFG1 (none) -> Lattice; MFG2 (none) -> Lattice; MNF1_URL (none) -> www.latticesemi.com; MNF2_URL (none) -> www.latticesemi.com; MP_N2 (none) -> LFE5U-12F-6BG381C; Mouser (none) -> 842-LFE5U85F6BG381C; Side (none) -> T; price100_Mouse (none) -> 22.82$
