File: gpdi.kicad_sch (KiCad schematic)
At the start: 45 parts, among them SW1 SW_DIP_x02, U1 LFE5U-85F-6BG381C

Commit message: fix #44
Other:
- company: EMARD -> Intergalaktik d.o.o.
- title: ULX3S -> ULX4M-LD
Changed lines of the file:
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@@
 	(paper "A4")
 	(title_block
-		(title "ULX3S")
-		(rev "1.0.5")
-		(company "EMARD")
+		(title "ULX4M-LD")
+		(date "2025-03-12")
+		(rev "0.0.3")
+		(company "Intergalaktik d.o.o.")
 		(comment 1 "General Purpose Differential Interface")
 		(comment 2 "License: CERN-OHL-S v2")

Commit message: fix #50
Connections:
- net SD_D0 renamed SD_DAT0
- net SD_D1 renamed SD_DAT1
- net SD_D2 renamed SD_DAT2
Changed lines of the file:
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@@
+	(wire
+		(pts
+			(xy 60.96 73.66) (xy 72.39 73.66)
+		)
+		(stroke
+			(width 0)
+			(type default)
+		)
+	)
 	(wire
 		(pts
@@
 	(wire
 		(pts
+			(xy 121.92 60.96) (xy 110.49 60.96)
+		)
+		(stroke
+			(width 0)
+			(type default)
+		)
+	)
+	(wire
+		(pts
 			(xy 185.42 93.98) (xy 190.5 93.98)
 		)
@@
 		(pts
 			(xy 69.85 55.88) (xy 72.39 55.88)
+		)
+		(stroke
+			(width 0)
+			(type default)
+		)
+	)
+	(wire
+		(pts
+			(xy 120.65 76.2) (xy 110.49 76.2)
 		)
 		(stroke
@@
 		)
 	)
+	(label "SD_D1"
+		(at 113.03 60.96 0)
+		(effects
+			(font
+				(size 1.524 1.524)
+			)
+			(justify left bottom)
+		)
+	)
+	(label "SD_D2"
+		(at 111.76 76.2 0)
+		(effects
+			(font
+				(size 1.524 1.524)
+			)
+			(justify left bottom)
+		)
+	)
+	(label "SD_D0"
+		(at 63.5 73.66 0)
+		(effects
+			(font
+				(size 1.524 1.524)
+			)
+			(justify left bottom)
+		)
+	)
 	(global_label "SW2"
 		(shape input)
@@
 		)
 	)
-	(global_label "SD_D0"
-		(shape input)
-		(at 72.39 73.66 180)
+	(global_label "SD_DAT0"
+		(shape input)
+		(at 60.96 73.66 180)
 		(effects
 			(font
@@
 		)
 		(property "Intersheetrefs" "${INTERSHEET_REFS}"
-			(at 72.39 73.66 0)
+			(at 60.96 73.66 0)
 			(effects
 				(font
@@
 		)
 	)
+	(global_label "SD_DAT2"
+		(shape input)
+		(at 120.65 76.2 0)
+		(effects
+			(font
+				(size 1.524 1.524)
+			)
+			(justify left)
+		)
+		(property "Intersheetrefs" "${INTERSHEET_REFS}"
+			(at 120.65 76.2 0)
+			(effects
+				(font
+					(size 1.27 1.27)
+				)
+				(hide yes)
+			)
+		)
+	)
 	(global_label "DSI0_D0_P"
 		(shape input)
@@
 		)
 	)
-	(global_label "SD_D1"
-		(shape input)
-		(at 110.49 60.96 0)
-		(effects
-			(font
-				(size 1.524 1.524)
-			)
-			(justify left)
-		)
-		(property "Intersheetrefs" "${INTERSHEET_REFS}"
-			(at 110.49 60.96 0)
+	(global_label "SD_DAT1"
+		(shape input)
+		(at 121.92 60.96 0)
+		(effects
+			(font
+				(size 1.524 1.524)
+			)
+			(justify left)
+		)
+		(property "Intersheetrefs" "${INTERSHEET_REFS}"
+			(at 121.92 60.96 0)
 			(effects
 				(font
@@
 			(effects
 				(font
-					(size 1.27 1.27)
-				)
-				(hide yes)
-			)
-		)
-	)
-	(global_label "SD_D2"
-		(shape input)
-		(at 110.49 76.2 0)
-		(effects
-			(font
-				(size 1.524 1.524)
-			)
-			(justify left)
-		)
-		(property "Intersheetrefs" "${INTERSHEET_REFS}"
-			(at 110.49 76.2 0)
-			(effects
-				(font

Commit message: Cleanup
Connections:
- no-connect marks 3 -> 11
Changed lines of the file:
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@@
+	)
+	(no_connect
+		(at 110.49 63.5)
 	)
 	(no_connect
@@
 	)
 	(no_connect
+		(at 110.49 91.44)
+	)
+	(no_connect
 		(at 110.49 93.98)
+	)
+	(no_connect
+		(at 72.39 63.5)
+	)
+	(no_connect
+		(at 72.39 71.12)
+	)
+	(no_connect
+		(at 72.39 91.44)
+	)
+	(no_connect
+		(at 110.49 73.66)
+	)
+	(no_connect
+		(at 72.39 68.58)
+	)
+	(no_connect
+		(at 110.49 68.58)
 	)
 	(wire
@@
 			(effects
 				(font
-					(size 1.27 1.27)
-				)
-				(hide yes)
-			)
-		)
-	)
-	(global_label "nEXTRST"
-		(shape input)
-		(at 60.96 138.43 180)
-		(effects
-			(font
-				(size 1.524 1.524)
-			)
-			(justify right)
-		)
-		(property "Intersheetrefs" "${INTERSHEET_REFS}"
-			(at 60.96 138.43 0)
-			(effects
-				(font

Commit message: Improving schematics
Other:
- company: Intergalaktik d.o.o. -> ${project_creator}
- title: ULX4M-LD -> ${project_name}
Changed lines of the file:
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@@
 	(paper "A4")
 	(title_block
-		(title "ULX4M-LD")
+		(title "${project_name}")
 		(date "2025-03-12")
-		(rev "0.0.3")
-		(company "Intergalaktik d.o.o.")
+		(rev "${project_version}")
+		(company "${project_creator}")
 		(comment 1 "General Purpose Differential Interface")
-		(comment 2 "License: CERN-OHL-S v2")
+		(comment 2 "License: ${project_license}")
 	)
 	(junction
