File: gpio.kicad_sch (KiCad schematic)
At the start: 7 parts, among them J1 DF40C-100DP-0.4V(51), J2 DF40C-100DP-0.4V(51), U1 LFE5U-85F-6BG381C

Commit message: fix #44
Other:
- company: EMARD -> Intergalaktik d.o.o.
- title: ULX3S -> ULX4M-LD
Changed lines of the file:
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@@
 	(paper "A4")
 	(title_block
-		(title "ULX3S")
-		(rev "1.0.2")
-		(company "EMARD")
+		(title "ULX4M-LD")
+		(date "2025-03-12")
+		(rev "0.0.3")
+		(company "Intergalaktik d.o.o.")
 		(comment 1 "GPIO 2.54 mm connectors")
 		(comment 2 "License: CERN-OHL-S v2")

Commit message: fix #50
Changed lines of the file:
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@@
 	(wire
 		(pts
-			(xy 134.62 105.41) (xy 136.525 105.41)
+			(xy 93.98 166.37) (xy 106.68 166.37)
 		)
 		(stroke
@@
 	(wire
 		(pts
-			(xy 134.62 102.87) (xy 136.525 102.87)
+			(xy 92.71 163.83) (xy 106.68 163.83)
 		)
 		(stroke
@@
 	(wire
 		(pts
-			(xy 134.62 95.25) (xy 136.525 95.25)
+			(xy 93.98 156.21) (xy 106.68 156.21)
 		)
 		(stroke
@@
 	(wire
 		(pts
-			(xy 136.525 100.33) (xy 134.62 100.33)
+			(xy 106.68 161.29) (xy 93.98 161.29)
 		)
 		(stroke
@@
 	(wire
 		(pts
-			(xy 135.255 92.71) (xy 136.525 92.71)
+			(xy 94.615 153.67) (xy 106.68 153.67)
 		)
 		(stroke
@@
 	(wire
 		(pts
-			(xy 134.62 97.79) (xy 136.525 97.79)
+			(xy 93.98 158.75) (xy 106.68 158.75)
 		)
 		(stroke
@@
 		)
 	)
+	(label "SD_D3"
+		(at 96.52 156.21 0)
+		(effects
+			(font
+				(size 1.524 1.524)
+			)
+			(justify left bottom)
+		)
+	)
+	(label "SD_CMD"
+		(at 96.52 166.37 0)
+		(effects
+			(font
+				(size 1.524 1.524)
+			)
+			(justify left bottom)
+		)
+	)
+	(label "SD_D2"
+		(at 96.52 163.83 0)
+		(effects
+			(font
+				(size 1.524 1.524)
+			)
+			(justify left bottom)
+		)
+	)
 	(label "CAM0_D0_LP"
 		(at 48.26 82.55 180)
@@
 		)
 	)
+	(label "SD_CLK"
+		(at 96.52 153.67 0)
+		(effects
+			(font
+				(size 1.524 1.524)
+			)
+			(justify left bottom)
+		)
+	)
+	(label "SD_D0"
+		(at 96.52 158.75 0)
+		(effects
+			(font
+				(size 1.524 1.524)
+			)
+			(justify left bottom)
+		)
+	)
+	(label "SD_D1"
+		(at 96.52 161.29 0)
+		(effects
+			(font
+				(size 1.524 1.524)
+			)
+			(justify left bottom)
+		)
+	)
 	(global_label "USB_OTG_ID"
 		(shape input)
@@
 	(global_label "SD_CMD"
 		(shape input)
-		(at 136.525 105.41 0)
+		(at 106.68 166.37 0)
 		(effects
 			(font
@@
 		)
 		(property "Intersheetrefs" "${INTERSHEET_REFS}"
-			(at 136.525 105.41 0)
+			(at 106.68 166.37 0)
 			(effects
 				(font
@@
 	(global_label "SD_CLK"
 		(shape input)
-		(at 136.525 92.71 0)
+		(at 106.68 153.67 0)
 		(effects
 			(font
@@
 		)
 		(property "Intersheetrefs" "${INTERSHEET_REFS}"
-			(at 136.525 92.71 0)
+			(at 106.68 153.67 0)
 			(effects
 				(font
@@
 	(global_label "SD_DAT0"
 		(shape input)
-		(at 136.525 97.79 0)
+		(at 106.68 158.75 0)
 		(effects
 			(font
@@
 		)
 		(property "Intersheetrefs" "${INTERSHEET_REFS}"
-			(at 136.525 97.79 0)
+			(at 106.68 158.75 0)
 			(effects
 				(font
@@
 	(global_label "SD_DAT1"
 		(shape input)
-		(at 136.525 100.33 0)
+		(at 106.68 161.29 0)
 		(effects
 			(font
@@
 		)
 		(property "Intersheetrefs" "${INTERSHEET_REFS}"
-			(at 136.525 100.33 0)
+			(at 106.68 161.29 0)
 			(effects
 				(font
@@
 	(global_label "GPIO14"
 		(shape input)
-		(at 134.62 95.25 180)
+		(at 93.98 156.21 180)
 		(effects
 			(font
@@
 		)
 		(property "Intersheetrefs" "${INTERSHEET_REFS}"
-			(at 134.62 95.25 0)
+			(at 93.98 156.21 0)
 			(effects
 				(font
@@
 	(global_label "SD_DAT2"
 		(shape input)
-		(at 136.525 102.87 0)
+		(at 106.68 163.83 0)
 		(effects
 			(font
@@
 		)
 		(property "Intersheetrefs" "${INTERSHEET_REFS}"
-			(at 136.525 102.87 0)
+			(at 106.68 163.83 0)
 			(effects
 				(font
@@
 	(global_label "GPIO2"
 		(shape input)
-		(at 134.62 102.87 180)
+		(at 92.71 163.83 180)
 		(effects
 			(font
@@
 		)
 		(property "Intersheetrefs" "${INTERSHEET_REFS}"
-			(at 134.62 102.87 0)
+			(at 92.71 163.83 0)
 			(effects
 				(font
@@
 	(global_label "GPIO3"
 		(shape input)
-		(at 134.62 100.33 180)
+		(at 93.98 161.29 180)
 		(effects
 			(font
@@
 		)
 		(property "Intersheetrefs" "${INTERSHEET_REFS}"
-			(at 134.62 100.33 0)
+			(at 93.98 161.29 0)
 			(effects
 				(font
@@
 	(global_label "SD_DAT3"
 		(shape input)
-		(at 136.525 95.25 0)
+		(at 106.68 156.21 0)
 		(effects
 			(font
@@
 		)
 		(property "Intersheetrefs" "${INTERSHEET_REFS}"
-			(at 136.525 95.25 0)
+			(at 106.68 156.21 0)
 			(effects
 				(font
@@
 	(global_label "GPIO4"
 		(shape input)
-		(at 134.62 97.79 180)
+		(at 93.98 158.75 180)
 		(effects
 			(font
@@
 		)
 		(property "Intersheetrefs" "${INTERSHEET_REFS}"
-			(at 134.62 97.79 0)
+			(at 93.98 158.75 0)
 			(effects
 				(font
@@
 	(global_label "GPIO27"
 		(shape input)
-		(at 134.62 105.41 180)
+		(at 93.98 166.37 180)
 		(effects
 			(font
@@
 		)
 		(property "Intersheetrefs" "${INTERSHEET_REFS}"
-			(at 134.62 105.41 0)
+			(at 93.98 166.37 0)
 			(effects
 				(font
@@
 	(global_label "GPIO15"
 		(shape input)
-		(at 135.255 92.71 180)
+		(at 94.615 153.67 180)
 		(effects
 			(font
@@
 		)
 		(property "Intersheetrefs" "${INTERSHEET_REFS}"
-			(at 135.255 92.71 0)
+			(at 94.615 153.67 0)
 			(effects
 				(font

Commit message: Cleanup
Connections:
- net PCIe_nRST: now also TP_D8.1, U1.D8 (PT13B); no longer U1.A9 (GR_PCLK0_1)
- no-connect marks 3 -> 16
Other:
- moved on the sheet: R21, TP_D8, TP_E8, TP_E9, U1A, U1F

Commit message: Improving schematics
Other:
- company: Intergalaktik d.o.o. -> ${project_creator}
- title: ULX4M-LD -> ${project_name}
Changed lines of the file:
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@@
 	(paper "A4")
 	(title_block
-		(title "ULX4M-LD")
+		(title "${project_name}")
 		(date "2025-03-12")
-		(rev "0.0.3")
-		(company "Intergalaktik d.o.o.")
+		(rev "${project_version}")
+		(company "${project_creator}")
 		(comment 1 "GPIO 2.54 mm connectors")
-		(comment 2 "License: CERN-OHL-S v2")
+		(comment 2 "License: ${project_license}")
 	)
 	(junction
