File: power.kicad_sch (KiCad schematic)
At the start: 68 parts, among them U1 LFE5U-85F-6BG381C, U5 TLV62569DBV, U6 TLV62569DBV, U7 TLV62569DBV, U8 TLV62569DBV

Commit message: Before graphical cleanup
Parts:
- renumbered C39 to C30, C14 to C31, C13 to C32, C38 to C47, C60 to C?, C76 to C?, C77 to C?, C95 to C?, C96 to C?, C98 to C?, C97 to C?, RA4 to RA?, RC2 to RB?, RB4 to RB?, RC1 to RC?
