File: power.kicad_sch (KiCad schematic)
At the start: 68 parts, among them U1 LFE5U-85F-6BG381C, U5 TLV62569DBV, U6 TLV62569DBV, U7 TLV62569DBV, U8 TLV62569DBV

Commit message: Updating schematics
Parts:
- C?: footprint (none) -> Capacitor_SMD:C_0402_1005Metric
- D14: renamed from D17; footprint (none) -> Diode_SMD:D_SOD-323
- R3: footprint (none) -> Resistor_SMD:R_0402_1005Metric
- U1: Digike_y2 (none) -> 220-2071-ND; Digikey (none) -> 220-2177-ND; Koncar (none) -> FU004; LCSC (none) -> C446029; LowCost (none) -> 842-LFE5U12F6BG381C; MFG1 (none) -> Lattice; MFG2 (none) -> Lattice; MNF2_URL (none) -> www.latticesemi.com; MP_N2 (none) -> LFE5U-12F-6BG381C; Mouser (none) -> 842-LFE5U85F6BG381C; Mouser_URL (none) -> www.mouser.com; Side (none) -> T; price100_Mouse (none) -> 22.82$
Other:
- moved on the sheet: 1.1V_1, C25, C26, C27, C28, C29, C30, C31, C32, C48, C49, C50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

Commit message: Errors cleanup
Parts:
- C?: footprint Capacitor_SMD:C_0402_1005Metric -> (none)
- D14: footprint Diode_SMD:D_SOD-323 -> (none)
- R3: footprint Resistor_SMD:R_0402_1005Metric -> (none)
Connections:
- net P1V35 is gone; now on net +1V35: C?.1, C?.1, C?.1, C?.1, L4.2, RA?.1, RP4.1
- net P2V5 is gone; now on net +2V5: C10.1, C11.1, C12.1, C23.1, L2.2, RA2.1, RP2.1
- net P3V3 is gone; now on net +3V3: C24.1, C6.1, C7.1, C8.1, L3.2, RA3.1, RP3.1
Other:
- moved on the sheet: C?, L4, RA?, RB?, RP4, U8

Commit message: Cleanup
Parts:
- C?, D14, R3: now not fitted; now left out of the parts list
Changed lines of the file:
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@@
 		(at 72.39 94.615 270)
 		(unit 1)
-		(exclude_from_sim no)
-		(in_bom yes)
-		(on_board yes)
-		(dnp no)
+		(exclude_from_sim yes)
+		(in_bom no)
+		(on_board no)
+		(dnp yes)
 		(property "Reference" "R3"
 			(at 72.39 97.155 90)
@@
 		(at 72.39 88.265 0)
 		(unit 1)
-		(exclude_from_sim no)
-		(in_bom yes)
-		(on_board yes)
-		(dnp no)
+		(exclude_from_sim yes)
+		(in_bom no)
+		(on_board no)
+		(dnp yes)
 		(property "Reference" "D14"
 			(at 72.39 90.805 0)
@@
 		(at 48.26 103.505 270)
 		(unit 1)
-		(exclude_from_sim no)
-		(in_bom yes)
-		(on_board yes)
-		(dnp no)
+		(exclude_from_sim yes)
+		(in_bom no)
+		(on_board no)
+		(dnp yes)
 		(property "Reference" "C?"
 			(at 49.53 102.235 90)
