File: ram.kicad_sch (KiCad schematic)
At the start: 7 parts, among them U1 LFE5U-85F-6BG381C

Commit message: Updating schematics
Parts:
- U1: Digike_y2 (none) -> 220-2071-ND; Digikey (none) -> 220-2177-ND; Koncar (none) -> FU004; LCSC (none) -> C446029; LowCost (none) -> 842-LFE5U12F6BG381C; MFG1 (none) -> Lattice; MFG2 (none) -> Lattice; MNF1_URL (none) -> www.latticesemi.com; MNF2_URL (none) -> www.latticesemi.com; MP_N2 (none) -> LFE5U-12F-6BG381C; Mouser (none) -> 842-LFE5U85F6BG381C; Mouser_URL (none) -> www.mouser.com; Side (none) -> T; price100_Mouse (none) -> 22.82$
Other:
- moved on the sheet: R?

Commit message: Cleanup
Connections:
- no-connect marks 3 -> 5
Changed lines of the file:
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@@
+	)
+	(no_connect
+		(at 205.74 66.04)
+	)
+	(no_connect
+		(at 205.74 104.14)
 	)
 	(no_connect
