File: ram.kicad_sch (KiCad schematic)
At the start: 7 parts, among them U1 LFE5U-85F-6BG381C

Commit message: fix #44
Other:
- title: ULX4M -> ULX4M-LD
Changed lines of the file:
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@@
 	(paper "A4")
 	(title_block
-		(title "ULX4M")
-		(date "2021-11-08")
-		(rev "0.0.2")
+		(title "ULX4M-LD")
+		(date "2025-03-12")
+		(rev "0.0.3")
 		(company "Intergalaktik d.o.o.")
 		(comment 1 "SDRAM memory")

Commit message: Cleanup
Connections:
- no-connect marks 3 -> 7
Changed lines of the file:
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@@
+	)
+	(no_connect
+		(at 205.74 48.26)
+	)
+	(no_connect
+		(at 205.74 104.14)
+	)
+	(no_connect
+		(at 167.64 127)
 	)
 	(no_connect
 		(at 167.64 83.82)
 	)
+	(no_connect
+		(at 167.64 99.06)
+	)
 	(global_label "DDR3_DQ14"

Commit message: Improving schematics
Other:
- company: Intergalaktik d.o.o. -> ${project_creator}
- title: ULX4M-LD -> ${project_name}
Changed lines of the file:
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@@
 	(paper "A4")
 	(title_block
-		(title "ULX4M-LD")
+		(title "${project_name}")
 		(date "2025-03-12")
-		(rev "0.0.3")
-		(company "Intergalaktik d.o.o.")
+		(rev "${project_version}")
+		(company "${project_creator}")
 		(comment 1 "SDRAM memory")
-		(comment 2 "License: CERN-OHL-S v2")
+		(comment 2 "License: ${project_license}")
 	)
 	(no_connect
