File: serdes.kicad_sch (KiCad schematic)
At the start: 26 parts, among them J4 Antenna

Commit message: Before graphical cleanup
Parts:
- renumbered C59 to C?, C61 to C?, C62 to C?, C66 to C?, C67 to C?, C68 to C?, C64 to C?, C65 to C?, C70 to C?, C71 to C?, C63 to C?, C69 to C?, C55 to C?, C56 to C?, C73 to C?, C72 to C?, C58 to C?, C57 to C?, C74 to C?, C75 to C?, C91 to C?, C92 to C?, C93 to C?, C94 to C?
Changed lines of the file:
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@@
 	(label "S_5_N"
 		(at 168.91 96.52 0)
+		(fields_autoplaced yes)
 		(effects
 			(font
@@
 	(label "2N"
 		(at 180.34 120.015 0)
+		(fields_autoplaced yes)
 		(effects
 			(font
@@
 	(label "S_7_P"
 		(at 113.03 93.98 0)
+		(fields_autoplaced yes)
 		(effects
 			(font
@@
 	(label "CLK_1_P"
 		(at 111.76 86.36 0)
+		(fields_autoplaced yes)
 		(effects
 			(font
@@
 	(label "2P"
 		(at 179.705 122.555 0)
+		(fields_autoplaced yes)
 		(effects
 			(font
@@
 	(label "S_5_P"
 		(at 194.945 126.365 0)
+		(fields_autoplaced yes)
 		(effects
 			(font
@@
 	(label "S_1_P"
 		(at 113.03 59.69 0)
+		(fields_autoplaced yes)
 		(effects
 			(font
@@
 	(label "S_3_P"
 		(at 113.03 57.15 0)
+		(fields_autoplaced yes)
 		(effects
 			(font
@@
 	(label "CLK_0_P"
 		(at 113.03 49.53 0)
+		(fields_autoplaced yes)
 		(effects
 			(font
@@
 	(label "S_0_P"
 		(at 113.03 54.61 0)
+		(fields_autoplaced yes)
 		(effects
 			(font
@@
 	(label "S_6_P"
 		(at 113.03 88.9 0)
+		(fields_autoplaced yes)
 		(effects
 			(font
@@
 	(label "S_2_P"
 		(at 113.03 52.07 0)
+		(fields_autoplaced yes)
 		(effects
 			(font
@@
 	(label "S_4_P"
 		(at 113.03 91.44 0)
+		(fields_autoplaced yes)
 		(effects
 			(font
@@
 	(label "S_7_P"
 		(at 194.945 117.475 0)
+		(fields_autoplaced yes)
 		(effects
 			(font
@@
 	(label "S_1_N"
 		(at 168.91 59.69 0)
+		(fields_autoplaced yes)
 		(effects
 			(font
@@
 	(label "S_3_N"
 		(at 168.91 57.15 0)
+		(fields_autoplaced yes)
 		(effects
 			(font
@@
 	(label "CLK_0_N"
 		(at 168.91 49.53 0)
+		(fields_autoplaced yes)
 		(effects
 			(font
@@
 	(label "S_2_N"
 		(at 168.91 52.07 0)
+		(fields_autoplaced yes)
 		(effects
 			(font
@@
 	(label "S_7_N"
 		(at 194.945 113.03 0)
+		(fields_autoplaced yes)
 		(effects
 			(font
@@
 	(label "CLK_1_N"
 		(at 168.91 86.36 0)
+		(fields_autoplaced yes)
 		(effects
 			(font
@@
 	(label "S_7_N"
 		(at 168.91 93.98 0)
+		(fields_autoplaced yes)
 		(effects
 			(font
@@
 	(label "S_4_N"
 		(at 168.91 91.44 0)
+		(fields_autoplaced yes)
 		(effects
 			(font
@@
 	(label "S_6_N"
 		(at 168.91 88.9 0)
+		(fields_autoplaced yes)
 		(effects
 			(font
@@
 	(label "1P"
 		(at 180.34 117.475 0)
+		(fields_autoplaced yes)
 		(effects
 			(font
@@
 	(label "S_5_P"
 		(at 113.03 96.52 0)
+		(fields_autoplaced yes)
 		(effects
 			(font
@@
 	(label "S_5_N"
 		(at 194.945 121.92 0)
+		(fields_autoplaced yes)
 		(effects
 			(font
@@
 	(label "S_0_N"
 		(at 168.91 54.61 0)
+		(fields_autoplaced yes)
 		(effects
 			(font
@@
 	(label "1N"
 		(at 180.34 113.03 0)
+		(fields_autoplaced yes)
 		(effects
 			(font
@@
 		(pin "1"
 		)
+		(instances
+			(project ""
+				(path "/1876dd7c-56e8-4d11-a76e-0d3f3f8be70a/00000000-0000-0000-0000-000058da7327"
+					(reference "#PWR0147")
+					(unit 1)
+				)
+			)
+		)
 	)
 	(symbol
@@
 		(on_board yes)
 		(dnp no)
-		(property "Reference" "#PWR0179"
+		(property "Reference" "#PWR?"
 			(at 167.64 64.77 0)
 			(effects
@@
 		(on_board yes)
 		(dnp no)
-		(property "Reference" "#PWR0180"
+		(property "Reference" "#PWR?"
 			(at 121.92 71.12 0)
 			(effects
@@
 		(on_board yes)
 		(dnp no)
-		(property "Reference" "#PWR0181"
+		(property "Reference" "#PWR?"
 			(at 167.64 81.28 0)
 			(effects
@@
 		(on_board yes)
 		(dnp no)
-		(property "Reference" "C59"
+		(property "Reference" "C?"
 			(at 109.22 48.26 90)
 			(effects
@@
 		(on_board yes)
 		(dnp no)
-		(property "Reference" "C61"
+		(property "Reference" "C?"
 			(at 109.22 53.34 90)
 			(effects
@@
 		(on_board yes)
 		(dnp no)
-		(property "Reference" "C62"
+		(property "Reference" "C?"
 			(at 109.22 58.42 90)
 			(effects
@@
 		(on_board yes)
 		(dnp no)
-		(property "Reference" "C66"
+		(property "Reference" "C?"
 			(at 185.42 48.26 90)
 			(effects
@@
 		(on_board yes)
 		(dnp no)
-		(property "Reference" "C67"
+		(property "Reference" "C?"
 			(at 185.42 53.34 90)
 			(effects
@@
 		(on_board yes)
 		(dnp no)
-		(property "Reference" "C68"
+		(property "Reference" "C?"
 			(at 185.42 58.42 90)
 			(effects
@@
 		(on_board yes)
 		(dnp no)
-		(property "Reference" "C64"
+		(property "Reference" "C?"
 			(at 109.22 90.17 90)
 			(effects
@@
 		(on_board yes)
 		(dnp no)
-		(property "Reference" "C65"
+		(property "Reference" "C?"
 			(at 109.22 95.25 90)
 			(effects
@@
 		(on_board yes)
 		(dnp no)
-		(property "Reference" "C70"
+		(property "Reference" "C?"
 			(at 185.42 90.17 90)
 			(effects
@@
 		(on_board yes)
 		(dnp no)
-		(property "Reference" "C71"
+		(property "Reference" "C?"
 			(at 185.42 95.25 90)
 			(effects
@@
 		(on_board yes)
 		(dnp no)
-		(property "Reference" "C63"
+		(property "Reference" "C?"
 			(at 109.22 85.09 90)
 			(effects
@@
 		(on_board yes)
 		(dnp no)
-		(property "Reference" "C69"
+		(property "Reference" "C?"
 			(at 185.42 85.09 90)
 			(effects
@@
 		(on_board yes)
 		(dnp no)
-		(property "Reference" "C55"
+		(property "Reference" "C?"
 			(at 87.63 50.8 90)
 			(effects
@@
 		(on_board yes)
 		(dnp no)
-		(property "Reference" "C56"
+		(property "Reference" "C?"
 			(at 87.63 55.88 90)
 			(effects
@@
 		(on_board yes)
 		(dnp no)
-		(property "Reference" "C73"
+		(property "Reference" "C?"
 			(at 203.2 55.88 90)
 			(effects
@@
 		(on_board yes)
 		(dnp no)
-		(property "Reference" "C72"
+		(property "Reference" "C?"
 			(at 203.2 50.8 90)
 			(effects
@@
 		(on_board yes)
 		(dnp no)
-		(property "Reference" "C58"
+		(property "Reference" "C?"
 			(at 87.63 92.71 90)
 			(effects
@@
 		(on_board yes)
 		(dnp no)
-		(property "Reference" "C57"
+		(property "Reference" "C?"
 			(at 87.63 87.63 90)
 			(effects
@@
 		(on_board yes)
 		(dnp no)
-		(property "Reference" "C74"
+		(property "Reference" "C?"
 			(at 203.2 87.63 90)
 			(effects
@@
 		(on_board yes)
 		(dnp no)
-		(property "Reference" "C75"
+		(property "Reference" "C?"
 			(at 203.2 92.71 90)
 			(effects
@@
 		(on_board yes)
 		(dnp no)
-		(property "Reference" "C91"
+		(property "Reference" "C?"
 			(at 187.96 111.76 90)
 			(effects
@@
 		(on_board yes)
 		(dnp no)
-		(property "Reference" "C92"
+		(property "Reference" "C?"
 			(at 187.96 116.205 90)
 			(effects
@@
 		(on_board yes)
 		(dnp no)
-		(property "Reference" "C93"
+		(property "Reference" "C?"
 			(at 187.96 120.65 90)
 			(effects
@@
 		(on_board yes)
 		(dnp no)
-		(property "Reference" "C94"
+		(property "Reference" "C?"
 			(at 187.96 125.095 90)
 			(effects
