File: serdes.kicad_sch (KiCad schematic)
At the start: 26 parts, among them J4 Antenna

Commit message: Updating schematics
Parts:
- C? (x4): footprint (none) -> Capacitor_SMD:C_0402_1005Metric
- U?: Mouser_URL (none) -> www.mouser.com
Connections:
- net ETH_0N: now also C?.2
- net ETH_0P: now also C?.1
- net ETH_1N: now also C?.2
- net ETH_1P: now also C?.1
- net S_4_N: now also C?.1
- net S_4_P: now also C?.2
- net S_6_N: now also C?.1
- net S_6_P: now also C?.2
Other:
- moved on the sheet: C?
Changed lines of the file:
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@@
 	(label "S_5_N"
 		(at 168.91 96.52 0)
-		(fields_autoplaced yes)
 		(effects
 			(font
@@
 	(label "2N"
 		(at 180.34 120.015 0)
-		(fields_autoplaced yes)
 		(effects
 			(font
@@
 	(label "S_7_P"
 		(at 113.03 93.98 0)
-		(fields_autoplaced yes)
 		(effects
 			(font
@@
 	(label "CLK_1_P"
 		(at 111.76 86.36 0)
-		(fields_autoplaced yes)
 		(effects
 			(font
@@
 	(label "2P"
 		(at 179.705 122.555 0)
-		(fields_autoplaced yes)
 		(effects
 			(font
@@
 	(label "S_5_P"
 		(at 194.945 126.365 0)
-		(fields_autoplaced yes)
 		(effects
 			(font
@@
 	(label "S_1_P"
 		(at 113.03 59.69 0)
-		(fields_autoplaced yes)
 		(effects
 			(font
@@
 	(label "S_3_P"
 		(at 113.03 57.15 0)
-		(fields_autoplaced yes)
 		(effects
 			(font
@@
 	(label "CLK_0_P"
 		(at 113.03 49.53 0)
-		(fields_autoplaced yes)
 		(effects
 			(font
@@
 	(label "S_0_P"
 		(at 113.03 54.61 0)
-		(fields_autoplaced yes)
 		(effects
 			(font
@@
 	(label "S_6_P"
 		(at 113.03 88.9 0)
-		(fields_autoplaced yes)
 		(effects
 			(font
@@
 	(label "S_2_P"
 		(at 113.03 52.07 0)
-		(fields_autoplaced yes)
 		(effects
 			(font
@@
 	(label "S_4_P"
 		(at 113.03 91.44 0)
-		(fields_autoplaced yes)
 		(effects
 			(font
@@
 	(label "S_7_P"
 		(at 194.945 117.475 0)
-		(fields_autoplaced yes)
 		(effects
 			(font
@@
 	(label "S_1_N"
 		(at 168.91 59.69 0)
-		(fields_autoplaced yes)
 		(effects
 			(font
@@
 	(label "S_3_N"
 		(at 168.91 57.15 0)
-		(fields_autoplaced yes)
 		(effects
 			(font
@@
 	(label "CLK_0_N"
 		(at 168.91 49.53 0)
-		(fields_autoplaced yes)
 		(effects
 			(font
@@
 	(label "S_2_N"
 		(at 168.91 52.07 0)
-		(fields_autoplaced yes)
 		(effects
 			(font
@@
 	(label "S_7_N"
 		(at 194.945 113.03 0)
-		(fields_autoplaced yes)
 		(effects
 			(font
@@
 	(label "CLK_1_N"
 		(at 168.91 86.36 0)
-		(fields_autoplaced yes)
 		(effects
 			(font
@@
 	(label "S_7_N"
 		(at 168.91 93.98 0)
-		(fields_autoplaced yes)
 		(effects
 			(font
@@
 	(label "S_4_N"
 		(at 168.91 91.44 0)
-		(fields_autoplaced yes)
 		(effects
 			(font
@@
 	(label "S_6_N"
 		(at 168.91 88.9 0)
-		(fields_autoplaced yes)
 		(effects
 			(font
@@
 	(label "1P"
 		(at 180.34 117.475 0)
-		(fields_autoplaced yes)
 		(effects
 			(font
@@
 	(label "S_5_P"
 		(at 113.03 96.52 0)
-		(fields_autoplaced yes)
 		(effects
 			(font
@@
 	(label "S_5_N"
 		(at 194.945 121.92 0)
-		(fields_autoplaced yes)
 		(effects
 			(font
@@
 	(label "S_0_N"
 		(at 168.91 54.61 0)
-		(fields_autoplaced yes)
 		(effects
 			(font
@@
 	(label "1N"
 		(at 180.34 113.03 0)
-		(fields_autoplaced yes)
 		(effects
 			(font
@@
 			)
 		)
-		(property "Datasheet" "http://www.latticesemi.com/~/media/LatticeSemi/Documents/ApplicationNotes/EH/TN1261.pdf?document_id=50463"
+		(property "Datasheet" "http://www.latticesemi.com/~/media/LatticeSemi/Documents/DataSheets/ECP5/FPGA-DS-02012.pdf"
 			(at 118.11 48.26 0)
 			(effects
@@
 			)
 		)
+		(property "Mouser_URL" "www.mouser.com"
+			(at 0 144.78 0)
+			(effects
+				(font
+					(size 1.27 1.27)
+				)
+				(hide yes)
+			)
+		)
 		(pin "A11"
 		)
@@
 	(symbol
 		(lib_id "Device:C_Small")
-		(at 100.33 110.49 90)
+		(at 90.17 88.9 90)
 		(unit 1)
 		(exclude_from_sim no)
@@
 		(dnp no)
 		(property "Reference" "C?"
-			(at 102.87 109.22 90)
+			(at 92.71 87.63 90)
 			(effects
 				(font
@@
 		)
 		(property "Value" "22n"
-			(at 104.14 111.76 90)
+			(at 93.98 90.17 90)
 			(effects
 				(font
@@
 			)
 		)
-		(property "Footprint" ""
-			(at 100.33 110.49 0)
+		(property "Footprint" "Capacitor_SMD:C_0402_1005Metric"
+			(at 90.17 88.9 0)
 			(effects
 				(font
@@
 		)
 		(property "Datasheet" "~"
-			(at 100.33 110.49 0)
+			(at 90.17 88.9 0)
 			(effects
 				(font
@@
 		)
 		(property "Description" ""
-			(at 100.33 110.49 0)
+			(at 90.17 88.9 0)
 			(effects
 				(font
@@
 	(symbol
 		(lib_id "Device:C_Small")
-		(at 102.87 115.57 90)
+		(at 200.66 88.9 90)
 		(unit 1)
 		(exclude_from_sim no)
@@
 		(dnp no)
 		(property "Reference" "C?"
-			(at 105.41 114.3 90)
+			(at 203.2 87.63 90)
 			(effects
 				(font
@@
 		)
 		(property "Value" "22n"
-			(at 106.68 116.84 90)
+			(at 204.47 90.17 90)
 			(effects
 				(font
@@
 			)
 		)
-		(property "Footprint" ""
-			(at 102.87 115.57 0)
+		(property "Footprint" "Capacitor_SMD:C_0402_1005Metric"
+			(at 200.66 88.9 0)
 			(effects
 				(font
@@
 		)
 		(property "Datasheet" "~"
-			(at 102.87 115.57 0)
+			(at 200.66 88.9 0)
 			(effects
 				(font
@@
 		)
 		(property "Description" ""
-			(at 102.87 115.57 0)
+			(at 200.66 88.9 0)
 			(effects
 				(font
@@
 	(symbol
 		(lib_id "Device:C_Small")
-		(at 95.25 114.3 90)
+		(at 106.68 91.44 90)
 		(unit 1)
 		(exclude_from_sim no)
@@
 		(dnp no)
 		(property "Reference" "C?"
-			(at 92.71 113.03 90)
+			(at 104.14 90.17 90)
 			(effects
 				(font
@@
 		)
 		(property "Value" "22n"
-			(at 92.71 115.57 90)
+			(at 104.14 92.71 90)
 			(effects
 				(font
@@
 			)
 		)
-		(property "Footprint" ""
-			(at 95.25 114.3 0)
+		(property "Footprint" "Capacitor_SMD:C_0402_1005Metric"
+			(at 106.68 91.44 0)
 			(effects
 				(font
@@
 		)
 		(property "Datasheet" "~"
-			(at 95.25 114.3 0)
+			(at 106.68 91.44 0)
 			(effects
 				(font
@@
 		)
 		(property "Description" ""
-			(at 95.25 114.3 0)
+			(at 106.68 91.44 0)
 			(effects
 				(font
@@
 	(symbol
 		(lib_id "Device:C_Small")
-		(at 97.79 119.38 90)
+		(at 182.88 91.44 90)
 		(unit 1)
 		(exclude_from_sim no)
@@
 		(dnp no)
 		(property "Reference" "C?"
-			(at 100.33 118.11 90)
+			(at 185.42 90.17 90)
 			(effects
 				(font
@@
 		)
 		(property "Value" "22n"
-			(at 101.6 120.65 90)
+			(at 186.69 92.71 90)
 			(effects
 				(font
@@
 			)
 		)
-		(property "Footprint" ""
-			(at 97.79 119.38 0)
+		(property "Footprint" "Capacitor_SMD:C_0402_1005Metric"
+			(at 182.88 91.44 0)
 			(effects
 				(font
@@
 		)
 		(property "Datasheet" "~"
-			(at 97.79 119.38 0)
+			(at 182.88 91.44 0)
 			(effects
 				(font
@@
 		)
 		(property "Description" ""
-			(at 97.79 119.38 0)
+			(at 182.88 91.44 0)
 			(effects
 				(font
@@
 		(pin "4"
 		)
+		(instances
+			(project "ulx4m"
+				(path "/1876dd7c-56e8-4d11-a76e-0d3f3f8be70a/00000000-0000-0000-0000-000058da7327"
+					(reference "J4")
+					(unit 1)
+				)
+			)
+		)
 	)

Commit message: Errors cleanup
Parts:
- C? (x4): footprint Capacitor_SMD:C_0402_1005Metric -> (none)
Changed lines of the file:
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@@
 			)
 		)
-		(property "Footprint" "Capacitor_SMD:C_0402_1005Metric"
+		(property "Footprint" ""
 			(at 90.17 88.9 0)
 			(effects
@@
 			)
 		)
-		(property "Footprint" "Capacitor_SMD:C_0402_1005Metric"
+		(property "Footprint" ""
 			(at 200.66 88.9 0)
 			(effects
@@
 			)
 		)
-		(property "Footprint" "Capacitor_SMD:C_0402_1005Metric"
+		(property "Footprint" ""
 			(at 106.68 91.44 0)
 			(effects
@@
 			)
 		)
-		(property "Footprint" "Capacitor_SMD:C_0402_1005Metric"
+		(property "Footprint" ""
 			(at 182.88 91.44 0)
 			(effects

Commit message: Cleanup
Parts:
- C? (x4): now not fitted; now left out of the parts list
