File: ethernet.kicad_sch (KiCad schematic)
At the start: 21 parts, among them U4 LAN8720A

Commit message: Connecting Ethernt LEDs to CM4 GPIO pins fix #51
Connections:
- net ACTLED renamed GPIO10
- net LINKLED renamed GPIO21
Changed lines of the file:
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@@
+	(wire
+		(pts
+			(xy 220.98 167.64) (xy 226.06 167.64)
+		)
+		(stroke
+			(width 0)
+			(type default)
+		)
+	)
 	(wire
 		(pts
@@
 		(pts
 			(xy 128.905 151.13) (xy 128.905 146.05)
+		)
+		(stroke
+			(width 0)
+			(type default)
+		)
+	)
+	(wire
+		(pts
+			(xy 220.98 163.83) (xy 226.06 163.83)
 		)
 		(stroke
@@
 		)
 	)
+	(label "ACTLED"
+		(at 226.06 167.64 0)
+		(fields_autoplaced yes)
+		(effects
+			(font
+				(size 1.27 1.27)
+			)
+			(justify left bottom)
+		)
+	)
 	(label "RXD0"
 		(at 154.305 138.43 180)
@@
 			)
 			(justify right bottom)
+		)
+	)
+	(label "LINKLED"
+		(at 226.06 163.83 0)
+		(fields_autoplaced yes)
+		(effects
+			(font
+				(size 1.27 1.27)
+			)
+			(justify left bottom)
 		)
 	)
@@
 		)
 	)
+	(global_label "GPIO21"
+		(shape input)
+		(at 220.98 163.83 180)
+		(effects
+			(font
+				(size 1.524 1.524)
+			)
+			(justify right)
+		)
+		(property "Intersheetrefs" "${INTERSHEET_REFS}"
+			(at 220.98 163.83 0)
+			(effects
+				(font
+					(size 1.27 1.27)
+				)
+				(hide yes)
+			)
+		)
+	)
 	(global_label "RGMII_RXD1"
 		(shape output)
@@
 			(effects
 				(font
+					(size 1.27 1.27)
+				)
+				(hide yes)
+			)
+		)
+	)
+	(global_label "GPIO10"
+		(shape input)
+		(at 220.98 167.64 180)
+		(effects
+			(font
+				(size 1.524 1.524)
+			)
+			(justify right)
+		)
+		(property "Intersheetrefs" "${INTERSHEET_REFS}"
+			(at 220.98 167.64 0)
+			(effects
+				(font
