File: ethernet.kicad_sch (KiCad schematic)
At the start: 21 parts, among them U4 LAN8720A

Commit message: LS Adding resistor to ethernet #50
Parts:
- added R64, R65, R66, R67: 300, Resistor_SMD:R_0402_1005Metric, symbol ecp5-dc-scm:R_1k_0402
Connections:
- net +3V3: now also R64.2, R65.2, R66.2, R67.2
- net ETH_0N: now also R65.1
- net ETH_0P: now also R64.1
- net ETH_1N: now also R67.1
- net ETH_1P: now also R66.1
