File: ethernet.kicad_sch (KiCad schematic)
At the start: 47 parts, among them U4 KSZ9031RNXCA, Y2 ASEMB-25.000MHZ-LC-T

Commit message: fix #44
Other:
- company: (none) -> Intergalaktik d.o.o.
- title: Ethernet -> ULX4M-LD
Changed lines of the file:
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@@
 	(paper "A3")
 	(title_block
-		(title "Ethernet")
-		(rev "1.0.3")
+		(title "ULX4M-LD")
+		(date "2025-03-12")
+		(rev "0.0.3")
+		(company "Intergalaktik d.o.o.")
 		(comment 1 "Reference - ecp5-dc-scm")
-		(comment 2 "License: Apache License 2.0")
+		(comment 2 "License: CERN-OHL-S v2")
 	)
 	(junction

Commit message: Changing ethernet resistor value to 0R fix #54
Parts:
- R66: value 300 -> 0R; Val 300 -> 0R
- R67: Val 300 -> 0R
Changed lines of the file:
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@@
 			)
 		)
-		(property "Value" "300"
+		(property "Value" "0R"
 			(at 330.835 102.235 0)
 			(effects
@@
 			)
 		)
-		(property "Val" "300"
+		(property "Val" "0R"
 			(at 330.835 98.425 0)
 			(effects
@@
 			)
 		)
-		(property "Val" "300"
+		(property "Val" "0R"
 			(at 330.835 107.315 0)
 			(effects

Commit message: Placing all components
Parts:
- removed R66: 0R, Resistor_SMD:R_0402_1005Metric, symbol ecp5-dc-scm:R_1k_0402
- removed R67: 300, Resistor_SMD:R_0402_1005Metric, symbol ecp5-dc-scm:R_1k_0402
- added R72, R73: 10k2, Resistor_SMD:R_0402_1005Metric, symbol ecp5-dc-scm:R_10k2_0402
- added R74, R75, R76, R77, R84, R85, R86, R87: 10k2, Resistor_SMD:R_0201_0603Metric, symbol ecp5-dc-scm:R_10k2_0402
Connections:
- net ETH_LED1 is gone; now on net ETH_nLED2: R63.1, U4.17 (LED1/PHAD0/PME_N1)
- net ETH_LED2 is gone; now on net ETH_nLED1: R64.1, U4.15 (LED2/PHYAD1)
- net +3V3: now also R72.2, R73.2, R74.2, R75.2, R76.2, R77.2, R84.2, R85.2, R86.2, R87.2
- net ETH_0N: now also R75.1
- net ETH_0P: now also R74.1
- net ETH_1N: now also R77.1
- net ETH_1P: now also R76.1
- net ETH_2N: now also R85.1
- net ETH_2P: now also R84.1
- net ETH_3N: now also R87.1
- net ETH_3P: now also R86.1
- net ETH_nLED1: now also R72.1
- net ETH_nLED2: now also R73.1
Other:
- note added: "PHY ADDRESS"
- note added: "Use FPGA PULL-UP/DOWN"

Commit message: Cleanup
Parts:
- R53, R54, R55, R56, R57, R59, R60, R61, R62, R63, R64: now not fitted; now left out of the parts list
Other:
- note added: "Not connected"
- note added: "Pull up resistors - not conected use FPGA internal PULLs"
- note removed: "Pull up resistors - we will try internal"
Changed lines of the file:
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@@
 		)
 	)
-	(polyline
-		(pts
-			(xy 151.13 281.94) (xy 24.13 281.94)
-		)
-		(stroke
-			(width 0)
-			(type dash)
-		)
-	)
 	(wire
 		(pts
@@
 		)
 	)
-	(polyline
-		(pts
-			(xy 24.13 281.94) (xy 24.13 194.31)
-		)
-		(stroke
-			(width 0)
-			(type dash)
-		)
-	)
 	(wire
 		(pts
@@
 		)
 	)
-	(polyline
-		(pts
-			(xy 151.13 194.31) (xy 151.13 281.94)
-		)
-		(stroke
-			(width 0)
-			(type dash)
-		)
-	)
 	(wire
 		(pts
@@
 		)
 	)
-	(polyline
-		(pts
-			(xy 24.13 194.31) (xy 151.13 194.31)
-		)
-		(stroke
-			(width 0)
-			(type dash)
-		)
-	)
 	(wire
 		(pts
@@
 	)
 	(rectangle
+		(start 27.178 191.516)
+		(end 150.368 282.702)
+		(stroke
+			(width 0)
+			(type dot)
+			(color 0 0 0 1)
+		)
+		(fill
+			(type color)
+			(color 255 0 255 1)
+		)
+	)
+	(rectangle
 		(start 192.786 221.742)
 		(end 259.842 276.606)
@@
 		)
 	)
-	(text "Pull up resistors - we will try internal"
+	(text "Pull up resistors - not conected use FPGA internal PULLs"
 		(exclude_from_sim no)
-		(at 86.36 201.295 0)
+		(at 58.674 196.596 0)
 		(effects
 			(font
@@
 		)
 	)
+	(text "Not connected"
+		(exclude_from_sim no)
+		(at 120.396 157.734 0)
+		(effects
+			(font
+				(size 1.524 1.524)
+			)
+		)
+	)
 	(text "Use FPGA PULL-UP/DOWN"
 		(exclude_from_sim no)
@@
 		(at 108.585 229.235 270)
 		(unit 1)
-		(exclude_from_sim no)
-		(in_bom yes)
-		(on_board yes)
-		(dnp no)
+		(exclude_from_sim yes)
+		(in_bom no)
+		(on_board no)
+		(dnp yes)
 		(property "Reference" "R61"
 			(at 110.49 226.06 90)
@@
 		(at 52.705 229.235 90)
 		(unit 1)
-		(exclude_from_sim no)
-		(in_bom yes)
-		(on_board yes)
-		(dnp no)
+		(exclude_from_sim yes)
+		(in_bom no)
+		(on_board no)
+		(dnp yes)
 		(property "Reference" "R53"
 			(at 53.975 226.06 90)
@@
 		(at 59.69 229.235 90)
 		(unit 1)
-		(exclude_from_sim no)
-		(in_bom yes)
-		(on_board yes)
-		(dnp no)
+		(exclude_from_sim yes)
+		(in_bom no)
+		(on_board no)
+		(dnp yes)
 		(property "Reference" "R54"
 			(at 60.96 226.06 90)
@@
 		(at 66.675 229.235 90)
 		(unit 1)
-		(exclude_from_sim no)
-		(in_bom yes)
-		(on_board yes)
-		(dnp no)
+		(exclude_from_sim yes)
+		(in_bom no)
+		(on_board no)
+		(dnp yes)
 		(property "Reference" "R55"
 			(at 67.945 226.06 90)
@@
 		(at 73.66 229.235 90)
 		(unit 1)
-		(exclude_from_sim no)
-		(in_bom yes)
-		(on_board yes)
-		(dnp no)
+		(exclude_from_sim yes)
+		(in_bom no)
+		(on_board no)
+		(dnp yes)
 		(property "Reference" "R56"
 			(at 74.93 226.06 90)
@@
 		(at 80.645 229.235 90)
 		(unit 1)
-		(exclude_from_sim no)
-		(in_bom yes)
-		(on_board yes)
-		(dnp no)
+		(exclude_from_sim yes)
+		(in_bom no)
+		(on_board no)
+		(dnp yes)
 		(property "Reference" "R57"
 			(at 81.915 226.06 90)
@@
 		(at 87.63 229.235 90)
 		(unit 1)
-		(exclude_from_sim no)
-		(in_bom yes)
-		(on_board yes)
-		(dnp no)
+		(exclude_from_sim yes)
+		(in_bom no)
+		(on_board no)
+		(dnp yes)
 		(property "Reference" "R59"
 			(at 88.9 226.06 90)
@@
 		(at 94.615 229.235 90)
 		(unit 1)
-		(exclude_from_sim no)
-		(in_bom yes)
-		(on_board yes)
-		(dnp no)
+		(exclude_from_sim yes)
+		(in_bom no)
+		(on_board no)
+		(dnp yes)
 		(property "Reference" "R60"
 			(at 95.885 226.06 90)
@@
 		(at 115.57 229.235 90)
 		(unit 1)
-		(exclude_from_sim no)
-		(in_bom yes)
-		(on_board yes)
-		(dnp no)
+		(exclude_from_sim yes)
+		(in_bom no)
+		(on_board no)
+		(dnp yes)
 		(property "Reference" "R62"
 			(at 116.84 226.06 90)
@@
 		(at 129.54 229.235 90)
 		(unit 1)
-		(exclude_from_sim no)
-		(in_bom yes)
-		(on_board yes)
-		(dnp no)
+		(exclude_from_sim yes)
+		(in_bom no)
+		(on_board no)
+		(dnp yes)
 		(property "Reference" "R64"
 			(at 130.81 226.06 90)
@@
 		(at 122.555 229.235 90)
 		(unit 1)
-		(exclude_from_sim no)
-		(in_bom yes)
-		(on_board yes)
-		(dnp no)
+		(exclude_from_sim yes)
+		(in_bom no)
+		(on_board no)
+		(dnp yes)
 		(property "Reference" "R63"
 			(at 123.825 226.06 90)

Commit message: Improving schematics
Parts:
- R74, R75, R76, R77, R84, R85, R86, R87: footprint Resistor_SMD:R_0201_0603Metric -> Resistor_SMD:R_0402_1005Metric
Other:
- company: Intergalaktik d.o.o. -> ${project_creator}
- title: ULX4M-LD -> ${project_name}
Changed lines of the file:
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@@
 	(paper "A3")
 	(title_block
-		(title "ULX4M-LD")
+		(title "${project_name}")
 		(date "2025-03-12")
-		(rev "0.0.3")
-		(company "Intergalaktik d.o.o.")
+		(rev "${project_version}")
+		(company "${project_creator}")
 		(comment 1 "Reference - ecp5-dc-scm")
-		(comment 2 "License: CERN-OHL-S v2")
+		(comment 2 "License: ${project_license}")
 	)
 	(junction
@@
 			)
 		)
-		(property "Footprint" "Resistor_SMD:R_0201_0603Metric"
+		(property "Footprint" "Resistor_SMD:R_0402_1005Metric"
 			(at 321.31 148.59 0)
 			(effects
@@
 			)
 		)
-		(property "Footprint" "Resistor_SMD:R_0201_0603Metric"
+		(property "Footprint" "Resistor_SMD:R_0402_1005Metric"
 			(at 316.23 148.59 0)
 			(effects
@@
 			)
 		)
-		(property "Footprint" "Resistor_SMD:R_0201_0603Metric"
+		(property "Footprint" "Resistor_SMD:R_0402_1005Metric"
 			(at 311.15 148.59 0)
 			(effects
@@
 			)
 		)
-		(property "Footprint" "Resistor_SMD:R_0201_0603Metric"
+		(property "Footprint" "Resistor_SMD:R_0402_1005Metric"
 			(at 323.85 148.59 0)
 			(effects
@@
 			)
 		)
-		(property "Footprint" "Resistor_SMD:R_0201_0603Metric"
+		(property "Footprint" "Resistor_SMD:R_0402_1005Metric"
 			(at 313.69 148.59 0)
 			(effects
@@
 			)
 		)
-		(property "Footprint" "Resistor_SMD:R_0201_0603Metric"
+		(property "Footprint" "Resistor_SMD:R_0402_1005Metric"
 			(at 306.07 148.59 0)
 			(effects
@@
 			)
 		)
-		(property "Footprint" "Resistor_SMD:R_0201_0603Metric"
+		(property "Footprint" "Resistor_SMD:R_0402_1005Metric"
 			(at 318.77 148.59 0)
 			(effects
@@
 			)
 		)
-		(property "Footprint" "Resistor_SMD:R_0201_0603Metric"
+		(property "Footprint" "Resistor_SMD:R_0402_1005Metric"
 			(at 308.61 148.59 0)
 			(effects
