File: blinkey.kicad_sch (KiCad schematic)
At the start: 21 parts

Commit message: Updating schematics
Other:
- note removed: "ST7789/SSD1331/SSD1351/SSD1306 compatible LCD/OLED 0.96/1.3/1.54" PCB 14x14 units 1 unit = 2.54 mm"
- moved on the sheet: BTN1, BTN2, BTN3, R18
