File: blinkey.kicad_sch (KiCad schematic)
At the start: 21 parts

Commit message: fix #44
Other:
- company: EMARD -> Intergalaktik d.o.o.
- title: ULX3S -> ULX4M-LD
Changed lines of the file:
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@@
 	(paper "A4")
 	(title_block
-		(title "ULX3S")
-		(rev "1.0.3")
-		(company "EMARD")
+		(title "ULX4M-LD")
+		(date "2025-03-12")
+		(rev "0.0.3")
+		(company "Intergalaktik d.o.o.")
 		(comment 1 "Buttons, LEDs, OLED display")
 		(comment 2 "License: CERN-OHL-S v2")

Commit message: Improving schematics
Other:
- company: Intergalaktik d.o.o. -> ${project_creator}
- title: ULX4M-LD -> ${project_name}
Changed lines of the file:
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@@
 	(paper "A4")
 	(title_block
-		(title "ULX4M-LD")
+		(title "${project_name}")
 		(date "2025-03-12")
-		(rev "0.0.3")
-		(company "Intergalaktik d.o.o.")
+		(rev "${project_version}")
+		(company "${project_creator}")
 		(comment 1 "Buttons, LEDs, OLED display")
-		(comment 2 "License: CERN-OHL-S v2")
+		(comment 2 "License: ${project_license}")
 	)
 	(junction
