File: ulx4m.kicad_sch (KiCad schematic)
At the start: 10 parts

Commit message: Updating schematics
Other:
- sheet DDR3 renamed SDRAM
- note added: "3X BTN 8X LED"
- note added: "BANK POWER 3V3 2V5 1V1/1V2 1V35(DNP)"
- note added: "BANK0 BANK7 CM4 connector"
- note added: "BANK1 SW DSI"
- note added: "BANK2 BANK3"
- note added: "BANK6 CLK25 USB JTAG"
- note added: "BANK8 FLASH (IS25LP128F)"
- note added: "ETHERNET (LAN8720A)"
- note added: "Mounting holes"
- note added: "SDRAM (IS42S16320D)"
- note added: "SERDES"
- note removed: "click on mouse pointer arrow on top of right toolbar and double-click on sheet to open"
- moved on the sheet: H1, H2, H3, H4
