File: ulx4m.kicad_sch (KiCad schematic)
At the start: 10 parts

Commit message: fix #44
Other:
- title: ULX4M-LS -> ULX4M-LD
Changed lines of the file:
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@@
 	(paper "A4")
 	(title_block
-		(title "ULX4M-LS")
-		(date "2021-11-05")
-		(rev "0.0.2")
+		(title "ULX4M-LD")
+		(date "2025-03-12")
+		(rev "0.0.3")
 		(company "Intergalaktik d.o.o.")
-		(comment 1 "Root sheet")
 		(comment 2 "License: CERN-OHL-S v2")
 	)

Commit message: Adding schematics
Other:
- note added: "3X BTN 8X LED"
- note added: "BANK 50 BANK 51 SERDES"
- note added: "BANK POWER 1V1/1V2 1V35 2V5 3V3"
- note added: "BANK0 BANK7 CM4 connector"
- note added: "BANK1 DSI SD GPDI"
- note added: "BANK2 BANK3 DDR3 GPDI0"
- note added: "BANK6 CLK25 JTAG USB"
- note added: "BANK8 FLASH-IS25LP128F"
- note added: "DDR3-AS4C256M16D3"
- note added: "Ethernet-KSZ9031RNXCA"
- moved on the sheet: H1, H2, H3, H4
