File: usb.kicad_sch (KiCad schematic)
At the start: 18 parts, among them J3 JTAG, J6 GPIO>>JTAG, P1 USB_OTG, U1 LFE5U-85F-6BG381C, Y1 FNETHE025

Commit message: Updating schematics
Parts:
- U1: Digike_y2 (none) -> 220-2071-ND; Digikey (none) -> 220-2177-ND; Koncar (none) -> FU004; LCSC (none) -> C446029; LowCost (none) -> 842-LFE5U12F6BG381C; MFG1 (none) -> Lattice; MFG2 (none) -> Lattice; MNF1_URL (none) -> www.latticesemi.com; MNF2_URL (none) -> www.latticesemi.com; MP_N2 (none) -> LFE5U-12F-6BG381C; Mouser (none) -> 842-LFE5U85F6BG381C; Mouser_URL (none) -> www.mouser.com; Side (none) -> T; price100_Mouse (none) -> 22.82$
Other:
- note removed: "VNC2 programming pins: TXD RXD TXDEN"
- note removed: "WiFi programming pins: TXD RXD RTS DTR"
- moved on the sheet: J3, J6, U1J

Commit message: Cleanup
Connections:
- no-connect marks 1 -> 2
Changed lines of the file:
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@@
+	)
+	(no_connect
+		(at 257.81 67.31)
 	)
 	(no_connect
