File: ulx4m-ld.kicad_pcb (KiCad board)
At the start: 6 copper layers, 55.6 x 40.6 mm, 275 parts, among them J1 DF40C-100DP-0.4V(51), J2 DF40C-100DP-0.4V(51), J3 JTAG, J4 Antenna, P1 USB_OTG, SW1 SW_DIP_x02, U1 LFE5U-85F-6BG381C, U2 AS4C256M16D3, U3 IS25LP128F-JBLE, U4 KSZ9031RNXCA, U5 TLV62569DBV, U6 TLV62569DBV, U7 TLV62569DBV, U8 TLV62569DBV, Y1 FNETHE025, Y2 ASEMB-25.000MHZ-LC-T

Commit message: Improving schematics
Parts:
- C56, C57, C62, C64, C68, C70, C73, C74: footprint Capacitor_SMD:C_0201_0603Metric -> Capacitor_SMD:C_0402_1005Metric
- R74, R75, R76, R77, R84, R85, R86, R87: footprint Resistor_SMD:R_0201_0603Metric -> Resistor_SMD:R_0402_1005Metric
- moved C57 3.78 mm to (119.1, 101.3), turned to 0 degrees
- moved R86 2.62 mm to (110.3, 105.6), turned to 0 degrees
- moved R76 2.60 mm to (117.3, 102.2), turned to 180 degrees
- moved C62 1.70 mm to (111.8, 104.6), turned to 0 degrees
- moved R31 1.45 mm to (108.0, 102.9)
- moved C64 1.37 mm to (120.2, 103.3)
- moved R74 1.33 mm to (121.3, 105.5)
- moved C56 0.80 mm to (116.6, 104.6), turned to 180 degrees
- moved C68 0.60 mm to (113.7, 104.4), turned to 180 degrees
- moved R75 0.58 mm to (119.6, 106.2), turned to 90 degrees
- moved C70 0.57 mm to (119.7, 104.7), turned to 0 degrees
- moved R85 0.30 mm to (102.8, 106.9), turned to 180 degrees
- moved R87 0.30 mm to (114.1, 105.9)
- moved C119 0.29 mm to (102.3, 103.4)
- moved R77 0.21 mm to (118.2, 106.4), turned to 180 degrees
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Routing:
- net ETH_1P: track 28.2 -> 31.7 mm
- net ETH_MDIO: track 28.1 -> 24.9 mm
- net CM4_3.3V: track 253.3 -> 250.4 mm
- net ETH_3P: track 21.1 -> 24.0 mm
- net ETH_0P: track 33.6 -> 36.3 mm
- net GPIO12: track 40.3 -> 38.2 mm
- net /serdes/S_6_P: track 4.16 -> 6.05 mm
- net DDR3_VREF: track 71.6 -> 69.8 mm
- net /serdes/S_1_P: track 3.11 -> 4.85 mm
- net GND: track 409.1 -> 407.6 mm
- net Net-(BTN1-Pad1): track 29.9 -> 28.5 mm
- net /flash/FPGA_PROGRAMN: track 7.95 -> 9.41 mm
- net ETH_2P: track 28.6 -> 30.0 mm
- net GPIO11: track 19.0 -> 20.3 mm
- net ETH_3N: track 21.0 -> 22.3 mm
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Other:
- board text added: "PCB3D_BR_ULX4M-LD"
- board text added: "PCB3D_TL_ULX4M-LD"
