File: ulx4m-ld.kicad_sch (KiCad schematic)
At the start: 10 parts

Commit message: Improving schematics
Other:
- added sheet drawings (drawings.kicad_sch)
- note added: "${CURRENT_DATE}"
- note added: "${project_name} ${project_version}"
- note added: "......"
- note added: "......."
- note added: "1"
- note added: "10"
- note added: "11"
- note added: "12"
- note added: "2"
- note added: "3"
- note added: "4"
- note added: "5"
- note added: "6"
- note added: "7"
- note added: "8"
- note added: "9"
- note added: "Blender render top side"
- note added: "Blinkey"
- note added: "CoverPage"
- note added: "DDR3"
- note added: "DDR3 FPGA"
- note added: "Ethernet"
- note added: "Flash"
- note added: "GPDI"
- note added: "GPIO"
- note added: "Index"
- note added: "MehanicalDrawing"
- note added: "Page"
- note added: "PowerPage"
- note added: "SerDes"
- note added: "USB"
- company: Intergalaktik d.o.o. -> ${project_creator}
- title: ULX4M-LD -> ${project_name}
- moved on the sheet: H1, H2, H3, H4
